Commit message: git-svn-id: file:///home/svn/meka-ros-pkg@21 cfd446f6-b9c6-49ad-a440-209cd04d0f1d

File: trunk/m3_description/robots/irr.urdf.xacro (robot description, xacro)
@@ -6,9 +6,11 @@
        name="m3" >
  <property name="M_PI" value="3.1415926535897931" />
- <property name="R_ARM" value="ma10" />
- <property name="TORSO" value="mt3" />
- <property name="MESH" value="low_res" />
+ <property name="R_ARM" value="ma12" />
+ <property name="L_ARM" value="ma14" />
+ <property name="TORSO" value="mt4" />
+ <property name="MESH" value="m3_description/meshes/low_res" />
 <!-- M3 Arm -->
-  <include filename="$(find m3_description)/urdf/A2R2_r_arm_defs.urdf.xacro" />
+  <include filename="$(find m3_description)/urdf/A2R3_r_arm_defs.urdf.xacro" />
+  <include filename="$(find m3_description)/urdf/A2R3_l_arm_defs.urdf.xacro" />
   <material name="GreyA"> <!-- darkest -->
 	  <color rgba="0.3 0.3 0.3 1.0"/>
@@ -43,5 +45,5 @@
       <origin xyz="0 0 0" rpy="0 0 0 " />
       <geometry name="panplate_geom">
-	      <mesh filename="package://${MESH}/T2R2_panplate.mesh" />
+	      <mesh filename="package://${MESH}/T2R3_panplate.mesh" />
       </geometry>
     </visual>
@@ -69,5 +71,5 @@
       <origin xyz="0 0 0" rpy="0 0 0 " />
       <geometry name="torso_geom">
-	      <mesh filename="package://${MESH}/T2R2_torso.mesh" />
+	      <mesh filename="package://${MESH}/T2R3_torso.mesh" />
       </geometry>
     </visual>
@@ -95,5 +97,5 @@
       <origin xyz="0 0 0" rpy="0 0 0" />
       <geometry name="mid_geom">
-	      <mesh filename="package://${MESH}/T2R2_mid.mesh" />
+	      <mesh filename="package://${MESH}/T2R3_mid.mesh" />
       </geometry>
     </visual>
@@ -121,5 +123,5 @@
       <origin xyz="0 0 0" rpy="0 0 3.14159" />
       <geometry name="upper_geom">
-	      <mesh filename="package://${MESH}/T2R2_upper.mesh" />
+	      <mesh filename="package://${MESH}/T2R3_upper.mesh" />
       </geometry>
     </visual>

File: trunk/m3_description/robots/iss.urdf.xacro (robot description, xacro)
@@ -6,9 +6,11 @@
        name="m3" >
  <property name="M_PI" value="3.1415926535897931" />
- <property name="R_ARM" value="ma10" />
- <property name="TORSO" value="mt3" />
- <property name="MESH" value="low_res" />
+ <property name="R_ARM" value="ma8" />
+ <property name="L_ARM" value="ma9" />
+ <property name="TORSO" value="mt2" />
+ <property name="MESH" value="m3_description/meshes/low_res" />
 <!-- M3 Arm -->
   <include filename="$(find m3_description)/urdf/A2R2_r_arm_defs.urdf.xacro" />
+  <include filename="$(find m3_description)/urdf/A2R2_l_arm_defs.urdf.xacro" />
   <material name="GreyA"> <!-- darkest -->
 	  <color rgba="0.3 0.3 0.3 1.0"/>

File: trunk/m3_description/robots/m3.urdf.xacro (robot description, xacro)
@@ -1,18 +1,16 @@
 <?xml version="1.0"?>
-<robot name="m3"
-       xmlns:xi="http://www.w3.org/2001/XInclude"
-       xmlns:gazebo="http://playerstage.sourceforge.net/gazebo/xmlschema/#gz"
-       xmlns:model="http://playerstage.sourceforge.net/gazebo/xmlschema/#model"
-       xmlns:sensor="http://playerstage.sourceforge.net/gazebo/xmlschema/#sensor"
-       xmlns:body="http://playerstage.sourceforge.net/gazebo/xmlschema/#body"
-       xmlns:geom="http://playerstage.sourceforge.net/gazebo/xmlschema/#geom"
-       xmlns:joint="http://playerstage.sourceforge.net/gazebo/xmlschema/#joint"
+<robot xmlns:sensor="http://playerstage.sourceforge.net/gazebo/xmlschema/#sensor"
+       xmlns:controller="http://playerstage.sourceforge.net/gazebo/xmlschema/#controller"
        xmlns:interface="http://playerstage.sourceforge.net/gazebo/xmlschema/#interface"
-       xmlns:rendering="http://playerstage.sourceforge.net/gazebo/xmlschema/#rendering"
-       xmlns:renderable="http://playerstage.sourceforge.net/gazebo/xmlschema/#renderable"
-       xmlns:controller="http://playerstage.sourceforge.net/gazebo/xmlschema/#controller"
-       xmlns:physics="http://playerstage.sourceforge.net/gazebo/xmlschema/#physics">
-	<include filename="$(find m3_defs_ros)/defs/A2R2_r_arm_defs.urdf.xacro" />
-  <property name="M_PI" value="3.1415926535897931" />
+       xmlns:xacro="http://playerstage.sourceforge.net/gazebo/xmlschema/#interface"
+       name="m3" >
+ <property name="M_PI" value="3.1415926535897931" />
+ <property name="R_ARM" value="ma8" />
+ <property name="L_ARM" value="ma9" />
+ <property name="TORSO" value="mt2" />
+ <property name="MESH" value="m3_description/meshes/low_res" />
+<!-- M3 Arm -->
+  <include filename="$(find m3_description)/urdf/A2R2_r_arm_defs.urdf.xacro" />
+  <include filename="$(find m3_description)/urdf/A2R2_l_arm_defs.urdf.xacro" />
   <material name="GreyA"> <!-- darkest -->
 	  <color rgba="0.3 0.3 0.3 1.0"/>
@@ -30,4 +28,5 @@
 	  <origin xyz="0.0 0.18465 0.2337" rpy="0 0 0" />
   </m3_l_arm>
+  <link name="world" />
   <!-- Solid Base -->
   <joint name="base_joint" type="fixed">
@@ -46,5 +45,5 @@
       <origin xyz="0 0 0" rpy="0 0 0 " />
       <geometry name="panplate_geom">
-	      <mesh filename="package://m3_defs_ros/meshes/T2R2_panplate.mesh" />
+	      <mesh filename="package://${MESH}/T2R2_panplate.mesh" />
       </geometry>
     </visual>
@@ -56,5 +55,5 @@
     </collision>
   </link>
-  <joint name="m3joint_mt3_j0" type="continuous">
+  <joint name="m3joint_${TORSO}_j0" type="continuous">
     <axis xyz="0 0 1"/>
     <origin xyz="0 0 0.1493" rpy="0 0 0" />
@@ -72,5 +71,5 @@
       <origin xyz="0 0 0" rpy="0 0 0 " />
       <geometry name="torso_geom">
-	      <mesh filename="package://m3_defs_ros/meshes/T2R2_torso.mesh" />
+	      <mesh filename="package://${MESH}/T2R2_torso.mesh" />
       </geometry>
     </visual>
@@ -82,5 +81,5 @@
     </collision>
   </link>
-  <joint name="m3joint_mt3_j1" type="continuous">
+  <joint name="m3joint_${TORSO}_j1" type="continuous">
     <axis xyz="0 1 0"/>
     <origin xyz="0 0 0" rpy="0 0 0" />
@@ -98,5 +97,5 @@
       <origin xyz="0 0 0" rpy="0 0 0" />
       <geometry name="mid_geom">
-	      <mesh filename="package://m3_defs_ros/meshes/T2R2_mid.mesh" />
+	      <mesh filename="package://${MESH}/T2R2_mid.mesh" />
       </geometry>
     </visual>
@@ -108,5 +107,5 @@
     </collision>
   </link>
-  <joint name="m3joint_slave_mt3_j2" type="continuous">
+  <joint name="m3joint_slave_${TORSO}_j2" type="continuous">
     <axis xyz="0 1 0"/>
     <origin xyz="0 0 0.1397" rpy="0 0 0" />
@@ -124,5 +123,5 @@
       <origin xyz="0 0 0" rpy="0 0 3.14159" />
       <geometry name="upper_geom">
-	      <mesh filename="package://m3_defs_ros/meshes/T2R2_upper.mesh" />
+	      <mesh filename="package://${MESH}/T2R2_upper.mesh" />
       </geometry>
     </visual>

Commit message: git-svn-id: file:///home/svn/meka-ros-pkg@22 cfd446f6-b9c6-49ad-a440-209cd04d0f1d

File: trunk/m3_description/robots/irr.urdf.xacro (robot description, xacro)
@@ -45,5 +45,5 @@
       <origin xyz="0 0 0" rpy="0 0 0 " />
       <geometry name="panplate_geom">
-	      <mesh filename="package://${MESH}/T2R3_panplate.mesh" />
+	      <mesh filename="package://${MESH}/T2R3/T2R3_panplate.mesh" />
       </geometry>
     </visual>
@@ -71,5 +71,5 @@
       <origin xyz="0 0 0" rpy="0 0 0 " />
       <geometry name="torso_geom">
-	      <mesh filename="package://${MESH}/T2R3_torso.mesh" />
+	      <mesh filename="package://${MESH}/T2R3/T2R3_torso.mesh" />
       </geometry>
     </visual>
@@ -97,5 +97,5 @@
       <origin xyz="0 0 0" rpy="0 0 0" />
       <geometry name="mid_geom">
-	      <mesh filename="package://${MESH}/T2R3_mid.mesh" />
+	      <mesh filename="package://${MESH}/T2R3/T2R3_mid.mesh" />
       </geometry>
     </visual>
@@ -123,5 +123,5 @@
       <origin xyz="0 0 0" rpy="0 0 3.14159" />
       <geometry name="upper_geom">
-	      <mesh filename="package://${MESH}/T2R3_upper.mesh" />
+	      <mesh filename="package://${MESH}/T2R3/T2R3_upper.mesh" />
       </geometry>
     </visual>

File: trunk/m3_description/robots/iss.urdf.xacro (robot description, xacro)
@@ -45,5 +45,5 @@
       <origin xyz="0 0 0" rpy="0 0 0 " />
       <geometry name="panplate_geom">
-	      <mesh filename="package://${MESH}/T2R2_panplate.mesh" />
+	      <mesh filename="package://${MESH}/T2R2/T2R2_panplate.mesh" />
       </geometry>
     </visual>
@@ -71,5 +71,5 @@
       <origin xyz="0 0 0" rpy="0 0 0 " />
       <geometry name="torso_geom">
-	      <mesh filename="package://${MESH}/T2R2_torso.mesh" />
+	      <mesh filename="package://${MESH}/T2R2/T2R2_torso.mesh" />
       </geometry>
     </visual>
@@ -97,5 +97,5 @@
       <origin xyz="0 0 0" rpy="0 0 0" />
       <geometry name="mid_geom">
-	      <mesh filename="package://${MESH}/T2R2_mid.mesh" />
+	      <mesh filename="package://${MESH}/T2R2/T2R2_mid.mesh" />
       </geometry>
     </visual>
@@ -123,5 +123,5 @@
       <origin xyz="0 0 0" rpy="0 0 3.14159" />
       <geometry name="upper_geom">
-	      <mesh filename="package://${MESH}/T2R2_upper.mesh" />
+	      <mesh filename="package://${MESH}/T2R2/T2R2_upper.mesh" />
       </geometry>
     </visual>

File: trunk/m3_description/robots/m3.urdf.xacro (robot description, xacro)
@@ -45,5 +45,5 @@
       <origin xyz="0 0 0" rpy="0 0 0 " />
       <geometry name="panplate_geom">
-	      <mesh filename="package://${MESH}/T2R2_panplate.mesh" />
+	      <mesh filename="package://${MESH}/T2R2/T2R2_panplate.mesh" />
       </geometry>
     </visual>
@@ -71,5 +71,5 @@
       <origin xyz="0 0 0" rpy="0 0 0 " />
       <geometry name="torso_geom">
-	      <mesh filename="package://${MESH}/T2R2_torso.mesh" />
+	      <mesh filename="package://${MESH}/T2R2/T2R2_torso.mesh" />
       </geometry>
     </visual>
@@ -97,5 +97,5 @@
       <origin xyz="0 0 0" rpy="0 0 0" />
       <geometry name="mid_geom">
-	      <mesh filename="package://${MESH}/T2R2_mid.mesh" />
+	      <mesh filename="package://${MESH}/T2R2/T2R2_mid.mesh" />
       </geometry>
     </visual>
@@ -123,5 +123,5 @@
       <origin xyz="0 0 0" rpy="0 0 3.14159" />
       <geometry name="upper_geom">
-	      <mesh filename="package://${MESH}/T2R2_upper.mesh" />
+	      <mesh filename="package://${MESH}/T2R2/T2R2_upper.mesh" />
       </geometry>
     </visual>

File: trunk/m3_description/robots/uta.urdf.xacro (robot description, xacro)
@@ -43,5 +43,5 @@
       <origin xyz="0 0 0" rpy="0 0 0 " />
       <geometry name="panplate_geom">
-	      <mesh filename="package://${MESH}/T2R2_panplate.mesh" />
+	      <mesh filename="package://${MESH}/T2R2/T2R2_panplate.mesh" />
       </geometry>
     </visual>
