Commit message: git-svn-id: file:///home/svn/meka-ros-pkg@28 cfd446f6-b9c6-49ad-a440-209cd04d0f1d

File: trunk/m3_description/robots/m3.urdf.xacro (robot description, xacro)
@@ -6,11 +6,11 @@
        name="m3" >
  <property name="M_PI" value="3.1415926535897931" />
- <property name="R_ARM" value="ma8" />
- <property name="L_ARM" value="ma9" />
- <property name="TORSO" value="mt2" />
+ <property name="R_ARM" value="ma12" />
+ <property name="L_ARM" value="ma14" />
+ <property name="TORSO" value="mt4" />
  <property name="MESH" value="m3_description/meshes/low_res" />
 <!-- M3 Arm -->
-  <include filename="$(find m3_description)/urdf/A2R2_r_arm_defs.urdf.xacro" />
-  <include filename="$(find m3_description)/urdf/A2R2_l_arm_defs.urdf.xacro" />
+  <include filename="$(find m3_description)/urdf/A2R3_r_arm_defs.urdf.xacro" />
+  <include filename="$(find m3_description)/urdf/A2R3_l_arm_defs.urdf.xacro" />
   <material name="GreyA"> <!-- darkest -->
 	  <color rgba="0.3 0.3 0.3 1.0"/>
@@ -45,5 +45,5 @@
       <origin xyz="0 0 0" rpy="0 0 0 " />
       <geometry name="panplate_geom">
-	      <mesh filename="package://${MESH}/T2R2/T2R2_panplate.mesh" />
+	      <mesh filename="package://${MESH}/T2R3/T2R3_panplate.mesh" />
       </geometry>
     </visual>
@@ -71,5 +71,5 @@
       <origin xyz="0 0 0" rpy="0 0 0 " />
       <geometry name="torso_geom">
-	      <mesh filename="package://${MESH}/T2R2/T2R2_torso.mesh" />
+	      <mesh filename="package://${MESH}/T2R3/T2R3_torso.mesh" />
       </geometry>
     </visual>
@@ -97,5 +97,5 @@
       <origin xyz="0 0 0" rpy="0 0 0" />
       <geometry name="mid_geom">
-	      <mesh filename="package://${MESH}/T2R2/T2R2_mid.mesh" />
+	      <mesh filename="package://${MESH}/T2R3/T2R3_mid.mesh" />
       </geometry>
     </visual>
@@ -123,5 +123,5 @@
       <origin xyz="0 0 0" rpy="0 0 3.14159" />
       <geometry name="upper_geom">
-	      <mesh filename="package://${MESH}/T2R2/T2R2_upper.mesh" />
+	      <mesh filename="package://${MESH}/T2R3/T2R3_upper.mesh" />
       </geometry>
     </visual>
