Commit message: updated urdfs and meshes
git-svn-id: file:///home/svn/meka-ros-pkg@31 cfd446f6-b9c6-49ad-a440-209cd04d0f1d

File: trunk/m3_description/robots/uta.urdf.xacro (robot description, xacro)
@@ -23,7 +23,7 @@
 	  <origin xyz="0.0 -0.18465 0.2337" rpy="0 0 0" />
   </m3_r_arm>
-  <m3_l_arm side="l" reflect="1" parent="upper">
+  <!--<m3_l_arm side="l" reflect="1" parent="upper">
 	  <origin xyz="0.0 0.18465 0.2337" rpy="0 0 0" />
-  </m3_l_arm>
+  </m3_l_arm>-->
   <link name="world" />
   <!-- Solid Base -->
@@ -55,13 +55,14 @@
   <joint name="m3joint_${TORSO}_j0" type="continuous">
     <axis xyz="0 0 1"/>
-    <origin xyz="0 0 0.1493" rpy="0 0 0" />
+    <origin xyz="0 0 0.1678" rpy="0 0 0" />
     <parent link="panplate" />
     <child link="torso" />
+    <limit effort="25" velocity="${25.0*M_PI/180}" lower="${-120*M_PI/180}" upper="${120*M_PI/180}" />
   </joint>
   <link name="torso">
     <inertial>
-      <mass value="1000" />
-      <origin xyz="0 0 0" />
-      <inertia ixx="1000"  ixy="0"  ixz="0" iyy="1000" iyz="0" izz="1000" />
+      <mass value="4.411" />
+      <origin xyz="0.00011774 0.0038073 -0.0522753" />
+      <inertia ixx="0.026360"  ixy="-0.0000024"  ixz="-0.0000508" iyy="0.0134266" iyz="0.0006839" izz="0.0229879" />
     </inertial>
     <visual>
@@ -84,10 +85,16 @@
     <parent link="torso" />
     <child link="mid" />
+    <limit effort="200" velocity="${10.0*M_PI/180}" lower="${-11.79349*M_PI/180}" upper="${53.29349*M_PI/180}" />
   </joint>
   <link name="mid">
     <inertial>
-      <mass value="1000" />
-      <origin xyz="0 0 0" />
-      <inertia ixx="1000"  ixy="0"  ixz="0" iyy="1000" iyz="0" izz="1000" />
+      <mass value="4.934" />
+      <origin xyz="0.001179 -0.002993 0.046259"/>
+      <inertia ixx="0.041106"
+      iyy="0.026009"
+      izz="0.025902"
+      ixy="0.000135"
+      ixz="0.000505"
+      iyz="0.002396" />
     </inertial>
     <visual>
@@ -110,14 +117,20 @@
     <parent link="mid" />
     <child link="upper" />
+    <limit effort="200" velocity="${10.0*M_PI/180}" lower="${-11.79349*M_PI/180}" upper="${53.29349*M_PI/180}" />
   </joint>
   <link name="upper">
     <inertial>
-      <mass value="1000" />
-      <origin xyz="0 0 0" />
-      <inertia ixx="1000"  ixy="0"  ixz="0" iyy="1000" iyz="0" izz="1000" />
+      <mass value="6.245" />
+      <origin xyz="0.008700 0.011470 0.129740"/>
+      <inertia ixx="0.069760"
+      iyy="0.048010"
+      izz="0.040590"
+      ixy="-0.000400"
+      ixz="0.001300"
+      iyz="0.005100" />
     </inertial>
     <visual>
       <material name="GreyC" />
-      <origin xyz="0 0 0" rpy="0 0 3.14159" />
+      <origin xyz="0 0 0" rpy="0 0 0" />
       <geometry name="upper_geom">
 	      <mesh filename="package://${MESH}/T2R2/T2R2_upper.mesh" />

File: trunk/m3_description/urdf/A2R2_r_arm_defs.urdf.xacro (robot description, xacro)
@@ -4,26 +4,4 @@
        xmlns:interface="http://playerstage.sourceforge.net/gazebo/xmlschema/#interface">
   <property name="M_PI" value="3.1415926535897931" />
-  <property name="VELOCITY_LIMIT_SCALE" value="0.6" />
-  <property name="shoulder_lift_length" value="0.10" />
-  <property name="shoulder_lift_radius" value="0.12" />
-  <!-- for non-symmetric upper arm -->
-  <property name="uar_xyz1" value= "0.21398" />
-  <property name="uar_xyz2" value="-0.01621" />
-  <property name="uar_xyz3" value="-0.00020" />
-  <property name="uar_ixx"  value= "0.01537748957" />
-  <property name="uar_ixy"  value= "0.00375711247" />
-  <property name="uar_ixz"  value="-0.00070852914" />
-  <property name="uar_iyy"  value= "0.07473670440" />
-  <property name="uar_iyz"  value="-0.00017936450" />
-  <property name="uar_izz"  value= "0.07608763307" />
-  <property name="ual_xyz1" value= "0.21405" />
-  <property name="ual_xyz2" value= "0.01658" />
-  <property name="ual_xyz3" value="-0.00057" />
-  <property name="ual_ixx"  value= "0.01530603856" />
-  <property name="ual_ixy"  value="-0.00339324862" />
-  <property name="ual_ixz"  value= "0.00060765455" />
-  <property name="ual_iyy"  value= "0.07473694455" />
-  <property name="ual_iyz"  value="-0.00019953729" />
-  <property name="ual_izz"  value= "0.07601594191" />
   <macro name="m3_r_shoulder" params="side parent reflect *origin">
     <!-- Shoulder pan -->
@@ -33,19 +11,16 @@
       <parent link="${parent}"/>
       <child link="shoulderupper_RIGHT"/>
-      <limit lower="${reflect*M_PI/4-1.5}"  upper="${reflect*M_PI/4+1.5}"
-             effort="30" velocity="${VELOCITY_LIMIT_SCALE*3.48}" />
-      <dynamics damping="10.0" />
-      <safety_controller k_position="100" k_velocity="10"
-                         soft_lower_limit="${reflect*M_PI/4-1.5+0.15}"
-                         soft_upper_limit="${reflect*M_PI/4+1.5-0.15}" />
-      <!-- joint angle when the rising or the falling flag is activated on PR2 -->
+      <limit effort="40" velocity="${30.0*M_PI/180}" lower="${-80*M_PI/180}" upper="${200*M_PI/180}" />
     </joint>
     <link name="shoulderupper_RIGHT">
       <inertial>
-        <mass value="25.799322" />
-        <origin xyz="-0.001201 0.024513 -0.098231" rpy="0 0 0"/>
-        <inertia ixx="0.866179142480"  ixy="-0.06086507933"  ixz="-0.12118061183"
-                 iyy="0.87421714893"  iyz="-0.05886609911"
-                 izz="0.27353821674" />
+        <mass value="2.0310" />
+	<origin xyz="-0.010946 0.025127 0.000022"/>
+	<inertia ixx="0.003461"
+	iyy="0.003097"
+	izz="0.005416"
+	ixy="0.000428"
+	ixz="0.000002"
+	iyz="0.000000" />
       </inertial>
       <visual>
@@ -63,13 +38,7 @@
       </collision>
     </link>
-    <!-- Shoulder lift -->
     <joint name="m3joint_${R_ARM}_j1" type="revolute">
       <axis xyz="-1 0 0"/>
-      <!-- Limits updated from Function's CAD values as of 2009_02_24 (link_data.xls) -->
-      <limit lower="-0.5236" upper="1.3963"
-             effort="30" velocity="${VELOCITY_LIMIT_SCALE*3.47}" />
-      <safety_controller k_position="100" k_velocity="10"
-                         soft_lower_limit="${-0.5236+0.17}" soft_upper_limit="${1.3963-0.05}" />
-      <dynamics damping="10.0" />
+     <limit effort="40" velocity="${30*M_PI/180}" lower="${-24*M_PI/180}" upper="${150*M_PI/180}" />
       <origin xyz="0 0 0" rpy="0 0 0" />
       <parent link="shoulderupper_RIGHT"/>
@@ -78,9 +47,12 @@
     <link name="shoulderpitch_RIGHT">
       <inertial>
-        <mass value="2.74988" />
-        <origin xyz="0.02195 -0.02664 -0.03127" rpy="0 0 0"/>
-        <inertia ixx="0.02105584615" ixy="0.00496704022"  ixz="-0.00194808955"
-                 iyy="0.02127223737" iyz="0.00110425490"
-                 izz="0.01975753814" />
+        <mass value="0.566" />
+        <origin xyz="0.000944 -0.026331 -0.043257"/>
+	<inertia ixx="0.000754"
+	iyy="0.000921"
+	izz="0.000834"
+	ixy="0.000015"
+	ixz="0.000014"
+	iyz="0.000142" />
       </inertial>
       <visual>
@@ -98,5 +70,4 @@
       </collision>
     </link>
-    <!-- Upperarm roll: internal fixed attchment point for upper arm -->
     <joint name="m3joint_${R_ARM}_j2" type="revolute">
       <axis xyz="0 0 -1" />
@@ -104,16 +75,16 @@
       <parent link="shoulderpitch_RIGHT" />
       <child link="bicep_RIGHT"/>
-      <limit lower="${reflect*1.55-2.35}" upper="${reflect*1.55+2.35}" effort="30" velocity="${VELOCITY_LIMIT_SCALE*5.45}" />
-      <safety_controller k_position="100" k_velocity="2" soft_lower_limit="${reflect*1.55-2.35+0.15}" soft_upper_limit="${reflect*1.55+2.35-0.15}" />
-      <dynamics damping="0.1" />
+      <limit effort="20" velocity="${50*M_PI/180}" lower="${-85*M_PI/180}" upper="${85*M_PI/180}" />
     </joint>
     <link name="bicep_RIGHT">
       <inertial>
-        <!-- dummy mass, to be removed -->
-        <mass value="0.1" />
-        <origin xyz="0.0 0 0" rpy="0 0 0" />
-        <inertia  ixx="0.01" ixy="0.00"  ixz="0.00"
-                  iyy="0.01" iyz="0.00"
-                  izz="0.01" />
+        <mass value="2.296" />
+        <origin xyz="-0.005767 0.084539 0.001385"/>
+	<inertia ixx="0.013031"
+	iyy="0.002070"
+	izz="0.013173"
+	ixy="-0.000564"
+	ixz="-0.000077"
+	iyz="0.000162" />
       </inertial>
       <visual>
@@ -139,18 +110,16 @@
       <parent link="${parent}"/>
       <child link="elbowclevis_RIGHT"/>
-	<limit lower="${reflect*M_PI/4-1.5}"  upper="${reflect*M_PI/4+1.5}"
-             effort="30" velocity="${VELOCITY_LIMIT_SCALE*3.48}" />
+	<limit effort="20" velocity="${50*M_PI/180}" lower="${ 0.182*M_PI/180}" upper="${132.8175*M_PI/180}" />
     </joint>
     <link name="elbowclevis_RIGHT">
       <inertial>
-        <!-- NOTE:reflect==-1 for right side, reflect==1 for the left side -->
-        <mass value="6.01769" />
-        <origin xyz="${0.5*((reflect+1)*ual_xyz1+(1-reflect)*uar_xyz1)} ${0.5*((reflect+1)*ual_xyz2+(1-reflect)*uar_xyz2)} ${0.5*((reflect+1)*ual_xyz3+(1-reflect)*uar_xyz3)}" />
-        <inertia  ixx="${0.5*((reflect+1)*ual_ixx+(1-reflect)*uar_ixx)}"
-                  ixy="${0.5*((reflect+1)*ual_ixy+(1-reflect)*uar_ixy)}"
-                  ixz="${0.5*((reflect+1)*ual_ixz+(1-reflect)*uar_ixz)}"
-                  iyy="${0.5*((reflect+1)*ual_iyy+(1-reflect)*uar_iyy)}"
-                  iyz="${0.5*((reflect+1)*ual_iyz+(1-reflect)*uar_iyz)}"
-                  izz="${0.5*((reflect+1)*ual_izz+(1-reflect)*uar_izz)}" />
+        <mass value="0.223" />
+        <origin xyz="-0.000002 0.000278 -0.026124"/>
+	<inertia ixx="0.000470"
+	iyy="0.000233"
+	izz="0.000425"
+	ixy="0.000000"
+	ixz="0.000000"
+	iyz="0.000019" />
       </inertial>
       <visual>
@@ -168,10 +137,7 @@
       </collision>
     </link>
-    <!-- Elbow flex -->
     <joint name="m3joint_${R_ARM}_j4" type="revolute">
 	    <axis xyz="0 0 -1" />
-      <limit lower="-2.3" upper="0.1" effort="30" velocity="${VELOCITY_LIMIT_SCALE*5.5}" />
-      <safety_controller k_position="100" k_velocity="3" soft_lower_limit="${-2.3+0.25}" soft_upper_limit="${0.1-0.1}" />
-      <dynamics damping="1.0" />
+      <limit effort="4" velocity="${150*M_PI/180}" lower="${-49.4*M_PI/180}" upper="${229.4*M_PI/180}" />
       <origin xyz="0 0 -0.27747" rpy="0 0 0" />
       <parent link="elbowclevis_RIGHT"/>
@@ -180,9 +146,12 @@
     <link name="wrist_RIGHT">
       <inertial>
-        <mass value="1.90327" />
-        <origin xyz="0.01014 0.00032 -0.01211" />
-        <inertia  ixx="0.00346541989" ixy="0.00004066825"  ixz="0.00043171614"
-                  iyy="0.00441606455"  iyz="-0.00003968914"
-                  izz="0.00359156824" />
+        <mass value="1.468" />
+        <origin xyz="-0.004404 0.000124 0.130931"/>
+	<inertia ixx="0.006099"
+	iyy="0.006120"
+	izz="0.001179"
+	ixy="0.000004"
+	ixz="-0.000043"
+	iyz="0.000015" />
       </inertial>
       <visual>
@@ -208,14 +177,13 @@
       <parent link="${parent}"/>
       <child link="w_differential_RIGHT"/>
-	<limit lower="${reflect*M_PI/4-1.5}"  upper="${reflect*M_PI/4+1.5}"
-             effort="30" velocity="${VELOCITY_LIMIT_SCALE*3.48}" />
+	<limit effort="8" velocity="${40*M_PI/180}" lower="${-58.83*M_PI/180}" upper="${58.83*M_PI/180}" />
     </joint>
     <link name="w_differential_RIGHT">
       <inertial>
-        <mass value="2.57968" />
-        <origin xyz="0.18791 -0.00017 -0.00912" />
-        <inertia ixx="0.00364857222" ixy="0.00005215877" ixz="0.00071534842"
-                 iyy="0.01507736897" iyz="-0.00001310770"
-                 izz="0.01659310749" />
+        <mass value="0.278" />
+        <origin xyz="0 0 0" />
+        <inertia ixx="0" ixy="0" ixz="0"
+                 iyy="0" iyz="0"
+                 izz="0" />
       </inertial>
       <visual>
@@ -233,10 +201,7 @@
       </collision>
     </link>
-    <!-- Wrist flex -->
     <joint name="m3joint_${R_ARM}_j6" type="revolute">
 	    <axis xyz="-1 0 0" />
-      <limit lower="-0.1" upper="2.2" effort="200" velocity="${VELOCITY_LIMIT_SCALE*5.13}" />
-      <safety_controller k_position="20" k_velocity="4" soft_lower_limit="${-0.1+0.2}" soft_upper_limit="${2.2-0.2}" />
-      <dynamics damping="0.1" />
+      <limit effort="8" velocity="${40*M_PI/180}" lower="${-60*M_PI/180}" upper="${60*M_PI/180}" />
       <origin xyz="0 0 0" rpy="0 0 0" />
       <parent link="w_differential_RIGHT"/>
@@ -245,9 +210,9 @@
     <link name="handmount_RIGHT">
       <inertial>
-        <mass value="0.61402" />
-        <origin xyz="-0.00157 0.0 -0.00075" />
-        <inertia ixx="0.00065165722" ixy="0.00000028864" ixz="0.00000303477"
-                 iyy="0.00019824443" iyz="-0.00000022645"
-                 izz="0.00064450498" />
+        <mass value="0.093" />
+        <origin xyz="0 0 0" />
+        <inertia ixx="0" ixy="0" ixz="0"
+                 iyy="0" iyz="0"
+                 izz="0" />
       </inertial>
       <visual>

Commit message: adding inertials
git-svn-id: file:///home/svn/meka-ros-pkg@33 cfd446f6-b9c6-49ad-a440-209cd04d0f1d

File: trunk/m3_description/robots/uta.urdf.xacro (robot description, xacro)
@@ -8,7 +8,11 @@
  <property name="R_ARM" value="ma10" />
  <property name="TORSO" value="mt3" />
+ <property name="HEAD" value="ms2" />
  <property name="MESH" value="m3_description/meshes/low_res" />
-<!-- M3 Arm -->
+<!-- Meka Arm -->
   <include filename="$(find m3_description)/urdf/A2R2_r_arm_defs.urdf.xacro" />
+<!-- Meka Head -->
+  <include filename="$(find m3_description)/urdf/S2R1_head_defs.urdf.xacro" />
+   <property name="M_PI" value="3.1415926535897931" />
   <material name="GreyA"> <!-- darkest -->
 	  <color rgba="0.3 0.3 0.3 1.0"/>
@@ -23,4 +27,7 @@
 	  <origin xyz="0.0 -0.18465 0.2337" rpy="0 0 0" />
   </m3_r_arm>
+  <m3_head side="r" reflect="1" parent="upper">
+	  <origin xyz="0.0 0.0 0.31155" rpy="0 0 0" />
+  </m3_head>
   <!--<m3_l_arm side="l" reflect="1" parent="upper">
 	  <origin xyz="0.0 0.18465 0.2337" rpy="0 0 0" />
@@ -58,5 +65,5 @@
     <parent link="panplate" />
     <child link="torso" />
-    <limit effort="25" velocity="${25.0*M_PI/180}" lower="${-120*M_PI/180}" upper="${120*M_PI/180}" />
+    <limit effort="25" velocity="${25.0*M_PI/180}" lower="${-120*M_PI/180.0}" upper="${120*M_PI/180}" />
   </joint>
   <link name="torso">
@@ -121,5 +128,5 @@
   <link name="upper">
     <inertial>
-      <mass value="6.245" />
+      <mass value="6.534" /> <!-- torso with motors, bottom pullies, and neck mount -->
       <origin xyz="0.008700 0.011470 0.129740"/>
       <inertia ixx="0.069760"
@@ -134,5 +141,5 @@
       <origin xyz="0 0 0" rpy="0 0 0" />
       <geometry name="upper_geom">
-	      <mesh filename="package://${MESH}/T2R2/T2R2_upper.mesh" />
+	      <mesh filename="package://${MESH}/T2R2/T2R2_upper_neck.mesh" />
       </geometry>
     </visual>

Commit message: adding hand
git-svn-id: file:///home/svn/meka-ros-pkg@36 cfd446f6-b9c6-49ad-a440-209cd04d0f1d

File: trunk/m3_description/robots/uta.urdf.xacro (robot description, xacro)
@@ -7,4 +7,5 @@
  <property name="M_PI" value="3.1415926535897931" />
  <property name="R_ARM" value="ma10" />
+ <property name="R_HAND" value="mh8" />
  <property name="TORSO" value="mt3" />
  <property name="HEAD" value="ms2" />
@@ -12,4 +13,6 @@
 <!-- Meka Arm -->
   <include filename="$(find m3_description)/urdf/A2R2_r_arm_defs.urdf.xacro" />
+<!-- Meka Hand -->
+  <include filename="$(find m3_description)/urdf/H2R2_r_hand_defs.urdf.xacro" />
 <!-- Meka Head -->
   <include filename="$(find m3_description)/urdf/S2R1_head_defs.urdf.xacro" />
@@ -30,4 +33,7 @@
 	  <origin xyz="0.0 0.0 0.31155" rpy="0 0 0" />
   </m3_head>
+  <m3_r_hand side="r" reflect="1" parent="handmount_RIGHT">
+	  <origin xyz="0.0 0.0 0.0" rpy="0 0 0" />
+  </m3_r_hand>
   <!--<m3_l_arm side="l" reflect="1" parent="upper">
 	  <origin xyz="0.0 0.18465 0.2337" rpy="0 0 0" />

Commit message: git-svn-id: file:///home/svn/meka-ros-pkg@44 cfd446f6-b9c6-49ad-a440-209cd04d0f1d

File: trunk/m3_description/robots/uta.urdf.xacro (robot description, xacro)
@@ -10,5 +10,9 @@
  <property name="TORSO" value="mt3" />
  <property name="HEAD" value="ms2" />
- <property name="MESH" value="m3_description/meshes/low_res" />
+ <property name="MESH" value="m3_description/meshes/mid_res" />
+ <property name="MESH_COLL" value="m3_description/meshes/low_res" />
+<!-- generic simulator_gazebo plugins for starting mechanism control, ros time, ros battery -->
+  <include filename="$(find m3_full_description)/gazebo/gazebo.urdf.xacro" />
+  <include filename="$(find m3_full_description)/transmissions/uta.transmission.xacro" />
 <!-- Meka Arm -->
   <include filename="$(find m3_description)/urdf/A2R2_r_arm_defs.urdf.xacro" />
@@ -17,32 +21,41 @@
 <!-- Meka Head -->
   <include filename="$(find m3_description)/urdf/S2R1_head_defs.urdf.xacro" />
+  <!-- john added transmissions -->
+  <include filename="$(find m3_full_description)/transmissions/A2R2_r_arm_defs.transmission.xacro" />
+  <include filename="$(find m3_full_description)/transmissions/H2R2_r_hand_defs.transmission.xacro" />
+  <include filename="$(find m3_full_description)/transmissions/S2R1_head_defs.transmission.xacro" />
    <property name="M_PI" value="3.1415926535897931" />
   <material name="GreyA"> <!-- darkest -->
-	  <color rgba="0.3 0.3 0.3 1.0"/>
+    <color rgba="0.3 0.3 0.3 1.0"/>
   </material>
   <material name="GreyB">
-	  <color rgba="0.5 0.5 0.5 1.0"/>
+    <color rgba="0.5 0.5 0.5 1.0"/>
   </material>
   <material name="GreyC">
-	  <color rgba="0.7 0.7 0.7 1.0"/>
+    <color rgba="0.7 0.7 0.7 1.0"/>
   </material>
  <m3_r_arm side="r" reflect="1" parent="upper">
-	  <origin xyz="0.0 -0.18465 0.2337" rpy="0 0 0" />
+    <origin xyz="0.0 -0.18465 0.2337" rpy="0 0 0" />
   </m3_r_arm>
+  <!-- john added transmissions -->
+  <m3_r_arm_transmission side="r" reflect="1" parent="upper"/>
+  <m3_r_hand_transmission/>
+  <m3_head_transmission/>
   <m3_head side="r" reflect="1" parent="upper">
-	  <origin xyz="0.0 0.0 0.31155" rpy="0 0 0" />
+    <origin xyz="0.0 0.0 0.31155" rpy="0 0 0" />
   </m3_head>
   <m3_r_hand side="r" reflect="1" parent="handmount_RIGHT">
-	  <origin xyz="0.0 0.0 0.0" rpy="0 0 0" />
+    <origin xyz="0.0 0.0 0.0" rpy="0 0 0" />
   </m3_r_hand>
   <!--<m3_l_arm side="l" reflect="1" parent="upper">
-	  <origin xyz="0.0 0.18465 0.2337" rpy="0 0 0" />
+    <origin xyz="0.0 0.18465 0.2337" rpy="0 0 0" />
   </m3_l_arm>-->
   <link name="world" />
   <!-- Solid Base -->
   <joint name="base_joint" type="fixed">
-    <origin xyz="0 0 0" rpy="0 0 0" />
+    <origin xyz="0 0 1" rpy="0 0 0" />
     <parent link="world" />
     <child link="panplate" />
+    <dynamics damping="1.0"/>
   </joint>
   <link name="panplate">
@@ -50,5 +63,5 @@
       <mass value="1000" />
       <origin xyz="0 0 0" />
-      <inertia ixx="1000"  ixy="0"  ixz="0" iyy="1000" iyz="0" izz="1000" />
+      <inertia ixx="100"  ixy="0"  ixz="0" iyy="100" iyz="0" izz="100" />
     </inertial>
     <visual>
@@ -56,5 +69,5 @@
       <origin xyz="0 0 0" rpy="0 0 0 " />
       <geometry name="panplate_geom">
-	      <mesh filename="package://${MESH}/T2R2/T2R2_panplate.mesh" />
+        <mesh filename="package://${MESH}/T2R3/T2R3_TJ0_base.dae" />
       </geometry>
     </visual>
@@ -62,5 +75,5 @@
       <origin xyz="0 0 0" rpy="0.0 0.0 0.0 " />
       <geometry name="base_collision_geom">
-        <box size="0.01 0.01 0.01" />
+        <mesh filename="package://${MESH_COLL}/T2R3/T2R3_TJ0_base.stl" />
       </geometry>
     </collision>
@@ -72,4 +85,5 @@
     <child link="torso" />
     <limit effort="25" velocity="${25.0*M_PI/180}" lower="${-120*M_PI/180.0}" upper="${120*M_PI/180}" />
+    <dynamics damping="1.0"/>
   </joint>
   <link name="torso">
@@ -83,5 +97,5 @@
       <origin xyz="0 0 0" rpy="0 0 0 " />
       <geometry name="torso_geom">
-	      <mesh filename="package://${MESH}/T2R2/T2R2_torso.mesh" />
+        <mesh filename="package://${MESH}/T2R3/T2R3_TJ1_pan.dae" />
       </geometry>
     </visual>
@@ -89,5 +103,5 @@
       <origin xyz="0 0 0" rpy="0.0 0.0 0.0 " />
       <geometry name="torso_collision_geom">
-        <box size="0.01 0.01 0.01" />
+        <mesh filename="package://${MESH_COLL}/T2R3/T2R3_TJ1_pan.stl" />
       </geometry>
     </collision>
@@ -99,4 +113,5 @@
     <child link="mid" />
     <limit effort="200" velocity="${10.0*M_PI/180}" lower="${-11.79349*M_PI/180}" upper="${53.29349*M_PI/180}" />
+    <dynamics damping="1.0"/>
   </joint>
   <link name="mid">
@@ -115,5 +130,5 @@
       <origin xyz="0 0 0" rpy="0 0 0" />
       <geometry name="mid_geom">
-	      <mesh filename="package://${MESH}/T2R2/T2R2_mid.mesh" />
+        <mesh filename="package://${MESH}/T2R3/T2R3_TJ2.dae" />
       </geometry>
     </visual>
@@ -121,5 +136,5 @@
       <origin xyz="0 0 0" rpy="0.0 0.0 0.0 " />
       <geometry name="mid_collision_geom">
-        <box size="0.01 0.01 0.01" />
+        <mesh filename="package://${MESH_COLL}/T2R3/T2R3_TJ2.stl" />
       </geometry>
     </collision>
@@ -131,4 +146,5 @@
     <child link="upper" />
     <limit effort="200" velocity="${10.0*M_PI/180}" lower="${-11.79349*M_PI/180}" upper="${53.29349*M_PI/180}" />
+    <dynamics damping="1.0"/>
   </joint>
   <link name="upper">
@@ -147,5 +163,5 @@
       <origin xyz="0 0 0" rpy="0 0 0" />
       <geometry name="upper_geom">
-	      <mesh filename="package://${MESH}/T2R2/T2R2_upper_neck.mesh" />
+        <mesh filename="package://${MESH}/T2R3/T2R3_TJ3_chest_waist_neck.dae" />
       </geometry>
     </visual>
@@ -153,5 +169,5 @@
       <origin xyz="0 0 0" rpy="0.0 0.0 0.0 " />
       <geometry name="upper_collision_geom">
-        <box size="0.01 0.01 0.01" />
+        <mesh filename="package://${MESH_COLL}/T2R3/T2R3_TJ3_chest_waist_neck.stl" />
       </geometry>
     </collision>
