Commit message: git-svn-id: file:///home/svn/meka-ros-pkg@20 cfd446f6-b9c6-49ad-a440-209cd04d0f1d

File: trunk/m3_description/robots/esp.urdf.xacro (robot description, xacro)
@@ -9,5 +9,5 @@
  <property name="MESH" value="m3_description/meshes/low_res" />
 <!-- M3 Arm -->
-  <include filename="$(find m3_description)/urdf/A2R1_r_arm_defs.urdf.xacro" />
+  <include filename="$(find m3_description)/urdf/A2R3_r_arm_defs.urdf.xacro" />
   <property name="M_PI" value="3.1415926535897931" />
   <material name="GreyA"> <!-- darkest -->
@@ -43,5 +43,5 @@
 		  <origin xyz="0 0 0" rpy="0 0 0" />
 		  <geometry name="upper_geom">
-			  <mesh filename="package://${MESH}/A2R2/A2R2_upper.mesh" />
+			  <mesh filename="package://${MESH}/A2R3/A2R3_upper.mesh" />
 		  </geometry>
 	  </visual>

Commit message: switching to A1R1 for now
git-svn-id: file:///home/svn/meka-ros-pkg@55 cfd446f6-b9c6-49ad-a440-209cd04d0f1d

File: trunk/m3_description/robots/esp.urdf.xacro (robot description, xacro)
@@ -7,7 +7,7 @@
  <property name="M_PI" value="3.1415926535897931" />
  <property name="R_ARM" value="ma11" />
- <property name="MESH" value="m3_description/meshes/low_res" />
+ <property name="MESH" value="m3_description/meshes/mid_res" />
 <!-- M3 Arm -->
-  <include filename="$(find m3_description)/urdf/A2R3_r_arm_defs.urdf.xacro" />
+  <include filename="$(find m3_description)/urdf/A1R1_r_arm_defs.urdf.xacro" />
   <property name="M_PI" value="3.1415926535897931" />
   <material name="GreyA"> <!-- darkest -->
@@ -43,5 +43,5 @@
 		  <origin xyz="0 0 0" rpy="0 0 0" />
 		  <geometry name="upper_geom">
-			  <mesh filename="package://${MESH}/A2R3/A2R3_upper.mesh" />
+			  <mesh filename="package://${MESH}/A2R2/A2R2_upper.mesh" />
 		  </geometry>
 	  </visual>
