Commit message: git-svn-id: file:///home/svn/meka-ros-pkg@54 cfd446f6-b9c6-49ad-a440-209cd04d0f1d

File: trunk/m3_description/robots/hrl.urdf.xacro (robot description, xacro)
@@ -8,18 +8,8 @@
  <property name="R_ARM" value="ma1" />
  <property name="L_ARM" value="ma2" />
- <!--<property name="R_HAND" value="mh8" />-->
- <property name="MESH" value="m3_description/meshes/low_res" />
-<!-- generic simulator_gazebo plugins for starting mechanism control, ros time, ros battery -->
-  <!--<include filename="$(find m3_full_description)/gazebo/gazebo.urdf.xacro" />-->
-  <!--<include filename="$(find m3_full_description)/transmissions/uta.transmission.xacro" />-->
+ <property name="MESH" value="m3_description/meshes/mid_res" />
 <!-- Meka Arm -->
   <include filename="$(find m3_description)/urdf/A1R1_r_arm_defs.urdf.xacro" />
   <include filename="$(find m3_description)/urdf/A1R1_l_arm_defs.urdf.xacro" />
-<!-- Meka Hand -->
-<!--  <include filename="$(find m3_description)/urdf/H2R2_r_hand_defs.urdf.xacro" />-->
-  <!-- john added transmissions -->
-  <!--<include filename="$(find m3_full_description)/transmissions/A2R2_r_arm_defs.transmission.xacro" />
-  <include filename="$(find m3_full_description)/transmissions/H2R2_r_hand_defs.transmission.xacro" />
-  <include filename="$(find m3_full_description)/transmissions/S2R1_head_defs.transmission.xacro" />-->
    <property name="M_PI" value="3.1415926535897931" />
   <material name="GreyA"> <!-- darkest -->
@@ -51,5 +41,5 @@
   <!-- Solid Base -->
   <joint name="base_joint" type="fixed">
-	  <origin xyz="0 0 -0.2341" rpy="0 0 0" />
+	  <origin xyz="0 0 -0.2337" rpy="0 0 0" />
     <parent link="world" />
     <child link="upper" />
@@ -65,5 +55,6 @@
 		  <origin xyz="0 0 0" rpy="0 0 0" />
 		  <geometry name="upper_geom">
-			  <mesh filename="package://${MESH}/A1R1/A1R1_upper.mesh" />
+			  <!--<mesh filename="package://${MESH}/A2R3/A2R3_T4_Chest.mesh" />-->
+			  <mesh filename="package://${MESH}/A2R2/A2R2_upper.mesh" />
 		  </geometry>
 	  </visual>

Commit message: git-svn-id: file:///home/svn/meka-ros-pkg@71 cfd446f6-b9c6-49ad-a440-209cd04d0f1d

File: trunk/m3_description/robots/hrl.urdf.xacro (robot description, xacro)
@@ -9,4 +9,5 @@
  <property name="L_ARM" value="ma2" />
  <property name="MESH" value="m3_description/meshes/mid_res" />
+ <property name="MESH_COLL" value="m3_description/meshes/low_res" />
 <!-- Meka Arm -->
   <include filename="$(find m3_description)/urdf/A1R1_r_arm_defs.urdf.xacro" />
@@ -23,23 +24,13 @@
   </material>
  <m3_r_arm side="r" reflect="1" parent="upper">
-    <origin xyz="0.0 -0.18465 0.2337" rpy="0 0 0" />
+    <origin xyz="0.0 -0.18465 0.0" rpy="0 0 0" />
   </m3_r_arm>
   <m3_l_arm side="l" reflect="1" parent="upper">
-    <origin xyz="0.0 0.18465 0.2337" rpy="0 0 0" />
+    <origin xyz="0.0 0.184 0.0" rpy="0 0 0" />
   </m3_l_arm>
-  <!-- john added transmissions -->
-  <!--<m3_r_arm_transmission side="r" reflect="1" parent="upper"/>
-  <m3_r_hand_transmission/>
-  <m3_head_transmission/>
-  <m3_head side="r" reflect="1" parent="upper">
-    <origin xyz="0.0 0.0 0.31155" rpy="0 0 0" />
-  </m3_head>
-  <m3_r_hand side="r" reflect="1" parent="handmount_RIGHT">
-    <origin xyz="0.0 0.0 0.0" rpy="0 0 0" />
-  </m3_r_hand>-->
   <link name="world" />
   <!-- Solid Base -->
   <joint name="base_joint" type="fixed">
-	  <origin xyz="0 0 -0.2337" rpy="0 0 0" />
+	  <origin xyz="0 0 0.0" rpy="0 0 0" />
     <parent link="world" />
     <child link="upper" />
@@ -55,6 +46,5 @@
 		  <origin xyz="0 0 0" rpy="0 0 0" />
 		  <geometry name="upper_geom">
-			  <!--<mesh filename="package://${MESH}/A2R3/A2R3_T4_Chest.mesh" />-->
-			  <mesh filename="package://${MESH}/A2R2/A2R2_upper.mesh" />
+			  <mesh filename="package://${MESH}/A1R1/A1R1_T4_Chest.dae" />
 		  </geometry>
 	  </visual>
@@ -62,5 +52,5 @@
 		  <origin xyz="0 0 0" rpy="0.0 0.0 0.0 " />
 		  <geometry name="upper_collision_geom">
-			  <box size="0.01 0.01 0.01" />
+			  <mesh filename="package://${MESH_COLL}/A1R1/A1R1_T4_Chest.dae" />
 		  </geometry>
 	  </collision>
