Commit message: adding left hand
git-svn-id: file:///home/svn/meka-ros-pkg@93 cfd446f6-b9c6-49ad-a440-209cd04d0f1d

File: trunk/m3_description/robots/fts.urdf.xacro (robot description, xacro)
@@ -7,8 +7,10 @@
  <property name="M_PI" value="3.1415926535897931" />
  <property name="R_HAND" value="mh12" />
+ <property name="L_HAND" value="mh14" />
  <property name="MESH" value="m3_description/meshes/mid_res" />
  <property name="MESH_COLL" value="m3_description/meshes/low_res" />
 <!-- Meka Hand -->
-  <include filename="$(find m3_description)/urdf/H2R2_r_hand_defs.urdf.xacro" />
+<include filename="$(find m3_description)/urdf/H2R2_r_hand_defs.urdf.xacro" />
+  <include filename="$(find m3_description)/urdf/H2R2_l_hand_defs.urdf.xacro" />
   <material name="GreyA"> <!-- darkest -->
 	  <color rgba="0.3 0.3 0.3 1.0"/>
@@ -21,6 +23,9 @@
   </material>
   <link name="world" />
-   <m3_r_hand side="r" reflect="0" parent="world">
-    <origin xyz="0.0 0.0 0.0" rpy="0 0 0" />
+  <m3_r_hand side="r" reflect="0" parent="world">
+    <origin xyz="0.0 0.2 0.0" rpy="0 0 0" />
   </m3_r_hand>
+<m3_l_hand side="l" reflect="0" parent="world">
+    <origin xyz="0.0 -0.2 0.0" rpy="0 0 0" />
+  </m3_l_hand>
 </robot>
