Commit message: Updated SIM to M3 1.3 RVIZ working.
git-svn-id: file:///home/svn/meka-ros-pkg@98 cfd446f6-b9c6-49ad-a440-209cd04d0f1d

File: trunk/m3_description/robots/sim.urdf.xacro (robot description, xacro)
@@ -8,4 +8,8 @@
  <property name="R_ARM" value="ma4" />
  <property name="L_ARM" value="ma3" />
+ <property name="R_HAND" value="mh1" />
+ <property name="L_HAND" value="mh2" />
+ <property name="TORSO" value="mt0" />
+ <property name="HEAD" value="mc0" />
  <property name="MESH" value="m3_description/meshes/mid_res" />
  <property name="MESH_COLL" value="m3_description/meshes/low_res" />
@@ -24,35 +28,113 @@
   </material>
  <m3_r_arm side="r" reflect="1" parent="upper">
-    <origin xyz="0.0 -0.18465 0.0" rpy="0 0 0" />
+    <origin xyz="0.0 -0.18465 0.2337" rpy="0 0 0" />
   </m3_r_arm>
   <m3_l_arm side="l" reflect="1" parent="upper">
-    <origin xyz="0.0 0.184 0.0" rpy="0 0 0" />
+    <origin xyz="0.0 0.18465 0.2337" rpy="0 0 0" />
   </m3_l_arm>
-  <link name="world" />
+<link name="world" />
   <!-- Solid Base -->
   <joint name="base_joint" type="fixed">
-	  <origin xyz="0 0 0.0" rpy="0 0 0" />
+    <origin xyz="0 0 0" rpy="0 0 0" />
     <parent link="world" />
+    <child link="panplate" />
+  </joint>
+  <link name="panplate">
+    <inertial>
+      <mass value="1000" />
+      <origin xyz="0 0 0" />
+      <inertia ixx="1000"  ixy="0"  ixz="0" iyy="1000" iyz="0" izz="1000" />
+    </inertial>
+    <visual>
+      <material name="GreyA" />
+      <origin xyz="0 0 0" rpy="0 0 0 " />
+      <geometry name="panplate_geom">
+	      <mesh filename="package://${MESH}/T2R2/T2R2_panplate.mesh" />
+      </geometry>
+    </visual>
+    <collision>
+      <origin xyz="0 0 0" rpy="0.0 0.0 0.0 " />
+      <geometry name="base_collision_geom">
+        <box size="0.01 0.01 0.01" />
+      </geometry>
+    </collision>
+  </link>
+  <joint name="m3joint_${TORSO}_j0" type="continuous">
+    <axis xyz="0 0 1"/>
+    <origin xyz="0 0 0.1678" rpy="0 0 0" />
+    <parent link="panplate" />
+    <child link="torso" />
+  </joint>
+  <link name="torso">
+    <inertial>
+      <mass value="1000" />
+      <origin xyz="0 0 0" />
+      <inertia ixx="1000"  ixy="0"  ixz="0" iyy="1000" iyz="0" izz="1000" />
+    </inertial>
+    <visual>
+      <material name="GreyC" />
+      <origin xyz="0 0 0" rpy="0 0 0 " />
+      <geometry name="torso_geom">
+	      <mesh filename="package://${MESH}/T2R2/T2R2_torso.mesh" />
+      </geometry>
+    </visual>
+    <collision>
+      <origin xyz="0 0 0" rpy="0.0 0.0 0.0 " />
+      <geometry name="torso_collision_geom">
+        <box size="0.01 0.01 0.01" />
+      </geometry>
+    </collision>
+  </link>
+  <joint name="m3joint_${TORSO}_j1" type="continuous">
+    <axis xyz="0 1 0"/>
+    <origin xyz="0 0 0" rpy="0 0 0" />
+    <parent link="torso" />
+    <child link="mid" />
+  </joint>
+  <link name="mid">
+    <inertial>
+      <mass value="1000" />
+      <origin xyz="0 0 0" />
+      <inertia ixx="1000"  ixy="0"  ixz="0" iyy="1000" iyz="0" izz="1000" />
+    </inertial>
+    <visual>
+      <material name="GreyB" />
+      <origin xyz="0 0 0" rpy="0 0 0" />
+      <geometry name="mid_geom">
+	      <mesh filename="package://${MESH}/T2R2/T2R2_mid.mesh" />
+      </geometry>
+    </visual>
+    <collision>
+      <origin xyz="0 0 0" rpy="0.0 0.0 0.0 " />
+      <geometry name="mid_collision_geom">
+        <box size="0.01 0.01 0.01" />
+      </geometry>
+    </collision>
+  </link>
+  <joint name="m3joint_slave_${TORSO}_j2" type="continuous">
+    <axis xyz="0 1 0"/>
+    <origin xyz="0 0 0.1397" rpy="0 0 0" />
+    <parent link="mid" />
     <child link="upper" />
   </joint>
   <link name="upper">
-	  <inertial>
-		  <mass value="1000" />
-		  <origin xyz="0 0 0" />
-		  <inertia ixx="1000"  ixy="0"  ixz="0" iyy="1000" iyz="0" izz="1000" />
-	  </inertial>
-	  <visual>
-		  <material name="GreyC" />
-		  <origin xyz="0 0 0" rpy="0 0 0" />
-		  <geometry name="upper_geom">
-			  <mesh filename="package://${MESH}/A1R1/A1R1_T4_Chest.dae" />
-		  </geometry>
-	  </visual>
-	  <collision>
-		  <origin xyz="0 0 0" rpy="0.0 0.0 0.0 " />
-		  <geometry name="upper_collision_geom">
-			  <mesh filename="package://${MESH_COLL}/A1R1/A1R1_T4_Chest.dae" />
-		  </geometry>
-	  </collision>
+    <inertial>
+      <mass value="1000" />
+      <origin xyz="0 0 0" />
+      <inertia ixx="1000"  ixy="0"  ixz="0" iyy="1000" iyz="0" izz="1000" />
+    </inertial>
+    <visual>
+      <material name="GreyC" />
+      <origin xyz="0 0 0" rpy="0 0 0" />
+      <geometry name="upper_geom">
+	      <mesh filename="package://${MESH}/T2R2/T2R2_upper.mesh" />
+      </geometry>
+    </visual>
+    <collision>
+      <origin xyz="0 0 0" rpy="0.0 0.0 0.0 " />
+      <geometry name="upper_collision_geom">
+        <box size="0.01 0.01 0.01" />
+      </geometry>
+    </collision>
   </link>
 </robot>
