Commit message: git-svn-id: file:///home/svn/meka-ros-pkg@100 cfd446f6-b9c6-49ad-a440-209cd04d0f1d

File: trunk/m3_description/robots/htl.urdf.xacro (robot description, xacro)
@@ -6,38 +6,30 @@
        name="m3" >
  <property name="M_PI" value="3.1415926535897931" />
- <property name="R_ARM" value="ma5" />
+  <property name="R_ARM" value="ma5" />
  <property name="MESH" value="m3_description/meshes/mid_res" />
-<!-- Meka Arm -->
-  <include filename="$(find m3_description)/urdf/A2R1_r_arm_defs.urdf.xacro" />
-   <property name="M_PI" value="3.1415926535897931" />
+ <property name="MESH_COLL" value="m3_description/meshes/low_res" />
+<!-- M3 Arm -->
+  <!--<include filename="$(find m3_description)/urdf/A1R1_r_arm_defs.urdf.xacro" />-->
+  <include filename="$(find m3_description)/urdf/A2R2_r_arm_defs.urdf.xacro" />
+  <property name="M_PI" value="3.1415926535897931" />
   <material name="GreyA"> <!-- darkest -->
-    <color rgba="0.3 0.3 0.3 1.0"/>
+	  <color rgba="0.3 0.3 0.3 1.0"/>
   </material>
   <material name="GreyB">
-    <color rgba="0.5 0.5 0.5 1.0"/>
+	  <color rgba="0.5 0.5 0.5 1.0"/>
   </material>
   <material name="GreyC">
-    <color rgba="0.7 0.7 0.7 1.0"/>
+	  <color rgba="0.7 0.7 0.7 1.0"/>
   </material>
- <m3_r_arm side="r" reflect="1" parent="upper">
-    <origin xyz="0.0 -0.18465 0.2337" rpy="0 0 0" />
+  <m3_r_arm side="r" reflect="1" parent="upper">
+	  <origin xyz="0.0 -0.18493 0.2341" rpy="0 0 0" />
   </m3_r_arm>
-  <m3_l_arm side="l" reflect="1" parent="upper">
-    <origin xyz="0.0 0.18465 0.2337" rpy="0 0 0" />
-  </m3_l_arm>
-  <!-- john added transmissions -->
-  <!--<m3_r_arm_transmission side="r" reflect="1" parent="upper"/>
-  <m3_r_hand_transmission/>
-  <m3_head_transmission/>
-  <m3_head side="r" reflect="1" parent="upper">
-    <origin xyz="0.0 0.0 0.31155" rpy="0 0 0" />
-  </m3_head>
-  <m3_r_hand side="r" reflect="1" parent="handmount_RIGHT">
-    <origin xyz="0.0 0.0 0.0" rpy="0 0 0" />
-  </m3_r_hand>-->
-  <link name="world" />
+<!--  <m3_l_arm side="l" reflect="1" parent="upper">
+	  <origin xyz="0.0 0.18493 0.2341" rpy="0 0 0" />
+  </m3_l_arm>-->
+   <link name="world" />
   <!-- Solid Base -->
   <joint name="base_joint" type="fixed">
-	  <origin xyz="0 0 -0.2337" rpy="0 0 0" />
+	  <origin xyz="0 0 -0.2341" rpy="0 0 0" />
     <parent link="world" />
     <child link="upper" />
@@ -53,5 +45,4 @@
 		  <origin xyz="0 0 0" rpy="0 0 0" />
 		  <geometry name="upper_geom">
-			  <!--<mesh filename="package://${MESH}/A2R3/A2R3_T4_Chest.mesh" />-->
 			  <mesh filename="package://${MESH}/A2R2/A2R2_upper.mesh" />
 		  </geometry>
