Commit message: git-svn-id: file:///home/svn/meka-ros-pkg@29 cfd446f6-b9c6-49ad-a440-209cd04d0f1d

File: trunk/m3_description/urdf/A2R3_r_arm_defs.urdf.xacro (robot description, xacro)
@@ -88,5 +88,5 @@
 	      <origin xyz="0 0 0" rpy="0 0 0 " />
 	      <geometry name="shoulderpitch_RIGHT">
-		      <mesh filename="package://${MESH}/A2R3/A2R3/A2R3_shoulderpitch_RIGHT.mesh" />
+		      <mesh filename="package://${MESH}/A2R3/A2R3_shoulderpitch_RIGHT.mesh" />
 	      </geometry>
       </visual>
@@ -121,5 +121,5 @@
 	      <origin xyz="0 0 0" rpy="0 0 0 " />
 	      <geometry name="bicep_RIGHT_geom">
-		      <mesh filename="package://${MESH}/A2R3/A2R3/A2R3_bicep_RIGHT.mesh" />
+		      <mesh filename="package://${MESH}/A2R3/A2R3_bicep_RIGHT.mesh" />
 	      </geometry>
       </visual>
@@ -158,5 +158,5 @@
 	      <origin xyz="0 0 0" rpy="0 0 0 " />
 	      <geometry name="elbowclevis_RIGHT_geom">
-		      <mesh filename="package://${MESH}/A2R3/A2R3/A2R3_elbowclevis_RIGHT.mesh" />
+		      <mesh filename="package://${MESH}/A2R3/A2R3_elbowclevis_RIGHT.mesh" />
 	      </geometry>
       </visual>
@@ -190,5 +190,5 @@
 	      <origin xyz="0 0 0" rpy="0 0 0 " />
 	      <geometry name="wrist_RIGHT_geom">
-		      <mesh filename="package://${MESH}/A2R3/A2R3/A2R3_wrist.mesh" />
+		      <mesh filename="package://${MESH}/A2R3/A2R3_wrist.mesh" />
 	      </geometry>
       </visual>
@@ -223,5 +223,5 @@
 	      <origin xyz="0 0 0" rpy="0 0 0 " />
 	      <geometry name="w_differential_RIGHT_geom">
-		      <mesh filename="package://${MESH}/A2R3/A2R3/A2R3_w_differential.mesh" />
+		      <mesh filename="package://${MESH}/A2R3/A2R3_w_differential.mesh" />
 	      </geometry>
       </visual>
@@ -255,5 +255,5 @@
 	      <origin xyz="0 0 0" rpy="0 0 0 " />
 	      <geometry name="handmount_RIGHT_geom">
-		      <mesh filename="package://${MESH}/A2R3/A2R3/A2R3_handmount.mesh" />
+		      <mesh filename="package://${MESH}/A2R3/A2R3_handmount.mesh" />
 	      </geometry>
       </visual>
