Commit message: added joint limits for head..
git-svn-id: file:///home/svn/meka-ros-pkg@34 cfd446f6-b9c6-49ad-a440-209cd04d0f1d

File: trunk/m3_description/urdf/S2R1_head_defs.urdf.xacro (robot description, xacro)
@@ -10,5 +10,5 @@
       <parent link="${parent}"/>
       <child link="neck_tilt"/>
-      <limit effort="40" velocity="${30.0*M_PI/180}" lower="${-80*M_PI/180}" upper="${200*M_PI/180}" />
+      <limit velocity="${20.0*M_PI/180}" lower="${-40*M_PI/180}" upper="${15*M_PI/180}" />
     </joint>
     <link name="neck_tilt">
@@ -39,5 +39,5 @@
     <joint name="m3joint_${HEAD}_j1" type="revolute">
       <axis xyz="0 0 1"/>
-     <limit effort="40" velocity="${30*M_PI/180}" lower="${-24*M_PI/180}" upper="${150*M_PI/180}" />
+     <limit velocity="${75*M_PI/180}" lower="${-80.919*M_PI/180}" upper="${80.91*M_PI/180}" />
       <origin xyz="0 0 0.13849" rpy="0 0 0" />
       <parent link="neck_tilt"/>
@@ -67,5 +67,5 @@
       <parent link="neck_roll" />
       <child link="neck_yaw"/>
-      <limit effort="20" velocity="${50*M_PI/180}" lower="${-85*M_PI/180}" upper="${85*M_PI/180}" />
+      <limit velocity="${50*M_PI/180}" lower="${-14.94*M_PI/180}" upper="${14.94*M_PI/180}" />
     </joint>
     <link name="neck_yaw">
@@ -99,5 +99,5 @@
       <parent link="neck_yaw" />
       <child link="head_shell"/>
-	<limit effort="20" velocity="${50*M_PI/180}" lower="${ 0.182*M_PI/180}" upper="${132.8175*M_PI/180}" />
+	<limit velocity="${50*M_PI/180}" lower="${-7.072*M_PI/180}" upper="${37.072*M_PI/180}" />
     </joint>
     <link name="head_shell">
@@ -128,5 +128,5 @@
     <joint name="m3joint_${HEAD}_j4" type="revolute">
 	    <axis xyz="0 -1 0" />
-      <limit effort="4" velocity="${150*M_PI/180}" lower="${-49.4*M_PI/180}" upper="${229.4*M_PI/180}" />
+      <limit velocity="${1600*M_PI/180}" lower="${-34.99*M_PI/180}" upper="${34.99*M_PI/180}" />
       <origin xyz="0.12508 0 0" rpy="0 0 0" />
       <parent link="head_shell"/>
@@ -150,5 +150,5 @@
     <joint name="m3joint_${HEAD}_j5" type="revolute">
 	    <axis xyz="0 0 1" />
-      <limit effort="4" velocity="${150*M_PI/180}" lower="${-49.4*M_PI/180}" upper="${229.4*M_PI/180}" />
+      <limit velocity="${1600*M_PI/180}" lower="${-34.21*M_PI/180}" upper="${34.213*M_PI/180}" />
       <origin xyz="0 -0.053 0" rpy="0 0 0" />
       <parent link="eye_tilt"/>
@@ -172,5 +172,5 @@
     <joint name="m3joint_${HEAD}_j6" type="revolute">
 	    <axis xyz="0 0 1" />
-      <limit effort="4" velocity="${150*M_PI/180}" lower="${-49.4*M_PI/180}" upper="${229.4*M_PI/180}" />
+      <limit velocity="${1600*M_PI/180}" lower="${-35.12*M_PI/180}" upper="${35.125*M_PI/180}" />
       <origin xyz="0 0.053 0" rpy="0 0 0" />
       <parent link="eye_tilt"/>

Commit message: fixing urdf for head
git-svn-id: file:///home/svn/meka-ros-pkg@35 cfd446f6-b9c6-49ad-a440-209cd04d0f1d

File: trunk/m3_description/urdf/S2R1_head_defs.urdf.xacro (robot description, xacro)
@@ -10,5 +10,5 @@
       <parent link="${parent}"/>
       <child link="neck_tilt"/>
-      <limit velocity="${20.0*M_PI/180}" lower="${-40*M_PI/180}" upper="${15*M_PI/180}" />
+      <limit effort="100" velocity="${20.0*M_PI/180}" lower="${-40*M_PI/180}" upper="${15*M_PI/180}" />
     </joint>
     <link name="neck_tilt">
@@ -39,5 +39,5 @@
     <joint name="m3joint_${HEAD}_j1" type="revolute">
       <axis xyz="0 0 1"/>
-     <limit velocity="${75*M_PI/180}" lower="${-80.919*M_PI/180}" upper="${80.91*M_PI/180}" />
+     <limit effort="100" velocity="${75*M_PI/180}" lower="${-80.919*M_PI/180}" upper="${80.91*M_PI/180}" />
       <origin xyz="0 0 0.13849" rpy="0 0 0" />
       <parent link="neck_tilt"/>
@@ -47,4 +47,11 @@
       <inertial>
         <mass value="0.409" />
+	<origin xyz="0.0 0.0 0.0"/>
+	<inertia ixx="0.0"
+	iyy="0.0"
+	izz="0.0"
+	ixy="0.0"
+	ixz="0.0"
+	iyz="0.0" />
       </inertial>
       <visual>
@@ -67,5 +74,5 @@
       <parent link="neck_roll" />
       <child link="neck_yaw"/>
-      <limit velocity="${50*M_PI/180}" lower="${-14.94*M_PI/180}" upper="${14.94*M_PI/180}" />
+      <limit effort="100" velocity="${50*M_PI/180}" lower="${-14.94*M_PI/180}" upper="${14.94*M_PI/180}" />
     </joint>
     <link name="neck_yaw">
@@ -99,5 +106,5 @@
       <parent link="neck_yaw" />
       <child link="head_shell"/>
-	<limit velocity="${50*M_PI/180}" lower="${-7.072*M_PI/180}" upper="${37.072*M_PI/180}" />
+	<limit effort="100" velocity="${50*M_PI/180}" lower="${-7.072*M_PI/180}" upper="${37.072*M_PI/180}" />
     </joint>
     <link name="head_shell">
@@ -128,5 +135,5 @@
     <joint name="m3joint_${HEAD}_j4" type="revolute">
 	    <axis xyz="0 -1 0" />
-      <limit velocity="${1600*M_PI/180}" lower="${-34.99*M_PI/180}" upper="${34.99*M_PI/180}" />
+      <limit effort="100" velocity="${1600*M_PI/180}" lower="${-34.99*M_PI/180}" upper="${34.99*M_PI/180}" />
       <origin xyz="0.12508 0 0" rpy="0 0 0" />
       <parent link="head_shell"/>
@@ -150,5 +157,5 @@
     <joint name="m3joint_${HEAD}_j5" type="revolute">
 	    <axis xyz="0 0 1" />
-      <limit velocity="${1600*M_PI/180}" lower="${-34.21*M_PI/180}" upper="${34.213*M_PI/180}" />
+      <limit effort="100" velocity="${1600*M_PI/180}" lower="${-34.21*M_PI/180}" upper="${34.213*M_PI/180}" />
       <origin xyz="0 -0.053 0" rpy="0 0 0" />
       <parent link="eye_tilt"/>
@@ -172,5 +179,5 @@
     <joint name="m3joint_${HEAD}_j6" type="revolute">
 	    <axis xyz="0 0 1" />
-      <limit velocity="${1600*M_PI/180}" lower="${-35.12*M_PI/180}" upper="${35.125*M_PI/180}" />
+      <limit effort="100" velocity="${1600*M_PI/180}" lower="${-35.12*M_PI/180}" upper="${35.125*M_PI/180}" />
       <origin xyz="0 0.053 0" rpy="0 0 0" />
       <parent link="eye_tilt"/>
