Commit message: adding damping for A2R2 j3 and j5, previously not specified.
git-svn-id: file:///home/svn/meka-ros-pkg@38 cfd446f6-b9c6-49ad-a440-209cd04d0f1d

File: trunk/m3_description/urdf/A2R2_l_arm_defs.urdf.xacro (robot description, xacro)
@@ -141,4 +141,5 @@
 	<limit lower="${reflect*M_PI/4-1.5}"  upper="${reflect*M_PI/4+1.5}"
              effort="30" velocity="${VELOCITY_LIMIT_SCALE*3.48}" />
+      <dynamics damping="10.0" />
     </joint>
     <link name="elbowclevis_LEFT">
@@ -204,4 +205,5 @@
   <macro name="m3_l_forearm" params="side parent reflect">
 	  <joint name="m3joint_${L_ARM}_j5" type="revolute">
+      <dynamics damping="1.0" />
 		  <axis xyz="0 -1 0" />
       <origin xyz="0 0 0" rpy="0 0 0" />

File: trunk/m3_description/urdf/A2R2_r_arm_defs.urdf.xacro (robot description, xacro)
@@ -111,4 +111,5 @@
       <child link="elbowclevis_RIGHT"/>
 	<limit effort="20" velocity="${50*M_PI/180}" lower="${ 0.182*M_PI/180}" upper="${132.8175*M_PI/180}" />
+      <dynamics damping="10.0" />
     </joint>
     <link name="elbowclevis_RIGHT">
@@ -173,4 +174,5 @@
   <macro name="m3_r_forearm" params="side parent reflect">
 	  <joint name="m3joint_${R_ARM}_j5" type="revolute">
+      <dynamics damping="1.0" />
 		  <axis xyz="0 -1 0" />
       <origin xyz="0 0 0" rpy="0 0 0" />
