Commit message: git-svn-id: file:///home/svn/meka-ros-pkg@24 cfd446f6-b9c6-49ad-a440-209cd04d0f1d

File: trunk/m3_description/urdf/A2R2_r_arm_defs.urdf.xacro (robot description, xacro)
@@ -53,5 +53,5 @@
 	      <origin xyz="0 0 0" rpy="0 0 0 " />
 	      <geometry name="r_shoulder_geom">
-		      <mesh filename="package://${MESH}/A2R2_shoulderupper_RIGHT.mesh" />
+		      <mesh filename="package://${MESH}/A2R2/A2R2_shoulderupper_RIGHT.mesh" />
 	      </geometry>
       </visual>

Commit message: We need some finite damping for simulation to behave better, adding default damping of 1.0 for simulation.
git-svn-id: file:///home/svn/meka-ros-pkg@43 cfd446f6-b9c6-49ad-a440-209cd04d0f1d

File: trunk/m3_description/urdf/A2R2_r_arm_defs.urdf.xacro (robot description, xacro)
@@ -12,4 +12,5 @@
       <child link="shoulderupper_RIGHT"/>
       <limit effort="40" velocity="${30.0*M_PI/180}" lower="${-80*M_PI/180}" upper="${200*M_PI/180}" />
+      <dynamics damping="1.0"/>
     </joint>
     <link name="shoulderupper_RIGHT">
@@ -44,4 +45,5 @@
       <parent link="shoulderupper_RIGHT"/>
       <child link="shoulderpitch_RIGHT"/>
+      <dynamics damping="1.0"/>
     </joint>
     <link name="shoulderpitch_RIGHT">
@@ -76,4 +78,5 @@
       <child link="bicep_RIGHT"/>
       <limit effort="20" velocity="${50*M_PI/180}" lower="${-85*M_PI/180}" upper="${85*M_PI/180}" />
+      <dynamics damping="1.0"/>
     </joint>
     <link name="bicep_RIGHT">
@@ -144,4 +147,5 @@
       <parent link="elbowclevis_RIGHT"/>
       <child link="wrist_RIGHT"/>
+      <dynamics damping="1.0"/>
     </joint>
     <link name="wrist_RIGHT">
@@ -180,4 +184,5 @@
       <child link="w_differential_RIGHT"/>
 	<limit effort="8" velocity="${40*M_PI/180}" lower="${-58.83*M_PI/180}" upper="${58.83*M_PI/180}" />
+      <dynamics damping="1.0"/>
     </joint>
     <link name="w_differential_RIGHT">
@@ -209,4 +214,5 @@
       <parent link="w_differential_RIGHT"/>
       <child link="handmount_RIGHT"/>
+      <dynamics damping="1.0"/>
     </joint>
     <link name="handmount_RIGHT">

Commit message: added collisions and switched to dae meshes
git-svn-id: file:///home/svn/meka-ros-pkg@45 cfd446f6-b9c6-49ad-a440-209cd04d0f1d

File: trunk/m3_description/urdf/A2R2_r_arm_defs.urdf.xacro (robot description, xacro)
@@ -29,5 +29,5 @@
 	      <origin xyz="0 0 0" rpy="0 0 0 " />
 	      <geometry name="r_shoulder_geom">
-		      <mesh filename="package://${MESH}/A2R2/A2R2_shoulderupper_RIGHT.mesh" />
+		      <mesh filename="package://${MESH}/A2R3/A2R3_RT1_shoulderRoll.dae" />
 	      </geometry>
       </visual>
@@ -35,5 +35,5 @@
 	      <origin xyz="0 0 0" rpy="0.0 0.0 0.0 " />
 	      <geometry name="r_shoulder_collision_geom">
-		      <box size="0.01 0.01 0.01" />
+		      <mesh filename="package://${MESH_COLL}/A2R3/A2R3_RT1_shoulderRoll.stl" />
 	      </geometry>
       </collision>
@@ -62,5 +62,5 @@
 	      <origin xyz="0 0 0" rpy="0 0 0 " />
 	      <geometry name="shoulderpitch_RIGHT">
-		      <mesh filename="package://${MESH}/A2R2/A2R2_shoulderpitch_RIGHT.mesh" />
+		      <mesh filename="package://${MESH}/A2R3/A2R3_RT2_shoulderPitch.dae" />
 	      </geometry>
       </visual>
@@ -68,5 +68,5 @@
 	      <origin xyz="0 0 0" rpy="0.0 0.0 0.0 " />
 	      <geometry name="shoulderpitch_RIGHT_collision">
-		      <box size="0.01 0.01 0.01" />
+		      <mesh filename="package://${MESH_COLL}/A2R3/A2R3_RT2_shoulderPitch.stl" />
 	      </geometry>
       </collision>
@@ -95,5 +95,5 @@
 	      <origin xyz="0 0 0" rpy="0 0 0 " />
 	      <geometry name="bicep_RIGHT_geom">
-		      <mesh filename="package://${MESH}/A2R2/A2R2_bicep_RIGHT.mesh" />
+		      <mesh filename="package://${MESH}/A2R3/A2R3_RT3_bicep.dae" />
 	      </geometry>
       </visual>
@@ -101,5 +101,5 @@
 	      <origin xyz="0 0 0" rpy="0.0 0.0 0.0 " />
 	      <geometry name="bicep_RIGHT_geom_collision">
-		      <box size="0.01 0.01 0.01" />
+		      <mesh filename="package://${MESH_COLL}/A2R3/A2R3_RT3_bicep.stl" />
 	      </geometry>
       </collision>
@@ -131,5 +131,5 @@
 	      <origin xyz="0 0 0" rpy="0 0 0 " />
 	      <geometry name="elbowclevis_RIGHT_geom">
-		      <mesh filename="package://${MESH}/A2R2/A2R2_elbowclevis_RIGHT.mesh" />
+		      <mesh filename="package://${MESH}/A2R3/A2R3_RT4_elbow.dae" />
 	      </geometry>
       </visual>
@@ -137,5 +137,5 @@
 	      <origin xyz="0 0 0" rpy="0.0 0.0 0.0 " />
 	      <geometry name="elbowclevis_RIGHT_collision">
-		      <box size="0.01 0.01 0.01" />
+		      <mesh filename="package://${MESH_COLL}/A2R3/A2R3_RT4_elbow.stl" />
 	      </geometry>
       </collision>
@@ -164,5 +164,5 @@
 	      <origin xyz="0 0 0" rpy="0 0 0 " />
 	      <geometry name="wrist_RIGHT_geom">
-		      <mesh filename="package://${MESH}/A2R2/A2R2_wrist.mesh" />
+		      <mesh filename="package://${MESH}/A2R3/A2R3_T5_forearmRoll.dae" />
 	      </geometry>
       </visual>
@@ -170,5 +170,5 @@
 	      <origin xyz="0 0 0" rpy="0.0 0.0 0.0 " />
 	      <geometry name="wrist_RIGHT_collision">
-		      <box size="0.01 0.01 0.01" />
+		      <mesh filename="package://${MESH_COLL}/A2R3/A2R3_T5_forearmRoll.stl" />
 	      </geometry>
       </collision>
@@ -198,5 +198,5 @@
 	      <origin xyz="0 0 0" rpy="0 0 0 " />
 	      <geometry name="w_differential_RIGHT_geom">
-		      <mesh filename="package://${MESH}/A2R2/A2R2_w_differential.mesh" />
+		      <mesh filename="package://${MESH}/A2R3/A2R3_T6_wristDiff.dae" />
 	      </geometry>
       </visual>
@@ -228,5 +228,5 @@
 	      <origin xyz="0 0 0" rpy="0 0 0 " />
 	      <geometry name="handmount_RIGHT_geom">
-		      <mesh filename="package://${MESH}/A2R2/A2R2_handmount.mesh" />
+		       <mesh filename="package://${MESH}/A2R3/A2R3_T7_wristYaw.dae" />
 	      </geometry>
       </visual>
@@ -234,5 +234,5 @@
 	      <origin xyz="0 0 0" rpy="0.0 0.0 0.0 " />
 	      <geometry name="handmount_RIGHT_collision">
-		      <box size="0.01 0.01 0.01" />
+		      <mesh filename="package://${MESH_COLL}/A2R3/A2R3_T7_wristYaw.stl" />
 	      </geometry>
       </collision>

File: trunk/m3_description/urdf/H2R2_r_hand_defs.urdf.xacro (robot description, xacro)
@@ -25,5 +25,5 @@
 	      <origin xyz="0 0 0" rpy="0 0 0 " />
 	      <geometry name="palm_geom">
-		      <mesh filename="package://${MESH}/H2R3/H2R3_RT8_palm_right.mesh" />
+		      <mesh filename="package://${MESH}/H2R3/H2R3_RT8_palm_right.dae" />
 	      </geometry>
       </visual>
@@ -31,5 +31,5 @@
 	      <origin xyz="0 0 0" rpy="0.0 0.0 0.0 " />
 	      <geometry name="palm_collision">
-		      <box size="0.01 0.01 0.01" />
+		      <mesh filename="package://${MESH_COLL}/H2R3/H2R3_RT8_palm_right.stl" />
 	      </geometry>
       </collision>
@@ -58,5 +58,5 @@
 	      <origin xyz="0 0 0" rpy="0 0 0 " />
 	      <geometry name="thumb0_geom">
-		      <mesh filename="package://${MESH}/H2R3/H2R3_RJ0_thumb_abductlink.mesh" />
+		      <mesh filename="package://${MESH}/H2R3/H2R3_RJ0_thumb_abductlink.dae" />
 	      </geometry>
       </visual>
@@ -64,5 +64,5 @@
 	      <origin xyz="0 0 0" rpy="0.0 0.0 0.0 " />
 	      <geometry name="thumb0_collision">
-		      <box size="0.01 0.01 0.01" />
+		      <mesh filename="package://${MESH_COLL}/H2R3/H2R3_RJ0_thumb_abductlink.stl" />
 	      </geometry>
       </collision>
@@ -90,5 +90,5 @@
 	      <origin xyz="0 0 0" rpy="0 0 0 " />
 	      <geometry name="thumb1_geom">
-		      <mesh filename="package://${MESH}/H2R3/H2R3_thumb_knuckle1.mesh" />
+		      <mesh filename="package://${MESH}/H2R3/H2R3_thumb_knuckle1.dae" />
 	      </geometry>
       </visual>
@@ -96,5 +96,5 @@
 	      <origin xyz="0 0 0" rpy="0.0 0.0 0.0 " />
 	      <geometry name="thumb1_collision">
-		      <box size="0.01 0.01 0.01" />
+		      <mesh filename="package://${MESH_COLL}/H2R3/H2R3_thumb_knuckle1.stl" />
 	      </geometry>
       </collision>
@@ -112,5 +112,5 @@
 	      <origin xyz="0 0 0" rpy="0 0 0 " />
 	      <geometry name="thumb_knuckle2_geom">
-		      <mesh filename="package://${MESH}/H2R3/H2R3_thumb_knuckle2.mesh" />
+		      <mesh filename="package://${MESH}/H2R3/H2R3_thumb_knuckle2.dae" />
 	      </geometry>
       </visual>
@@ -118,5 +118,5 @@
 	      <origin xyz="0 0 0" rpy="0.0 0.0 0.0 " />
 	      <geometry name="thumb_knuckle2_collision">
-		      <box size="0.01 0.01 0.01" />
+		      <mesh filename="package://${MESH_COLL}/H2R3/H2R3_thumb_knuckle2.stl" />
 	      </geometry>
       </collision>
@@ -135,5 +135,5 @@
 	      <origin xyz="0 0 0" rpy="0 0 0 " />
 	      <geometry name="index0_geom">
-		     <mesh filename="package://${MESH}/H2R3/H2R3_finger_knuckle1.mesh" />
+		     <mesh filename="package://${MESH}/H2R3/H2R3_finger_knuckle1.dae" />
 	      </geometry>
       </visual>
@@ -141,5 +141,5 @@
 	      <origin xyz="0 0 0" rpy="0.0 0.0 0.0 " />
 	      <geometry name="index0__collision">
-		      <box size="0.01 0.01 0.01" />
+		      <mesh filename="package://${MESH_COLL}/H2R3/H2R3_finger_knuckle1.stl" />
 	      </geometry>
       </collision>
@@ -167,5 +167,5 @@
 	      <origin xyz="0 0 0" rpy="0 0 0 " />
 	      <geometry name="index1_geom">
-		      <mesh filename="package://${MESH}/H2R3/H2R3_finger_knuckle2.mesh" />
+		      <mesh filename="package://${MESH}/H2R3/H2R3_finger_knuckle2.dae" />
 	      </geometry>
       </visual>
@@ -173,5 +173,5 @@
 	      <origin xyz="0 0 0" rpy="0.0 0.0 0.0 " />
 	      <geometry name="index1_collision">
-		      <box size="0.01 0.01 0.01" />
+		      <mesh filename="package://${MESH_COLL}/H2R3/H2R3_finger_knuckle2.stl" />
 	      </geometry>
       </collision>
@@ -189,5 +189,5 @@
 	      <origin xyz="0 0 0" rpy="0 0 0 " />
 	      <geometry name="index2_geom">
-		      <mesh filename="package://${MESH}/H2R3/H2R3_finger_knuckle3.mesh" />
+		      <mesh filename="package://${MESH}/H2R3/H2R3_finger_knuckle3.dae" />
 	      </geometry>
       </visual>
@@ -195,5 +195,5 @@
 	      <origin xyz="0 0 0" rpy="0.0 0.0 0.0 " />
 	      <geometry name="index2_collision">
-		      <box size="0.01 0.01 0.01" />
+		      <mesh filename="package://${MESH_COLL}/H2R3/H2R3_finger_knuckle3.stl" />
 	      </geometry>
       </collision>
@@ -212,5 +212,5 @@
 	      <origin xyz="0 0 0" rpy="0 0 0 " />
 	      <geometry name="ring0_geom">
-		     <mesh filename="package://${MESH}/H2R3/H2R3_finger_knuckle1.mesh" />
+		     <mesh filename="package://${MESH}/H2R3/H2R3_finger_knuckle1.dae" />
 	      </geometry>
       </visual>
@@ -218,5 +218,5 @@
 	      <origin xyz="0 0 0" rpy="0.0 0.0 0.0 " />
 	      <geometry name="ring0__collision">
-		      <box size="0.01 0.01 0.01" />
+		      <mesh filename="package://${MESH_COLL}/H2R3/H2R3_finger_knuckle1.stl" />
 	      </geometry>
       </collision>
@@ -244,5 +244,5 @@
 	      <origin xyz="0 0 0" rpy="0 0 0 " />
 	      <geometry name="ring1_geom">
-		      <mesh filename="package://${MESH}/H2R3/H2R3_finger_knuckle2.mesh" />
+		      <mesh filename="package://${MESH}/H2R3/H2R3_finger_knuckle2.dae" />
 	      </geometry>
       </visual>
@@ -250,5 +250,5 @@
 	      <origin xyz="0 0 0" rpy="0.0 0.0 0.0 " />
 	      <geometry name="ring1_collision">
-		      <box size="0.01 0.01 0.01" />
+		      <mesh filename="package://${MESH_COLL}/H2R3/H2R3_finger_knuckle2.stl" />
 	      </geometry>
       </collision>
@@ -266,5 +266,5 @@
 	      <origin xyz="0 0 0" rpy="0 0 0 " />
 	      <geometry name="ring2_geom">
-		      <mesh filename="package://${MESH}/H2R3/H2R3_finger_knuckle3.mesh" />
+		      <mesh filename="package://${MESH}/H2R3/H2R3_finger_knuckle3.dae" />
 	      </geometry>
       </visual>
@@ -272,5 +272,5 @@
 	      <origin xyz="0 0 0" rpy="0.0 0.0 0.0 " />
 	      <geometry name="ring2_collision">
-		      <box size="0.01 0.01 0.01" />
+		      <mesh filename="package://${MESH_COLL}/H2R3/H2R3_finger_knuckle3.stl" />
 	      </geometry>
       </collision>
@@ -289,5 +289,5 @@
 	      <origin xyz="0 0 0" rpy="0 0 0 " />
 	      <geometry name="pinky0_geom">
-		     <mesh filename="package://${MESH}/H2R3/H2R3_finger_knuckle1.mesh" />
+		     <mesh filename="package://${MESH}/H2R3/H2R3_finger_knuckle1.dae" />
 	      </geometry>
       </visual>
@@ -295,5 +295,5 @@
 	      <origin xyz="0 0 0" rpy="0.0 0.0 0.0 " />
 	      <geometry name="pinky0__collision">
-		      <box size="0.01 0.01 0.01" />
+		      <mesh filename="package://${MESH_COLL}/H2R3/H2R3_finger_knuckle1.stl" />
 	      </geometry>
       </collision>
@@ -321,5 +321,5 @@
 	      <origin xyz="0 0 0" rpy="0 0 0 " />
 	      <geometry name="pinky1_geom">
-		      <mesh filename="package://${MESH}/H2R3/H2R3_finger_knuckle2.mesh" />
+		      <mesh filename="package://${MESH}/H2R3/H2R3_finger_knuckle2.dae" />
 	      </geometry>
       </visual>
@@ -327,5 +327,5 @@
 	      <origin xyz="0 0 0" rpy="0.0 0.0 0.0 " />
 	      <geometry name="pinky1_collision">
-		      <box size="0.01 0.01 0.01" />
+		      <mesh filename="package://${MESH_COLL}/H2R3/H2R3_finger_knuckle2.stl" />
 	      </geometry>
       </collision>
@@ -343,5 +343,5 @@
 	      <origin xyz="0 0 0" rpy="0 0 0 " />
 	      <geometry name="pinky2_geom">
-		      <mesh filename="package://${MESH}/H2R3/H2R3_finger_knuckle3.mesh" />
+		      <mesh filename="package://${MESH}/H2R3/H2R3_finger_knuckle3.dae" />
 	      </geometry>
       </visual>
@@ -349,5 +349,5 @@
 	      <origin xyz="0 0 0" rpy="0.0 0.0 0.0 " />
 	      <geometry name="pinky2_collision">
-		      <box size="0.01 0.01 0.01" />
+		      <mesh filename="package://${MESH_COLL}/H2R3/H2R3_finger_knuckle3.stl" />
 	      </geometry>
       </collision>

File: trunk/m3_description/urdf/S2R1_head_defs.urdf.xacro (robot description, xacro)
@@ -27,5 +27,5 @@
 	      <origin xyz="0 0 0" rpy="0 0 0 " />
 	      <geometry name="neck_tilt_geom">
-		      <mesh filename="package://${MESH}/S2R1/S2R1_SH1_neckTilt.mesh" />
+		      <mesh filename="package://${MESH}/S2R1/S2R1_SH1_neckTilt.dae" />
 	      </geometry>
       </visual>
@@ -33,5 +33,5 @@
 	      <origin xyz="0 0 0" rpy="0.0 0.0 0.0 " />
 	      <geometry name="neck_tilt_geom_collison">
-		      <box size="0.01 0.01 0.01" />
+		      <mesh filename="package://${MESH_COLL}/S2R1/S2R1_SH1_neckTilt.stl" />
 	      </geometry>
       </collision>
@@ -59,5 +59,5 @@
 	      <origin xyz="0 0 0" rpy="0 0 0 " />
 	      <geometry name="neck_roll_geom">
-		      <mesh filename="package://${MESH}/S2R1/S2R1_SH2_neckRoll.mesh" />
+		      <mesh filename="package://${MESH}/S2R1/S2R1_SH2_neckRoll.dae" />
 	      </geometry>
       </visual>
@@ -91,5 +91,5 @@
 	      <origin xyz="0 0 0" rpy="0 0 0 " />
 	      <geometry name="S2R1_H3_neckYaw_geom">
-		      <mesh filename="package://${MESH}/S2R1/S2R1_H3_neckYaw.mesh" />
+		      <mesh filename="package://${MESH}/S2R1/S2R1_H3_neckYaw.dae" />
 	      </geometry>
       </visual>
@@ -123,5 +123,5 @@
 	      <origin xyz="0 0 0" rpy="0 0 0 " />
 	      <geometry name="head_shell_geom">
-		      <mesh filename="package://${MESH}/S2R1/S2R1_H4_UTA_head.mesh" />
+		      <mesh filename="package://${MESH}/S2R1/S2R1_H4_UTA_head.dae" />
 	      </geometry>
       </visual>
@@ -129,5 +129,5 @@
 	      <origin xyz="0 0 0" rpy="0.0 0.0 0.0 " />
 	      <geometry name="head_shell_collision">
-		      <box size="0.01 0.01 0.01" />
+		      <mesh filename="package://${MESH_COLL}/S2R1/S2R1_H4_UTA_head.stl" />
 	      </geometry>
       </collision>
@@ -145,5 +145,5 @@
 	      <origin xyz="0 0 0" rpy="0 0 0 " />
 	      <geometry name="eye_tilt_geom">
-		      <mesh filename="package://${MESH}/S2R1/S2R1_SH5_eyeTilt.mesh" />
+		      <mesh filename="package://${MESH}/S2R1/S2R1_SH5_eyeTilt.dae" />
 	      </geometry>
       </visual>
@@ -167,5 +167,5 @@
 	      <origin xyz="0 0 0" rpy="0 0 0 " />
 	      <geometry name="right_eye_geom">
-		      <mesh filename="package://${MESH}/S2R1/S2R1_eye.mesh" />
+		      <mesh filename="package://${MESH}/S2R1/S2R1_eye.dae" />
 	      </geometry>
       </visual>
@@ -173,5 +173,5 @@
 	      <origin xyz="0 0 0" rpy="0.0 0.0 0.0 " />
 	      <geometry name="right_eye_collision">
-		      <box size="0.01 0.01 0.01" />
+		      <mesh filename="package://${MESH_COLL}/S2R1/S2R1_eye.stl" />
 	      </geometry>
       </collision>
@@ -189,5 +189,5 @@
 	      <origin xyz="0 0 0" rpy="0 0 0 " />
 	      <geometry name="left_eye_geom">
-		      <mesh filename="package://${MESH}/S2R1/S2R1_eye.mesh" />
+		      <mesh filename="package://${MESH}/S2R1/S2R1_eye.dae" />
 	      </geometry>
       </visual>
@@ -195,5 +195,5 @@
 	      <origin xyz="0 0 0" rpy="0.0 0.0 0.0 " />
 	      <geometry name="left_eye_collision">
-		      <box size="0.01 0.01 0.01" />
+		      <mesh filename="package://${MESH_COLL}/S2R1/S2R1_eye.stl" />
 	      </geometry>
       </collision>
