Commit message: added mass for fingers
git-svn-id: file:///home/svn/meka-ros-pkg@51 cfd446f6-b9c6-49ad-a440-209cd04d0f1d

File: trunk/m3_description/urdf/H2R2_r_hand_defs.urdf.xacro (robot description, xacro)
@@ -108,4 +108,14 @@
     </joint>
     <link name="thumb2">
+      <inertial>
+        <mass value="0.01" />
+	<origin xyz="0.0 0.0 0.0"/>
+	<inertia ixx="0.0"
+	iyy="0.0"
+	izz="0.0"
+	ixy="0.0"
+	ixz="0.0"
+	iyz="0.0" />
+      </inertial>
       <visual>
 	      <material name="GreyC" />
@@ -131,4 +141,14 @@
     </joint>
     <link name="index0">
+      <inertial>
+        <mass value="0.01" />
+	<origin xyz="0.0 0.0 0.0"/>
+	<inertia ixx="0.0"
+	iyy="0.0"
+	izz="0.0"
+	ixy="0.0"
+	ixz="0.0"
+	iyz="0.0" />
+      </inertial>
       <visual>
 	      <material name="GreyA" />
@@ -185,4 +205,14 @@
     </joint>
     <link name="index2">
+      <inertial>
+        <mass value="0.01" />
+	<origin xyz="0.0 0.0 0.0"/>
+	<inertia ixx="0.0"
+	iyy="0.0"
+	izz="0.0"
+	ixy="0.0"
+	ixz="0.0"
+	iyz="0.0" />
+      </inertial>
       <visual>
 	      <material name="GreyC" />
@@ -208,4 +238,14 @@
     </joint>
     <link name="ring0">
+      <inertial>
+        <mass value="0.01" />
+	<origin xyz="0.0 0.0 0.0"/>
+	<inertia ixx="0.0"
+	iyy="0.0"
+	izz="0.0"
+	ixy="0.0"
+	ixz="0.0"
+	iyz="0.0" />
+      </inertial>
       <visual>
 	      <material name="GreyA" />
@@ -262,4 +302,14 @@
     </joint>
     <link name="ring2">
+      <inertial>
+        <mass value="0.01" />
+	<origin xyz="0.0 0.0 0.0"/>
+	<inertia ixx="0.0"
+	iyy="0.0"
+	izz="0.0"
+	ixy="0.0"
+	ixz="0.0"
+	iyz="0.0" />
+      </inertial>
       <visual>
 	      <material name="GreyC" />
@@ -285,4 +335,14 @@
     </joint>
     <link name="pinky0">
+      <inertial>
+        <mass value="0.01" />
+	<origin xyz="0.0 0.0 0.0"/>
+	<inertia ixx="0.0"
+	iyy="0.0"
+	izz="0.0"
+	ixy="0.0"
+	ixz="0.0"
+	iyz="0.0" />
+      </inertial>
       <visual>
 	      <material name="GreyA" />
@@ -339,4 +399,14 @@
     </joint>
     <link name="pinky2">
+      <inertial>
+        <mass value="0.01" />
+	<origin xyz="0.0 0.0 0.0"/>
+	<inertia ixx="0.0"
+	iyy="0.0"
+	izz="0.0"
+	ixy="0.0"
+	ixz="0.0"
+	iyz="0.0" />
+      </inertial>
       <visual>
 	      <material name="GreyC" />
