Commit message: git-svn-id: file:///home/svn/meka-ros-pkg@70 cfd446f6-b9c6-49ad-a440-209cd04d0f1d

File: trunk/m3_description/urdf/A1R1_l_arm_defs.urdf.xacro (robot description, xacro)
@@ -53,5 +53,5 @@
 	      <origin xyz="0 0 0" rpy="0 0 0 " />
 	      <geometry name="l_shoulder_geom">
-		      <mesh filename="package://${MESH}/A2R2/A2R2_shoulderupper_LEFT.mesh" />
+		      <mesh filename="package://${MESH}/A1R1/A1R1_LT1_shoulderRoll.dae" />
 	      </geometry>
       </visual>
@@ -59,5 +59,5 @@
 	      <origin xyz="0 0 0" rpy="0.0 0.0 0.0 " />
 	      <geometry name="l_shoulder_collision_geom">
-		      <box size="0.01 0.01 0.01" />
+		      <mesh filename="package://${MESH_COLL}/A1R1/A1R1_LT1_shoulderRoll.dae" />
 	      </geometry>
       </collision>
@@ -88,5 +88,5 @@
 	      <origin xyz="0 0 0" rpy="0 0 0 " />
 	      <geometry name="shoulderpitch_LEFT">
-		      <mesh filename="package://${MESH}/A2R2/A2R2_shoulderpitch_LEFT.mesh" />
+		      <mesh filename="package://${MESH}/A1R1/A1R1_LT2_shoulderPitch.dae" />
 	      </geometry>
       </visual>
@@ -94,5 +94,5 @@
 	      <origin xyz="0 0 0" rpy="0.0 0.0 0.0 " />
 	      <geometry name="shoulderpitch_LEFT_collision">
-		      <box size="0.01 0.01 0.01" />
+		      <mesh filename="package://${MESH_COLL}/A1R1/A1R1_LT2_shoulderPitch.dae" />
 	      </geometry>
       </collision>
@@ -121,5 +121,5 @@
 	      <origin xyz="0 0 0" rpy="0 0 0 " />
 	      <geometry name="bicep_l_geom">
-		      <mesh filename="package://${MESH}/A2R2/A2R2_bicep_LEFT.mesh" />
+		      <mesh filename="package://${MESH}/A1R1/A1R1_LT3_bicep.dae" />
 	      </geometry>
       </visual>
@@ -127,5 +127,5 @@
 	      <origin xyz="0 0 0" rpy="0.0 0.0 0.0 " />
 	      <geometry name="bicep_l_geom_collision">
-		      <box size="0.01 0.01 0.01" />
+		      <mesh filename="package://${MESH_COLL}/A1R1/A1R1_LT3_bicep.dae" />
 	      </geometry>
       </collision>
@@ -159,5 +159,5 @@
 	      <origin xyz="0 0 0" rpy="0 0 0 " />
 	      <geometry name="elbowclevis_l_geom">
-		      <mesh filename="package://${MESH}/A2R2/A2R2_elbowclevis_LEFT.mesh" />
+		      <mesh filename="package://${MESH}/A1R1/A1R1_LT4_elbow.dae" />
 	      </geometry>
       </visual>
@@ -165,5 +165,5 @@
 	      <origin xyz="0 0 0" rpy="0.0 0.0 0.0 " />
 	      <geometry name="elbowclevis_l_collision">
-		      <box size="0.01 0.01 0.01" />
+		      <mesh filename="package://${MESH_COLL}/A1R1/A1R1_LT4_elbow.dae" />
 	      </geometry>
       </collision>
@@ -191,5 +191,5 @@
 	      <origin xyz="0 0 0" rpy="0 0 0 " />
 	      <geometry name="wrist_l_geom">
-		      <mesh filename="package://${MESH}/A2R2/A2R2_wrist.mesh" />
+		      <mesh filename="package://${MESH}/A1R1/A1R1_LT5_forearmRoll.dae" />
 	      </geometry>
       </visual>
@@ -197,5 +197,5 @@
 	      <origin xyz="0 0 0" rpy="0.0 0.0 0.0 " />
 	      <geometry name="wrist_l_collision">
-		      <box size="0.01 0.01 0.01" />
+		      <mesh filename="package://${MESH_COLL}/A1R1/A1R1_LT5_forearmRoll.dae" />
 	      </geometry>
       </collision>
@@ -225,5 +225,5 @@
 	      <origin xyz="0 0 0" rpy="0 0 0 " />
 	      <geometry name="w_differential_l_geom">
-		      <mesh filename="package://${MESH}/A2R2/A2R2_w_differential.mesh" />
+		      <box size="0.01 0.01 0.01" />
 	      </geometry>
       </visual>
@@ -257,5 +257,5 @@
 	      <origin xyz="0 0 0" rpy="0 0 0 " />
 	      <geometry name="handmount_l_geom">
-		      <mesh filename="package://${MESH}/A2R2/A2R2_handmount.mesh" />
+		      <mesh filename="package://${MESH}/A1R1/A1R1_T7_wristYaw.dae" />
 	      </geometry>
       </visual>
@@ -263,5 +263,5 @@
 	      <origin xyz="0 0 0" rpy="0.0 0.0 0.0 " />
 	      <geometry name="handmount_l_collision">
-		      <box size="0.01 0.01 0.01" />
+		      <mesh filename="package://${MESH_COLL}/A1R1/A1R1_T7_wristYaw.dae" />
 	      </geometry>
       </collision>

File: trunk/m3_description/urdf/A1R1_r_arm_defs.urdf.xacro (robot description, xacro)
@@ -29,5 +29,5 @@
 	      <origin xyz="0 0 0" rpy="0 0 0 " />
 	      <geometry name="r_shoulder_geom">
-		      <mesh filename="package://${MESH}/A2R2/A2R2_shoulderupper_RIGHT.mesh" />
+		      <mesh filename="package://${MESH}/A1R1/A1R1_RT1_shoulderRoll.dae" />
 	      </geometry>
       </visual>
@@ -35,5 +35,5 @@
 	      <origin xyz="0 0 0" rpy="0.0 0.0 0.0 " />
 	      <geometry name="r_shoulder_collision_geom">
-		      <box size="0.01 0.01 0.01" />
+		      <mesh filename="package://${MESH_COLL}/A1R1/A1R1_RT1_shoulderRoll.dae" />
 	      </geometry>
       </collision>
@@ -62,5 +62,5 @@
 	      <origin xyz="0 0 0" rpy="0 0 0 " />
 	      <geometry name="shoulderpitch_RIGHT">
-		      <mesh filename="package://${MESH}/A2R2/A2R2_shoulderpitch_RIGHT.mesh" />
+		      <mesh filename="package://${MESH}/A1R1/A1R1_RT2_shoulderPitch.dae" />
 	      </geometry>
       </visual>
@@ -68,5 +68,5 @@
 	      <origin xyz="0 0 0" rpy="0.0 0.0 0.0 " />
 	      <geometry name="shoulderpitch_RIGHT_collision">
-		      <box size="0.01 0.01 0.01" />
+		      <mesh filename="package://${MESH_COLL}/A1R1/A1R1_RT2_shoulderPitch.dae" />
 	      </geometry>
       </collision>
@@ -74,5 +74,5 @@
     <joint name="m3joint_${R_ARM}_j2" type="revolute">
       <axis xyz="0 0 -1" />
-      <origin xyz="0 -0.03175 -0.27857" rpy="0 0 0" />
+      <origin xyz="0 -0.03175 -0.278" rpy="0 0 0" />
       <parent link="shoulderpitch_RIGHT" />
       <child link="bicep_RIGHT"/>
@@ -95,5 +95,5 @@
 	      <origin xyz="0 0 0" rpy="0 0 0 " />
 	      <geometry name="bicep_RIGHT_geom">
-		      <mesh filename="package://${MESH}/A2R2/A2R2_bicep_RIGHT.mesh" />
+		      <mesh filename="package://${MESH}/A1R1/A1R1_RT3_bicep.dae" />
 	      </geometry>
       </visual>
@@ -101,5 +101,5 @@
 	      <origin xyz="0 0 0" rpy="0.0 0.0 0.0 " />
 	      <geometry name="bicep_RIGHT_geom_collision">
-		      <box size="0.01 0.01 0.01" />
+		      <mesh filename="package://${MESH_COLL}/A1R1/A1R1_RT3_bicep.dae" />
 	      </geometry>
       </collision>
@@ -110,5 +110,5 @@
 	  <joint name="m3joint_${R_ARM}_j3" type="revolute">
 		  <axis xyz="0 -1 0" />
-		  <origin xyz="0.00502 0  0" rpy="0 0 0" />
+		  <origin xyz="0.00635 0  0" rpy="0 0 0" />
       <parent link="${parent}"/>
       <child link="elbowclevis_RIGHT"/>
@@ -131,5 +131,5 @@
 	      <origin xyz="0 0 0" rpy="0 0 0 " />
 	      <geometry name="elbowclevis_RIGHT_geom">
-		      <mesh filename="package://${MESH}/A2R2/A2R2_elbowclevis_RIGHT.mesh" />
+		      <mesh filename="package://${MESH}/A1R1/A1R1_RT4_elbow.dae" />
 	      </geometry>
       </visual>
@@ -137,5 +137,5 @@
 	      <origin xyz="0 0 0" rpy="0.0 0.0 0.0 " />
 	      <geometry name="elbowclevis_RIGHT_collision">
-		      <box size="0.01 0.01 0.01" />
+		      <mesh filename="package://${MESH_COLL}/A1R1/A1R1_RT4_elbow.dae" />
 	      </geometry>
       </collision>
@@ -164,5 +164,5 @@
 	      <origin xyz="0 0 0" rpy="0 0 0 " />
 	      <geometry name="wrist_RIGHT_geom">
-		      <mesh filename="package://${MESH}/A2R2/A2R2_wrist.mesh" />
+		      <mesh filename="package://${MESH}/A1R1/A1R1_RT5_forearmRoll.dae" />
 	      </geometry>
       </visual>
@@ -170,5 +170,5 @@
 	      <origin xyz="0 0 0" rpy="0.0 0.0 0.0 " />
 	      <geometry name="wrist_RIGHT_collision">
-		      <box size="0.01 0.01 0.01" />
+		      <mesh filename="package://${MESH_COLL}/A1R1/A1R1_RT5_forearmRoll.dae" />
 	      </geometry>
       </collision>
@@ -198,5 +198,5 @@
 	      <origin xyz="0 0 0" rpy="0 0 0 " />
 	      <geometry name="w_differential_RIGHT_geom">
-		      <mesh filename="package://${MESH}/A2R2/A2R2_w_differential.mesh" />
+		      <box size="0.01 0.01 0.01" />
 	      </geometry>
       </visual>
@@ -228,5 +228,5 @@
 	      <origin xyz="0 0 0" rpy="0 0 0 " />
 	      <geometry name="handmount_RIGHT_geom">
-		      <mesh filename="package://${MESH}/A2R2/A2R2_handmount.mesh" />
+		       <mesh filename="package://${MESH}/A1R1/A1R1_T7_wristYaw.dae" />
 	      </geometry>
       </visual>
@@ -234,5 +234,5 @@
 	      <origin xyz="0 0 0" rpy="0.0 0.0 0.0 " />
 	      <geometry name="handmount_RIGHT_collision">
-		      <box size="0.01 0.01 0.01" />
+		      <mesh filename="package://${MESH_COLL}/A1R1/A1R1_T7_wristYaw.dae" />
 	      </geometry>
       </collision>
