Commit message: git-svn-id: file:///home/svn/meka-ros-pkg@108 cfd446f6-b9c6-49ad-a440-209cd04d0f1d

File: trunk/meka_description/urdf/A2R3_r_arm_defs.urdf.xacro (robot description, xacro)
@@ -4,26 +4,4 @@
        xmlns:interface="http://playerstage.sourceforge.net/gazebo/xmlschema/#interface">
   <property name="M_PI" value="3.1415926535897931" />
-  <property name="VELOCITY_LIMIT_SCALE" value="0.6" />
-  <property name="shoulder_lift_length" value="0.10" />
-  <property name="shoulder_lift_radius" value="0.12" />
-  <!-- for non-symmetric upper arm -->
-  <property name="uar_xyz1" value= "0.21398" />
-  <property name="uar_xyz2" value="-0.01621" />
-  <property name="uar_xyz3" value="-0.00020" />
-  <property name="uar_ixx"  value= "0.01537748957" />
-  <property name="uar_ixy"  value= "0.00375711247" />
-  <property name="uar_ixz"  value="-0.00070852914" />
-  <property name="uar_iyy"  value= "0.07473670440" />
-  <property name="uar_iyz"  value="-0.00017936450" />
-  <property name="uar_izz"  value= "0.07608763307" />
-  <property name="ual_xyz1" value= "0.21405" />
-  <property name="ual_xyz2" value= "0.01658" />
-  <property name="ual_xyz3" value="-0.00057" />
-  <property name="ual_ixx"  value= "0.01530603856" />
-  <property name="ual_ixy"  value="-0.00339324862" />
-  <property name="ual_ixz"  value= "0.00060765455" />
-  <property name="ual_iyy"  value= "0.07473694455" />
-  <property name="ual_iyz"  value="-0.00019953729" />
-  <property name="ual_izz"  value= "0.07601594191" />
   <macro name="m3_r_shoulder" params="side parent reflect *origin">
     <!-- Shoulder pan -->
@@ -33,19 +11,17 @@
       <parent link="${parent}"/>
       <child link="shoulderupper_RIGHT"/>
-      <limit lower="${reflect*M_PI/4-1.5}"  upper="${reflect*M_PI/4+1.5}"
-             effort="30" velocity="${VELOCITY_LIMIT_SCALE*3.48}" />
-      <dynamics damping="10.0" />
-      <safety_controller k_position="100" k_velocity="10"
-                         soft_lower_limit="${reflect*M_PI/4-1.5+0.15}"
-                         soft_upper_limit="${reflect*M_PI/4+1.5-0.15}" />
-      <!-- joint angle when the rising or the falling flag is activated on PR2 -->
+      <limit effort="40" velocity="${30.0*M_PI/180}" lower="${-80*M_PI/180}" upper="${200*M_PI/180}" />
+      <dynamics damping="1.0"/>
     </joint>
     <link name="shoulderupper_RIGHT">
       <inertial>
-        <mass value="25.799322" />
-        <origin xyz="-0.001201 0.024513 -0.098231" rpy="0 0 0"/>
-        <inertia ixx="0.866179142480"  ixy="-0.06086507933"  ixz="-0.12118061183"
-                 iyy="0.87421714893"  iyz="-0.05886609911"
-                 izz="0.27353821674" />
+        <mass value="2.0310" />
+	<origin xyz="-0.010946 0.025127 0.000022"/>
+	<inertia ixx="0.003461"
+	iyy="0.003097"
+	izz="0.005416"
+	ixy="0.000428"
+	ixz="0.000002"
+	iyz="0.000000" />
       </inertial>
       <visual>
@@ -53,5 +29,5 @@
 	      <origin xyz="0 0 0" rpy="0 0 0 " />
 	      <geometry name="r_shoulder_geom">
-		      <mesh filename="package://${MESH}/A2R3/A2R3_shoulderupper_RIGHT.mesh" />
+		      <mesh filename="package://${MESH}/A2R3/A2R3_RT1_shoulderRoll.dae" />
 	      </geometry>
       </visual>
@@ -59,28 +35,26 @@
 	      <origin xyz="0 0 0" rpy="0.0 0.0 0.0 " />
 	      <geometry name="r_shoulder_collision_geom">
-		      <box size="0.01 0.01 0.01" />
-	      </geometry>
-      </collision>
-    </link>
-    <!-- Shoulder lift -->
+		      <mesh filename="package://${MESH_COLL}/A2R3/A2R3_RT1_shoulderRoll.stl" />
+	      </geometry>
+      </collision>
+    </link>
     <joint name="m3joint_${R_ARM}_j1" type="revolute">
       <axis xyz="-1 0 0"/>
-      <!-- Limits updated from Function's CAD values as of 2009_02_24 (link_data.xls) -->
-      <limit lower="-0.5236" upper="1.3963"
-             effort="30" velocity="${VELOCITY_LIMIT_SCALE*3.47}" />
-      <safety_controller k_position="100" k_velocity="10"
-                         soft_lower_limit="${-0.5236+0.17}" soft_upper_limit="${1.3963-0.05}" />
-      <dynamics damping="10.0" />
+     <limit effort="40" velocity="${30*M_PI/180}" lower="${-24*M_PI/180}" upper="${150*M_PI/180}" />
       <origin xyz="0 0 0" rpy="0 0 0" />
       <parent link="shoulderupper_RIGHT"/>
       <child link="shoulderpitch_RIGHT"/>
+      <dynamics damping="1.0"/>
     </joint>
     <link name="shoulderpitch_RIGHT">
       <inertial>
-        <mass value="2.74988" />
-        <origin xyz="0.02195 -0.02664 -0.03127" rpy="0 0 0"/>
-        <inertia ixx="0.02105584615" ixy="0.00496704022"  ixz="-0.00194808955"
-                 iyy="0.02127223737" iyz="0.00110425490"
-                 izz="0.01975753814" />
+        <mass value="0.566" />
+        <origin xyz="0.000944 -0.026331 -0.043257"/>
+	<inertia ixx="0.000754"
+	iyy="0.000921"
+	izz="0.000834"
+	ixy="0.000015"
+	ixz="0.000014"
+	iyz="0.000142" />
       </inertial>
       <visual>
@@ -88,5 +62,5 @@
 	      <origin xyz="0 0 0" rpy="0 0 0 " />
 	      <geometry name="shoulderpitch_RIGHT">
-		      <mesh filename="package://${MESH}/A2R3/A2R3_shoulderpitch_RIGHT.mesh" />
+		      <mesh filename="package://${MESH}/A2R3/A2R3_RT2_shoulderPitch.dae" />
 	      </geometry>
       </visual>
@@ -94,9 +68,8 @@
 	      <origin xyz="0 0 0" rpy="0.0 0.0 0.0 " />
 	      <geometry name="shoulderpitch_RIGHT_collision">
-		      <box size="0.01 0.01 0.01" />
-	      </geometry>
-      </collision>
-    </link>
-    <!-- Upperarm roll: internal fixed attchment point for upper arm -->
+		      <mesh filename="package://${MESH_COLL}/A2R3/A2R3_RT2_shoulderPitch.stl" />
+	      </geometry>
+      </collision>
+    </link>
     <joint name="m3joint_${R_ARM}_j2" type="revolute">
       <axis xyz="0 0 -1" />
@@ -104,16 +77,17 @@
       <parent link="shoulderpitch_RIGHT" />
       <child link="bicep_RIGHT"/>
-      <limit lower="${reflect*1.55-2.35}" upper="${reflect*1.55+2.35}" effort="30" velocity="${VELOCITY_LIMIT_SCALE*5.45}" />
-      <safety_controller k_position="100" k_velocity="2" soft_lower_limit="${reflect*1.55-2.35+0.15}" soft_upper_limit="${reflect*1.55+2.35-0.15}" />
-      <dynamics damping="0.1" />
+      <limit effort="20" velocity="${50*M_PI/180}" lower="${-85*M_PI/180}" upper="${85*M_PI/180}" />
+      <dynamics damping="1.0"/>
     </joint>
     <link name="bicep_RIGHT">
       <inertial>
-        <!-- dummy mass, to be removed -->
-        <mass value="0.1" />
-        <origin xyz="0.0 0 0" rpy="0 0 0" />
-        <inertia  ixx="0.01" ixy="0.00"  ixz="0.00"
-                  iyy="0.01" iyz="0.00"
-                  izz="0.01" />
+        <mass value="2.296" />
+        <origin xyz="-0.005767 0.084539 0.001385"/>
+	<inertia ixx="0.013031"
+	iyy="0.002070"
+	izz="0.013173"
+	ixy="-0.000564"
+	ixz="-0.000077"
+	iyz="0.000162" />
       </inertial>
       <visual>
@@ -121,5 +95,5 @@
 	      <origin xyz="0 0 0" rpy="0 0 0 " />
 	      <geometry name="bicep_RIGHT_geom">
-		      <mesh filename="package://${MESH}/A2R3/A2R3_bicep_RIGHT.mesh" />
+		      <mesh filename="package://${MESH}/A2R3/A2R3_RT3_bicep.dae" />
 	      </geometry>
       </visual>
@@ -127,5 +101,5 @@
 	      <origin xyz="0 0 0" rpy="0.0 0.0 0.0 " />
 	      <geometry name="bicep_RIGHT_geom_collision">
-		      <box size="0.01 0.01 0.01" />
+		      <mesh filename="package://${MESH_COLL}/A2R3/A2R3_RT3_bicep.stl" />
 	      </geometry>
       </collision>
@@ -139,18 +113,17 @@
       <parent link="${parent}"/>
       <child link="elbowclevis_RIGHT"/>
-	<limit lower="${reflect*M_PI/4-1.5}"  upper="${reflect*M_PI/4+1.5}"
-             effort="30" velocity="${VELOCITY_LIMIT_SCALE*3.48}" />
+	<limit effort="20" velocity="${50*M_PI/180}" lower="${ 0.182*M_PI/180}" upper="${132.8175*M_PI/180}" />
+      <dynamics damping="10.0" />
     </joint>
     <link name="elbowclevis_RIGHT">
       <inertial>
-        <!-- NOTE:reflect==-1 for right side, reflect==1 for the left side -->
-        <mass value="6.01769" />
-        <origin xyz="${0.5*((reflect+1)*ual_xyz1+(1-reflect)*uar_xyz1)} ${0.5*((reflect+1)*ual_xyz2+(1-reflect)*uar_xyz2)} ${0.5*((reflect+1)*ual_xyz3+(1-reflect)*uar_xyz3)}" />
-        <inertia  ixx="${0.5*((reflect+1)*ual_ixx+(1-reflect)*uar_ixx)}"
-                  ixy="${0.5*((reflect+1)*ual_ixy+(1-reflect)*uar_ixy)}"
-                  ixz="${0.5*((reflect+1)*ual_ixz+(1-reflect)*uar_ixz)}"
-                  iyy="${0.5*((reflect+1)*ual_iyy+(1-reflect)*uar_iyy)}"
-                  iyz="${0.5*((reflect+1)*ual_iyz+(1-reflect)*uar_iyz)}"
-                  izz="${0.5*((reflect+1)*ual_izz+(1-reflect)*uar_izz)}" />
+        <mass value="0.223" />
+        <origin xyz="-0.000002 0.000278 -0.026124"/>
+	<inertia ixx="0.000470"
+	iyy="0.000233"
+	izz="0.000425"
+	ixy="0.000000"
+	ixz="0.000000"
+	iyz="0.000019" />
       </inertial>
       <visual>
@@ -158,5 +131,5 @@
 	      <origin xyz="0 0 0" rpy="0 0 0 " />
 	      <geometry name="elbowclevis_RIGHT_geom">
-		      <mesh filename="package://${MESH}/A2R3/A2R3_elbowclevis_RIGHT.mesh" />
+		      <mesh filename="package://${MESH}/A2R3/A2R3_RT4_elbow.dae" />
 	      </geometry>
       </visual>
@@ -164,25 +137,26 @@
 	      <origin xyz="0 0 0" rpy="0.0 0.0 0.0 " />
 	      <geometry name="elbowclevis_RIGHT_collision">
-		      <box size="0.01 0.01 0.01" />
-	      </geometry>
-      </collision>
-    </link>
-    <!-- Elbow flex -->
+		      <mesh filename="package://${MESH_COLL}/A2R3/A2R3_RT4_elbow.stl" />
+	      </geometry>
+      </collision>
+    </link>
     <joint name="m3joint_${R_ARM}_j4" type="revolute">
 	    <axis xyz="0 0 -1" />
-      <limit lower="-2.3" upper="0.1" effort="30" velocity="${VELOCITY_LIMIT_SCALE*5.5}" />
-      <safety_controller k_position="100" k_velocity="3" soft_lower_limit="${-2.3+0.25}" soft_upper_limit="${0.1-0.1}" />
-      <dynamics damping="1.0" />
+      <limit effort="4" velocity="${150*M_PI/180}" lower="${-49.4*M_PI/180}" upper="${229.4*M_PI/180}" />
       <origin xyz="0 0 -0.27747" rpy="0 0 0" />
       <parent link="elbowclevis_RIGHT"/>
       <child link="wrist_RIGHT"/>
+      <dynamics damping="1.0"/>
     </joint>
     <link name="wrist_RIGHT">
       <inertial>
-        <mass value="1.90327" />
-        <origin xyz="0.01014 0.00032 -0.01211" />
-        <inertia  ixx="0.00346541989" ixy="0.00004066825"  ixz="0.00043171614"
-                  iyy="0.00441606455"  iyz="-0.00003968914"
-                  izz="0.00359156824" />
+        <mass value="1.468" />
+        <origin xyz="-0.004404 0.000124 0.130931"/>
+	<inertia ixx="0.006099"
+	iyy="0.006120"
+	izz="0.001179"
+	ixy="0.000004"
+	ixz="-0.000043"
+	iyz="0.000015" />
       </inertial>
       <visual>
@@ -190,5 +164,5 @@
 	      <origin xyz="0 0 0" rpy="0 0 0 " />
 	      <geometry name="wrist_RIGHT_geom">
-		      <mesh filename="package://${MESH}/A2R3/A2R3_wrist.mesh" />
+		      <mesh filename="package://${MESH}/A2R3/A2R3_T5_forearmRoll.dae" />
 	      </geometry>
       </visual>
@@ -196,5 +170,5 @@
 	      <origin xyz="0 0 0" rpy="0.0 0.0 0.0 " />
 	      <geometry name="wrist_RIGHT_collision">
-		      <box size="0.01 0.01 0.01" />
+		      <mesh filename="package://${MESH_COLL}/A2R3/A2R3_T5_forearmRoll.stl" />
 	      </geometry>
       </collision>
@@ -204,18 +178,19 @@
   <macro name="m3_r_forearm" params="side parent reflect">
 	  <joint name="m3joint_${R_ARM}_j5" type="revolute">
+      <dynamics damping="1.0" />
 		  <axis xyz="0 -1 0" />
       <origin xyz="0 0 0" rpy="0 0 0" />
       <parent link="${parent}"/>
       <child link="w_differential_RIGHT"/>
-	<limit lower="${reflect*M_PI/4-1.5}"  upper="${reflect*M_PI/4+1.5}"
-             effort="30" velocity="${VELOCITY_LIMIT_SCALE*3.48}" />
+	<limit effort="8" velocity="${40*M_PI/180}" lower="${-58.83*M_PI/180}" upper="${58.83*M_PI/180}" />
+      <dynamics damping="1.0"/>
     </joint>
     <link name="w_differential_RIGHT">
       <inertial>
-        <mass value="2.57968" />
-        <origin xyz="0.18791 -0.00017 -0.00912" />
-        <inertia ixx="0.00364857222" ixy="0.00005215877" ixz="0.00071534842"
-                 iyy="0.01507736897" iyz="-0.00001310770"
-                 izz="0.01659310749" />
+        <mass value="0.278" />
+        <origin xyz="0 0 0" />
+        <inertia ixx="0" ixy="0" ixz="0"
+                 iyy="0" iyz="0"
+                 izz="0" />
       </inertial>
       <visual>
@@ -223,5 +198,5 @@
 	      <origin xyz="0 0 0" rpy="0 0 0 " />
 	      <geometry name="w_differential_RIGHT_geom">
-		      <mesh filename="package://${MESH}/A2R3/A2R3_w_differential.mesh" />
+		      <mesh filename="package://${MESH}/A2R3/A2R3_T6_wristDiff.dae" />
 	      </geometry>
       </visual>
@@ -233,21 +208,19 @@
       </collision>
     </link>
-    <!-- Wrist flex -->
     <joint name="m3joint_${R_ARM}_j6" type="revolute">
 	    <axis xyz="-1 0 0" />
-      <limit lower="-0.1" upper="2.2" effort="200" velocity="${VELOCITY_LIMIT_SCALE*5.13}" />
-      <safety_controller k_position="20" k_velocity="4" soft_lower_limit="${-0.1+0.2}" soft_upper_limit="${2.2-0.2}" />
-      <dynamics damping="0.1" />
+      <limit effort="8" velocity="${40*M_PI/180}" lower="${-60*M_PI/180}" upper="${60*M_PI/180}" />
       <origin xyz="0 0 0" rpy="0 0 0" />
       <parent link="w_differential_RIGHT"/>
       <child link="handmount_RIGHT"/>
+      <dynamics damping="1.0"/>
     </joint>
     <link name="handmount_RIGHT">
       <inertial>
-        <mass value="0.61402" />
-        <origin xyz="-0.00157 0.0 -0.00075" />
-        <inertia ixx="0.00065165722" ixy="0.00000028864" ixz="0.00000303477"
-                 iyy="0.00019824443" iyz="-0.00000022645"
-                 izz="0.00064450498" />
+        <mass value="0.093" />
+        <origin xyz="0 0 0" />
+        <inertia ixx="0" ixy="0" ixz="0"
+                 iyy="0" iyz="0"
+                 izz="0" />
       </inertial>
       <visual>
@@ -255,5 +228,5 @@
 	      <origin xyz="0 0 0" rpy="0 0 0 " />
 	      <geometry name="handmount_RIGHT_geom">
-		      <mesh filename="package://${MESH}/A2R3/A2R3_handmount.mesh" />
+		       <mesh filename="package://${MESH}/A2R3/A2R3_T7_wristYaw.dae" />
 	      </geometry>
       </visual>
@@ -261,5 +234,5 @@
 	      <origin xyz="0 0 0" rpy="0.0 0.0 0.0 " />
 	      <geometry name="handmount_RIGHT_collision">
-		      <box size="0.01 0.01 0.01" />
+		      <mesh filename="package://${MESH_COLL}/A2R3/A2R3_T7_wristYaw.stl" />
 	      </geometry>
       </collision>

Commit message: git-svn-id: file:///home/svn/meka-ros-pkg@130 cfd446f6-b9c6-49ad-a440-209cd04d0f1d

File: trunk/meka_description/urdf/A2R3_r_arm_defs.urdf.xacro (robot description, xacro)
@@ -113,5 +113,5 @@
       <parent link="${parent}"/>
       <child link="elbowclevis_RIGHT"/>
-	<limit effort="20" velocity="${50*M_PI/180}" lower="${ 0.182*M_PI/180}" upper="${132.8175*M_PI/180}" />
+	<limit effort="20" velocity="${50*M_PI/180}" lower="${-0.278978*M_PI/180}" upper="${132.8175*M_PI/180}" />
       <dynamics damping="10.0" />
     </joint>
