Commit message: git-svn-id: file:///home/svn/meka-ros-pkg@141 cfd446f6-b9c6-49ad-a440-209cd04d0f1d

File: trunk/meka_description/urdf/Z1R2_defs.urdf.xacro (robot description, xacro)
@@ -7,5 +7,5 @@
     <!-- Shoulder pan -->
     <joint name="zlift_z" type="prismatic">
-      <axis xyz="0 1 0" />
+      <axis xyz="0 0 1" />
       <insert_block name="origin" /> <!-- transform from parent link to this joint frame -->
       <parent link="${parent}"/>
