Commit message: git-svn-id: file:///home/svn/meka-ros-pkg@149 cfd446f6-b9c6-49ad-a440-209cd04d0f1d

File: trunk/meka_description/urdf/H2R4_l_hand_defs.urdf.xacro (robot description, xacro)
@@ -4,11 +4,11 @@
        xmlns:interface="http://playerstage.sourceforge.net/gazebo/xmlschema/#interface">
   <property name="M_PI" value="3.1415926535897931" />
-  <macro name="m3_r_palm" params="side parent reflect *origin">
-  <joint name="palm_joint" type="fixed">
+  <macro name="m3_l_palm" params="side parent reflect *origin">
+  <joint name="l_palm_joint" type="fixed">
     <origin xyz="0 0 -0.04414" rpy="0 0 0" />
     <parent link="${parent}"/>
-    <child link="palm" />
+    <child link="l_palm" />
   </joint>
-     <link name="palm">
+     <link name="l_palm">
       <inertial>
         <mass value="0.663" />
@@ -24,5 +24,5 @@
 	      <material name="GreyA" />
 	      <origin xyz="0 0 0" rpy="0 0 0 " />
-	      <geometry name="palm_geom">
+	      <geometry name="l_palm_geom">
 		      <mesh filename="package://${MESH}/H2R3/H2R3_RT8_palm_right.dae" />
 	      </geometry>
@@ -30,5 +30,5 @@
       <collision>
 	      <origin xyz="0 0 0" rpy="0.0 0.0 0.0 " />
-	      <geometry name="palm_collision">
+	      <geometry name="l_palm_collision">
 		      <mesh filename="package://${MESH_COLL}/H2R3/H2R3_RT8_palm_right.stl" />
 	      </geometry>
@@ -36,12 +36,12 @@
     </link>
 <!-- Start Thumb -->
-    <joint name="right_hand_j0" type="revolute">
+    <joint name="left_hand_j0" type="revolute">
       <axis xyz="0 0 -1" />
       <origin xyz="-0.02 0.028 -0.03" rpy="0 0 0" />
-      <parent link="palm"/>
-      <child link="thumb0"/>
+      <parent link="l_palm"/>
+      <child link="l_thumb0"/>
       <limit effort="100" velocity="${20.0*M_PI/180}" lower="${-40*M_PI/180}" upper="${15*M_PI/180}" />
     </joint>
-    <link name="thumb0">
+    <link name="l_thumb0">
       <inertial>
         <mass value="0.0117" />
@@ -57,5 +57,5 @@
 	      <material name="GreyA" />
 	      <origin xyz="0 0 0" rpy="0 0 0 " />
-	      <geometry name="thumb0_geom">
+	      <geometry name="l_thumb0_geom">
 		      <mesh filename="package://${MESH}/H2R3/H2R3_RJ0_thumb_abductlink.dae" />
 	      </geometry>
@@ -63,17 +63,17 @@
       <collision>
 	      <origin xyz="0 0 0" rpy="0.0 0.0 0.0 " />
-	      <geometry name="thumb0_collision">
+	      <geometry name="l_thumb0_collision">
 		      <mesh filename="package://${MESH_COLL}/H2R3/H2R3_RJ0_thumb_abductlink.stl" />
 	      </geometry>
       </collision>
     </link>
-    <joint name="right_hand_j1" type="revolute">
+    <joint name="left_hand_j1" type="revolute">
       <axis xyz="0 -1 0"/>
      <limit effort="100" velocity="${75*M_PI/180}" lower="${-80.919*M_PI/180}" upper="${80.91*M_PI/180}" />
       <origin xyz="-0.018 0 0" rpy="0 0 0" />
-      <parent link="thumb0"/>
-      <child link="thumb1"/>
-    </joint>
-    <link name="thumb1">
+      <parent link="l_thumb0"/>
+      <child link="l_thumb1"/>
+    </joint>
+    <link name="l_thumb1">
       <inertial>
         <mass value="0.0344" />
@@ -89,5 +89,5 @@
 	      <material name="GreyB" />
 	      <origin xyz="0 0 0" rpy="0 0 0 " />
-	      <geometry name="thumb1_geom">
+	      <geometry name="l_thumb1_geom">
 		      <mesh filename="package://${MESH}/H2R3/H2R3_thumb_knuckle1.dae" />
 	      </geometry>
@@ -95,31 +95,31 @@
       <collision>
 	      <origin xyz="0 0 0" rpy="0.0 0.0 0.0 " />
-	      <geometry name="thumb1_collision">
+	      <geometry name="l_thumb1_collision">
 		      <mesh filename="package://${MESH_COLL}/H2R3/H2R3_thumb_knuckle1.stl" />
 	      </geometry>
       </collision>
     </link>
-    <joint name="right_hand_j2" type="revolute">
+    <joint name="left_hand_j2" type="revolute">
       <axis xyz="0 -1 0" />
       <origin xyz="-0.044 0 0" rpy="0 0 0" />
-      <parent link="thumb1" />
-      <child link="thumb2"/>
+      <parent link="l_thumb1" />
+      <child link="l_thumb2"/>
       <limit effort="100" velocity="${50*M_PI/180}" lower="${-14.94*M_PI/180}" upper="${14.94*M_PI/180}" />
     </joint>
-    <link name="thumb2">
-      <inertial>
-        <mass value="0.01" />
-	<origin xyz="0.0 0.0 0.0"/>
-	<inertia ixx="0.0"
-	iyy="0.0"
-	izz="0.0"
-	ixy="0.0"
-	ixz="0.0"
-	iyz="0.0" />
-      </inertial>
-      <visual>
-	      <material name="GreyC" />
-	      <origin xyz="0 0 0" rpy="0 0 0 " />
-	      <geometry name="thumb_knuckle2_geom">
+    <link name="l_thumb2">
+      <inertial>
+        <mass value="0.01" />
+	<origin xyz="0.0 0.0 0.0"/>
+	<inertia ixx="0.0"
+	iyy="0.0"
+	izz="0.0"
+	ixy="0.0"
+	ixz="0.0"
+	iyz="0.0" />
+      </inertial>
+      <visual>
+	      <material name="GreyC" />
+	      <origin xyz="0 0 0" rpy="0 0 0 " />
+	      <geometry name="l_thumb_knuckle2_geom">
 		      <mesh filename="package://${MESH}/H2R3/H2R3_thumb_knuckle2.dae" />
 	      </geometry>
@@ -127,5 +127,5 @@
       <collision>
 	      <origin xyz="0 0 0" rpy="0.0 0.0 0.0 " />
-	      <geometry name="thumb_knuckle2_collision">
+	      <geometry name="l_thumb_knuckle2_collision">
 		      <mesh filename="package://${MESH_COLL}/H2R3/H2R3_thumb_knuckle2.stl" />
 	      </geometry>
@@ -133,12 +133,12 @@
     </link>
 <!-- Start Index Finger -->
-    <joint name="right_hand_j3" type="revolute">
+    <joint name="left_hand_j3" type="revolute">
       <axis xyz="0 1 0" />
       <origin xyz="0 0.028 -0.101" rpy="0 0 0" />
-      <parent link="palm" />
-      <child link="index0"/>
+      <parent link="l_palm" />
+      <child link="l_index0"/>
 	<limit effort="100" velocity="${50*M_PI/180}" lower="${-7.072*M_PI/180}" upper="${37.072*M_PI/180}" />
     </joint>
-    <link name="index0">
+    <link name="l_index0">
       <inertial>
         <mass value="0.01" />
@@ -154,5 +154,5 @@
 	      <material name="GreyA" />
 	      <origin xyz="0 0 0" rpy="0 0 0 " />
-	      <geometry name="index0_geom">
+	      <geometry name="l_index0_geom">
 		     <mesh filename="package://${MESH}/H2R3/H2R3_finger_knuckle1.dae" />
 	      </geometry>
@@ -160,17 +160,17 @@
       <collision>
 	      <origin xyz="0 0 0" rpy="0.0 0.0 0.0 " />
-	      <geometry name="index0__collision">
+	      <geometry name="l_index0__collision">
 		      <mesh filename="package://${MESH_COLL}/H2R3/H2R3_finger_knuckle1.stl" />
 	      </geometry>
       </collision>
     </link>
-    <joint name="right_hand_j4" type="revolute">
+    <joint name="left_hand_j4" type="revolute">
       <axis xyz="0 1 0" />
       <limit effort="100" velocity="${1600*M_PI/180}" lower="${-34.99*M_PI/180}" upper="${34.99*M_PI/180}" />
       <origin xyz="0 0 -0.044" rpy="0 0 0" />
-      <parent link="index0"/>
-      <child link="index1"/>
-    </joint>
-    <link name="index1">
+      <parent link="l_index0"/>
+      <child link="l_index1"/>
+    </joint>
+    <link name="l_index1">
       <inertial>
         <mass value="0.0429" />
@@ -186,5 +186,5 @@
 	      <material name="GreyC" />
 	      <origin xyz="0 0 0" rpy="0 0 0 " />
-	      <geometry name="index1_geom">
+	      <geometry name="l_index1_geom">
 		      <mesh filename="package://${MESH}/H2R3/H2R3_finger_knuckle2.dae" />
 	      </geometry>
@@ -192,31 +192,31 @@
       <collision>
 	      <origin xyz="0 0 0" rpy="0.0 0.0 0.0 " />
-	      <geometry name="index1_collision">
+	      <geometry name="l_index1_collision">
 		      <mesh filename="package://${MESH_COLL}/H2R3/H2R3_finger_knuckle2.stl" />
 	      </geometry>
       </collision>
     </link>
-    <joint name="right_hand_j5" type="revolute">
+    <joint name="left_hand_j5" type="revolute">
       <axis xyz="0 1 0" />
       <limit effort="100" velocity="${1600*M_PI/180}" lower="${-34.21*M_PI/180}" upper="${34.213*M_PI/180}" />
       <origin xyz="0 0 -0.032" rpy="0 0 0" />
-      <parent link="index1"/>
-      <child link="index2"/>
-    </joint>
-    <link name="index2">
-      <inertial>
-        <mass value="0.01" />
-	<origin xyz="0.0 0.0 0.0"/>
-	<inertia ixx="0.0"
-	iyy="0.0"
-	izz="0.0"
-	ixy="0.0"
-	ixz="0.0"
-	iyz="0.0" />
-      </inertial>
-      <visual>
-	      <material name="GreyC" />
-	      <origin xyz="0 0 0" rpy="0 0 0 " />
-	      <geometry name="index2_geom">
+      <parent link="l_index1"/>
+      <child link="l_index2"/>
+    </joint>
+    <link name="l_index2">
+      <inertial>
+        <mass value="0.01" />
+	<origin xyz="0.0 0.0 0.0"/>
+	<inertia ixx="0.0"
+	iyy="0.0"
+	izz="0.0"
+	ixy="0.0"
+	ixz="0.0"
+	iyz="0.0" />
+      </inertial>
+      <visual>
+	      <material name="GreyC" />
+	      <origin xyz="0 0 0" rpy="0 0 0 " />
+	      <geometry name="l_index2_geom">
 		      <mesh filename="package://${MESH}/H2R3/H2R3_finger_knuckle3.dae" />
 	      </geometry>
@@ -224,5 +224,5 @@
       <collision>
 	      <origin xyz="0 0 0" rpy="0.0 0.0 0.0 " />
-	      <geometry name="index2_collision">
+	      <geometry name="l_index2_collision">
 		      <mesh filename="package://${MESH_COLL}/H2R3/H2R3_finger_knuckle3.stl" />
 	      </geometry>
@@ -230,12 +230,12 @@
     </link>
 <!-- Start Ring Finger -->
-    <joint name="right_hand_j6" type="revolute">
+    <joint name="left_hand_j6" type="revolute">
       <axis xyz="0 1 0" />
       <origin xyz="0 0 -0.101" rpy="0 0 0" />
-      <parent link="palm" />
-      <child link="ring0"/>
+      <parent link="l_palm" />
+      <child link="l_ring0"/>
 	<limit effort="100" velocity="${50*M_PI/180}" lower="${-7.072*M_PI/180}" upper="${37.072*M_PI/180}" />
     </joint>
-    <link name="ring0">
+    <link name="l_ring0">
       <inertial>
         <mass value="0.01" />
@@ -251,5 +251,5 @@
 	      <material name="GreyA" />
 	      <origin xyz="0 0 0" rpy="0 0 0 " />
-	      <geometry name="ring0_geom">
+	      <geometry name="l_ring0_geom">
 		     <mesh filename="package://${MESH}/H2R3/H2R3_finger_knuckle1.dae" />
 	      </geometry>
@@ -257,17 +257,17 @@
       <collision>
 	      <origin xyz="0 0 0" rpy="0.0 0.0 0.0 " />
-	      <geometry name="ring0__collision">
+	      <geometry name="l_ring0__collision">
 		      <mesh filename="package://${MESH_COLL}/H2R3/H2R3_finger_knuckle1.stl" />
 	      </geometry>
       </collision>
     </link>
-    <joint name="right_hand_j7" type="revolute">
+    <joint name="left_hand_j7" type="revolute">
       <axis xyz="0 1 0" />
       <limit effort="100" velocity="${1600*M_PI/180}" lower="${-34.99*M_PI/180}" upper="${34.99*M_PI/180}" />
       <origin xyz="0 0 -0.044" rpy="0 0 0" />
-      <parent link="ring0"/>
-      <child link="ring1"/>
-    </joint>
-    <link name="ring1">
+      <parent link="l_ring0"/>
+      <child link="l_ring1"/>
+    </joint>
+    <link name="l_ring1">
       <inertial>
         <mass value="0.0429" />
@@ -283,5 +283,5 @@
 	      <material name="GreyC" />
 	      <origin xyz="0 0 0" rpy="0 0 0 " />
-	      <geometry name="ring1_geom">
+	      <geometry name="l_ring1_geom">
 		      <mesh filename="package://${MESH}/H2R3/H2R3_finger_knuckle2.dae" />
 	      </geometry>
@@ -289,31 +289,31 @@
       <collision>
 	      <origin xyz="0 0 0" rpy="0.0 0.0 0.0 " />
-	      <geometry name="ring1_collision">
+	      <geometry name="l_ring1_collision">
 		      <mesh filename="package://${MESH_COLL}/H2R3/H2R3_finger_knuckle2.stl" />
 	      </geometry>
       </collision>
     </link>
-    <joint name="right_hand_j8" type="revolute">
+    <joint name="left_hand_j8" type="revolute">
       <axis xyz="0 1 0" />
       <limit effort="100" velocity="${1600*M_PI/180}" lower="${-34.21*M_PI/180}" upper="${34.213*M_PI/180}" />
       <origin xyz="0 0 -0.032" rpy="0 0 0" />
-      <parent link="ring1"/>
-      <child link="ring2"/>
-    </joint>
-    <link name="ring2">
-      <inertial>
-        <mass value="0.01" />
-	<origin xyz="0.0 0.0 0.0"/>
-	<inertia ixx="0.0"
-	iyy="0.0"
-	izz="0.0"
-	ixy="0.0"
-	ixz="0.0"
-	iyz="0.0" />
-      </inertial>
-      <visual>
-	      <material name="GreyC" />
-	      <origin xyz="0 0 0" rpy="0 0 0 " />
-	      <geometry name="ring2_geom">
+      <parent link="l_ring1"/>
+      <child link="l_ring2"/>
+    </joint>
+    <link name="l_ring2">
+      <inertial>
+        <mass value="0.01" />
+	<origin xyz="0.0 0.0 0.0"/>
+	<inertia ixx="0.0"
+	iyy="0.0"
+	izz="0.0"
+	ixy="0.0"
+	ixz="0.0"
+	iyz="0.0" />
+      </inertial>
+      <visual>
+	      <material name="GreyC" />
+	      <origin xyz="0 0 0" rpy="0 0 0 " />
+	      <geometry name="l_ring2_geom">
 		      <mesh filename="package://${MESH}/H2R3/H2R3_finger_knuckle3.dae" />
 	      </geometry>
@@ -321,5 +321,5 @@
       <collision>
 	      <origin xyz="0 0 0" rpy="0.0 0.0 0.0 " />
-	      <geometry name="ring2_collision">
+	      <geometry name="l_ring2_collision">
 		      <mesh filename="package://${MESH_COLL}/H2R3/H2R3_finger_knuckle3.stl" />
 	      </geometry>
@@ -327,12 +327,12 @@
     </link>
 <!-- Start Pinky Finger -->
-    <joint name="right_hand_j9" type="revolute">
+    <joint name="left_hand_j9" type="revolute">
       <axis xyz="0 1 0" />
       <origin xyz="0 -0.028 -0.101" rpy="0 0 0" />
-      <parent link="palm" />
-      <child link="pinky0"/>
+      <parent link="l_palm" />
+      <child link="l_pinky0"/>
 	<limit effort="100" velocity="${50*M_PI/180}" lower="${-7.072*M_PI/180}" upper="${37.072*M_PI/180}" />
     </joint>
-    <link name="pinky0">
+    <link name="l_pinky0">
       <inertial>
         <mass value="0.01" />
@@ -348,5 +348,5 @@
 	      <material name="GreyA" />
 	      <origin xyz="0 0 0" rpy="0 0 0 " />
-	      <geometry name="pinky0_geom">
+	      <geometry name="l_pinky0_geom">
 		     <mesh filename="package://${MESH}/H2R3/H2R3_finger_knuckle1.dae" />
 	      </geometry>
@@ -354,17 +354,17 @@
       <collision>
 	      <origin xyz="0 0 0" rpy="0.0 0.0 0.0 " />
-	      <geometry name="pinky0__collision">
+	      <geometry name="l_pinky0__collision">
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
Commit message: git-svn-id: file:///home/svn/meka-ros-pkg@155 cfd446f6-b9c6-49ad-a440-209cd04d0f1d

File: trunk/meka_description/urdf/H2R4_l_hand_defs.urdf.xacro (robot description, xacro)
@@ -25,5 +25,5 @@
 	      <origin xyz="0 0 0" rpy="0 0 0 " />
 	      <geometry name="l_palm_geom">
-		      <mesh filename="package://${MESH}/H2R3/H2R3_RT8_palm_right.dae" />
+		      <mesh filename="package://${MESH}/H2R3/H2R3_LT8_palm_left.dae" />
 	      </geometry>
       </visual>
@@ -38,5 +38,5 @@
     <joint name="left_hand_j0" type="revolute">
       <axis xyz="0 0 -1" />
-      <origin xyz="-0.02 0.028 -0.03" rpy="0 0 0" />
+      <origin xyz="-0.02 -0.028 -0.03" rpy="0 0 0" />
       <parent link="l_palm"/>
       <child link="l_thumb0"/>
