Commit message: git-svn-id: file:///home/svn/meka-ros-pkg@171 cfd446f6-b9c6-49ad-a440-209cd04d0f1d

File: trunk/meka_description/urdf/A2R4_l_arm_defs.urdf.xacro (robot description, xacro)
@@ -33,6 +33,5 @@
       <parent link="${parent}"/>
       <child link="shoulderupper_LEFT"/>
-      <limit lower="${reflect*M_PI/4-1.5}"  upper="${reflect*M_PI/4+1.5}"
-             effort="30" velocity="${VELOCITY_LIMIT_SCALE*3.48}" />
+      <limit effort="40" velocity="${30.0*M_PI/180}" lower="${-80*M_PI/180}" upper="${200*M_PI/180}" />
       <dynamics damping="10.0" />
       <safety_controller k_position="100" k_velocity="10"
@@ -67,6 +66,5 @@
       <axis xyz="-1 0 0"/>
       <!-- Limits updated from Function's CAD values as of 2009_02_24 (link_data.xls) -->
-      <limit lower="-0.5236" upper="1.3963"
-             effort="30" velocity="${VELOCITY_LIMIT_SCALE*3.47}" />
+      <limit effort="40" velocity="${30*M_PI/180}" upper="${24*M_PI/180}"  lower="${-150*M_PI/180}" />
       <safety_controller k_position="100" k_velocity="10"
                          soft_lower_limit="${-0.5236+0.17}" soft_upper_limit="${1.3963-0.05}" />
@@ -104,5 +102,5 @@
       <parent link="shoulderpitch_LEFT" />
       <child link="bicep_LEFT"/>
-      <limit lower="${reflect*1.55-2.35}" upper="${reflect*1.55+2.35}" effort="30" velocity="${VELOCITY_LIMIT_SCALE*5.45}" />
+     <limit effort="20" velocity="${50*M_PI/180}" lower="${-85*M_PI/180}" upper="${85*M_PI/180}" />
       <safety_controller k_position="100" k_velocity="2" soft_lower_limit="${reflect*1.55-2.35+0.15}" soft_upper_limit="${reflect*1.55+2.35-0.15}" />
       <dynamics damping="0.1" />
@@ -139,6 +137,5 @@
       <parent link="${parent}"/>
       <child link="elbowclevis_LEFT"/>
-	<limit lower="${reflect*M_PI/4-1.5}"  upper="${reflect*M_PI/4+1.5}"
-             effort="30" velocity="${VELOCITY_LIMIT_SCALE*3.48}" />
+	<limit effort="20" velocity="${50*M_PI/180}" lower="${-0.278978*M_PI/180}" upper="${132.8175*M_PI/180}" />
     </joint>
     <link name="elbowclevis_LEFT">
@@ -171,5 +168,5 @@
     <joint name="left_arm_j4" type="revolute">
 	    <axis xyz="0 0 -1" />
-      <limit lower="-2.3" upper="0.1" effort="30" velocity="${VELOCITY_LIMIT_SCALE*5.5}" />
+     <limit effort="4" velocity="${150*M_PI/180}" lower="${-190.7*M_PI/180}" upper="${19.7*M_PI/180}" />
       <safety_controller k_position="100" k_velocity="3" soft_lower_limit="${-2.3+0.25}" soft_upper_limit="${0.1-0.1}" />
       <dynamics damping="1.0" />
@@ -208,6 +205,5 @@
       <parent link="${parent}"/>
       <child link="w_differential_LEFT"/>
-	<limit lower="${reflect*M_PI/4-1.5}"  upper="${reflect*M_PI/4+1.5}"
-             effort="30" velocity="${VELOCITY_LIMIT_SCALE*3.48}" />
+	<limit effort="8" velocity="${40*M_PI/180}" lower="${-58.83*M_PI/180}" upper="${58.83*M_PI/180}" />
     </joint>
     <link name="w_differential_LEFT">
@@ -236,5 +232,5 @@
     <joint name="left_arm_j6" type="revolute">
 	    <axis xyz="-1 0 0" />
-      <limit lower="-0.1" upper="2.2" effort="200" velocity="${VELOCITY_LIMIT_SCALE*5.13}" />
+      <limit effort="8" velocity="${40*M_PI/180}" lower="${-60*M_PI/180}" upper="${60*M_PI/180}" />
       <safety_controller k_position="20" k_velocity="4" soft_lower_limit="${-0.1+0.2}" soft_upper_limit="${2.2-0.2}" />
       <dynamics damping="0.1" />

File: trunk/meka_description/urdf/A2R4_r_arm_defs.urdf.xacro (robot description, xacro)
@@ -143,5 +143,5 @@
     <joint name="right_arm_j4" type="revolute">
 	    <axis xyz="0 0 -1" />
-      <limit effort="4" velocity="${150*M_PI/180}" lower="${-49.4*M_PI/180}" upper="${229.4*M_PI/180}" />
+      <limit effort="4" velocity="${150*M_PI/180}" lower="${-19.7*M_PI/180}" upper="${199.7*M_PI/180}" />
       <origin xyz="0 0 -0.27747" rpy="0 0 0" />
       <parent link="elbowclevis_RIGHT"/>
@@ -177,5 +177,5 @@
   <!-- ============================   Forearm   ============================ -->
   <macro name="m3_r_forearm" params="side parent reflect">
-	  <joint name="right_arm_j5" type="revolute">
+    <joint name="right_arm_j5" type="revolute">
       <dynamics damping="1.0" />
 		  <axis xyz="0 -1 0" />

File: trunk/meka_description/urdf/Z1R2B_defs.urdf.xacro (robot description, xacro)
@@ -11,5 +11,5 @@
       <parent link="${parent}"/>
       <child link="zlift_link"/>
-      <limit lower="${reflect*M_PI/4-1.5}"  upper="${reflect*M_PI/4+1.5}"
+      <limit lower="${0.0*M_PI/180.0}"  upper="${31965.0*M_PI/180.0}"
              effort="30" velocity="${3.48}" />
       <dynamics damping="10.0" />
