Commit message: git-svn-id: file:///home/svn/meka-ros-pkg@154 cfd446f6-b9c6-49ad-a440-209cd04d0f1d

File: trunk/meka_description/robots/m1.urdf.xacro (robot description, xacro)
@@ -20,5 +20,5 @@
   <!-- Meka Hand -->
   <include filename="$(find meka_description)/urdf/H2R4_r_hand_defs.urdf.xacro" />
-  <!--<include filename="$(find meka_description)/urdf/H2R4_l_hand_defs.urdf.xacro" />-->
+  <include filename="$(find meka_description)/urdf/H2R4_l_hand_defs.urdf.xacro" />
 <!-- Meka Head -->
   <include filename="$(find meka_description)/urdf/S2R1B_head_defs.urdf.xacro" />
@@ -43,4 +43,7 @@
     <origin xyz="0.0 0.0 0.0" rpy="0 0 0" />
   </m3_r_hand>
+  <m3_l_hand side="l" reflect="1" parent="handmount_LEFT">
+    <origin xyz="0.0 0.0 0.0" rpy="0 0 0" />
+  </m3_l_hand>
   <m3_head side="r" reflect="1" parent="upper">
     <origin xyz="0.0 0.0 0.31155" rpy="0 0 0" />
@@ -49,7 +52,10 @@
     <origin xyz="0.0 -0.18465 0.2337" rpy="0 0 0" />
   </m3_r_arm>
+ <m3_l_arm side="l" reflect="1" parent="upper">
+    <origin xyz="0.0 0.18465 0.2337" rpy="0 0 0" />
+  </m3_l_arm>
   <link name="world" />
   <link name="base_link" />
-<!-- Solid Base -->
+  <!-- Solid Base -->
   <joint name="base_joint" type="fixed">
 	  <origin xyz="0 0 1" rpy="0 0 0" />

File: trunk/meka_description/urdf/A2R4_l_arm_defs.urdf.xacro (robot description, xacro)
@@ -51,13 +51,13 @@
       <visual>
 	      <material name="GreyA" />
-	      <origin xyz="0 0 0" rpy="0 0 0 " />
+	      <origin xyz="0 0 0" rpy="3.14 0 0 " />
 	      <geometry name="l_shoulder_geom">
-		      <mesh filename="package://${MESH}/A2R3/A2R3_shoulderupper_LEFT.mesh" />
-	      </geometry>
-      </visual>
-      <collision>
-	      <origin xyz="0 0 0" rpy="0.0 0.0 0.0 " />
+		      <mesh filename="package://${MESH}/A2R3/A2R3_RT1_shoulderRoll.dae" />
+	      </geometry>
+      </visual>
+      <collision>
+	      <origin xyz="0 0 0" rpy="3.14 0.0 0.0 " />
 	      <geometry name="l_shoulder_collision_geom">
-		      <box size="0.01 0.01 0.01" />
+		      <mesh filename="package://${MESH_COLL}/A2R3/A2R3_RT1_shoulderRoll.stl" />
 	      </geometry>
       </collision>
@@ -86,17 +86,17 @@
       <visual>
 	      <material name="GreyB" />
-	      <origin xyz="0 0 0" rpy="0 0 0 " />
-	      <geometry name="shoulderpitch_LEFT">
-		      <mesh filename="package://${MESH}/A2R3/A2R3_shoulderpitch_LEFT.mesh" />
-	      </geometry>
-      </visual>
-      <collision>
-	      <origin xyz="0 0 0" rpy="0.0 0.0 0.0 " />
-	      <geometry name="shoulderpitch_LEFT_collision">
-		      <box size="0.01 0.01 0.01" />
-	      </geometry>
-      </collision>
-    </link>
-    <!-- Upperarm roll: internal fixed attchment point for upper arm -->
+	      <origin xyz="0 0 0" rpy="0 0 3.14" />
+	      <geometry name="l_shoulderpitch_RIGHT">
+		      <mesh filename="package://${MESH}/A2R3/A2R3_RT2_shoulderPitch.dae" />
+	      </geometry>
+      </visual>
+      <collision>
+	      <origin xyz="0 0 0" rpy="0.0 0.0 3.14" />
+	      <geometry name="l_shoulderpitch_RIGHT_collision">
+		      <mesh filename="package://${MESH_COLL}/A2R3/A2R3_RT2_shoulderPitch.stl" />
+	      </geometry>
+      </collision>
+    </link>
+ <!-- Upperarm roll: internal fixed attchment point for upper arm -->
     <joint name="left_arm_j2" type="revolute">
       <axis xyz="0 0 -1" />
@@ -120,12 +120,12 @@
 	      <material name="GreyC" />
 	      <origin xyz="0 0 0" rpy="0 0 0 " />
-	      <geometry name="bicep_l_geom">
-		      <mesh filename="package://${MESH}/A2R3/A2R3_bicep_LEFT.mesh" />
-	      </geometry>
-      </visual>
-      <collision>
-	      <origin xyz="0 0 0" rpy="0.0 0.0 0.0 " />
-	      <geometry name="bicep_l_geom_collision">
-		      <box size="0.01 0.01 0.01" />
+	      <geometry name="bicep_LEFT_geom">
+		      <mesh filename="package://${MESH}/A2R3/A2R3_LT3_bicep.dae" />
+	      </geometry>
+      </visual>
+      <collision>
+	      <origin xyz="0 0 0" rpy="0.0 0.0 0.0 " />
+	      <geometry name="bicep_LEFT_geom_collision">
+		      <mesh filename="package://${MESH_COLL}/A2R3/A2R3_LT3_bicep.stl" />
 	      </geometry>
       </collision>
@@ -157,12 +157,12 @@
 	      <material name="GreyA" />
 	      <origin xyz="0 0 0" rpy="0 0 0 " />
-	      <geometry name="elbowclevis_l_geom">
-		      <mesh filename="package://${MESH}/A2R3/A2R3_elbowclevis_LEFT.mesh" />
-	      </geometry>
-      </visual>
-      <collision>
-	      <origin xyz="0 0 0" rpy="0.0 0.0 0.0 " />
-	      <geometry name="elbowclevis_l_collision">
-		      <box size="0.01 0.01 0.01" />
+	      <geometry name="elbowclevis_LEFT_geom">
+		      <mesh filename="package://${MESH}/A2R3/A2R3_LT4_elbow.dae" />
+	      </geometry>
+      </visual>
+      <collision>
+	      <origin xyz="0 0 0" rpy="0.0 0.0 0.0 " />
+	      <geometry name="elbowclevis_LEFT_collision">
+		      <mesh filename="package://${MESH_COLL}/A2R3/A2R3_RT4_elbow.stl" />
 	      </geometry>
       </collision>
@@ -189,12 +189,12 @@
 	      <material name="GreyC" />
 	      <origin xyz="0 0 0" rpy="0 0 0 " />
-	      <geometry name="wrist_l_geom">
-		      <mesh filename="package://${MESH}/A2R3/A2R3_wrist.mesh" />
-	      </geometry>
-      </visual>
-      <collision>
-	      <origin xyz="0 0 0" rpy="0.0 0.0 0.0 " />
-	      <geometry name="wrist_l_collision">
-		      <box size="0.01 0.01 0.01" />
+	      <geometry name="wrist_LEFT_geom">
+		      <mesh filename="package://${MESH}/A2R3/A2R3_T5_forearmRoll.dae" />
+	      </geometry>
+      </visual>
+      <collision>
+	      <origin xyz="0 0 0" rpy="0.0 0.0 0.0 " />
+	      <geometry name="wrist_LEFT_collision">
+		      <mesh filename="package://${MESH_COLL}/A2R3/A2R3_T5_forearmRoll.stl" />
 	      </geometry>
       </collision>
@@ -203,5 +203,5 @@
   <!-- ============================   Forearm   ============================ -->
   <macro name="m3_l_forearm" params="side parent reflect">
-	  <joint name="m3joint_${L_ARM}_j5" type="revolute">
+	  <joint name="left_arm_j5" type="revolute">
 		  <axis xyz="0 -1 0" />
       <origin xyz="0 0 0" rpy="0 0 0" />
@@ -219,20 +219,20 @@
                  izz="0.01659310749" />
       </inertial>
-      <visual>
+       <visual>
 	      <material name="GreyB" />
 	      <origin xyz="0 0 0" rpy="0 0 0 " />
-	      <geometry name="w_differential_l_geom">
-		      <mesh filename="package://${MESH}/A2R3/A2R3_w_differential.mesh" />
-	      </geometry>
-      </visual>
-      <collision>
-	      <origin xyz="0 0 0" rpy="0.0 0.0 0.0 " />
-	      <geometry name="w_differential_l_collision">
+	      <geometry name="w_differential_LEFT_geom">
+		      <mesh filename="package://${MESH}/A2R3/A2R3_T6_wristDiff.dae" />
+	      </geometry>
+      </visual>
+      <collision>
+	      <origin xyz="0 0 0" rpy="0.0 0.0 0.0 " />
+	      <geometry name="w_differential_LEFT_collision">
 		      <box size="0.01 0.01 0.01" />
 	      </geometry>
       </collision>
     </link>
-    <!-- Wrist flex -->
-    <joint name="m3joint_${L_ARM}_j6" type="revolute">
+  <!-- Wrist flex -->
+    <joint name="left_arm_j6" type="revolute">
 	    <axis xyz="-1 0 0" />
       <limit lower="-0.1" upper="2.2" effort="200" velocity="${VELOCITY_LIMIT_SCALE*5.13}" />
@@ -254,12 +254,12 @@
 	      <material name="GreyA" />
 	      <origin xyz="0 0 0" rpy="0 0 0 " />
-	      <geometry name="handmount_l_geom">
-		      <mesh filename="package://${MESH}/A2R3/A2R3_handmount.mesh" />
-	      </geometry>
-      </visual>
-      <collision>
-	      <origin xyz="0 0 0" rpy="0.0 0.0 0.0 " />
-	      <geometry name="handmount_l_collision">
-		      <box size="0.01 0.01 0.01" />
+	      <geometry name="handmount_LEFT_geom">
+		       <mesh filename="package://${MESH}/A2R3/A2R3_T7_wristYaw.dae" />
+	      </geometry>
+      </visual>
+      <collision>
+	      <origin xyz="0 0 0" rpy="0.0 0.0 0.0 " />
+	      <geometry name="handmount_LEFT_collision">
+		      <mesh filename="package://${MESH_COLL}/A2R3/A2R3_T7_wristYaw.stl" />
 	      </geometry>
       </collision>

Commit message: git-svn-id: file:///home/svn/meka-ros-pkg@164 cfd446f6-b9c6-49ad-a440-209cd04d0f1d

File: trunk/meka_description/robots/m1.urdf.xacro (robot description, xacro)
@@ -87,4 +87,5 @@
 			  <mesh filename="package://${MESH}/T2R3/T2R3_TJ3_chest_waist_neck.dae" />
 		  </geometry>
+		  <material name="Blue" />
 	  </visual>
 	  <collision>

Commit message: git-svn-id: file:///home/svn/meka-ros-pkg@167 cfd446f6-b9c6-49ad-a440-209cd04d0f1d

File: trunk/meka_description/robots/m1.urdf.xacro (robot description, xacro)
@@ -71,5 +71,5 @@
   <!-- Solid Base -->
   <joint name="chest_joint" type="fixed">
-	  <origin xyz="0 0 0.0" rpy="0 0 0" />
+	  <origin xyz="0 0 -0.03" rpy="0 0 0" />
     <parent link="zlift_link" />
     <child link="upper" />
@@ -85,5 +85,5 @@
 		  <origin xyz="0 0 0" rpy="0 0 0" />
 		  <geometry name="upper_geom">
-			  <mesh filename="package://${MESH}/T2R3/T2R3_TJ3_chest_waist_neck.dae" />
+			  <mesh filename="package://${MESH}/A2R3/A2R3_T4_Chest_Neck.dae" />
 		  </geometry>
 		  <material name="Blue" />

File: trunk/meka_description/robots/simc.urdf.xacro (robot description, xacro)
@@ -6,31 +6,25 @@
        name="meka" >
  <property name="M_PI" value="3.1415926535897931" />
- <property name="R_ARM" value="ma16" />
- <property name="R_HAND" value="mh12" />
- <property name="L_ARM" value="ma17" />
- <property name="L_HAND" value="mh13" />
- <property name="TORSO" value="mt5" />
-  <property name="HEAD" value="ms2" />
  <property name="MESH" value="meka_description/meshes/mid_res" />
  <property name="MESH_COLL" value="meka_description/meshes/low_res" />
 <!-- generic simulator_gazebo plugins for starting mechanism control, ros time, ros battery -->
   <include filename="$(find meka_description)/gazebo/gazebo.urdf.xacro" />
-  <include filename="$(find meka_description)/transmissions/uta.transmission.xacro" />
+  <!--<include filename="$(find meka_description)/transmissions/uta.transmission.xacro" />-->
 <!-- Meka Base -->
-  <include filename="$(find meka_description)/urdf/B1R2_defs.urdf.xacro" />
+  <include filename="$(find meka_description)/urdf/B1R2B_defs.urdf.xacro" />
 <!-- Meka Zlift -->
-  <include filename="$(find meka_description)/urdf/Z1R2_defs.urdf.xacro" />
+  <include filename="$(find meka_description)/urdf/Z1R2B_defs.urdf.xacro" />
 <!-- Meka Arm -->
-  <include filename="$(find meka_description)/urdf/A2R3_r_arm_defs.urdf.xacro" />
-  <include filename="$(find meka_description)/urdf/A2R3_l_arm_defs.urdf.xacro" />
+  <include filename="$(find meka_description)/urdf/A2R4_r_arm_defs.urdf.xacro" />
+  <include filename="$(find meka_description)/urdf/A2R4_l_arm_defs.urdf.xacro" />
   <!-- Meka Hand -->
-  <include filename="$(find meka_description)/urdf/H2R2_r_hand_defs.urdf.xacro" />
-  <include filename="$(find meka_description)/urdf/H2R2_l_hand_defs.urdf.xacro" />
+  <include filename="$(find meka_description)/urdf/H2R4_r_hand_defs.urdf.xacro" />
+  <include filename="$(find meka_description)/urdf/H2R4_l_hand_defs.urdf.xacro" />
 <!-- Meka Head -->
-  <include filename="$(find meka_description)/urdf/S2R1_head_defs.urdf.xacro" />
+  <include filename="$(find meka_description)/urdf/S2R1B_head_defs.urdf.xacro" />
   <!-- john added transmissions -->
-  <include filename="$(find meka_description)/transmissions/A2R3_r_arm_defs.transmission.xacro" />
-  <include filename="$(find meka_description)/transmissions/H2R2_r_hand_defs.transmission.xacro" />
-  <include filename="$(find meka_description)/transmissions/S2R1_head_defs.transmission.xacro" />
+  <include filename="$(find meka_description)/transmissions/A2R4_r_arm_defs.transmission.xacro" />
+  <!--<include filename="$(find meka_description)/transmissions/H2R2_r_hand_defs.transmission.xacro" />-->
+  <!--<include filename="$(find meka_description)/transmissions/S2R1_head_defs.transmission.xacro" />-->
    <property name="M_PI" value="3.1415926535897931" />
   <material name="GreyA"> <!-- darkest -->
@@ -49,16 +43,19 @@
     <origin xyz="0.0 0.0 0.0" rpy="0 0 0" />
   </m3_r_hand>
+  <m3_l_hand side="l" reflect="1" parent="handmount_LEFT">
+    <origin xyz="0.0 0.0 0.0" rpy="0 0 0" />
+  </m3_l_hand>
   <m3_head side="r" reflect="1" parent="upper">
     <origin xyz="0.0 0.0 0.31155" rpy="0 0 0" />
   </m3_head>
-  <!--<m3_l_arm side="l" reflect="1" parent="upper">
-    <origin xyz="0.0 0.18465 0.2337" rpy="0 0 0" />
-  </m3_l_arm>-->
  <m3_r_arm side="r" reflect="1" parent="upper">
     <origin xyz="0.0 -0.18465 0.2337" rpy="0 0 0" />
   </m3_r_arm>
+ <m3_l_arm side="l" reflect="1" parent="upper">
+    <origin xyz="0.0 0.18465 0.2337" rpy="0 0 0" />
+  </m3_l_arm>
   <link name="world" />
   <link name="base_link" />
-<!-- Solid Base -->
+  <!-- Solid Base -->
   <joint name="base_joint" type="fixed">
 	  <origin xyz="0 0 1" rpy="0 0 0" />
@@ -74,5 +71,5 @@
   <!-- Solid Base -->
   <joint name="chest_joint" type="fixed">
-	  <origin xyz="0 0 0.0" rpy="0 0 0" />
+	  <origin xyz="0 0 -0.03" rpy="0 0 0" />
     <parent link="zlift_link" />
     <child link="upper" />
@@ -88,6 +85,7 @@
 		  <origin xyz="0 0 0" rpy="0 0 0" />
 		  <geometry name="upper_geom">
-			  <mesh filename="package://${MESH}/T2R3/T2R3_TJ3_chest_waist_neck.dae" />
+			  <mesh filename="package://${MESH}/A2R3/A2R3_T4_Chest_Neck.dae" />
 		  </geometry>
+		  <material name="Blue" />
 	  </visual>
 	  <collision>

File: trunk/meka_description/urdf/A2R4_l_arm_defs.urdf.xacro (robot description, xacro)
@@ -156,7 +156,7 @@
       <visual>
 	      <material name="GreyA" />
-	      <origin xyz="0 0 0" rpy="0 0 0 " />
+	      <origin xyz="0 0 0" rpy="0 0 3.14 " />
 	      <geometry name="elbowclevis_LEFT_geom">
-		      <mesh filename="package://${MESH}/A2R3/A2R3_LT4_elbow.dae" />
+		      <mesh filename="package://${MESH}/A2R3/A2R3_RT4_elbow.dae" />
 	      </geometry>
       </visual>

File: trunk/meka_description/urdf/S2R1B_head_defs.urdf.xacro (robot description, xacro)
@@ -101,5 +101,5 @@
       </collision>
     </link>
-      <joint name="head_j3" type="revolute">
+    <joint name="head_j3" type="revolute">
 		  <axis xyz="0 -1 0" />
       <origin xyz="0 0 0" rpy="0 0 0" />
@@ -123,5 +123,6 @@
 	      <origin xyz="0 0 0" rpy="0 0 0 " />
 	      <geometry name="head_shell_geom">
-		      <mesh filename="package://${MESH}/S2R1/S2R1_H4_UTA_head.dae" />
+		<mesh filename="package://${MESH}/S2R1/S2R1_H4_SIMC_head.dae" />
+		<!--<mesh filename="package://${MESH}/S2R1/S2R1_H4_UTA_head.dae" />-->
 	      </geometry>
       </visual>
@@ -196,4 +197,180 @@
 	      <geometry name="left_eye_collision">
 		      <mesh filename="package://${MESH_COLL}/S2R1/S2R1_eye.stl" />
+	      </geometry>
+      </collision>
+    </link>
+    <joint name="head_j7_rt_eyelid_top" type="revolute">
+	    <axis xyz="0 -1 0" />
+      <limit effort="100" velocity="${1600*M_PI/180}" lower="${-35.12*M_PI/180}" upper="${35.125*M_PI/180}" />
+      <origin xyz="0 0.0 0" rpy="0 0.785 0" />
+      <parent link="right_eye"/>
+      <child link="rt_eyelid_top"/>
+    </joint>
+    <link name="rt_eyelid_top">
+      <visual>
+	      <material name="GreyC" />
+	      <origin xyz="0 0 0" rpy="0 0 0 " />
+	      <geometry name="rt_eyelid_top_geom">
+		      <mesh filename="package://${MESH}/S2R1/eyelid_top.dae" />
+	      </geometry>
+      </visual>
+      <collision>
+	      <origin xyz="0 0 0" rpy="0.0 0.0 0.0 " />
+	      <geometry name="rt_eyelid_top_collision">
+		      <box size="0.01 0.01 0.01" />
+	      </geometry>
+      </collision>
+    </link>
+    <joint name="head_j7_rt_eyelid_bottom" type="revolute">
+	    <axis xyz="0 1 0" />
+      <limit effort="100" velocity="${1600*M_PI/180}" lower="${-35.12*M_PI/180}" upper="${35.125*M_PI/180}" />
+      <origin xyz="0 0.0 0" rpy="0 -0.785 0" />
+      <parent link="right_eye"/>
+      <child link="rt_eyelid_bottom"/>
+    </joint>
+    <link name="rt_eyelid_bottom">
+      <visual>
+	      <material name="GreyC" />
+	      <origin xyz="0 0 0" rpy="0 0 0 " />
+	      <geometry name="eyelid_bottom_geom">
+		      <mesh filename="package://${MESH}/S2R1/eyelid_bottom.dae" />
+	      </geometry>
+      </visual>
+      <collision>
+	      <origin xyz="0 0 0" rpy="0.0 0.0 0.0 " />
+	      <geometry name="eyelid_bottom_collision">
+		      <box size="0.01 0.01 0.01" />
+	      </geometry>
+      </collision>
+    </link>
+    <joint name="head_j7_lt_eyelid_top" type="revolute">
+	    <axis xyz="0 -1 0" />
+      <limit effort="100" velocity="${1600*M_PI/180}" lower="${-35.12*M_PI/180}" upper="${35.125*M_PI/180}" />
+      <origin xyz="0 0.0 0" rpy="0 0.785 0" />
+      <parent link="left_eye"/>
+      <child link="lt_eyelid_top"/>
+    </joint>
+    <link name="lt_eyelid_top">
+      <visual>
+	      <material name="GreyC" />
+	      <origin xyz="0 0 0" rpy="0 0 0 " />
+	      <geometry name="lt_eyelid_top_geom">
+		      <mesh filename="package://${MESH}/S2R1/eyelid_top.dae" />
+	      </geometry>
+      </visual>
+      <collision>
+	      <origin xyz="0 0 0" rpy="0.0 0.0 0.0 " />
+	      <geometry name="lt_eyelid_top_collision">
+		      <box size="0.01 0.01 0.01" />
+	      </geometry>
+      </collision>
+    </link>
+    <joint name="head_j7_lt_eyelid_bottom" type="revolute">
+	    <axis xyz="0 1 0" />
+      <limit effort="100" velocity="${1600*M_PI/180}" lower="${-35.12*M_PI/180}" upper="${35.125*M_PI/180}" />
+      <origin xyz="0 0.0 0" rpy="0 -0.785 0" />
+      <parent link="left_eye"/>
+      <child link="lt_eyelid_bottom"/>
+    </joint>
+    <link name="lt_eyelid_bottom">
+      <visual>
+	      <material name="GreyC" />
+	      <origin xyz="0 0 0" rpy="0 0 0 " />
+	      <geometry name="eyelid_bottom_geom2">
+		      <mesh filename="package://${MESH}/S2R1/eyelid_bottom.dae" />
+	      </geometry>
+      </visual>
+      <collision>
+	      <origin xyz="0 0 0" rpy="0.0 0.0 0.0 " />
+	      <geometry name="eyelid_bottom_collision2">
+		      <box size="0.01 0.01 0.01" />
+	      </geometry>
+      </collision>
+    </link>
+     <joint name="head_j8" type="revolute">
+	    <axis xyz="0 0 1" />
+      <limit effort="100" velocity="${1600*M_PI/180}" lower="${-34.99*M_PI/180}" upper="${34.99*M_PI/180}" />
+      <origin xyz="0.022 0.138 0.120" rpy="-1.13 0 0" />
+      <parent link="head_shell"/>
+      <child link="ear_roll"/>
+    </joint>
+    <link name="ear_roll">
+      <visual>
+	      <material name="GreyC" />
+	      <origin xyz="0 0 0" rpy="0 0 0 " />
+	      <geometry name="ear_roll_geom">
+		      <mesh filename="package://${MESH}/S2R1/ear_mount.dae" />
+	      </geometry>
+      </visual>
+      <collision>
+	      <origin xyz="0 0 0" rpy="0.0 0.0 0.0 " />
+	      <geometry name="ear_roll_collision">
+		      <box size="0.01 0.01 0.01" />
+	      </geometry>
+      </collision>
+    </link>
+    <joint name="head_j9" type="revolute">
+	    <axis xyz="0 -1 0" />
+      <limit effort="100" velocity="${1600*M_PI/180}" lower="${-34.99*M_PI/180}" upper="${34.99*M_PI/180}" />
+      <origin xyz="0.0 0.0 0.0" rpy="0 1.07 0" />
+      <parent link="ear_roll"/>
+      <child link="ear1"/>
+    </joint>
+    <link name="ear1">
+      <visual>
+	      <material name="GreyC" />
+	      <origin xyz="0 0 0" rpy="0 0 0 " />
+	      <geometry name="ear1_geom">
+		      <mesh filename="package://${MESH}/S2R1/ear.dae" />
+	      </geometry>
+      </visual>
+      <collision>
+	      <origin xyz="0 0 0" rpy="0.0 0.0 0.0 " />
+	      <geometry name="ear1_collision">
+		      <box size="0.01 0.01 0.01" />
+	      </geometry>
+      </collision>
+    </link>
+    <joint name="head_j10" type="revolute">
+	    <axis xyz="0 0 1" />
+      <limit effort="100" velocity="${1600*M_PI/180}" lower="${-34.99*M_PI/180}" upper="${34.99*M_PI/180}" />
+      <origin xyz="0.022 -0.138 0.120" rpy="1.13 0 0" />
+      <parent link="head_shell"/>
+      <child link="ear_roll2"/>
+    </joint>
+    <link name="ear_roll2">
+      <visual>
+	      <material name="GreyC" />
+	      <origin xyz="0 0 0" rpy="0 0 0 " />
+	      <geometry name="ear_roll_geom2">
+		      <mesh filename="package://${MESH}/S2R1/ear_mount.dae" />
+	      </geometry>
+      </visual>
+      <collision>
+	      <origin xyz="0 0 0" rpy="0.0 0.0 0.0 " />
+	      <geometry name="ear_roll_collision2">
+		      <box size="0.01 0.01 0.01" />
+	      </geometry>
+      </collision>
+    </link>
+    <joint name="head_j11" type="revolute">
+	    <axis xyz="0 -1 0" />
+      <limit effort="100" velocity="${1600*M_PI/180}" lower="${-34.99*M_PI/180}" upper="${34.99*M_PI/180}" />
+      <origin xyz="0.0 0.0 0.0" rpy="0 1.07 0" />
+      <parent link="ear_roll2"/>
+      <child link="ear2"/>
+    </joint>
+    <link name="ear2">
+      <visual>
+	      <material name="GreyC" />
+	      <origin xyz="0 0 0" rpy="0 0 0 " />
+	      <geometry name="ear2_geom">
+		      <mesh filename="package://${MESH}/S2R1/ear.dae" />
+	      </geometry>
+      </visual>
+      <collision>
+	      <origin xyz="0 0 0" rpy="0.0 0.0 0.0 " />
+	      <geometry name="ear2_collision">
+		      <box size="0.01 0.01 0.01" />
 	      </geometry>
       </collision>
