Commit message: git-svn-id: file:///home/svn/meka-ros-pkg@138 cfd446f6-b9c6-49ad-a440-209cd04d0f1d

File: trunk/meka_description/robots/simc.urdf.xacro (robot description, xacro)
@@ -8,5 +8,8 @@
  <property name="R_ARM" value="ma16" />
  <property name="R_HAND" value="mh12" />
+ <property name="L_ARM" value="ma17" />
+ <property name="L_HAND" value="mh13" />
  <property name="TORSO" value="mt5" />
+  <property name="HEAD" value="ms2" />
  <property name="MESH" value="meka_description/meshes/mid_res" />
  <property name="MESH_COLL" value="meka_description/meshes/low_res" />
@@ -20,9 +23,14 @@
 <!-- Meka Arm -->
   <include filename="$(find meka_description)/urdf/A2R3_r_arm_defs.urdf.xacro" />
+  <include filename="$(find meka_description)/urdf/A2R3_l_arm_defs.urdf.xacro" />
   <!-- Meka Hand -->
   <include filename="$(find meka_description)/urdf/H2R2_r_hand_defs.urdf.xacro" />
+  <include filename="$(find meka_description)/urdf/H2R2_l_hand_defs.urdf.xacro" />
+<!-- Meka Head -->
+  <include filename="$(find meka_description)/urdf/S2R1_head_defs.urdf.xacro" />
   <!-- john added transmissions -->
   <include filename="$(find meka_description)/transmissions/A2R3_r_arm_defs.transmission.xacro" />
   <include filename="$(find meka_description)/transmissions/H2R2_r_hand_defs.transmission.xacro" />
+  <include filename="$(find meka_description)/transmissions/S2R1_head_defs.transmission.xacro" />
    <property name="M_PI" value="3.1415926535897931" />
   <material name="GreyA"> <!-- darkest -->
@@ -38,7 +46,10 @@
   <m3_r_arm_transmission side="r" reflect="1" parent="upper"/>
   <m3_r_hand_transmission/>
-  <!--<m3_r_hand side="r" reflect="1" parent="handmount_RIGHT">
+  <m3_r_hand side="r" reflect="1" parent="handmount_RIGHT">
     <origin xyz="0.0 0.0 0.0" rpy="0 0 0" />
-  </m3_r_hand>-->
+  </m3_r_hand>
+  <m3_head side="r" reflect="1" parent="upper">
+    <origin xyz="0.0 0.0 0.31155" rpy="0 0 0" />
+  </m3_head>
   <!--<m3_l_arm side="l" reflect="1" parent="upper">
     <origin xyz="0.0 0.18465 0.2337" rpy="0 0 0" />

Commit message: git-svn-id: file:///home/svn/meka-ros-pkg@170 cfd446f6-b9c6-49ad-a440-209cd04d0f1d

File: trunk/meka_description/robots/simc.urdf.xacro (robot description, xacro)
@@ -22,5 +22,5 @@
   <include filename="$(find meka_description)/urdf/H2R4_l_hand_defs.urdf.xacro" />
 <!-- Meka Head -->
-  <include filename="$(find meka_description)/urdf/S2R1B_head_defs.urdf.xacro" />
+  <include filename="$(find meka_description)/urdf/SIMC_head_defs.urdf.xacro" />
   <!-- john added transmissions -->
   <include filename="$(find meka_description)/transmissions/A2R4_r_arm_defs.transmission.xacro" />
@@ -92,5 +92,5 @@
 		  <origin xyz="0 0 0" rpy="0.0 0.0 0.0 " />
 		  <geometry name="upper_collision_geom">
-			  <mesh filename="package://${MESH_COLL}/T2R3/T2R3_TJ3_chest_waist_neck.stl" />
+			  <mesh filename="package://${MESH_COLL}/A2R3/A2R3_T4_Chest_Neck.stl" />
 		  </geometry>
 	  </collision>

File: trunk/meka_description/urdf/B1R2B_defs.urdf.xacro (robot description, xacro)
@@ -97,5 +97,5 @@
 		  <origin xyz="0 0 0" rpy="0.0 0.0 0.0 " />
 		  <geometry name="b1r1_3_geom">
-			  <box size="0.01 0.01 0.01" />
+			  <mesh filename="package://${MESH_COLL}/B1R1/MB1_00_000_meka_mobile_base+backpack+zlift.stl" />
 		  </geometry>
 	  </collision>

File: trunk/meka_description/urdf/Z1R2B_defs.urdf.xacro (robot description, xacro)
@@ -36,5 +36,5 @@
 	      <origin xyz="0 0 0" rpy="0.0 0.0 0.0 " />
 	      <geometry name="z_lift_geom_collision_geom">
-		      <box size="0.01 0.01 0.01" />
+		      <mesh filename="package://${MESH_COLL}/B1R1/MB1_00_011_festo-chest_mount_assy+spacer.stl" />
 	      </geometry>
       </collision>
