Commit message: git-svn-id: file:///home/svn/meka-ros-pkg@192 cfd446f6-b9c6-49ad-a440-209cd04d0f1d

File: trunk/meka_description/robots/gai.urdf.xacro (robot description, xacro)
@@ -21,4 +21,6 @@
   <include filename="$(find meka_description)/urdf/H2R4_r_hand_defs.urdf.xacro" />
  <!--<include filename="$(find meka_description)/urdf/H2R4_l_hand_defs.urdf.xacro" />-->
+    <!-- Meka Head -->
+  <include filename="$(find meka_description)/urdf/S3R1_head_defs.urdf.xacro" />
 <!-- Meka Head -->
 <!--<include filename="$(find meka_description)/urdf/SIMC_head_defs.urdf.xacro" />-->
@@ -46,7 +48,7 @@
     <origin xyz="0.0 0.0 0.0" rpy="0 0 0" />
   </m3_l_hand>-->
-  <m3_head side="r" reflect="1" parent="upper">
+<!--  <m3_head side="r" reflect="1" parent="upper">
     <origin xyz="0.0 0.0 0.31155" rpy="0 0 0" />
-  </m3_head>
+  </m3_head>-->
  <m3_r_arm side="r" reflect="1" parent="upper">
     <origin xyz="0.0 -0.18465 0.2337" rpy="0 0 0" />
@@ -55,4 +57,7 @@
     <origin xyz="0.0 0.18465 0.2337" rpy="0 0 0" />
   </m3_l_arm>
+   <m3_head side="r" reflect="1" parent="upper">
+    <origin xyz="0.0 0.0 0.2337" rpy="0 0 0" />
+  </m3_head>
   <link name="world" />
   <link name="base_link" />
@@ -85,5 +90,5 @@
 		  <origin xyz="0 0 0" rpy="0 0 0" />
 		  <geometry name="upper_geom">
-			  <mesh filename="package://${MESH}/A2R3/A2R3_T4_Chest_Neck.dae" />
+			  <mesh filename="package://${MESH}/A2R3/A2R3_T4_Chest2.dae" />
 		  </geometry>
 		  <material name="Blue" />

Commit message: git-svn-id: file:///home/svn/meka-ros-pkg@194 cfd446f6-b9c6-49ad-a440-209cd04d0f1d

File: trunk/meka_description/robots/gai.urdf.xacro (robot description, xacro)
@@ -20,5 +20,6 @@
   <!-- Meka Hand -->
   <include filename="$(find meka_description)/urdf/H2R4_r_hand_defs.urdf.xacro" />
- <!--<include filename="$(find meka_description)/urdf/H2R4_l_hand_defs.urdf.xacro" />-->
+  <!-- Meka Gripper -->
+  <include filename="$(find meka_description)/urdf/G2R1_l_gripper_defs.urdf.xacro" />
     <!-- Meka Head -->
   <include filename="$(find meka_description)/urdf/S3R1_head_defs.urdf.xacro" />
@@ -45,10 +46,7 @@
     <origin xyz="0.0 0.0 0.0" rpy="0 0 0" />
   </m3_r_hand>
-  <!--<m3_l_hand side="l" reflect="1" parent="handmount_LEFT">
+  <m3_l_gripper side="r" reflect="1" parent="handmount_LEFT">
     <origin xyz="0.0 0.0 0.0" rpy="0 0 0" />
-  </m3_l_hand>-->
-<!--  <m3_head side="r" reflect="1" parent="upper">
-    <origin xyz="0.0 0.0 0.31155" rpy="0 0 0" />
-  </m3_head>-->
+  </m3_l_gripper>
  <m3_r_arm side="r" reflect="1" parent="upper">
     <origin xyz="0.0 -0.18465 0.2337" rpy="0 0 0" />

File: trunk/meka_description/urdf/G2R1_l_gripper_defs.urdf.xacro (robot description, xacro)
@@ -4,11 +4,11 @@
        xmlns:interface="http://playerstage.sourceforge.net/gazebo/xmlschema/#interface">
   <property name="M_PI" value="3.1415926535897931" />
-  <macro name="m3_l_palm" params="side parent reflect *origin">
-  <joint name="l_palm_joint" type="fixed">
+  <macro name="m3_l_chassis" params="side parent reflect *origin">
+  <joint name="l_chassis_joint" type="fixed">
     <origin xyz="0 0 -0.04414" rpy="0 0 0" />
     <parent link="${parent}"/>
-    <child link="l_palm" />
+    <child link="l_chassis" />
   </joint>
-     <link name="l_palm">
+     <link name="l_chassis">
       <inertial>
         <mass value="0.663" />
@@ -24,24 +24,23 @@
 	      <material name="GreyA" />
 	      <origin xyz="0 0 0" rpy="0 0 0 " />
-	      <geometry name="l_palm_geom">
-		      <mesh filename="package://${MESH}/H2R3/H2R3_LT8_palm_left.dae" />
+	      <geometry name="l_chassis_geom">
+		      <mesh filename="package://${MESH}/G2R1/chassis.dae" />
 	      </geometry>
       </visual>
       <collision>
 	      <origin xyz="0 0 0" rpy="0.0 0.0 0.0 " />
-	      <geometry name="l_palm_collision">
-		      <mesh filename="package://${MESH_COLL}/H2R3/H2R3_RT8_palm_right.stl" />
+	      <geometry name="l_chassis_collision">
+		      <box size="0.01 0.01 0.01" />
 	      </geometry>
       </collision>
     </link>
-<!-- Start Thumb -->
-    <joint name="left_hand_j0" type="revolute">
-      <axis xyz="0 0 -1" />
-      <origin xyz="-0.02 -0.028 -0.03" rpy="0 0 0" />
-      <parent link="l_palm"/>
-      <child link="l_thumb0"/>
+    <joint name="left_gripper_j0" type="revolute">
+      <axis xyz="1 0 0" />
+      <origin xyz="0 0.021 -0.09013" rpy="0 0 0" />
+      <parent link="l_chassis"/>
+      <child link="l_base_0"/>
       <limit effort="100" velocity="${20.0*M_PI/180}" lower="${-40*M_PI/180}" upper="${15*M_PI/180}" />
     </joint>
-    <link name="l_thumb0">
+    <link name="l_base_0">
       <inertial>
         <mass value="0.0117" />
@@ -57,25 +56,25 @@
 	      <material name="GreyA" />
 	      <origin xyz="0 0 0" rpy="0 0 0 " />
-	      <geometry name="l_thumb0_geom">
-		      <mesh filename="package://${MESH}/H2R3/H2R3_RJ0_thumb_abductlink.dae" />
+	      <geometry name="l_base0_geom">
+		      <mesh filename="package://${MESH}/G2R1/base.dae" />
 	      </geometry>
       </visual>
       <collision>
 	      <origin xyz="0 0 0" rpy="0.0 0.0 0.0 " />
-	      <geometry name="l_thumb0_collision">
-		      <mesh filename="package://${MESH_COLL}/H2R3/H2R3_RJ0_thumb_abductlink.stl" />
+	      <geometry name="l_base0_collision">
+		      <box size="0.01 0.01 0.01" />
 	      </geometry>
       </collision>
     </link>
-    <joint name="left_hand_j1" type="revolute">
-      <axis xyz="0 -1 0"/>
-     <limit effort="100" velocity="${75*M_PI/180}" lower="${-80.919*M_PI/180}" upper="${80.91*M_PI/180}" />
-      <origin xyz="-0.018 0 0" rpy="0 0 0" />
-      <parent link="l_thumb0"/>
-      <child link="l_thumb1"/>
+    <joint name="left_gripper_j1" type="revolute">
+      <axis xyz="1 0 0" />
+      <origin xyz="0 -0.021 -0.09013" rpy="0 0 0" />
+      <parent link="l_chassis"/>
+      <child link="l_base_1"/>
+      <limit effort="100" velocity="${20.0*M_PI/180}" lower="${-40*M_PI/180}" upper="${15*M_PI/180}" />
     </joint>
-    <link name="l_thumb1">
+    <link name="l_base_1">
       <inertial>
-        <mass value="0.0344" />
+        <mass value="0.0117" />
 	<origin xyz="0.0 0.0 0.0"/>
 	<inertia ixx="0.0"
@@ -87,27 +86,27 @@
       </inertial>
       <visual>
-	      <material name="GreyB" />
-	      <origin xyz="0 0 0" rpy="0 0 0 " />
-	      <geometry name="l_thumb1_geom">
-		      <mesh filename="package://${MESH}/H2R3/H2R3_thumb_knuckle1.dae" />
+	      <material name="GreyA" />
+	      <origin xyz="0 0 0" rpy="0 0 3.14 " />
+	      <geometry name="l_base1_geom">
+		      <mesh filename="package://${MESH}/G2R1/base.dae" />
 	      </geometry>
       </visual>
       <collision>
 	      <origin xyz="0 0 0" rpy="0.0 0.0 0.0 " />
-	      <geometry name="l_thumb1_collision">
-		      <mesh filename="package://${MESH_COLL}/H2R3/H2R3_thumb_knuckle1.stl" />
+	      <geometry name="l_base1_collision">
+		      <box size="0.01 0.01 0.01" />
 	      </geometry>
       </collision>
     </link>
-    <joint name="left_hand_j2" type="revolute">
-      <axis xyz="0 -1 0" />
-      <origin xyz="-0.044 0 0" rpy="0 0 0" />
-      <parent link="l_thumb1" />
-      <child link="l_thumb2"/>
-      <limit effort="100" velocity="${50*M_PI/180}" lower="${-14.94*M_PI/180}" upper="${14.94*M_PI/180}" />
+     <joint name="left_gripper_j2" type="revolute">
+      <axis xyz="1 0 0" />
+      <origin xyz="0 0.0 -0.055" rpy="0 0 0" />
+      <parent link="l_base_0"/>
+      <child link="l_tip_0"/>
+      <limit effort="100" velocity="${20.0*M_PI/180}" lower="${-40*M_PI/180}" upper="${15*M_PI/180}" />
     </joint>
-    <link name="l_thumb2">
+    <link name="l_tip_0">
       <inertial>
-        <mass value="0.01" />
+        <mass value="0.0117" />
 	<origin xyz="0.0 0.0 0.0"/>
 	<inertia ixx="0.0"
@@ -119,28 +118,27 @@
       </inertial>
       <visual>
-	      <material name="GreyC" />
-	      <origin xyz="0 0 0" rpy="0 0 0 " />
-	      <geometry name="l_thumb_knuckle2_geom">
-		      <mesh filename="package://${MESH}/H2R3/H2R3_thumb_knuckle2.dae" />
+	      <material name="GreyA" />
+	      <origin xyz="0 0 0" rpy="0 0 3.14 " />
+	      <geometry name="l_tip0_geom">
+		      <mesh filename="package://${MESH}/G2R1/tip.dae" />
 	      </geometry>
       </visual>
       <collision>
 	      <origin xyz="0 0 0" rpy="0.0 0.0 0.0 " />
-	      <geometry name="l_thumb_knuckle2_collision">
-		      <mesh filename="package://${MESH_COLL}/H2R3/H2R3_thumb_knuckle2.stl" />
+	      <geometry name="l_tip0_collision">
+		      <box size="0.01 0.01 0.01" />
 	      </geometry>
       </collision>
     </link>
-<!-- Start Index Finger -->
-    <joint name="left_hand_j3" type="revolute">
-      <axis xyz="0 1 0" />
-      <origin xyz="0 0.028 -0.101" rpy="0 0 0" />
-      <parent link="l_palm" />
-      <child link="l_index0"/>
-	<limit effort="100" velocity="${50*M_PI/180}" lower="${-7.072*M_PI/180}" upper="${37.072*M_PI/180}" />
+    <joint name="left_gripper_j3" type="revolute">
+      <axis xyz="1 0 0" />
+      <origin xyz="0 0.0 -0.055" rpy="0 0 0" />
+      <parent link="l_base_1"/>
+      <child link="l_tip_1"/>
+      <limit effort="100" velocity="${20.0*M_PI/180}" lower="${-40*M_PI/180}" upper="${15*M_PI/180}" />
     </joint>
-    <link name="l_index0">
+    <link name="l_tip_1">
       <inertial>
-        <mass value="0.01" />
+        <mass value="0.0117" />
 	<origin xyz="0.0 0.0 0.0"/>
 	<inertia ixx="0.0"
@@ -154,278 +152,20 @@
 	      <material name="GreyA" />
 	      <origin xyz="0 0 0" rpy="0 0 0 " />
-	      <geometry name="l_index0_geom">
-		     <mesh filename="package://${MESH}/H2R3/H2R3_finger_knuckle1.dae" />
+	      <geometry name="l_tip1_geom">
+		      <mesh filename="package://${MESH}/G2R1/tip.dae" />
 	      </geometry>
       </visual>
       <collision>
 	      <origin xyz="0 0 0" rpy="0.0 0.0 0.0 " />
-	      <geometry name="l_index0__collision">
-		      <mesh filename="package://${MESH_COLL}/H2R3/H2R3_finger_knuckle1.stl" />
-	      </geometry>
-      </collision>
-    </link>
-    <joint name="left_hand_j4" type="revolute">
-      <axis xyz="0 1 0" />
-      <limit effort="100" velocity="${1600*M_PI/180}" lower="${-34.99*M_PI/180}" upper="${34.99*M_PI/180}" />
-      <origin xyz="0 0 -0.044" rpy="0 0 0" />
-      <parent link="l_index0"/>
-      <child link="l_index1"/>
-    </joint>
-    <link name="l_index1">
-      <inertial>
-        <mass value="0.0429" />
-	<origin xyz="0.0 0.0 0.0"/>
-	<inertia ixx="0.0"
-	iyy="0.0"
-	izz="0.0"
-	ixy="0.0"
-	ixz="0.0"
-	iyz="0.0" />
-      </inertial>
-      <visual>
-	      <material name="GreyC" />
-	      <origin xyz="0 0 0" rpy="0 0 0 " />
-	      <geometry name="l_index1_geom">
-		      <mesh filename="package://${MESH}/H2R3/H2R3_finger_knuckle2.dae" />
-	      </geometry>
-      </visual>
-      <collision>
-	      <origin xyz="0 0 0" rpy="0.0 0.0 0.0 " />
-	      <geometry name="l_index1_collision">
-		      <mesh filename="package://${MESH_COLL}/H2R3/H2R3_finger_knuckle2.stl" />
-	      </geometry>
-      </collision>
-    </link>
-    <joint name="left_hand_j5" type="revolute">
-      <axis xyz="0 1 0" />
-      <limit effort="100" velocity="${1600*M_PI/180}" lower="${-34.21*M_PI/180}" upper="${34.213*M_PI/180}" />
-      <origin xyz="0 0 -0.032" rpy="0 0 0" />
-      <parent link="l_index1"/>
-      <child link="l_index2"/>
-    </joint>
-    <link name="l_index2">
-      <inertial>
-        <mass value="0.01" />
-	<origin xyz="0.0 0.0 0.0"/>
-	<inertia ixx="0.0"
-	iyy="0.0"
-	izz="0.0"
-	ixy="0.0"
-	ixz="0.0"
-	iyz="0.0" />
-      </inertial>
-      <visual>
-	      <material name="GreyC" />
-	      <origin xyz="0 0 0" rpy="0 0 0 " />
-	      <geometry name="l_index2_geom">
-		      <mesh filename="package://${MESH}/H2R3/H2R3_finger_knuckle3.dae" />
-	      </geometry>
-      </visual>
-      <collision>
-	      <origin xyz="0 0 0" rpy="0.0 0.0 0.0 " />
-	      <geometry name="l_index2_collision">
-		      <mesh filename="package://${MESH_COLL}/H2R3/H2R3_finger_knuckle3.stl" />
-	      </geometry>
-      </collision>
-    </link>
-<!-- Start Ring Finger -->
-    <joint name="left_hand_j6" type="revolute">
-      <axis xyz="0 1 0" />
-      <origin xyz="0 0 -0.101" rpy="0 0 0" />
-      <parent link="l_palm" />
-      <child link="l_ring0"/>
-	<limit effort="100" velocity="${50*M_PI/180}" lower="${-7.072*M_PI/180}" upper="${37.072*M_PI/180}" />
-    </joint>
-    <link name="l_ring0">
-      <inertial>
-        <mass value="0.01" />
-	<origin xyz="0.0 0.0 0.0"/>
-	<inertia ixx="0.0"
-	iyy="0.0"
-	izz="0.0"
-	ixy="0.0"
-	ixz="0.0"
-	iyz="0.0" />
-      </inertial>
-      <visual>
-	      <material name="GreyA" />
-	      <origin xyz="0 0 0" rpy="0 0 0 " />
-	      <geometry name="l_ring0_geom">
-		     <mesh filename="package://${MESH}/H2R3/H2R3_finger_knuckle1.dae" />
-	      </geometry>
-      </visual>
-      <collision>
-	      <origin xyz="0 0 0" rpy="0.0 0.0 0.0 " />
-	      <geometry name="l_ring0__collision">
-		      <mesh filename="package://${MESH_COLL}/H2R3/H2R3_finger_knuckle1.stl" />
-	      </geometry>
-      </collision>
-    </link>
-    <joint name="left_hand_j7" type="revolute">
-      <axis xyz="0 1 0" />
-      <limit effort="100" velocity="${1600*M_PI/180}" lower="${-34.99*M_PI/180}" upper="${34.99*M_PI/180}" />
-      <origin xyz="0 0 -0.044" rpy="0 0 0" />
-      <parent link="l_ring0"/>
-      <child link="l_ring1"/>
-    </joint>
-    <link name="l_ring1">
-      <inertial>
-        <mass value="0.0429" />
-	<origin xyz="0.0 0.0 0.0"/>
-	<inertia ixx="0.0"
-	iyy="0.0"
-	izz="0.0"
-	ixy="0.0"
-	ixz="0.0"
-	iyz="0.0" />
-      </inertial>
-      <visual>
-	      <material name="GreyC" />
-	      <origin xyz="0 0 0" rpy="0 0 0 " />
-	      <geometry name="l_ring1_geom">
-		      <mesh filename="package://${MESH}/H2R3/H2R3_finger_knuckle2.dae" />
-	      </geometry>
-      </visual>
-      <collision>
-	      <origin xyz="0 0 0" rpy="0.0 0.0 0.0 " />
-	      <geometry name="l_ring1_collision">
-		      <mesh filename="package://${MESH_COLL}/H2R3/H2R3_finger_knuckle2.stl" />
-	      </geometry>
-      </collision>
-    </link>
-    <joint name="left_hand_j8" type="revolute">
-      <axis xyz="0 1 0" />
-      <limit effort="100" velocity="${1600*M_PI/180}" lower="${-34.21*M_PI/180}" upper="${34.213*M_PI/180}" />
-      <origin xyz="0 0 -0.032" rpy="0 0 0" />
-      <parent link="l_ring1"/>
-      <child link="l_ring2"/>
-    </joint>
-    <link name="l_ring2">
-      <inertial>
-        <mass value="0.01" />
-	<origin xyz="0.0 0.0 0.0"/>
-	<inertia ixx="0.0"
-	iyy="0.0"
-	izz="0.0"
-	ixy="0.0"
-	ixz="0.0"
-	iyz="0.0" />
-      </inertial>
-      <visual>
-	      <material name="GreyC" />
-	      <origin xyz="0 0 0" rpy="0 0 0 " />
-	      <geometry name="l_ring2_geom">
-		      <mesh filename="package://${MESH}/H2R3/H2R3_finger_knuckle3.dae" />
-	      </geometry>
-      </visual>
-      <collision>
-	      <origin xyz="0 0 0" rpy="0.0 0.0 0.0 " />
-	      <geometry name="l_ring2_collision">
-		      <mesh filename="package://${MESH_COLL}/H2R3/H2R3_finger_knuckle3.stl" />
-	      </geometry>
-      </collision>
-    </link>
-<!-- Start Pinky Finger -->
-    <joint name="left_hand_j9" type="revolute">
-      <axis xyz="0 1 0" />
-      <origin xyz="0 -0.028 -0.101" rpy="0 0 0" />
-      <parent link="l_palm" />
-      <child link="l_pinky0"/>
-	<limit effort="100" velocity="${50*M_PI/180}" lower="${-7.072*M_PI/180}" upper="${37.072*M_PI/180}" />
-    </joint>
-    <link name="l_pinky0">
-      <inertial>
-        <mass value="0.01" />
-	<origin xyz="0.0 0.0 0.0"/>
-	<inertia ixx="0.0"
-	iyy="0.0"
-	izz="0.0"
-	ixy="0.0"
-	ixz="0.0"
-	iyz="0.0" />
-      </inertial>
-      <visual>
-	      <material name="GreyA" />
-	      <origin xyz="0 0 0" rpy="0 0 0 " />
-	      <geometry name="l_pinky0_geom">
-		     <mesh filename="package://${MESH}/H2R3/H2R3_finger_knuckle1.dae" />
-	      </geometry>
-      </visual>
-      <collision>
-	      <origin xyz="0 0 0" rpy="0.0 0.0 0.0 " />
-	      <geometry name="l_pinky0__collision">
-		      <mesh filename="package://${MESH_COLL}/H2R3/H2R3_finger_knuckle1.stl" />
-	      </geometry>
-      </collision>
-    </link>
-    <joint name="left_hand_j10" type="revolute">
-      <axis xyz="0 1 0" />
-      <limit effort="100" velocity="${1600*M_PI/180}" lower="${-34.99*M_PI/180}" upper="${34.99*M_PI/180}" />
-      <origin xyz="0 0 -0.044" rpy="0 0 0" />
-      <parent link="l_pinky0"/>
-      <child link="l_pinky1"/>
-    </joint>
-    <link name="l_pinky1">
-      <inertial>
-        <mass value="0.0429" />
-	<origin xyz="0.0 0.0 0.0"/>
-	<inertia ixx="0.0"
-	iyy="0.0"
-	izz="0.0"
-	ixy="0.0"
-	ixz="0.0"
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