Commit message: git-svn-id: file:///home/svn/meka-ros-pkg@176 cfd446f6-b9c6-49ad-a440-209cd04d0f1d

File: trunk/meka_description/robots/bie.urdf.xacro (robot description, xacro)
@@ -22,5 +22,5 @@
   <include filename="$(find meka_description)/urdf/H2R4_l_hand_defs.urdf.xacro" />
 <!-- Meka Head -->
-  <include filename="$(find meka_description)/urdf/SIMC_head_defs.urdf.xacro" />
+  <include filename="$(find meka_description)/urdf/S3R1_head_defs.urdf.xacro" />
   <!-- john added transmissions -->
   <include filename="$(find meka_description)/transmissions/A2R4_r_arm_defs.transmission.xacro" />
@@ -73,26 +73,119 @@
 	  <origin xyz="0 0 -0.03" rpy="0 0 0" />
     <parent link="zlift_link" />
+    <child link="panplate" />
+  </joint>
+  <link name="panplate">
+    <inertial>
+      <mass value="1000" />
+      <origin xyz="0 0 0" />
+      <inertia ixx="100"  ixy="0"  ixz="0" iyy="100" iyz="0" izz="100" />
+    </inertial>
+    <visual>
+      <material name="GreyA" />
+      <origin xyz="0 0 0" rpy="0 0 0 " />
+      <geometry name="panplate_geom">
+        <mesh filename="package://${MESH}/T2R3/T2R3_TJ0_base.dae" />
+      </geometry>
+    </visual>
+    <collision>
+      <origin xyz="0 0 0" rpy="0.0 0.0 0.0 " />
+      <geometry name="base_collision_geom">
+        <mesh filename="package://${MESH_COLL}/T2R3/T2R3_TJ0_base.stl" />
+      </geometry>
+    </collision>
+  </link>
+  <joint name="m3joint_${TORSO}_j0" type="continuous">
+    <axis xyz="0 0 1"/>
+    <origin xyz="0 0 0.1678" rpy="0 0 0" />
+    <parent link="panplate" />
+    <child link="torso" />
+    <limit effort="25" velocity="${25.0*M_PI/180}" lower="${-120*M_PI/180.0}" upper="${120*M_PI/180}" />
+    <dynamics damping="1.0"/>
+  </joint>
+  <link name="torso">
+    <inertial>
+      <mass value="4.411" />
+      <origin xyz="0.00011774 0.0038073 -0.0522753" />
+      <inertia ixx="0.026360"  ixy="-0.0000024"  ixz="-0.0000508" iyy="0.0134266" iyz="0.0006839" izz="0.0229879" />
+    </inertial>
+    <visual>
+      <material name="GreyC" />
+      <origin xyz="0 0 0" rpy="0 0 0 " />
+      <geometry name="torso_geom">
+        <mesh filename="package://${MESH}/T2R3/T2R3_TJ1_pan.dae" />
+      </geometry>
+    </visual>
+    <collision>
+      <origin xyz="0 0 0" rpy="0.0 0.0 0.0 " />
+      <geometry name="torso_collision_geom">
+        <mesh filename="package://${MESH_COLL}/T2R3/T2R3_TJ1_pan.stl" />
+      </geometry>
+    </collision>
+  </link>
+  <joint name="m3joint_${TORSO}_j1" type="continuous">
+    <axis xyz="0 1 0"/>
+    <origin xyz="0 0 0" rpy="0 0 0" />
+    <parent link="torso" />
+    <child link="mid" />
+    <limit effort="200" velocity="${10.0*M_PI/180}" lower="${-11.79349*M_PI/180}" upper="${53.29349*M_PI/180}" />
+    <dynamics damping="1.0"/>
+  </joint>
+  <link name="mid">
+    <inertial>
+      <mass value="4.934" />
+      <origin xyz="0.001179 -0.002993 0.046259"/>
+      <inertia ixx="0.041106"
+      iyy="0.026009"
+      izz="0.025902"
+      ixy="0.000135"
+      ixz="0.000505"
+      iyz="0.002396" />
+    </inertial>
+    <visual>
+      <material name="GreyB" />
+      <origin xyz="0 0 0" rpy="0 0 0" />
+      <geometry name="mid_geom">
+        <mesh filename="package://${MESH}/T2R3/T2R3_TJ2.dae" />
+      </geometry>
+    </visual>
+    <collision>
+      <origin xyz="0 0 0" rpy="0.0 0.0 0.0 " />
+      <geometry name="mid_collision_geom">
+        <mesh filename="package://${MESH_COLL}/T2R3/T2R3_TJ2.stl" />
+      </geometry>
+    </collision>
+  </link>
+  <joint name="m3joint_slave_${TORSO}_j2" type="continuous">
+    <axis xyz="0 1 0"/>
+    <origin xyz="0 0 0.1397" rpy="0 0 0" />
+    <parent link="mid" />
     <child link="upper" />
+    <limit effort="200" velocity="${10.0*M_PI/180}" lower="${-11.79349*M_PI/180}" upper="${53.29349*M_PI/180}" />
+    <dynamics damping="1.0"/>
   </joint>
   <link name="upper">
-	  <inertial>
-		  <mass value="1000" />
-		  <origin xyz="0 0 0" />
-		  <inertia ixx="1000"  ixy="0"  ixz="0" iyy="1000" iyz="0" izz="1000" />
-	  </inertial>
-	  <visual>
-		  <material name="GreyC" />
-		  <origin xyz="0 0 0" rpy="0 0 0" />
-		  <geometry name="upper_geom">
-			  <mesh filename="package://${MESH}/A2R3/A2R3_T4_Chest_Neck.dae" />
-		  </geometry>
-		  <material name="Blue" />
-	  </visual>
-	  <collision>
-		  <origin xyz="0 0 0" rpy="0.0 0.0 0.0 " />
-		  <geometry name="upper_collision_geom">
-			  <mesh filename="package://${MESH_COLL}/A2R3/A2R3_T4_Chest_Neck.stl" />
-		  </geometry>
-	  </collision>
+    <inertial>
+      <mass value="6.534" /> <!-- torso with motors, bottom pullies, and neck mount -->
+      <origin xyz="0.008700 0.011470 0.129740"/>
+      <inertia ixx="0.069760"
+      iyy="0.048010"
+      izz="0.040590"
+      ixy="-0.000400"
+      ixz="0.001300"
+      iyz="0.005100" />
+    </inertial>
+    <visual>
+      <material name="GreyC" />
+      <origin xyz="0 0 0" rpy="0 0 0" />
+      <geometry name="upper_geom">
+        <mesh filename="package://${MESH}/T2R3/T2R3_TJ3_chest_waist_neck.dae" />
+      </geometry>
+    </visual>
+    <collision>
+      <origin xyz="0 0 0" rpy="0.0 0.0 0.0 " />
+      <geometry name="upper_collision_geom">
+        <mesh filename="package://${MESH_COLL}/T2R3/T2R3_TJ3_chest_waist_neck.stl" />
+      </geometry>
+    </collision>
   </link>
 </robot>

File: trunk/meka_description/urdf/S3R1_head_defs.urdf.xacro (robot description, xacro)
@@ -101,279 +101,4 @@
       </collision>
     </link>
-    <joint name="head_j3" type="revolute">
-		  <axis xyz="0 -1 0" />
-      <origin xyz="0 0 0" rpy="0 0 0" />
-      <parent link="neck_yaw" />
-      <child link="head_shell"/>
-	<limit effort="100" velocity="${50*M_PI/180}" lower="${-8.0*M_PI/180}" upper="${-2.0*M_PI/180}" />
-    </joint>
-    <link name="head_shell">
-      <inertial>
-        <mass value="3.178" />
-	<origin xyz="0.034944 0.000563 0.058668"/>
-	<inertia ixx="0.022924"
-	iyy="0.021814"
-	izz="0.026783"
-	ixy="-0.000034"
-	ixz="-0.002929"
-	iyz="-0.000235" />
-      </inertial>
-      <visual>
-	      <material name="GreyA" />
-	      <origin xyz="0 0 0" rpy="0 0 0 " />
-	      <geometry name="head_shell_geom">
-		<mesh filename="package://${MESH}/S2R1/S2R1_H4_SIMC_head.dae" />
-		<!--<mesh filename="package://${MESH}/S2R1/S2R1_H4_UTA_head.dae" />-->
-	      </geometry>
-      </visual>
-      <collision>
-	      <origin xyz="0 0 0" rpy="0.0 0.0 0.0 " />
-	      <geometry name="head_shell_collision">
-		      <mesh filename="package://${MESH_COLL}/S2R1/S2R1_H4_SIMC_head.stl" />
-	      </geometry>
-      </collision>
-    </link>
-    <joint name="head_j4" type="revolute">
-	    <axis xyz="0 -1 0" />
-      <limit effort="100" velocity="${1600*M_PI/180}" lower="${-70.1*M_PI/180}" upper="${70.1*M_PI/180}" />
-      <origin xyz="0.12508 0 0" rpy="0 0 0" />
-      <parent link="head_shell"/>
-      <child link="eye_tilt"/>
-    </joint>
-    <link name="eye_tilt">
-      <visual>
-	      <material name="GreyC" />
-	      <origin xyz="0 0 0" rpy="0 0 0 " />
-	      <geometry name="eye_tilt_geom">
-		      <mesh filename="package://${MESH}/S2R1/S2R1_SH5_eyeTilt.dae" />
-	      </geometry>
-      </visual>
-      <collision>
-	      <origin xyz="0 0 0" rpy="0.0 0.0 0.0 " />
-	      <geometry name="eye_tilt_collision">
-		      <box size="0.01 0.01 0.01" />
-	      </geometry>
-      </collision>
-    </link>
-    <joint name="head_j5" type="revolute">
-	    <axis xyz="0 0 1" />
-      <limit effort="100" velocity="${1600*M_PI/180}" lower="${-37.49*M_PI/180}" upper="${37.4*M_PI/180}" />
-      <origin xyz="0 -0.053 0" rpy="0 0 0" />
-      <parent link="eye_tilt"/>
-      <child link="right_eye"/>
-    </joint>
-    <link name="right_eye">
-      <visual>
-	      <material name="GreyC" />
-	      <origin xyz="0 0 0" rpy="0 0 0 " />
-	      <geometry name="right_eye_geom">
-		      <mesh filename="package://${MESH}/S2R1/S2R1_eye.dae" />
-	      </geometry>
-      </visual>
-      <collision>
-	      <origin xyz="0 0 0" rpy="0.0 0.0 0.0 " />
-	      <geometry name="right_eye_collision">
-		      <mesh filename="package://${MESH_COLL}/S2R1/S2R1_eye.stl" />
-	      </geometry>
-      </collision>
-    </link>
-    <joint name="head_j6" type="revolute">
-	    <axis xyz="0 0 1" />
-      <limit effort="100" velocity="${1600*M_PI/180}" lower="${-37.9*M_PI/180}" upper="${37.99*M_PI/180}" />
-      <origin xyz="0 0.053 0" rpy="0 0 0" />
-      <parent link="eye_tilt"/>
-      <child link="left_eye"/>
-    </joint>
-    <link name="left_eye">
-      <visual>
-	      <material name="GreyC" />
-	      <origin xyz="0 0 0" rpy="0 0 0 " />
-	      <geometry name="left_eye_geom">
-		      <mesh filename="package://${MESH}/S2R1/S2R1_eye.dae" />
-	      </geometry>
-      </visual>
-      <collision>
-	      <origin xyz="0 0 0" rpy="0.0 0.0 0.0 " />
-	      <geometry name="left_eye_collision">
-		      <mesh filename="package://${MESH_COLL}/S2R1/S2R1_eye.stl" />
-	      </geometry>
-      </collision>
-    </link>
-    <joint name="head_j7_rt_eyelid_top" type="revolute">
-	    <axis xyz="0 -1 0" />
-      <limit effort="100" velocity="${1600*M_PI/180}" lower="${2.0*M_PI/180}" upper="${68.0*M_PI/180}" />
-      <origin xyz="0 0.0 0" rpy="0 0.785 0" />
-      <parent link="right_eye"/>
-      <child link="rt_eyelid_top"/>
-    </joint>
-    <link name="rt_eyelid_top">
-      <visual>
-	      <material name="GreyC" />
-	      <origin xyz="0 0 0" rpy="0 0 0 " />
-	      <geometry name="rt_eyelid_top_geom">
-		      <mesh filename="package://${MESH}/S2R1/eyelid_top.dae" />
-	      </geometry>
-      </visual>
-      <collision>
-	      <origin xyz="0 0 0" rpy="0.0 0.0 0.0 " />
-	      <geometry name="rt_eyelid_top_collision">
-		      <box size="0.01 0.01 0.01" />
-	      </geometry>
-      </collision>
-    </link>
-    <joint name="head_j7_rt_eyelid_bottom" type="revolute">
-	    <axis xyz="0 1 0" />
-       <limit effort="100" velocity="${1600*M_PI/180}" lower="${2.0*M_PI/180}" upper="${68.0*M_PI/180}" />
-      <origin xyz="0 0.0 0" rpy="0 -0.785 0" />
-      <parent link="right_eye"/>
-      <child link="rt_eyelid_bottom"/>
-    </joint>
-    <link name="rt_eyelid_bottom">
-      <visual>
-	      <material name="GreyC" />
-	      <origin xyz="0 0 0" rpy="0 0 0 " />
-	      <geometry name="eyelid_bottom_geom">
-		      <mesh filename="package://${MESH}/S2R1/eyelid_bottom.dae" />
-	      </geometry>
-      </visual>
-      <collision>
-	      <origin xyz="0 0 0" rpy="0.0 0.0 0.0 " />
-	      <geometry name="eyelid_bottom_collision">
-		      <box size="0.01 0.01 0.01" />
-	      </geometry>
-      </collision>
-    </link>
-    <joint name="head_j7_lt_eyelid_top" type="revolute">
-	    <axis xyz="0 -1 0" />
-       <limit effort="100" velocity="${1600*M_PI/180}" lower="${2.0*M_PI/180}" upper="${68.0*M_PI/180}" />
-      <origin xyz="0 0.0 0" rpy="0 0.785 0" />
-      <parent link="left_eye"/>
-      <child link="lt_eyelid_top"/>
-    </joint>
-    <link name="lt_eyelid_top">
-      <visual>
-	      <material name="GreyC" />
-	      <origin xyz="0 0 0" rpy="0 0 0 " />
-	      <geometry name="lt_eyelid_top_geom">
-		      <mesh filename="package://${MESH}/S2R1/eyelid_top.dae" />
-	      </geometry>
-      </visual>
-      <collision>
-	      <origin xyz="0 0 0" rpy="0.0 0.0 0.0 " />
-	      <geometry name="lt_eyelid_top_collision">
-		      <box size="0.01 0.01 0.01" />
-	      </geometry>
-      </collision>
-    </link>
-    <joint name="head_j7_lt_eyelid_bottom" type="revolute">
-	    <axis xyz="0 1 0" />
-       <limit effort="100" velocity="${1600*M_PI/180}" lower="${2.0*M_PI/180}" upper="${68.0*M_PI/180}" />
-      <origin xyz="0 0.0 0" rpy="0 -0.785 0" />
-      <parent link="left_eye"/>
-      <child link="lt_eyelid_bottom"/>
-    </joint>
-    <link name="lt_eyelid_bottom">
-      <visual>
-	      <material name="GreyC" />
-	      <origin xyz="0 0 0" rpy="0 0 0 " />
-	      <geometry name="eyelid_bottom_geom2">
-		      <mesh filename="package://${MESH}/S2R1/eyelid_bottom.dae" />
-	      </geometry>
-      </visual>
-      <collision>
-	      <origin xyz="0 0 0" rpy="0.0 0.0 0.0 " />
-	      <geometry name="eyelid_bottom_collision2">
-		      <box size="0.01 0.01 0.01" />
-	      </geometry>
-      </collision>
-    </link>
-     <joint name="head_j8" type="revolute">
-	    <axis xyz="0 0 1" />
-      <limit effort="100" velocity="${1600*M_PI/180}" lower="${-150.0*M_PI/180}" upper="${150.0*M_PI/180}" />
-      <origin xyz="0.022 0.138 0.120" rpy="-1.13 0 0" />
-      <parent link="head_shell"/>
-      <child link="ear_roll"/>
-    </joint>
-    <link name="ear_roll">
-      <visual>
-	      <material name="GreyC" />
-	      <origin xyz="0 0 0" rpy="0 0 0 " />
-	      <geometry name="ear_roll_geom">
-		      <mesh filename="package://${MESH}/S2R1/ear_mount.dae" />
-	      </geometry>
-      </visual>
-      <collision>
-	      <origin xyz="0 0 0" rpy="0.0 0.0 0.0 " />
-	      <geometry name="ear_roll_collision">
-		      <box size="0.01 0.01 0.01" />
-	      </geometry>
-      </collision>
-    </link>
-    <joint name="head_j9" type="revolute">
-	    <axis xyz="0 -1 0" />
-      <limit effort="100" velocity="${1600*M_PI/180}" lower="${0.0*M_PI/180}" upper="${123.0*M_PI/180}" />
-      <origin xyz="0.0 0.0 0.0" rpy="0 1.07 0" />
-      <parent link="ear_roll"/>
-      <child link="ear1"/>
-    </joint>
-    <link name="ear1">
-      <visual>
-	      <material name="GreyC" />
-	      <origin xyz="0 0 0" rpy="0 0 0 " />
-	      <geometry name="ear1_geom">
-		      <mesh filename="package://${MESH}/S2R1/ear.dae" />
-	      </geometry>
-      </visual>
-      <collision>
-	      <origin xyz="0 0 0" rpy="0.0 0.0 0.0 " />
-	      <geometry name="ear1_collision">
-		      <box size="0.01 0.01 0.01" />
-	      </geometry>
-      </collision>
-    </link>
-    <joint name="head_j10" type="revolute">
-	    <axis xyz="0 0 1" />
-       <limit effort="100" velocity="${1600*M_PI/180}" lower="${-150.0*M_PI/180}" upper="${150.0*M_PI/180}" />
-      <origin xyz="0.022 -0.138 0.120" rpy="1.13 0 0" />
-      <parent link="head_shell"/>
-      <child link="ear_roll2"/>
-    </joint>
-    <link name="ear_roll2">
-      <visual>
-	      <material name="GreyC" />
-	      <origin xyz="0 0 0" rpy="0 0 0 " />
-	      <geometry name="ear_roll_geom2">
-		      <mesh filename="package://${MESH}/S2R1/ear_mount.dae" />
-	      </geometry>
-      </visual>
-      <collision>
-	      <origin xyz="0 0 0" rpy="0.0 0.0 0.0 " />
-	      <geometry name="ear_roll_collision2">
-		      <box size="0.01 0.01 0.01" />
-	      </geometry>
-      </collision>
-    </link>
-    <joint name="head_j11" type="revolute">
-	    <axis xyz="0 -1 0" />
-     <limit effort="100" velocity="${1600*M_PI/180}" lower="${0.0*M_PI/180}" upper="${123.0*M_PI/180}" />
-      <origin xyz="0.0 0.0 0.0" rpy="0 1.07 0" />
-      <parent link="ear_roll2"/>
-      <child link="ear2"/>
-    </joint>
-    <link name="ear2">
-      <visual>
-	      <material name="GreyC" />
-	      <origin xyz="0 0 0" rpy="0 0 0 " />
-	      <geometry name="ear2_geom">
-		      <mesh filename="package://${MESH}/S2R1/ear.dae" />
-	      </geometry>
-      </visual>
-      <collision>
-	      <origin xyz="0 0 0" rpy="0.0 0.0 0.0 " />
-	      <geometry name="ear2_collision">
-		      <box size="0.01 0.01 0.01" />
-	      </geometry>
-      </collision>
-    </link>
 </macro>
   <macro name="m3_head" params="side parent reflect *origin">

Commit message: git-svn-id: file:///home/svn/meka-ros-pkg@178 cfd446f6-b9c6-49ad-a440-209cd04d0f1d

File: trunk/meka_description/robots/bie.urdf.xacro (robot description, xacro)
@@ -71,5 +71,5 @@
   <!-- Solid Base -->
   <joint name="chest_joint" type="fixed">
-	  <origin xyz="0 0 -0.03" rpy="0 0 0" />
+	  <origin xyz="0.1 0.0 0.0" rpy="0 0 0" />
     <parent link="zlift_link" />
     <child link="panplate" />
@@ -95,5 +95,5 @@
     </collision>
   </link>
-  <joint name="m3joint_${TORSO}_j0" type="continuous">
+  <joint name="torso_j0" type="continuous">
     <axis xyz="0 0 1"/>
     <origin xyz="0 0 0.1678" rpy="0 0 0" />
@@ -123,5 +123,5 @@
     </collision>
   </link>
-  <joint name="m3joint_${TORSO}_j1" type="continuous">
+  <joint name="torso_j1" type="continuous">
     <axis xyz="0 1 0"/>
     <origin xyz="0 0 0" rpy="0 0 0" />
@@ -156,5 +156,5 @@
     </collision>
   </link>
-  <joint name="m3joint_slave_${TORSO}_j2" type="continuous">
+  <joint name="torso_j2" type="continuous">
     <axis xyz="0 1 0"/>
     <origin xyz="0 0 0.1397" rpy="0 0 0" />
@@ -179,5 +179,5 @@
       <origin xyz="0 0 0" rpy="0 0 0" />
       <geometry name="upper_geom">
-        <mesh filename="package://${MESH}/T2R3/T2R3_TJ3_chest_waist_neck.dae" />
+       <mesh filename="package://${MESH}/A2R3/A2R3_T4_Chest_Neck.dae" />
       </geometry>
     </visual>

File: trunk/meka_description/urdf/S3R1_head_defs.urdf.xacro (robot description, xacro)
@@ -69,36 +69,4 @@
       </collision>
     </link>
-    <joint name="head_j2" type="revolute">
-      <axis xyz="-1 0 0" />
-      <origin xyz="0 0 0" rpy="0 0 0" />
-      <parent link="neck_roll" />
-      <child link="neck_yaw"/>
-      <limit effort="100" velocity="${50*M_PI/180}" lower="${-15.87*M_PI/180}" upper="${15.87*M_PI/180}" />
-    </joint>
-    <link name="neck_yaw">
-      <inertial>
-        <mass value="0.496" />
-	<origin xyz="-0.010690 0.053982 0.000045"/>
-	<inertia ixx="0.001094"
-	iyy="0.000311"
-	izz="0.001222"
-	ixy="0.000284"
-	ixz="0.000000"
-	iyz="0.000000" />
-      </inertial>
-      <visual>
-	      <material name="GreyC" />
-	      <origin xyz="0 0 0" rpy="0 0 0 " />
-	      <geometry name="S2R1_H3_neckYaw_geom">
-		      <mesh filename="package://${MESH}/S2R1/S2R1_H3_neckYaw.dae" />
-	      </geometry>
-      </visual>
-      <collision>
-	      <origin xyz="0 0 0" rpy="0.0 0.0 0.0 " />
-	      <geometry name="S2R1_H3_neckYaw_collision">
-		      <box size="0.01 0.01 0.01" />
-	      </geometry>
-      </collision>
-    </link>
 </macro>
   <macro name="m3_head" params="side parent reflect *origin">

Commit message: git-svn-id: file:///home/svn/meka-ros-pkg@189 cfd446f6-b9c6-49ad-a440-209cd04d0f1d

File: trunk/meka_description/robots/bie.urdf.xacro (robot description, xacro)
@@ -47,5 +47,6 @@
   </m3_l_hand>
   <m3_head side="r" reflect="1" parent="upper">
-    <origin xyz="0.0 0.0 0.31155" rpy="0 0 0" />
+    <origin xyz="0.0 0.0 0.385987" rpy="0 0 0" />
+    <!--    <origin xyz="0.0 0.0 0.2337" rpy="0 0 0" />-->
   </m3_head>
  <m3_r_arm side="r" reflect="1" parent="upper">
@@ -179,5 +180,6 @@
       <origin xyz="0 0 0" rpy="0 0 0" />
       <geometry name="upper_geom">
-       <mesh filename="package://${MESH}/A2R3/A2R3_T4_Chest_Neck.dae" />
+	<!--<mesh filename="package://${MESH}/A2R3/A2R3_T4_Chest_Neck.dae" />-->
+	  <mesh filename="package://${MESH}/A2R3/A2R3_T4_Chest.dae" />
       </geometry>
     </visual>

File: trunk/meka_description/urdf/S3R1_head_defs.urdf.xacro (robot description, xacro)
@@ -5,12 +5,12 @@
   <property name="M_PI" value="3.1415926535897931" />
   <macro name="m3_neck" params="side parent reflect *origin">
-    <joint name="head_j0" type="revolute">
-      <axis xyz="0 -1 0" />
+     <joint name="head_j1" type="revolute">
+      <axis xyz="0 0 1"/>
+     <limit effort="100" velocity="${75*M_PI/180}" lower="${-56.0*M_PI/180}" upper="${56.0*M_PI/180}" />
       <insert_block name="origin" /> <!-- transform from parent link to this joint frame -->
       <parent link="${parent}"/>
-      <child link="neck_tilt"/>
-      <limit effort="100" velocity="${20.0*M_PI/180}" lower="${-18.0*M_PI/180}" upper="${1.0*M_PI/180}" />
+      <child link="neck_pan"/>
     </joint>
-    <link name="neck_tilt">
+    <link name="neck_pan">
       <inertial>
         <mass value="0.940" />
@@ -25,7 +25,10 @@
       <visual>
 	      <material name="GreyA" />
-	      <origin xyz="0 0 0" rpy="0 0 0 " />
+	      <!--<origin xyz="0 0 0.0" rpy="0 0 0 " />-->
+	      <origin xyz="0 0 -0.152287" rpy="0 0 0 " />
 	      <geometry name="neck_tilt_geom">
-		      <mesh filename="package://${MESH}/S2R1/S2R1_SH1_neckTilt.dae" />
+		<!--<box size="0.01 0.01 0.01" />-->
+		<!--<mesh filename="package://${MESH}/S2R1/S2R1_SH1_neckTilt.dae" />-->
+		<mesh filename="package://${MESH}/S3R1/neck.dae" />
 	      </geometry>
       </visual>
@@ -37,12 +40,12 @@
       </collision>
     </link>
-    <joint name="head_j1" type="revolute">
-      <axis xyz="0 0 1"/>
-     <limit effort="100" velocity="${75*M_PI/180}" lower="${-56.0*M_PI/180}" upper="${56.0*M_PI/180}" />
-      <origin xyz="0 0 0.13849" rpy="0 0 0" />
-      <parent link="neck_tilt"/>
-      <child link="neck_roll"/>
+    <joint name="head_j0" type="revolute">
+      <axis xyz="0 -1 0" />
+      <origin xyz="0 0 0.0" rpy="0 0 0" />
+      <parent link="neck_pan"/>
+      <child link="shell"/>
+      <limit effort="100" velocity="${20.0*M_PI/180}" lower="${-18.0*M_PI/180}" upper="${1.0*M_PI/180}" />
     </joint>
-    <link name="neck_roll">
+    <link name="shell">
       <inertial>
         <mass value="0.409" />
@@ -58,11 +61,43 @@
 	      <material name="GreyB" />
 	      <origin xyz="0 0 0" rpy="0 0 0 " />
-	      <geometry name="neck_roll_geom">
-		      <mesh filename="package://${MESH}/S2R1/S2R1_SH2_neckRoll.dae" />
+	      <geometry name="shell_geom">
+		      <mesh filename="package://${MESH}/S3R1/S3.dae" />
 	      </geometry>
       </visual>
       <collision>
 	      <origin xyz="0 0 0" rpy="0.0 0.0 0.0 " />
-	      <geometry name="S2R1_SH2_neckRoll_collision">
+	      <geometry name="S3_collision">
+		      <box size="0.01 0.01 0.01" />
+	      </geometry>
+      </collision>
+    </link>
+    <joint name="head_j2" type="revolute">
+      <axis xyz="0 -1 0" />
+      <origin xyz="0.07975 0 0.123536" rpy="0 0 0" />
+      <parent link="shell"/>
+      <child link="BB3"/>
+      <limit effort="100" velocity="${20.0*M_PI/180}" lower="${-18.0*M_PI/180}" upper="${1.0*M_PI/180}" />
+    </joint>
+    <link name="BB3">
+      <inertial>
+        <mass value="0.409" />
+	<origin xyz="0.0 0.0 0.0"/>
+	<inertia ixx="0.0"
+	iyy="0.0"
+	izz="0.0"
+	ixy="0.0"
+	ixz="0.0"
+	iyz="0.0" />
+      </inertial>
+      <visual>
+	      <material name="GreyB" />
+	      <origin xyz="0 0 0" rpy="0 0 0 " />
+	      <geometry name="shell_geom">
+		      <mesh filename="package://${MESH}/S3R1/BB3.dae" />
+	      </geometry>
+      </visual>
+      <collision>
+	      <origin xyz="0 0 0" rpy="0.0 0.0 0.0 " />
+	      <geometry name="S3_collision">
 		      <box size="0.01 0.01 0.01" />
 	      </geometry>
