Commit message: git-svn-id: file:///home/svn/meka-ros-pkg@190 cfd446f6-b9c6-49ad-a440-209cd04d0f1d

File: trunk/meka_description/robots/bie.urdf.xacro (robot description, xacro)
@@ -47,6 +47,6 @@
   </m3_l_hand>
   <m3_head side="r" reflect="1" parent="upper">
-    <origin xyz="0.0 0.0 0.385987" rpy="0 0 0" />
-    <!--    <origin xyz="0.0 0.0 0.2337" rpy="0 0 0" />-->
+    <!--<origin xyz="0.0 0.0 0.385987" rpy="0 0 0" />-->
+    <origin xyz="0.0 0.0 0.2337" rpy="0 0 0" />
   </m3_head>
  <m3_r_arm side="r" reflect="1" parent="upper">

File: trunk/meka_description/robots/utk.urdf.xacro (robot description, xacro)
@@ -25,4 +25,6 @@
   <!--<include filename="$(find meka_description)/transmissions/H2R2_r_hand_defs.transmission.xacro" />-->
   <!--<include filename="$(find meka_description)/transmissions/S2R1_head_defs.transmission.xacro" />-->
+  <!-- Meka Head -->
+  <include filename="$(find meka_description)/urdf/S3R1_head_defs.urdf.xacro" />
    <property name="M_PI" value="3.1415926535897931" />
   <material name="GreyA"> <!-- darkest -->
@@ -44,7 +46,4 @@
     <origin xyz="0.0 0.0 0.0" rpy="0 0 0" />
   </m3_l_hand>
-  <m3_head side="r" reflect="1" parent="upper">
-    <origin xyz="0.0 0.0 0.31155" rpy="0 0 0" />
-  </m3_head>
  <m3_r_arm side="r" reflect="1" parent="upper">
     <origin xyz="0.0 -0.18465 0.2337" rpy="0 0 0" />
@@ -53,4 +52,7 @@
     <origin xyz="0.0 0.18465 0.2337" rpy="0 0 0" />
   </m3_l_arm>
+  <m3_head side="r" reflect="1" parent="upper">
+    <origin xyz="0.0 0.0 0.2337" rpy="0 0 0" />
+  </m3_head>
   <link name="world" />
   <link name="base_link" />
@@ -83,5 +85,6 @@
 		  <origin xyz="0 0 0" rpy="0 0 0" />
 		  <geometry name="upper_geom">
-			  <mesh filename="package://${MESH}/A2R3/A2R3_T4_Chest_Neck.dae" />
+		    <!--<mesh filename="package://${MESH}/A2R3/A2R3_T4_Chest_Neck.dae" />-->
+		    <mesh filename="package://${MESH}/A2R3/A2R3_T4_Chest2.dae" />
 		  </geometry>
 		  <material name="Blue" />

File: trunk/meka_description/urdf/S3R1_head_defs.urdf.xacro (robot description, xacro)
@@ -26,5 +26,5 @@
 	      <material name="GreyA" />
 	      <!--<origin xyz="0 0 0.0" rpy="0 0 0 " />-->
-	      <origin xyz="0 0 -0.152287" rpy="0 0 0 " />
+	      <origin xyz="0 0 0" rpy="0 0 0 " />
 	      <geometry name="neck_tilt_geom">
 		<!--<box size="0.01 0.01 0.01" />-->
@@ -42,5 +42,5 @@
     <joint name="head_j0" type="revolute">
       <axis xyz="0 -1 0" />
-      <origin xyz="0 0 0.0" rpy="0 0 0" />
+      <origin xyz="0 0 0.152287" rpy="0 0 0" />
       <parent link="neck_pan"/>
       <child link="shell"/>

Commit message: git-svn-id: file:///home/svn/meka-ros-pkg@195 cfd446f6-b9c6-49ad-a440-209cd04d0f1d

File: trunk/meka_description/robots/bie.urdf.xacro (robot description, xacro)
@@ -68,5 +68,5 @@
   </meka_base>
   <meka_zlift  side="r" reflect="1" parent="dummy_3">
-    <origin xyz="0.43 0.0 0.75" rpy="0 0 0" />
+    <origin xyz="0.43 0.0 0.45" rpy="0 0 0" />
   </meka_zlift>
   <!-- Solid Base -->

File: trunk/meka_description/urdf/H2R4_l_hand_defs.urdf.xacro (robot description, xacro)
@@ -38,5 +38,5 @@
     <joint name="left_hand_j0" type="revolute">
       <axis xyz="0 0 -1" />
-      <origin xyz="-0.02 -0.028 -0.03" rpy="0 0 0" />
+      <origin xyz="-0.02 -0.028 -0.03" rpy="0 0 ${90.0*M_PI/180}" />
       <parent link="l_palm"/>
       <child link="l_thumb0"/>
@@ -56,5 +56,5 @@
       <visual>
 	      <material name="GreyA" />
-	      <origin xyz="0 0 0" rpy="0 0 0 " />
+	      <origin xyz="0 0 0" rpy="${0.0*M_PI/180} 0 0 " />
 	      <geometry name="l_thumb0_geom">
 		      <mesh filename="package://${MESH}/H2R3/H2R3_RJ0_thumb_abductlink.dae" />
