Commit message: git-svn-id: file:///home/svn/meka-ros-pkg@187 cfd446f6-b9c6-49ad-a440-209cd04d0f1d

File: trunk/meka_description/robots/uja.urdf.xacro (robot description, xacro)
@@ -41,16 +41,7 @@
     <origin xyz="0.0 0.0 0.0" rpy="0 0 0" />
   </m3_r_hand>
-  <m3_l_hand side="l" reflect="1" parent="handmount_LEFT">
-    <origin xyz="0.0 0.0 0.0" rpy="0 0 0" />
-  </m3_l_hand>
-  <m3_head side="r" reflect="1" parent="upper">
-    <origin xyz="0.0 0.0 0.31155" rpy="0 0 0" />
-  </m3_head>
  <m3_r_arm side="r" reflect="1" parent="upper">
     <origin xyz="0.0 -0.18465 0.2337" rpy="0 0 0" />
   </m3_r_arm>
- <m3_l_arm side="l" reflect="1" parent="upper">
-    <origin xyz="0.0 0.18465 0.2337" rpy="0 0 0" />
-  </m3_l_arm>
   <link name="world" />
   <link name="base_link" />
@@ -61,14 +52,8 @@
     <child link="base_link" />
   </joint>
-  <meka_base  side="r" reflect="1" parent="base_link">
-    <origin xyz="0.0 0.0 0.0" rpy="0 0 0" />
-  </meka_base>
-  <meka_zlift  side="r" reflect="1" parent="dummy_3">
-    <origin xyz="0.43 0.0 0.75" rpy="0 0 0" />
-  </meka_zlift>
   <!-- Solid Base -->
   <joint name="chest_joint" type="fixed">
 	  <origin xyz="0 0 -0.03" rpy="0 0 0" />
-    <parent link="zlift_link" />
+    <parent link="base_link" />
     <child link="upper" />
   </joint>

File: trunk/meka_description/urdf/H2R4_r_hand_defs.urdf.xacro (robot description, xacro)
@@ -37,6 +37,6 @@
 <!-- Start Thumb -->
     <joint name="right_hand_j0" type="revolute">
-      <axis xyz="0 0 -1" />
-      <origin xyz="-0.02 0.028 -0.03" rpy="0 0 0" />
+      <axis xyz="0 0 1" />
+      <origin xyz="-0.02 0.028 -0.03" rpy="0 0 -1.57" />
       <parent link="palm"/>
       <child link="thumb0"/>

Commit message: git-svn-id: file:///home/svn/meka-ros-pkg@197 cfd446f6-b9c6-49ad-a440-209cd04d0f1d

File: trunk/meka_description/robots/uja.urdf.xacro (robot description, xacro)
@@ -11,8 +11,4 @@
   <include filename="$(find meka_description)/gazebo/gazebo.urdf.xacro" />
   <!--<include filename="$(find meka_description)/transmissions/uta.transmission.xacro" />-->
-<!-- Meka Base -->
-  <include filename="$(find meka_description)/urdf/B1R2B_defs.urdf.xacro" />
-<!-- Meka Zlift -->
-  <include filename="$(find meka_description)/urdf/Z1R2B_defs.urdf.xacro" />
 <!-- Meka Arm -->
   <include filename="$(find meka_description)/urdf/A2R4_r_arm_defs.urdf.xacro" />
@@ -44,4 +40,10 @@
     <origin xyz="0.0 -0.18465 0.2337" rpy="0 0 0" />
   </m3_r_arm>
+  <m3_l_hand side="l" reflect="1" parent="handmount_LEFT">
+    <origin xyz="0.0 0.0 0.0" rpy="0 0 0" />
+  </m3_l_hand>
+   <m3_l_arm side="l" reflect="1" parent="upper">
+    <origin xyz="0.0 0.18465 0.2337" rpy="0 0 0" />
+  </m3_l_arm>
   <link name="world" />
   <link name="base_link" />
