Commit message: restored our head urdfs and meshes

File: meka_description/urdf/S3R1_simple_head_defs.urdf.xacro (robot description, xacro)
@@ -72,36 +72,4 @@
       </collision>
     </link>
-    <joint name="head_j2" type="revolute">
-      <axis xyz="0 -1 0" />
-      <origin xyz="0.07975 0 0.123536" rpy="0 0 0" />
-      <parent link="shell"/>
-      <child link="BB3"/>
-      <limit effort="100" velocity="${20.0*M_PI/180}" lower="${-18.0*M_PI/180}" upper="${1.0*M_PI/180}" />
-    </joint>
-    <link name="BB3">
-      <inertial>
-        <mass value="0.409" />
-	<origin xyz="0.0 0.0 0.0"/>
-	<inertia ixx="0.0"
-	iyy="0.0"
-	izz="0.0"
-	ixy="0.0"
-	ixz="0.0"
-	iyz="0.0" />
-      </inertial>
-      <visual>
-	      <material name="GreyB" />
-	      <origin xyz="0 0 0" rpy="0 0 0 " />
-	      <geometry name="shell_geom">
-		      <mesh filename="package://${MESH}/S3R1/BB3.dae" />
-	      </geometry>
-      </visual>
-      <collision>
-	      <origin xyz="0 0 0" rpy="0.0 0.0 0.0 " />
-	      <geometry name="S3_collision">
-		      <box size="0.01 0.01 0.01" />
-	      </geometry>
-      </collision>
-    </link>
 </macro>
   <macro name="m3_head" params="side parent reflect *origin">
