Commit message: modified hands urdf files to comply with joint denotation of the robot source

File: meka_description/urdf/H2R4_l_hand_defs.urdf.xacro (robot description, xacro)
@@ -100,5 +100,5 @@
       </collision>
     </link>
-    <joint name="left_hand_j2" type="revolute">
+    <joint name="left_hand_j5" type="revolute">
       <axis xyz="0 -1 0" />
       <origin xyz="-0.044 0 0" rpy="0 0 0" />
@@ -132,5 +132,5 @@
       </collision>
     </link>
-    <joint name="left_hand_j3" type="revolute">
+    <joint name="left_hand_j6" type="revolute">
       <axis xyz="0 -1 0" />
       <origin xyz="-0.035 0 0" rpy="0 0 0" />
@@ -141,5 +141,5 @@
     <link name="thumb_end_left"/>
 <!-- Start Index Finger -->
-    <joint name="left_hand_j4" type="revolute">
+    <joint name="left_hand_j2" type="revolute">
       <axis xyz="0 1 0" />
       <origin xyz="0 0.028 -0.101" rpy="0 0 0" />
@@ -173,5 +173,5 @@
       </collision>
     </link>
-    <joint name="left_hand_j5" type="revolute">
+    <joint name="left_hand_j7" type="revolute">
       <axis xyz="0 1 0" />
       <limit effort="100" velocity="${1600*M_PI/180}" lower="${-34.99*M_PI/180}" upper="${34.99*M_PI/180}" />
@@ -195,6 +195,6 @@
 	      <origin xyz="0 0 0" rpy="0 0 0 " />
 	      <geometry name="index1_geom_left">
+	      </geometry>
 		      <mesh filename="package://${MESH}/H2R3/H2R3_finger_knuckle2.dae" />
-	      </geometry>
       </visual>
       <collision>
@@ -205,5 +205,5 @@
       </collision>
     </link>
-    <joint name="left_hand_j6" type="revolute">
+    <joint name="left_hand_j8" type="revolute">
       <axis xyz="0 1 0" />
       <limit effort="100" velocity="${1600*M_PI/180}" lower="${-34.21*M_PI/180}" upper="${34.213*M_PI/180}" />
@@ -237,5 +237,5 @@
       </collision>
     </link>
-    <joint name="left_hand_j7" type="revolute">
+    <joint name="left_hand_j9" type="revolute">
       <axis xyz="0 1 0" />
       <limit effort="100" velocity="${1600*M_PI/180}" lower="${-34.21*M_PI/180}" upper="${34.213*M_PI/180}" />
@@ -246,5 +246,5 @@
     <link name="index_end_left"/>
 <!-- Start Ring Finger -->
-    <joint name="left_hand_j8" type="revolute">
+    <joint name="left_hand_j3" type="revolute">
       <axis xyz="0 1 0" />
       <origin xyz="0 0 -0.101" rpy="0 0 0" />
@@ -278,5 +278,5 @@
       </collision>
     </link>
-    <joint name="left_hand_j9" type="revolute">
+    <joint name="left_hand_j10" type="revolute">
       <axis xyz="0 1 0" />
       <limit effort="100" velocity="${1600*M_PI/180}" lower="${-34.99*M_PI/180}" upper="${34.99*M_PI/180}" />
@@ -310,5 +310,5 @@
       </collision>
     </link>
-    <joint name="left_hand_j10" type="revolute">
+    <joint name="left_hand_j11" type="revolute">
       <axis xyz="0 1 0" />
       <limit effort="100" velocity="${1600*M_PI/180}" lower="${-34.21*M_PI/180}" upper="${34.213*M_PI/180}" />
@@ -342,5 +342,5 @@
       </collision>
     </link>
-    <joint name="left_hand_j11" type="revolute">
+    <joint name="left_hand_j12" type="revolute">
       <axis xyz="0 1 0" />
       <limit effort="100" velocity="${1600*M_PI/180}" lower="${-34.21*M_PI/180}" upper="${34.213*M_PI/180}" />
@@ -351,5 +351,5 @@
     <link name="ring_end_left"/>
 <!-- Start Pinky Finger -->
-    <joint name="left_hand_j12" type="revolute">
+    <joint name="left_hand_j4" type="revolute">
       <axis xyz="0 1 0" />
       <origin xyz="0 -0.028 -0.101" rpy="0 0 0" />

File: meka_description/urdf/H2R4_r_hand_defs.urdf.xacro (robot description, xacro)
@@ -100,5 +100,5 @@
       </collision>
     </link>
-    <joint name="right_hand_j2" type="revolute">
+    <joint name="right_hand_j5" type="revolute">
       <axis xyz="0 -1 0" />
       <origin xyz="-0.044 0 0" rpy="0 0 0" />
@@ -132,5 +132,5 @@
       </collision>
     </link>
-    <joint name="right_hand_j3" type="revolute">
+    <joint name="right_hand_j6" type="revolute">
       <axis xyz="0 -1 0" />
       <origin xyz="-0.035 0 0" rpy="0 0 0" />
@@ -141,5 +141,5 @@
     <link name="thumb_end_right"/>
 <!-- Start Index Finger -->
-    <joint name="right_hand_j4" type="revolute">
+    <joint name="right_hand_j2" type="revolute">
       <axis xyz="0 1 0" />
       <origin xyz="0 0.028 -0.101" rpy="0 0 0" />
@@ -173,5 +173,5 @@
       </collision>
     </link>
-    <joint name="right_hand_j5" type="revolute">
+    <joint name="right_hand_j7" type="revolute">
       <axis xyz="0 1 0" />
       <limit effort="100" velocity="${1600*M_PI/180}" lower="${-34.99*M_PI/180}" upper="${34.99*M_PI/180}" />
@@ -205,5 +205,5 @@
       </collision>
     </link>
-    <joint name="right_hand_j6" type="revolute">
+    <joint name="right_hand_j8" type="revolute">
       <axis xyz="0 1 0" />
       <limit effort="100" velocity="${1600*M_PI/180}" lower="${-34.21*M_PI/180}" upper="${34.213*M_PI/180}" />
@@ -237,5 +237,5 @@
       </collision>
     </link>
-    <joint name="right_hand_j7" type="revolute">
+    <joint name="right_hand_j9" type="revolute">
       <axis xyz="0 1 0" />
       <limit effort="100" velocity="${1600*M_PI/180}" lower="${-34.21*M_PI/180}" upper="${34.213*M_PI/180}" />
@@ -246,5 +246,5 @@
     <link name="index_end_right"/>
 <!-- Start Ring Finger -->
-    <joint name="right_hand_j8" type="revolute">
+    <joint name="right_hand_j3" type="revolute">
       <axis xyz="0 1 0" />
       <origin xyz="0 0 -0.101" rpy="0 0 0" />
@@ -278,5 +278,5 @@
       </collision>
     </link>
-    <joint name="right_hand_j9" type="revolute">
+    <joint name="right_hand_j10" type="revolute">
       <axis xyz="0 1 0" />
       <limit effort="100" velocity="${1600*M_PI/180}" lower="${-34.99*M_PI/180}" upper="${34.99*M_PI/180}" />
@@ -310,5 +310,5 @@
       </collision>
     </link>
-    <joint name="right_hand_j10" type="revolute">
+    <joint name="right_hand_j11" type="revolute">
       <axis xyz="0 1 0" />
       <limit effort="100" velocity="${1600*M_PI/180}" lower="${-34.21*M_PI/180}" upper="${34.213*M_PI/180}" />
@@ -342,5 +342,5 @@
       </collision>
     </link>
-    <joint name="right_hand_j11" type="revolute">
+    <joint name="right_hand_j12" type="revolute">
       <axis xyz="0 1 0" />
       <limit effort="100" velocity="${1600*M_PI/180}" lower="${-34.21*M_PI/180}" upper="${34.213*M_PI/180}" />
@@ -351,5 +351,5 @@
     <link name="ring_end_right"/>
 <!-- Start Pinky Finger -->
-    <joint name="right_hand_j12" type="revolute">
+    <joint name="right_hand_j4" type="revolute">
       <axis xyz="0 1 0" />
       <origin xyz="0 -0.028 -0.101" rpy="0 0 0" />

Commit message: Changed end revolute joints to dummy fixed joints and renamed end as tip Removed wrong mimic for thumb Renumbered the joints to finish at j11

File: meka_description/urdf/H2R4_l_hand_defs.urdf.xacro (robot description, xacro)
@@ -140,19 +140,14 @@
       </collision>
     </link>
-    <joint name="left_hand_j6" type="revolute">
-      <axis xyz="0 -1 0" />
+    <joint name="left_hand_thumb_dummy" type="fixed">
       <origin xyz="-0.035 0 0" rpy="0 0 0" />
       <parent link="thumb2_left" />
-      <child link="thumb_end_left"/>
-      <limit effort="100" velocity="${50*M_PI/180}" lower="${-14.94*M_PI/180}" upper="${14.94*M_PI/180}" />
-      <xacro:if value="${use_mimic}">
-				<mimic joint="left_hand_j1" multiplier="${th_middist_coupling}"/>
-			</xacro:if>
-    </joint>
-    <link name="thumb_end_left"/>
+      <child link="thumb_tip_left"/>
+    </joint>
+    <link name="thumb_tip_left"/>
 <!-- Start Index Finger -->
     <joint name="left_hand_j2" type="revolute">
       <axis xyz="0 1 0" />
-      <origin xyz="0 0.028 -0.101" rpy="0 0 0" />
+      <origin xyz="0 -0.028 -0.101" rpy="0 0 0" />
       <parent link="palm_left" />
       <child link="index0_left"/>
@@ -184,5 +179,5 @@
       </collision>
     </link>
-    <joint name="left_hand_j7" type="revolute">
+    <joint name="left_hand_j6" type="revolute">
       <axis xyz="0 1 0" />
       <limit effort="100" velocity="${1600*M_PI/180}" lower="${-34.99*M_PI/180}" upper="${34.99*M_PI/180}" />
@@ -219,5 +214,5 @@
       </collision>
     </link>
-    <joint name="left_hand_j8" type="revolute">
+    <joint name="left_hand_j7" type="revolute">
       <axis xyz="0 1 0" />
       <limit effort="100" velocity="${1600*M_PI/180}" lower="${-34.21*M_PI/180}" upper="${34.213*M_PI/180}" />
@@ -254,12 +249,10 @@
       </collision>
     </link>
-    <joint name="left_hand_j9" type="revolute">
-      <axis xyz="0 1 0" />
-      <limit effort="100" velocity="${1600*M_PI/180}" lower="${-34.21*M_PI/180}" upper="${34.213*M_PI/180}" />
+    <joint name="left_hand_index_dummy" type="fixed">
       <origin xyz="0 0.008 -0.025" rpy="0 0 0" />
       <parent link="index2_left"/>
-      <child link="index_end_left"/>
-    </joint>
-    <link name="index_end_left"/>
+      <child link="index_tip_left"/>
+    </joint>
+    <link name="index_tip_left"/>
 <!-- Start Ring Finger -->
     <joint name="left_hand_j3" type="revolute">
@@ -295,5 +288,5 @@
       </collision>
     </link>
-    <joint name="left_hand_j10" type="revolute">
+    <joint name="left_hand_j8" type="revolute">
       <axis xyz="0 1 0" />
       <limit effort="100" velocity="${1600*M_PI/180}" lower="${-34.99*M_PI/180}" upper="${34.99*M_PI/180}" />
@@ -330,5 +323,5 @@
       </collision>
     </link>
-    <joint name="left_hand_j11" type="revolute">
+    <joint name="left_hand_j9" type="revolute">
       <axis xyz="0 1 0" />
       <limit effort="100" velocity="${1600*M_PI/180}" lower="${-34.21*M_PI/180}" upper="${34.213*M_PI/180}" />
@@ -365,16 +358,16 @@
       </collision>
     </link>
-    <joint name="left_hand_j12" type="revolute">
+    <joint name="left_hand_ring_dummy" type="fixed">
       <axis xyz="0 1 0" />
       <limit effort="100" velocity="${1600*M_PI/180}" lower="${-34.21*M_PI/180}" upper="${34.213*M_PI/180}" />
       <origin xyz="0 0.008 -0.025" rpy="0 0 0" />
       <parent link="ring2_left"/>
-      <child link="ring_end_left"/>
-    </joint>
-    <link name="ring_end_left"/>
+      <child link="ring_tip_left"/>
+    </joint>
+    <link name="ring_tip_left"/>
 <!-- Start Pinky Finger -->
     <joint name="left_hand_j4" type="revolute">
       <axis xyz="0 1 0" />
-      <origin xyz="0 -0.028 -0.101" rpy="0 0 0" />
+      <origin xyz="0 0.028 -0.101" rpy="0 0 0" />
       <parent link="palm_left" />
       <child link="pinky0_left"/>
@@ -406,5 +399,5 @@
       </collision>
     </link>
-    <joint name="left_hand_j13" type="revolute">
+    <joint name="left_hand_j10" type="revolute">
       <axis xyz="0 1 0" />
       <limit effort="100" velocity="${1600*M_PI/180}" lower="${-34.99*M_PI/180}" upper="${34.99*M_PI/180}" />
@@ -441,5 +434,5 @@
       </collision>
     </link>
-    <joint name="left_hand_j14" type="revolute">
+    <joint name="left_hand_j11" type="revolute">
       <axis xyz="0 1 0" />
       <limit effort="100" velocity="${1600*M_PI/180}" lower="${-34.21*M_PI/180}" upper="${34.213*M_PI/180}" />
@@ -476,12 +469,12 @@
       </collision>
     </link>
-    <joint name="left_hand_j15" type="revolute">
+    <joint name="left_hand_pinky_dummy" type="fixed">
       <axis xyz="0 1 0" />
       <limit effort="100" velocity="${1600*M_PI/180}" lower="${-34.21*M_PI/180}" upper="${34.213*M_PI/180}" />
       <origin xyz="0 0.008 -0.025" rpy="0 0 0" />
       <parent link="pinky2_left"/>
-      <child link="pinky_end_left"/>
-    </joint>
-    <link name="pinky_end_left"/>
+      <child link="pinky_tip_left"/>
+    </joint>
+    <link name="pinky_tip_left"/>
 </macro>
   <macro name="m3_l_hand" params="side parent reflect use_mimic:=false *origin">

File: meka_description/urdf/H2R4_r_hand_defs.urdf.xacro (robot description, xacro)
@@ -140,15 +140,10 @@
       </collision>
     </link>
-    <joint name="right_hand_j6" type="revolute">
-      <axis xyz="0 -1 0" />
+    <joint name="right_hand_thumb_dummy" type="fixed">
       <origin xyz="-0.035 0 0" rpy="0 0 0" />
       <parent link="thumb2_right" />
-      <child link="thumb_end_right"/>
-      <limit effort="100" velocity="${50*M_PI/180}" lower="${-14.94*M_PI/180}" upper="${14.94*M_PI/180}" />
-      <xacro:if value="${use_mimic}">
-				<mimic joint="right_hand_j1" multiplier="${th_middist_coupling}"/>
-			</xacro:if>
-    </joint>
-    <link name="thumb_end_right"/>
+      <child link="thumb_tip_right"/>
+    </joint>
+    <link name="thumb_tip_right"/>
 <!-- Start Index Finger -->
     <joint name="right_hand_j2" type="revolute">
@@ -184,5 +179,5 @@
       </collision>
     </link>
-    <joint name="right_hand_j7" type="revolute">
+    <joint name="right_hand_j6" type="revolute">
       <axis xyz="0 1 0" />
       <limit effort="100" velocity="${1600*M_PI/180}" lower="${-34.99*M_PI/180}" upper="${34.99*M_PI/180}" />
@@ -219,5 +214,5 @@
       </collision>
     </link>
-    <joint name="right_hand_j8" type="revolute">
+    <joint name="right_hand_j7" type="revolute">
       <axis xyz="0 1 0" />
       <limit effort="100" velocity="${1600*M_PI/180}" lower="${-34.21*M_PI/180}" upper="${34.213*M_PI/180}" />
@@ -254,12 +249,10 @@
       </collision>
     </link>
-    <joint name="right_hand_j9" type="revolute">
-      <axis xyz="0 1 0" />
-      <limit effort="100" velocity="${1600*M_PI/180}" lower="${-34.21*M_PI/180}" upper="${34.213*M_PI/180}" />
+    <joint name="right_hand_index_dummy" type="fixed">
       <origin xyz="0 0.008 -0.025" rpy="0 0 0" />
       <parent link="index2_right"/>
-      <child link="index_end_right"/>
-    </joint>
-    <link name="index_end_right"/>
+      <child link="index_tip_right"/>
+    </joint>
+    <link name="index_tip_right"/>
 <!-- Start Ring Finger -->
     <joint name="right_hand_j3" type="revolute">
@@ -295,5 +288,5 @@
       </collision>
     </link>
-    <joint name="right_hand_j10" type="revolute">
+    <joint name="right_hand_j8" type="revolute">
       <axis xyz="0 1 0" />
       <limit effort="100" velocity="${1600*M_PI/180}" lower="${-34.99*M_PI/180}" upper="${34.99*M_PI/180}" />
@@ -330,5 +323,5 @@
       </collision>
     </link>
-    <joint name="right_hand_j11" type="revolute">
+    <joint name="right_hand_j9" type="revolute">
       <axis xyz="0 1 0" />
       <limit effort="100" velocity="${1600*M_PI/180}" lower="${-34.21*M_PI/180}" upper="${34.213*M_PI/180}" />
@@ -365,12 +358,10 @@
       </collision>
     </link>
-    <joint name="right_hand_j12" type="revolute">
-      <axis xyz="0 1 0" />
-      <limit effort="100" velocity="${1600*M_PI/180}" lower="${-34.21*M_PI/180}" upper="${34.213*M_PI/180}" />
+    <joint name="right_hand_ring_dummy" type="fixed">
       <origin xyz="0 0.008 -0.025" rpy="0 0 0" />
       <parent link="ring2_right"/>
-      <child link="ring_end_right"/>
-    </joint>
-    <link name="ring_end_right"/>
+      <child link="ring_tip_right"/>
+    </joint>
+    <link name="ring_tip_right"/>
 <!-- Start Pinky Finger -->
     <joint name="right_hand_j4" type="revolute">
@@ -406,5 +397,5 @@
       </collision>
     </link>
-    <joint name="right_hand_j13" type="revolute">
+    <joint name="right_hand_j10" type="revolute">
       <axis xyz="0 1 0" />
       <limit effort="100" velocity="${1600*M_PI/180}" lower="${-34.99*M_PI/180}" upper="${34.99*M_PI/180}" />
@@ -441,5 +432,5 @@
       </collision>
     </link>
-    <joint name="right_hand_j14" type="revolute">
+    <joint name="right_hand_j11" type="revolute">
       <axis xyz="0 1 0" />
       <limit effort="100" velocity="${1600*M_PI/180}" lower="${-34.21*M_PI/180}" upper="${34.213*M_PI/180}" />
@@ -476,12 +467,10 @@
       </collision>
     </link>
-    <joint name="right_hand_j15" type="revolute">
-      <axis xyz="0 1 0" />
-      <limit effort="100" velocity="${1600*M_PI/180}" lower="${-34.21*M_PI/180}" upper="${34.213*M_PI/180}" />
+    <joint name="right_hand_pinky_dummy" type="fixed">
       <origin xyz="0 0.008 -0.025" rpy="0 0 0" />
       <parent link="pinky2_right"/>
-      <child link="pinky_end_right"/>
-    </joint>
-    <link name="pinky_end_right"/>
+      <child link="pinky_tip_right"/>
+    </joint>
+    <link name="pinky_tip_right"/>
 </macro>
   <macro name="m3_r_hand" params="side parent reflect use_mimic:=false *origin">

Commit message: added virtual link (TCP)

File: meka_description/urdf/H2R4_l_hand_defs.urdf.xacro (robot description, xacro)
@@ -79,4 +79,36 @@
       </collision>
     </link>
+    <!-- this defines TCP Tool Center Point as described in: https://groups.google.com/forum/m/#!topic/moveit-users/VB7VWsgV9-g -->
+  <joint name="hand_left_tool_frame_joint" type="fixed">
+    <parent link="${parent}"/>
+    <child link="hand_tool_frame_left" />
+    <origin xyz="-0.02 0 -0.12" rpy="0 -1.570796 0"/>
+  </joint>
+  <link name="hand_tool_frame_left">
+    <!-- This is the coordinate system of the end effector (this is the position
+         used in IK); there is no actual arm part attached to this link -->
+    <!-- The fake geometry here is only present to work around https://github.com/ros-planning/moveit_core/issues/158 -->
+    <visual>
+      <origin rpy="0 0 0" xyz="0 0 0"/>
+      <geometry>
+        <box size="0.01 0.01 0.01"/>
+      </geometry>
+      <material name="red" />
+    </visual>
+    <collision>
+      <origin rpy="0 0 0" xyz="0 0 -0.01"/>
+      <geometry>
+        <box size="0.001 0.001 0.001"/>
+      </geometry>
+      <material name="red" />
+    </collision>
+    <inertial>
+      <mass value="0.01" />
+      <origin xyz="0 0 0"/>
+      <inertia ixx="0.0" ixy="0.0" ixz="0.0"
+        iyy="0.0" iyz="0.0"
+        izz="0.0" />
+    </inertial>
+  </link>
 <!-- Start Thumb -->
     <joint name="left_hand_j0" type="revolute">

Commit message: Added a collision box to protect hand cables

File: meka_description/urdf/H2R4_l_hand_defs.urdf.xacro (robot description, xacro)
@@ -46,4 +46,10 @@
         <geometry>
           <box size="0.04 0.0972 0.07" />
+        </geometry>
+      </collision>
+      <collision>
+        <origin xyz="0.02 0.06 -0.030" rpy="0.0 0.0 0.0 " />
+        <geometry>
+          <box size="0.022 0.023 0.03" />
         </geometry>
       </collision>

File: meka_description/urdf/H2R4_r_hand_defs.urdf.xacro (robot description, xacro)
@@ -47,4 +47,10 @@
         <geometry>
           <box size="0.04 0.0972 0.07" />
+        </geometry>
+      </collision>
+      <collision>
+        <origin xyz="0.02 -0.06 -0.030" rpy="0.0 0.0 0.0 " />
+        <geometry>
+          <box size="0.022 0.023 0.03" />
         </geometry>
       </collision>

Commit message: adjusted hand coordinate system

File: meka_description/urdf/H2R4_l_hand_defs.urdf.xacro (robot description, xacro)
@@ -89,5 +89,5 @@
     <parent link="${parent}"/>
     <child link="hand_tool_frame_left" />
-    <origin xyz="-0.02 0 -0.12" rpy="0 -1.570796 0"/>
+    <origin xyz="-0.02 0 -0.12" rpy="-3.141592 1.570796 0"/>
   </joint>
   <link name="hand_tool_frame_left">

Commit message: Added and fixed tool frame Added install for meka_description

File: meka_description/urdf/H2R4_l_hand_defs.urdf.xacro (robot description, xacro)
@@ -89,5 +89,5 @@
     <parent link="${parent}"/>
     <child link="hand_tool_frame_left" />
-    <origin xyz="-0.02 0 -0.12" rpy="-3.141592 1.570796 0"/>
+    <origin xyz="-0.02 0 -0.12" rpy="-1.5708 0 1.5708"/>
   </joint>
   <link name="hand_tool_frame_left">

File: meka_description/urdf/H2R4_r_hand_defs.urdf.xacro (robot description, xacro)
@@ -85,4 +85,36 @@
         </geometry>
       </collision>
+    </link>
+      <!-- this defines TCP Tool Center Point as described in: https://groups.google.com/forum/m/#!topic/moveit-users/VB7VWsgV9-g -->
+    <joint name="hand_right_tool_frame_joint" type="fixed">
+      <parent link="${parent}"/>
+      <child link="hand_tool_frame_right" />
+      <origin xyz="-0.02 0 -0.12" rpy="-1.5708 0 1.5708"/>
+    </joint>
+    <link name="hand_tool_frame_right">
+      <!-- This is the coordinate system of the end effector (this is the position
+           used in IK); there is no actual arm part attached to this link -->
+      <!-- The fake geometry here is only present to work around https://github.com/ros-planning/moveit_core/issues/158 -->
+      <visual>
+        <origin rpy="0 0 0" xyz="0 0 0"/>
+        <geometry>
+          <box size="0.01 0.01 0.01"/>
+        </geometry>
+        <material name="red" />
+      </visual>
+      <collision>
+        <origin rpy="0 0 0" xyz="0 0 -0.01"/>
+        <geometry>
+          <box size="0.001 0.001 0.001"/>
+        </geometry>
+        <material name="red" />
+      </collision>
+      <inertial>
+        <mass value="0.01" />
+        <origin xyz="0 0 0"/>
+        <inertia ixx="0.0" ixy="0.0" ixz="0.0"
+          iyy="0.0" iyz="0.0"
+          izz="0.0" />
+      </inertial>
     </link>
 <!-- Start Thumb -->

Commit message: added ft-sensors to urdf

File: meka_description/urdf/H2R4_l_hand_defs.urdf.xacro (robot description, xacro)
@@ -85,4 +85,10 @@
       </collision>
     </link>
+    <joint name="fts_frame_joint_left" type="fixed">
+      <parent link="${parent}"/>
+      <child link="m3loadx6_ma30_l0" />
+      <origin xyz="0.0 0.0 -0.055" rpy="0.0 ${M_PI} 0.0"/>
+    </joint>
+    <link name="m3loadx6_ma30_l0"/>
     <!-- this defines TCP Tool Center Point as described in: https://groups.google.com/forum/m/#!topic/moveit-users/VB7VWsgV9-g -->
   <joint name="hand_left_tool_frame_joint" type="fixed">

File: meka_description/urdf/H2R4_r_hand_defs.urdf.xacro (robot description, xacro)
@@ -86,4 +86,10 @@
       </collision>
     </link>
+    <joint name="fts_frame_joint_right" type="fixed">
+      <parent link="${parent}"/>
+      <child link="m3loadx6_ma29_l0" />
+      <origin xyz="0.0 0.0 -0.055" rpy="0.0 ${M_PI} 0.0"/>
+    </joint>
+    <link name="m3loadx6_ma29_l0"/>
       <!-- this defines TCP Tool Center Point as described in: https://groups.google.com/forum/m/#!topic/moveit-users/VB7VWsgV9-g -->
     <joint name="hand_right_tool_frame_joint" type="fixed">
