Commit message: shifting the visual of the forearm to correct position

File: meka_description/urdf/A2R4_l_arm_defs.urdf.xacro (robot description, xacro)
@@ -150,5 +150,5 @@
       <visual>
 	      <material name="GreyC" />
-	      <origin xyz="0 0 0" rpy="0 0 0 " />
+	      <origin xyz="0.00502 0 0" rpy="0 0 0 " />
 	      <geometry name="bicep_LEFT_geom">
 		      <mesh filename="package://${MESH}/A2R3/A2R3_LT3_bicep.dae" />

File: meka_description/urdf/A2R4_r_arm_defs.urdf.xacro (robot description, xacro)
@@ -134,5 +134,5 @@
       <visual>
 	      <material name="GreyC" />
-	      <origin xyz="0 0 0" rpy="0 0 0 " />
+	      <origin xyz="0.00502 0 0" rpy="0 0 0 " />
 	      <geometry name="bicep_RIGHT_geom">
 		      <mesh filename="package://${MESH}/A2R3/A2R3_RT3_bicep.dae" />
