Commit message: Adapted collision primitives for new festo chest mount

File: meka_description/urdf/Z1R2B_defs.urdf.xacro (robot description, xacro)
@@ -41,5 +41,5 @@
       <!-- primitive meshes only -->
     <collision>
-		  <origin xyz="0 0 0.035" rpy="0.0 0.0 0.0 " />
+		  <origin xyz="0.108 0 0.035" rpy="0.0 0.0 0.0 " />
 		  <geometry>
 			  <box size="0.2 0.21 0.07" />
@@ -47,7 +47,7 @@
 	  </collision>
     <collision>
-		  <origin xyz="-0.105 0 0.09" rpy="0.0 0.0 0.0 " />
+		  <origin xyz="0.004 0 0.09" rpy="0.0 0.0 0.0 " />
 		  <geometry>
-			  <box size="0.03 0.08 0.18" />
+			  <box size="0.008 0.08 0.18" />
 		  </geometry>
 	  </collision>
