Commit message: new zlift light barrier height

File: meka_description/urdf/Z1R2_zlift_defs.urdf.xacro (robot description, xacro)
@@ -10,5 +10,5 @@
       <parent link="${parent}"/>
       <child link="zlift_link"/>
-      <limit lower="${0*M_PI/180}"  upper="${40.107*M_PI/180}"
+      <limit lower="${0*M_PI/180}"  upper="${38.9*M_PI/180}"
              effort="30" velocity="${34.8}" /> <!-- !!! this should be changed at some point !!! -->
       <dynamics damping="10.0" />
