Commit message: fixed left arm limits

File: meka_description/urdf/A2R4_arm_defs.urdf.xacro (robot description, xacro)
@@ -51,5 +51,10 @@
     <joint name="${lr}_arm_j1" type="revolute">
       <axis xyz="-1 0 0"/>
-     <limit effort="40" velocity="${30*M_PI/180}" lower="${-24*M_PI/180}" upper="${150*M_PI/180}" />
+      <xacro:if value="${lr == 'left'}">
+        <limit effort="40" velocity="${30*M_PI/180}" lower="${-150*M_PI/180}" upper="${24*M_PI/180}" />
+      </xacro:if>
+      <xacro:if value="${lr == 'right'}">
+        <limit effort="40" velocity="${30*M_PI/180}" lower="${-24*M_PI/180}" upper="${150*M_PI/180}" />
+      </xacro:if>
       <origin xyz="0 0 0" rpy="0 0 0" />
       <parent link="shoulderupper_${lr}"/>
@@ -74,5 +79,5 @@
       <!-- meshes
       <collision>
-	      <origin xyz="0 0 0" rpy="0.0 0.0 0.0 " />
+	      <origin xyz="0 0 0" rpy="0.0 0.0 ${rotate*M_PI} " />
 	      <geometry name="shoulderpitch_${lr}_collision">
 		      <mesh filename="package://${MESH_COLL}/A2R3/A2R3_RT2_shoulderPitch.stl" />
@@ -82,5 +87,5 @@
       <!-- primitive only -->
       <collision>
-        <origin xyz="0.0 ${reflect*-0.0256} -0.04" rpy="-0.58 0.0 0.0 " />
+        <origin xyz="0.0 ${reflect*-0.0256} -0.04" rpy="${reflect*-0.58} 0.0 0.0 " />
         <geometry>
           <box size="0.09 0.07 0.072" />
@@ -166,4 +171,5 @@
       <inertial>
         <mass value="0.223" />
+        <!--<origin xyz="${0.5*((reflect+1)*ual_xyz1+(1-reflect)*uar_xyz1)} ${0.5*((reflect+1)*ual_xyz2+(1-reflect)*uar_xyz2)} ${0.5*((reflect+1)*ual_xyz3+(1-reflect)*uar_xyz3)}" />-->
         <origin xyz="-0.000002 ${reflect*0.000278} -0.026124"/>
 	    <inertia ixx="0.000470" ixy="0.000000" ixz="0.000000"
@@ -180,5 +186,5 @@
       <!-- meshes
       <collision>
-	      <origin xyz="0 0 0" rpy="0.0 0.0 0.0 " />
+	      <origin xyz="0 0 0" rpy="0.0 0.0 ${rotate*M_PI}  " />
 	      <geometry name="elbowclevis_${lr}_collision">
 		      <mesh filename="package://${MESH_COLL}/A2R3/A2R3_RT4_elbow.stl" />
@@ -219,5 +225,10 @@
     <joint name="${lr}_arm_j4" type="revolute">
 	    <axis xyz="0 0 -1" />
-      <limit effort="4" velocity="${150*M_PI/180}" lower="${-19.7*M_PI/180}" upper="${199.7*M_PI/180}" />
+      <xacro:if value="${lr == 'left'}">
+        <limit effort="4" velocity="${150*M_PI/180}" lower="${-190.7*M_PI/180}" upper="${19.7*M_PI/180}" />
+      </xacro:if>
+      <xacro:if value="${lr == 'right'}">
+        <limit effort="4" velocity="${150*M_PI/180}" lower="${-19.7*M_PI/180}" upper="${190.7*M_PI/180}" />
+      </xacro:if>
       <origin xyz="0 0 -0.27747" rpy="0 0 0" />
       <parent link="elbowclevis_${lr}"/>

File: meka_description/urdf/H2R4_hand_defs.urdf.xacro (robot description, xacro)
@@ -17,7 +17,10 @@
      </joint>
      <link name="palm_${lr}">
-      <inertial>
+       <xacro:inertial_cuboid_with_pose mass="0.663" x_length="1.1" y_length="1.11" z_length="1.06">
+			<origin xyz="0.001459 0.001619 -0.051312"/>
+	   </xacro:inertial_cuboid_with_pose>
+      <!--inertial>
+        <origin xyz="0.001459 0.001619 -0.051312"/>
         <mass value="0.663" />
-	    <origin xyz="0.001459 0.001619 -0.051312"/>
 	    <inertia ixx="0.000873"
 	    iyy="0.000597"
@@ -26,5 +29,5 @@
 	    ixz="-0.000008"
 	    iyz="0.000016" />
-      </inertial>
+      </inertial-->
       <visual>
 	      <material name="GreyC" />
@@ -126,5 +129,5 @@
     </collision>
     <inertial>
-      <mass value="0.01" />
+      <mass value="1.01" />
       <origin xyz="0 0 0"/>
       <inertia ixx="0.0" ixy="0.0" ixz="0.0"

File: meka_description/urdf/T2R3_torso_defs.urdf.xacro (robot description, xacro)
@@ -47,9 +47,12 @@
 	</joint>
 	<link name="torso">
-		<inertial>
+		<xacro:inertial_cuboid_with_pose mass="4.411" x_length="0.1" y_length="0.24" z_length="0.25">
+			<origin xyz="0.00011774 0.0038073 -0.0522753" />
+	    </xacro:inertial_cuboid_with_pose>
+		<!--inertial>
 			<mass value="4.411" />
 			<origin xyz="0.00011774 0.0038073 -0.0522753" />
 			<inertia ixx="0.026360" ixy="-0.0000024" ixz="-0.0000508" iyy="0.0134266" iyz="0.0006839" izz="0.0229879" />
-		</inertial>
+		</inertial-->
 		<visual>
 			<material name="GreyC" />
