Commit message: turned laser upside down, inside out

File: meka_description/urdf/MEKA_BASIC.urdf.xacro (robot description, xacro)
@@ -44,5 +44,5 @@
 	</link>
 	<joint name="laser_rear_joint" type="fixed">
-	  <origin xyz="-0.306 0.0 0.4" rpy="0 ${M_PI} 0" />
+	  <origin xyz="-0.306 0.0 0.4" rpy="0 0 ${M_PI}" />
       <child link="laser_rear"/>
       <parent link="${base_link}"/>
