Commit message: Added consistent zlift parameter values and names.

File: meka_description/urdf/S3R1_head_defs.urdf.xacro (robot description, xacro)
@@ -56,5 +56,5 @@
     <joint name="head_j0" type="revolute">
       <axis xyz="0 -1 0" />
-      <origin xyz="0 0 0.1103" rpy="0 0 0" />
+      <origin xyz="0 0 0.1103" rpy="0 0.314159265 0" />
       <parent link="neck_pan"/>
       <child link="shell"/>

File: meka_description/urdf/Z1R2B_defs.urdf.xacro (robot description, xacro)
@@ -6,15 +6,15 @@
   <macro name="meka_zlift" params="side parent reflect *origin">
     <!-- Shoulder pan -->
-    <joint name="zlift_joint" type="prismatic">
+    <joint name="zlift_j0" type="prismatic">
       <axis xyz="0 0 1" />
       <insert_block name="origin" /> <!-- transform from parent link to this joint frame -->
       <parent link="${parent}"/>
       <child link="zlift_link"/>
-      <limit lower="${0.0*M_PI/180.0}"  upper="${31965.0*M_PI/180.0}"
-             effort="30" velocity="${3.48}" />
+      <limit lower="${0*M_PI/180}"  upper="${40107*M_PI/180}"
+             effort="30" velocity="${34.8}" /> <!-- !!! this should be changed at some point !!! -->
       <dynamics damping="10.0" />
-      <safety_controller k_position="100" k_velocity="10"
+      <!--safety_controller k_position="100" k_velocity="10"
                          soft_lower_limit="${reflect*M_PI/4-1.5+0.15}"
-                         soft_upper_limit="${reflect*M_PI/4+1.5-0.15}" />
+                         soft_upper_limit="${reflect*M_PI/4+1.5-0.15}" /-->
     </joint>
     <link name="zlift_link">

Commit message: increased head limits to their actual limits

File: meka_description/urdf/S3R1_head_defs.urdf.xacro (robot description, xacro)
@@ -59,5 +59,5 @@
       <parent link="neck_pan"/>
       <child link="shell"/>
-      <limit effort="100" velocity="${20.0*M_PI/180}" lower="${-18.0*M_PI/180}" upper="${1.0*M_PI/180}" />
+      <limit effort="100" velocity="${20.0*M_PI/180}" lower="${-40.0*M_PI/180}" upper="${2.0*M_PI/180}" />
     </joint>
     <link name="shell">
@@ -106,5 +106,5 @@
       <parent link="shell"/>
       <child link="BB2"/>
-      <limit effort="100" velocity="${20.0*M_PI/180}" lower="${-18.0*M_PI/180}" upper="${1.0*M_PI/180}" />
+      <limit effort="100" velocity="${20.0*M_PI/180}" lower="${-40.0*M_PI/180}" upper="${2.0*M_PI/180}" />
     </joint>
     <link name="BB2">

Commit message: added xtion to urdf

File: meka_description/urdf/S3R1_head_defs.urdf.xacro (robot description, xacro)
@@ -11,4 +11,5 @@
       <parent link="${parent}"/>
       <child link="neck_pan"/>
+      <child link="xtion"/>
     </joint>
     <link name="neck_pan">
@@ -66,9 +67,9 @@
 	<origin xyz="0.0 0.0 0.0"/>
 	<inertia ixx="0.0"
-	iyy="0.0"
-	izz="0.0"
-	ixy="0.0"
-	ixz="0.0"
-	iyz="0.0" />
+        iyy="0.0"
+        izz="0.0"
+        ixy="0.0"
+        ixz="0.0"
+        iyz="0.0" />
       </inertial>
       <visual>
@@ -101,9 +102,49 @@
       </collision>
     </link>
-    <joint name="head_j2" type="revolute">
+     <joint name="head_xtion_dummy" type="revolute">
+	<limit effort="100" velocity="${75*M_PI/180}" lower="${-56.0*M_PI/180}" upper="${56.0*M_PI/180}" />
+	<origin xyz="0.0865 0.0095 0.0542" rpy="-1.49304175558102 0.0465121191942754 -1.5830006092006217"/>
+      <axis xyz="0 0 1"/>
+      <parent link="shell"/>
+      <child link="_xtion_link"/>
+    </joint>
+    <link name="_xtion_link">
+	<parent link="shell"/>
+	<inertial>
+        <mass value="0.1" />
+	<origin xyz="0.0 0.0 0.0"/>
+      <inertia ixx="0.0"
+          iyy="0.0"
+          izz="0.0"
+          ixy="0.0"
+          ixz="0.0"
+          iyz="0.0" />
+      </inertial>
+    </link>
+     <joint name="head_xtion_dummy2" type="revolute">
+	<limit effort="100" velocity="${75*M_PI/180}" lower="${-56.0*M_PI/180}" upper="${56.0*M_PI/180}" />
+	<origin xyz="-0.04 0 0" rpy="0 -1.5708 1.5708"/>
+      <axis xyz="0 0 1"/>
+      <parent link="_xtion_link"/>
+      <child link="xtion_link"/>
+    </joint>
+    <link name="xtion_link">
+	<parent link="_xtion_link"/>
+	<inertial>
+        <mass value="0.1" />
+	<origin xyz="0.0 0.0 0.0"/>
+      <inertia ixx="0.0"
+          iyy="0.0"
+          izz="0.0"
+          ixy="0.0"
+          ixz="0.0"
+          iyz="0.0" />
+      </inertial>
+    </link>
+    <!--joint name="head_j2" type="revolute">
       <axis xyz="0 -1 0" />
       <origin xyz="0.07975 0 0.123536" rpy="0 0 0" />
       <parent link="shell"/>
-      <child link="BB2"/>
+	<child link="BB2"/>
       <limit effort="100" velocity="${20.0*M_PI/180}" lower="${-40.0*M_PI/180}" upper="${2.0*M_PI/180}" />
     </joint>
@@ -132,5 +173,5 @@
 	      </geometry>
       </collision>
-    </link>
+    </link> -->
 </macro>
   <macro name="m3_head" params="side parent reflect *origin">

Commit message: renamed _xtion_link to xtion_link_rot to match naming rules

File: meka_description/urdf/S3R1_head_defs.urdf.xacro (robot description, xacro)
@@ -93,7 +93,7 @@
       <axis xyz="0 0 1"/>
       <parent link="shell"/>
-      <child link="_xtion_link"/>
+      <child link="xtion_link_rot"/>
     </joint>
-    <link name="_xtion_link">
+    <link name="xtion_link_rot">
 	<parent link="shell"/>
 		<xacro:inertial_cuboid_with_pose mass="0.1" x_length="0.1" y_length="0.1" z_length="0.05">
@@ -105,9 +105,9 @@
 	<origin xyz="-0.04 0 0" rpy="0 -1.5708 1.5708"/>
       <axis xyz="0 0 1"/>
-      <parent link="_xtion_link"/>
+      <parent link="xtion_link_rot"/>
       <child link="xtion_link"/>
     </joint>
     <link name="xtion_link">
-	<parent link="_xtion_link"/>
+	<parent link="xtion_link_rot"/>
 		<xacro:inertial_cuboid_with_pose mass="0.1" x_length="0.1" y_length="0.1" z_length="0.05">
 			<origin xyz="0 0 0.0" rpy="0 0 0" />
