Commit message: add handover frame with resulting zero rot

File: meka_description/urdf/H2R4_hand_defs.urdf.xacro (robot description, xacro)
@@ -111,4 +111,36 @@
     </joint>
   <link name="hand_tool_frame_${lr}">
+    <!-- This is the coordinate system of the end effector (this is the position
+         used in IK); there is no actual arm part attached to this link -->
+    <!-- The fake geometry here is only present to work around https://github.com/ros-planning/moveit_core/issues/158 -->
+    <visual>
+      <origin rpy="0 0 0" xyz="0 0 0"/>
+      <geometry>
+        <box size="0.01 0.01 0.01"/>
+      </geometry>
+      <material name="red" />
+    </visual>
+    <collision>
+      <origin rpy="0 0 0" xyz="0 0 -0.01"/>
+      <geometry>
+        <box size="0.001 0.001 0.001"/>
+      </geometry>
+      <material name="red" />
+    </collision>
+    <inertial>
+      <mass value="1.01" />
+      <origin xyz="0 0 0"/>
+      <inertia ixx="0.0" ixy="0.0" ixz="0.0"
+        iyy="0.0" iyz="0.0"
+        izz="0.0" />
+    </inertial>
+  </link>
+    <!-- this defines handover point -->
+    <joint name="hand_${lr}_handover_frame_joint" type="fixed">
+        <parent link="${parent}"/>
+        <child link="handover_frame_${lr}" />
+        <origin xyz="-0.02 0 -0.12" rpy="-1.5708 1.5708 0"/>
+    </joint>
+  <link name="handover_frame_${lr}">
     <!-- This is the coordinate system of the end effector (this is the position
          used in IK); there is no actual arm part attached to this link -->

Commit message: update handover point in urdf

File: meka_description/urdf/H2R4_hand_defs.urdf.xacro (robot description, xacro)
@@ -136,36 +136,37 @@
     </inertial>
   </link>
-    <!-- this defines handover point -->
-    <joint name="hand_${lr}_handover_frame_joint" type="fixed">
-        <parent link="${parent}"/>
-        <child link="handover_frame_${lr}" />
-        <origin xyz="-0.02 0 -0.12" rpy="-1.5708 1.5708 0"/>
-    </joint>
-  <link name="handover_frame_${lr}">
-    <!-- This is the coordinate system of the end effector (this is the position
-         used in IK); there is no actual arm part attached to this link -->
-    <!-- The fake geometry here is only present to work around https://github.com/ros-planning/moveit_core/issues/158 -->
-    <visual>
-      <origin rpy="0 0 0" xyz="0 0 0"/>
-      <geometry>
-        <box size="0.01 0.01 0.01"/>
-      </geometry>
-      <material name="red" />
-    </visual>
-    <collision>
-      <origin rpy="0 0 0" xyz="0 0 -0.01"/>
-      <geometry>
-        <box size="0.001 0.001 0.001"/>
-      </geometry>
-      <material name="red" />
-    </collision>
-    <inertial>
-      <mass value="1.01" />
-      <origin xyz="0 0 0"/>
-      <inertia ixx="0.0" ixy="0.0" ixz="0.0"
-        iyy="0.0" iyz="0.0"
-        izz="0.0" />
-    </inertial>
-  </link>
+    <xacro:if value="${lr == 'right'}">
+        <!-- this defines handover point -->
+        <joint name="hand_${lr}_handover_frame_joint" type="fixed">
+            <parent link="${parent}"/>
+            <child link="handover_frame_${lr}" />
+            <origin xyz="-0.04 0.02 -0.13" rpy="-1.5708 1.5708 0"/>
+        </joint>
+    <link name="handover_frame_${lr}">
+        <!-- This is the coordinate system of the end effector (this is the position
+            used in IK); there is no actual arm part attached to this link -->
+        <visual>
+        <origin rpy="0 0 0" xyz="0 0 0"/>
+        <geometry>
+            <cylinder radius="0.02" length="0.15"/>
+        </geometry>
+        <material name="red" />
+        </visual>
+        <collision>
+        <origin rpy="0 0 0" xyz="0 0 0"/>
+        <geometry>
+            <cylinder radius="0.02" length="0.15"/>
+        </geometry>
+        <material name="red" />
+        </collision>
+        <inertial>
+        <mass value="1.01" />
+        <origin xyz="0 0 0"/>
+        <inertia ixx="0.0" ixy="0.0" ixz="0.0"
+            iyy="0.0" iyz="0.0"
+            izz="0.0" />
+        </inertial>
+    </link>
+  </xacro:if>
 <!-- Start Thumb -->
     <joint name="${lr}_hand_j0" type="revolute">
