Commit message: fixed robot model for bie robot

File: meka_description/robots/bie.urdf.xacro (robot description, xacro)
@@ -24,5 +24,5 @@
   <xacro:include filename="$(find meka_description)/urdf/S3R1_head_defs.urdf.xacro" />
   <!-- john added transmissions -->
-  <xacro:include filename="$(find meka_description)/transmissions/A2R4_r_arm_defs.transmission.xacro" />
+  <!-- <xacro:include filename="$(find meka_description)/transmissions/A2R4_r_arm_defs.transmission.xacro" /> -->
   <!--<xacro:include filename="$(find meka_description)/transmissions/H2R2_r_hand_defs.transmission.xacro" />-->
   <!--<xacro:include filename="$(find meka_description)/transmissions/S2R1_head_defs.transmission.xacro" />-->
@@ -95,5 +95,5 @@
     </collision>
   </link>
-  <joint name="torso_j0" type="continuous">
+  <joint name="torso_j0" type="revolute">
     <axis xyz="0 0 1"/>
     <origin xyz="0 0 0.1678" rpy="0 0 0" />
@@ -123,5 +123,5 @@
     </collision>
   </link>
-  <joint name="torso_j1" type="continuous">
+  <joint name="torso_j1" type="revolute">
     <axis xyz="0 1 0"/>
     <origin xyz="0 0 0" rpy="0 0 0" />
@@ -156,5 +156,5 @@
     </collision>
   </link>
-  <joint name="torso_j2" type="continuous">
+  <joint name="torso_j2" type="revolute">
     <axis xyz="0 1 0"/>
     <origin xyz="0 0 0.1397" rpy="0 0 0" />
@@ -166,5 +166,5 @@
   <link name="upper">
     <inertial>
-      <mass value="6.534" /> <!-- torso with motors, bottom pullies, and neck mount -->
+      <mass value="6.534" />
       <origin xyz="0.008700 0.011470 0.129740"/>
       <inertia ixx="0.069760"

File: meka_description/urdf/Z1R2B_defs.urdf.xacro (robot description, xacro)
@@ -40,5 +40,5 @@
       </collision>
     </link>
-  <link name="upper">
+  <!--link name="upper">
 	  <inertial>
 		  <mass value="1000" />
@@ -52,5 +52,5 @@
 			  <mesh filename="package://${MESH}/A2R3/A2R3_T4_Chest_Neck.dae" />
 		  </geometry>
-		  <!--material name="Blue" /-->
+		  <material name="Blue" />
 	  </visual>
 	  <collision>
@@ -60,16 +60,16 @@
 		  </geometry>
 	  </collision>
-  </link>
-    <joint name="chest_joint" type="fixed">
+  </link -->
+    <!--joint name="chest_joint" type="fixed">
 	<origin xyz="0 0 -0.03" rpy="0 0 0" />
 	<parent link="zlift_link" />
 	<child link="upper" />
-    </joint>
-    <joint name="origin_joint" type="fixed">
+    </joint-->
+    <!--joint name="origin_joint" type="fixed">
 	<origin xyz="0 0 0.2337" rpy="0 0 0" />
 	<parent link="upper" />
 	<child link="T0" />
-    </joint>
-    <link name="T0"/>
+    </joint-->
+    <!--link name="T0"/-->
   </macro>
 </robot>

Commit message: added meka base to urdf

File: meka_description/robots/bie.urdf.xacro (robot description, xacro)
@@ -55,12 +55,5 @@
     <origin xyz="0.0 0.18465 0.2337" rpy="0 0 0" />
   </m3_l_arm>
-  <link name="world" />
   <link name="base_link" />
-  <!-- Solid Base -->
-  <joint name="base_joint" type="fixed">
-	  <origin xyz="0 0 1" rpy="0 0 0" />
-    <parent link="world" />
-    <child link="base_link" />
-  </joint>
   <meka_base  side="r" reflect="1" parent="base_link">
     <origin xyz="0.0 0.0 0.0" rpy="0 0 0" />

File: meka_description/urdf/B1R2B_defs.urdf.xacro (robot description, xacro)
@@ -5,15 +5,15 @@
   <property name="M_PI" value="3.1415926535897931" />
   <macro name="meka_base" params="side parent reflect *origin">
-    <joint name="X" type="prismatic">
+    <joint name="X" type="fixed">  <!-- was prismatic -->
       <axis xyz="1 0 0" />
       <insert_block name="origin" />
       <parent link="${parent}"/>
       <child link="dummy_1"/>
-      <limit lower="${reflect*M_PI/4-1.5}"  upper="${reflect*M_PI/4+1.5}"
+      <!--limit lower="${reflect*M_PI/4-1.5}"  upper="${reflect*M_PI/4+1.5}"
              effort="30" velocity="${3.48}" />
       <dynamics damping="10.0" />
       <safety_controller k_position="100" k_velocity="10"
                          soft_lower_limit="${reflect*M_PI/4-1.5+0.15}"
-                         soft_upper_limit="${reflect*M_PI/4+1.5-0.15}" />
+                         soft_upper_limit="${reflect*M_PI/4+1.5-0.15}" /-->
     </joint>
     <link name="dummy_1">
@@ -39,11 +39,11 @@
       </collision>
     </link>
-    <joint name="Y" type="prismatic">
+    <joint name="Y" type="fixed"> <!-- was prismatic -->
       <axis xyz="0 1 0"/>
-      <limit lower="-0.5236" upper="1.3963"
+      <!-- limit lower="-0.5236" upper="1.3963"
              effort="30" velocity="${3.47}" />
       <safety_controller k_position="100" k_velocity="10"
                          soft_lower_limit="${-0.5236+0.17}" soft_upper_limit="${1.3963-0.05}" />
-      <dynamics damping="10.0" />
+      <dynamics damping="10.0" / -->
       <origin xyz="0 0 0" rpy="0 0 0" />
       <parent link="dummy_1"/>
@@ -72,12 +72,12 @@
       </collision>
     </link>
-    <joint name="yaw" type="revolute">
+    <joint name="yaw" type="fixed">  <!-- was revolute -->
       <axis xyz="0 0 1" />
       <origin xyz="0 0.0 0.0" rpy="0 0 0" />
       <parent link="dummy_2" />
       <child link="dummy_3"/>
-      <limit lower="${reflect*1.55-2.35}" upper="${reflect*1.55+2.35}" effort="30" velocity="${5.45}" />
+      <!-- limit lower="${reflect*1.55-2.35}" upper="${reflect*1.55+2.35}" effort="30" velocity="${5.45}" />
       <safety_controller k_position="100" k_velocity="2" soft_lower_limit="${reflect*1.55-2.35+0.15}" soft_upper_limit="${reflect*1.55+2.35-0.15}" />
-      <dynamics damping="0.1" />
+      <dynamics damping="0.1" / -->
     </joint>
   <link name="dummy_3">

Commit message: Added mimic joints (deactivated by default) Added a robot description visualizer with joint sliders Fixed a CMakeList bug

File: meka_description/robots/bie.urdf.xacro (robot description, xacro)
@@ -8,4 +8,6 @@
  <property name="MESH" value="meka_description/meshes/mid_res" />
  <property name="MESH_COLL" value="meka_description/meshes/low_res" />
+ <!-- synergy vector -->
+ <xacro:property name="torso_coupling" value="1.0" />
 <!-- generic simulator_gazebo plugins for starting mechanism control, ros time, ros battery -->
   <xacro:include filename="$(find meka_description)/gazebo/gazebo.urdf.xacro" />
@@ -40,5 +42,5 @@
   <m3_r_arm_transmission side="r" reflect="1" parent="upper"/>
   <m3_r_hand_transmission/>
-  <m3_r_hand side="r" reflect="1" parent="handmount_RIGHT">
+  <m3_r_hand side="r" reflect="1" parent="handmount_RIGHT" use_mimic="$(arg use_mimic)">
     <origin xyz="0.0 0.0 0.0" rpy="0 0 0" />
   </m3_r_hand>
@@ -156,4 +158,7 @@
     <limit effort="200" velocity="${10.0*M_PI/180}" lower="${-11.79349*M_PI/180}" upper="${53.29349*M_PI/180}" />
     <dynamics damping="1.0"/>
+    <xacro:if value="$(arg use_mimic)">
+      <mimic joint="torso_j1" multiplier="${torso_coupling}"/>
+		</xacro:if>
   </joint>
   <link name="upper">

File: meka_description/urdf/H2R4_r_hand_defs.urdf.xacro (robot description, xacro)
@@ -1,8 +1,11 @@
 <?xml version="1.0"?>
-<robot xmlns:sensor="http://playerstage.sourceforge.net/gazebo/xmlschema/#sensor"
+<robot xmlns:xacro="http://ros.org/wiki/xacro"
+       xmlns:sensor="http://playerstage.sourceforge.net/gazebo/xmlschema/#sensor"
        xmlns:controller="http://playerstage.sourceforge.net/gazebo/xmlschema/#controller"
        xmlns:interface="http://playerstage.sourceforge.net/gazebo/xmlschema/#interface">
   <property name="M_PI" value="3.1415926535897931" />
-  <macro name="m3_r_palm" params="side parent reflect *origin">
+  <property name="proxmid_coupling" value="1.0" />
+  <property name="middist_coupling" value="1.0" />
+  <macro name="m3_r_palm" params="side parent reflect *origin use_mimic:=false">
   <joint name="palm_joint_right" type="fixed">
     <origin xyz="0 0 -0.04414" rpy="0 0 0" />
@@ -179,4 +182,7 @@
       <parent link="index0_right"/>
       <child link="index1_right"/>
+      <xacro:if value="${use_mimic}">
+				<mimic joint="right_hand_j4" multiplier="${proxmid_coupling}"/>
+			</xacro:if>
     </joint>
     <link name="index1_right">
@@ -211,4 +217,7 @@
       <parent link="index1_right"/>
       <child link="index2_right"/>
+      <xacro:if value="${use_mimic}">
+				<mimic joint="right_hand_j4" multiplier="${middist_coupling}"/>
+			</xacro:if>
     </joint>
     <link name="index2_right">
@@ -284,4 +293,7 @@
       <parent link="ring0_right"/>
       <child link="ring1_right"/>
+      <xacro:if value="${use_mimic}">
+				<mimic joint="right_hand_j8" multiplier="${proxmid_coupling}"/>
+			</xacro:if>
     </joint>
     <link name="ring1_right">
@@ -316,4 +328,7 @@
       <parent link="ring1_right"/>
       <child link="ring2_right"/>
+      <xacro:if value="${use_mimic}">
+				<mimic joint="right_hand_j8" multiplier="${middist_coupling}"/>
+			</xacro:if>
     </joint>
     <link name="ring2_right">
@@ -389,4 +404,7 @@
       <parent link="pinky0_right"/>
       <child link="pinky1_right"/>
+      <xacro:if value="${use_mimic}">
+				<mimic joint="right_hand_j12" multiplier="${proxmid_coupling}"/>
+			</xacro:if>
     </joint>
     <link name="pinky1_right">
@@ -421,4 +439,7 @@
       <parent link="pinky1_right"/>
       <child link="pinky2_right"/>
+      <xacro:if value="${use_mimic}">
+				<mimic joint="right_hand_j12" multiplier="${middist_coupling}"/>
+			</xacro:if>
     </joint>
     <link name="pinky2_right">
@@ -456,6 +477,6 @@
     <link name="pinky_end_right"/>
 </macro>
-  <macro name="m3_r_hand" params="side parent reflect *origin">
-    <m3_r_palm side="${side}" reflect="${reflect}" parent="${parent}">
+  <macro name="m3_r_hand" params="side parent reflect use_mimic:=false *origin">
+    <m3_r_palm side="${side}" reflect="${reflect}" parent="${parent}" use_mimic="${use_mimic}">
       <insert_block name="origin" />
     </m3_r_palm>

Commit message: Added mimic for left hand, and thumb on both hands, fixed a misplaced geometry tag

File: meka_description/robots/bie.urdf.xacro (robot description, xacro)
@@ -45,5 +45,5 @@
     <origin xyz="0.0 0.0 0.0" rpy="0 0 0" />
   </m3_r_hand>
-  <m3_l_hand side="l" reflect="1" parent="handmount_LEFT">
+  <m3_l_hand side="l" reflect="1" parent="handmount_LEFT" use_mimic="$(arg use_mimic)">
     <origin xyz="0.0 0.0 0.0" rpy="0 0 0" />
   </m3_l_hand>

File: meka_description/urdf/H2R4_l_hand_defs.urdf.xacro (robot description, xacro)
@@ -1,8 +1,13 @@
 <?xml version="1.0"?>
-<robot xmlns:sensor="http://playerstage.sourceforge.net/gazebo/xmlschema/#sensor"
+<robot xmlns:xacro="http://ros.org/wiki/xacro"
+       xmlns:sensor="http://playerstage.sourceforge.net/gazebo/xmlschema/#sensor"
        xmlns:controller="http://playerstage.sourceforge.net/gazebo/xmlschema/#controller"
        xmlns:interface="http://playerstage.sourceforge.net/gazebo/xmlschema/#interface">
   <property name="M_PI" value="3.1415926535897931" />
-  <macro name="m3_l_palm" params="side parent reflect *origin">
+  <property name="proxmid_coupling" value="1.0" />
+  <property name="middist_coupling" value="1.0" />
+  <property name="th_proxmid_coupling" value="1.0" />
+  <property name="th_middist_coupling" value="1.0" />
+  <macro name="m3_l_palm" params="side parent reflect *origin use_mimic:=false">
   <joint name="palm_joint_left" type="fixed">
     <origin xyz="0 0 -0.04414" rpy="0 0 0" />
@@ -106,4 +111,7 @@
       <child link="thumb2_left"/>
       <limit effort="100" velocity="${50*M_PI/180}" lower="${-14.94*M_PI/180}" upper="${14.94*M_PI/180}" />
+      <xacro:if value="${use_mimic}">
+				<mimic joint="left_hand_j1" multiplier="${th_proxmid_coupling}"/>
+			</xacro:if>
     </joint>
     <link name="thumb2_left">
@@ -138,4 +146,7 @@
       <child link="thumb_end_left"/>
       <limit effort="100" velocity="${50*M_PI/180}" lower="${-14.94*M_PI/180}" upper="${14.94*M_PI/180}" />
+      <xacro:if value="${use_mimic}">
+				<mimic joint="left_hand_j1" multiplier="${th_middist_coupling}"/>
+			</xacro:if>
     </joint>
     <link name="thumb_end_left"/>
@@ -179,4 +190,7 @@
       <parent link="index0_left"/>
       <child link="index1_left"/>
+      <xacro:if value="${use_mimic}">
+				<mimic joint="left_hand_j2" multiplier="${proxmid_coupling}"/>
+			</xacro:if>
     </joint>
     <link name="index1_left">
@@ -195,6 +209,6 @@
 	      <origin xyz="0 0 0" rpy="0 0 0 " />
 	      <geometry name="index1_geom_left">
-	      </geometry>
 		      <mesh filename="package://${MESH}/H2R3/H2R3_finger_knuckle2.dae" />
+        </geometry>
       </visual>
       <collision>
@@ -211,4 +225,7 @@
       <parent link="index1_left"/>
       <child link="index2_left"/>
+      <xacro:if value="${use_mimic}">
+				<mimic joint="left_hand_j2" multiplier="${middist_coupling}"/>
+			</xacro:if>
     </joint>
     <link name="index2_left">
@@ -284,4 +301,7 @@
       <parent link="ring0_left"/>
       <child link="ring1_left"/>
+      <xacro:if value="${use_mimic}">
+				<mimic joint="left_hand_j3" multiplier="${proxmid_coupling}"/>
+			</xacro:if>
     </joint>
     <link name="ring1_left">
@@ -316,4 +336,7 @@
       <parent link="ring1_left"/>
       <child link="ring2_left"/>
+      <xacro:if value="${use_mimic}">
+				<mimic joint="left_hand_j3" multiplier="${middist_coupling}"/>
+			</xacro:if>
     </joint>
     <link name="ring2_left">
@@ -389,4 +412,7 @@
       <parent link="pinky0_left"/>
       <child link="pinky1_left"/>
+      <xacro:if value="${use_mimic}">
+				<mimic joint="left_hand_j4" multiplier="${proxmid_coupling}"/>
+			</xacro:if>
     </joint>
     <link name="pinky1_left">
@@ -421,4 +447,7 @@
       <parent link="pinky1_left"/>
       <child link="pinky2_left"/>
+      <xacro:if value="${use_mimic}">
+				<mimic joint="left_hand_j4" multiplier="${middist_coupling}"/>
+			</xacro:if>
     </joint>
     <link name="pinky2_left">
@@ -456,6 +485,6 @@
     <link name="pinky_end_left"/>
 </macro>
-  <macro name="m3_l_hand" params="side parent reflect *origin">
-    <m3_l_palm side="${side}" reflect="${reflect}" parent="${parent}">
+  <macro name="m3_l_hand" params="side parent reflect use_mimic:=false *origin">
+    <m3_l_palm side="${side}" reflect="${reflect}" parent="${parent}" use_mimic="${use_mimic}">
       <insert_block name="origin" />
     </m3_l_palm>

File: meka_description/urdf/H2R4_r_hand_defs.urdf.xacro (robot description, xacro)
@@ -7,4 +7,6 @@
   <property name="proxmid_coupling" value="1.0" />
   <property name="middist_coupling" value="1.0" />
+  <property name="th_proxmid_coupling" value="1.0" />
+  <property name="th_middist_coupling" value="1.0" />
   <macro name="m3_r_palm" params="side parent reflect *origin use_mimic:=false">
   <joint name="palm_joint_right" type="fixed">
@@ -109,4 +111,7 @@
       <child link="thumb2_right"/>
       <limit effort="100" velocity="${50*M_PI/180}" lower="${-14.94*M_PI/180}" upper="${14.94*M_PI/180}" />
+      <xacro:if value="${use_mimic}">
+				<mimic joint="right_hand_j1" multiplier="${th_proxmid_coupling}"/>
+			</xacro:if>
     </joint>
     <link name="thumb2_right">
@@ -141,4 +146,7 @@
       <child link="thumb_end_right"/>
       <limit effort="100" velocity="${50*M_PI/180}" lower="${-14.94*M_PI/180}" upper="${14.94*M_PI/180}" />
+      <xacro:if value="${use_mimic}">
+				<mimic joint="right_hand_j1" multiplier="${th_middist_coupling}"/>
+			</xacro:if>
     </joint>
     <link name="thumb_end_right"/>
@@ -183,5 +191,5 @@
       <child link="index1_right"/>
       <xacro:if value="${use_mimic}">
-				<mimic joint="right_hand_j4" multiplier="${proxmid_coupling}"/>
+				<mimic joint="right_hand_j2" multiplier="${proxmid_coupling}"/>
 			</xacro:if>
     </joint>
@@ -218,5 +226,5 @@
       <child link="index2_right"/>
       <xacro:if value="${use_mimic}">
-				<mimic joint="right_hand_j4" multiplier="${middist_coupling}"/>
+				<mimic joint="right_hand_j2" multiplier="${middist_coupling}"/>
 			</xacro:if>
     </joint>
@@ -294,5 +302,5 @@
       <child link="ring1_right"/>
       <xacro:if value="${use_mimic}">
-				<mimic joint="right_hand_j8" multiplier="${proxmid_coupling}"/>
+				<mimic joint="right_hand_j3" multiplier="${proxmid_coupling}"/>
 			</xacro:if>
     </joint>
@@ -329,5 +337,5 @@
       <child link="ring2_right"/>
       <xacro:if value="${use_mimic}">
-				<mimic joint="right_hand_j8" multiplier="${middist_coupling}"/>
+				<mimic joint="right_hand_j3" multiplier="${middist_coupling}"/>
 			</xacro:if>
     </joint>
@@ -405,5 +413,5 @@
       <child link="pinky1_right"/>
       <xacro:if value="${use_mimic}">
-				<mimic joint="right_hand_j12" multiplier="${proxmid_coupling}"/>
+				<mimic joint="right_hand_j4" multiplier="${proxmid_coupling}"/>
 			</xacro:if>
     </joint>
@@ -440,5 +448,5 @@
       <child link="pinky2_right"/>
       <xacro:if value="${use_mimic}">
-				<mimic joint="right_hand_j12" multiplier="${middist_coupling}"/>
+				<mimic joint="right_hand_j4" multiplier="${middist_coupling}"/>
 			</xacro:if>
     </joint>
