Commit message: Separated torso and hand for mimic (in real torso should not use mimic) Fixed thumb j0 direction and amplitude in URDF, corrected ranges Adapted m3viz to new mimic tags Style fix

File: meka_description/robots/bie.urdf.xacro (robot description, xacro)
@@ -8,6 +8,7 @@
  <property name="MESH" value="meka_description/meshes/mid_res" />
  <property name="MESH_COLL" value="meka_description/meshes/low_res" />
- <xacro:arg name="use_mimic" default="true"/>
- <!-- synergy vector -->
+ <xacro:arg name="hand_mimic" default="true"/>
+ <xacro:arg name="torso_mimic" default="true"/>
+<!-- synergy vector -->
  <xacro:property name="torso_coupling" value="1.0" />
 <!-- generic simulator_gazebo plugins for starting mechanism control, ros time, ros battery -->
@@ -43,8 +44,8 @@
   <m3_r_arm_transmission side="r" reflect="1" parent="upper"/>
   <m3_r_hand_transmission/>
-  <m3_r_hand side="r" reflect="1" parent="handmount_RIGHT" use_mimic="$(arg use_mimic)">
+  <m3_r_hand side="r" reflect="1" parent="handmount_RIGHT" use_mimic="$(arg hand_mimic)">
     <origin xyz="0.0 0.0 0.0" rpy="0 0 0" />
   </m3_r_hand>
-  <m3_l_hand side="l" reflect="1" parent="handmount_LEFT" use_mimic="$(arg use_mimic)">
+  <m3_l_hand side="l" reflect="1" parent="handmount_LEFT" use_mimic="$(arg hand_mimic)">
     <origin xyz="0.0 0.0 0.0" rpy="0 0 0" />
   </m3_l_hand>
@@ -93,15 +94,15 @@
     <!-- primitive only -->
     <collision>
-		  <origin xyz="-0.11 0 0.025" rpy="0.0 0.0 0.0 " />
-		  <geometry>
-			  <box size="0.22 0.19 0.05" />
-		  </geometry>
-	  </collision>
-    <collision>
-		  <origin xyz="0.0 0 0.05" rpy="0.0 0.0 0.0 " />
-		  <geometry>
-			  <cylinder radius="0.095" length="0.1" />
-		  </geometry>
-	  </collision>
+      <origin xyz="-0.11 0 0.025" rpy="0.0 0.0 0.0 " />
+      <geometry>
+        <box size="0.22 0.19 0.05" />
+      </geometry>
+    </collision>
+    <collision>
+      <origin xyz="0.0 0 0.05" rpy="0.0 0.0 0.0 " />
+      <geometry>
+        <cylinder radius="0.095" length="0.1" />
+      </geometry>
+    </collision>
   </link>
   <joint name="torso_j0" type="revolute">
@@ -136,27 +137,27 @@
     <!-- primitive only -->
     <collision>
-		  <origin xyz="0.0 0 -0.0615" rpy="0.0 0.0 0.0 " />
-		  <geometry>
-			  <cylinder radius="0.088" length="0.015" />
-		  </geometry>
-	  </collision>
-    <collision>
-		   <origin xyz="0.0 0 -0.0615" rpy="0.0 0.0 0.0 " />
-		  <geometry>
-			  <box size="0.08 0.23 0.015" />
-		  </geometry>
-	  </collision>
-    <collision>
-		  <origin xyz="0.0 0.105 0" rpy="1.5707 0.0 0.0 " />
-		  <geometry>
-			  <cylinder radius="0.052" length="0.02" />
-		  </geometry>
-	  </collision>
-    <collision>
-		  <origin xyz="0.0 -0.105 0" rpy="1.5707 0.0 0.0  " />
-		  <geometry>
-			  <cylinder radius="0.052" length="0.02" />
-		  </geometry>
-	  </collision>
+      <origin xyz="0.0 0 -0.0615" rpy="0.0 0.0 0.0 " />
+      <geometry>
+        <cylinder radius="0.088" length="0.015" />
+      </geometry>
+    </collision>
+    <collision>
+      <origin xyz="0.0 0 -0.0615" rpy="0.0 0.0 0.0 " />
+      <geometry>
+        <box size="0.08 0.23 0.015" />
+      </geometry>
+    </collision>
+    <collision>
+      <origin xyz="0.0 0.105 0" rpy="1.5707 0.0 0.0 " />
+      <geometry>
+        <cylinder radius="0.052" length="0.02" />
+      </geometry>
+    </collision>
+    <collision>
+      <origin xyz="0.0 -0.105 0" rpy="1.5707 0.0 0.0  " />
+      <geometry>
+        <cylinder radius="0.052" length="0.02" />
+      </geometry>
+  </collision>
   </link>
   <joint name="torso_j1" type="revolute">
@@ -196,21 +197,21 @@
     <!-- primitive only -->
     <collision>
-		  <origin xyz="0.0 0 0.0684" rpy="0.0 0.0 0.0 " />
-		  <geometry>
-			  <box size="0.114 0.241 0.1368" />
-		  </geometry>
-	  </collision>
-    <collision>
-		  <origin xyz="0.0 0.0 0" rpy="1.5707 0.0 0.0 " />
-		  <geometry>
-			  <cylinder radius="0.057" length="0.241" />
-		  </geometry>
-	  </collision>
-    <collision>
-		  <origin xyz="0.0 0.0 0.1368" rpy="1.5707 0.0 0.0 " />
-		  <geometry>
-			  <cylinder radius="0.057" length="0.241" />
-		  </geometry>
-	  </collision>
+      <origin xyz="0.0 0 0.0684" rpy="0.0 0.0 0.0 " />
+      <geometry>
+        <box size="0.114 0.241 0.1368" />
+      </geometry>
+    </collision>
+    <collision>
+      <origin xyz="0.0 0.0 0" rpy="1.5707 0.0 0.0 " />
+      <geometry>
+        <cylinder radius="0.057" length="0.241" />
+      </geometry>
+    </collision>
+    <collision>
+      <origin xyz="0.0 0.0 0.1368" rpy="1.5707 0.0 0.0 " />
+      <geometry>
+        <cylinder radius="0.057" length="0.241" />
+      </geometry>
+    </collision>
   </link>
   <joint name="torso_j2" type="revolute">
@@ -221,7 +222,7 @@
     <limit effort="200" velocity="${10.0*M_PI/180}" lower="${-11.79349*M_PI/180}" upper="${53.29349*M_PI/180}" />
     <dynamics damping="1.0"/>
-    <xacro:if value="$(arg use_mimic)">
+    <xacro:if value="$(arg torso_mimic)">
       <mimic joint="torso_j1" multiplier="${torso_coupling}"/>
-		</xacro:if>
+    </xacro:if>
   </joint>
   <link name="upper">
@@ -253,15 +254,15 @@
     <!-- primitive only -->
     <collision>
-		  <origin xyz="0.0 0 0.1346" rpy="0.0 0.0 0.0 " />
-		  <geometry>
-			  <box size="0.14 0.22 0.1978" />
-		  </geometry>
-	  </collision>
-    <collision>
-		  <origin xyz="0.0 0.0 0.2335" rpy="1.5707 0.0 0.0 " />
-		  <geometry>
-			  <cylinder radius="0.0644" length="0.22" />
-		  </geometry>
-	  </collision>
+      <origin xyz="0.0 0 0.1346" rpy="0.0 0.0 0.0 " />
+      <geometry>
+        <box size="0.14 0.22 0.1978" />
+      </geometry>
+    </collision>
+    <collision>
+      <origin xyz="0.0 0.0 0.2335" rpy="1.5707 0.0 0.0 " />
+      <geometry>
+        <cylinder radius="0.0644" length="0.22" />
+      </geometry>
+    </collision>
   </link>
 </robot>

File: meka_description/urdf/H2R4_l_hand_defs.urdf.xacro (robot description, xacro)
@@ -8,6 +8,6 @@
   <property name="proxmid_coupling" value="0.3" />
   <property name="middist_coupling" value="0.3" />
-  <property name="th_palmprox_coupling" value="0.5" />
-  <property name="th_proxdist_coupling" value="0.5" />
+  <property name="th_palmprox_coupling" value="0.4" />
+  <property name="th_proxdist_coupling" value="0.4" />
   <macro name="m3_l_palm" params="side parent reflect *origin use_mimic:=false">
   <joint name="palm_joint_left" type="fixed">
@@ -81,9 +81,9 @@
 <!-- Start Thumb -->
     <joint name="left_hand_j0" type="revolute">
-      <axis xyz="0 0 1" />
-      <origin xyz="-0.02 -0.028 -0.03" rpy="0 0 0" />
+      <axis xyz="0 0 -1" />
+      <origin xyz="-0.02 -0.028 -0.03" rpy="0 0 ${M_PI/2.0}" />
       <parent link="palm_left"/>
       <child link="thumb0_left"/>
-      <limit effort="100" velocity="${20.0*M_PI/180}" lower="${-40*M_PI/180}" upper="${15*M_PI/180}" />
+      <limit effort="100" velocity="${20.0*M_PI/180}" lower="${0.0*M_PI/180}" upper="${120.0*M_PI/180}" />
     </joint>
     <link name="thumb0_left">
@@ -145,10 +145,10 @@
       <parent link="palm_left" />
       <child link="thumb_motor_left"/>
-      <limit effort="100" velocity="${50*M_PI/180}" lower="${0*M_PI/180}" upper="${120.0*M_PI/180.0}" />
+      <limit effort="100" velocity="${50*M_PI/180}" lower="${0*M_PI/180}" upper="${170.0*M_PI/180.0}" />
     </joint>
     <link name="thumb_motor_left"/>
     <joint name="left_hand_j1a" type="revolute">
       <axis xyz="0 -1 0"/>
-      <limit effort="100" velocity="${75*M_PI/180}" lower="${-80.919*M_PI/180}" upper="${80.91*M_PI/180}" />
+      <limit effort="100" velocity="${75*M_PI/180}" lower="${0.0*M_PI/180}" upper="${85.0*M_PI/180}" />
       <origin xyz="-0.018 0 0" rpy="0 0 0" />
       <parent link="thumb0_left"/>
@@ -160,5 +160,5 @@
     <joint name="left_hand_j1" type="revolute">
       <axis xyz="0 -1 0"/>
-      <limit effort="100" velocity="${75*M_PI/180}" lower="${-80.919*M_PI/180}" upper="${80.91*M_PI/180}" />
+      <limit effort="100" velocity="${75*M_PI/180}" lower="${0.0*M_PI/180}" upper="${85.0*M_PI/180}" />
       <origin xyz="-0.018 0 0" rpy="0 0 0" />
       <parent link="thumb0_left"/>
@@ -218,5 +218,5 @@
       <parent link="thumb1_left" />
       <child link="thumb2_left"/>
-      <limit effort="100" velocity="${50*M_PI/180}" lower="${-14.94*M_PI/180}" upper="${14.94*M_PI/180}" />
+      <limit effort="100" velocity="${50*M_PI/180}" lower="${0.0*M_PI/180}" upper="${85.0*M_PI/180}" />
 			<mimic joint="left_hand_j1" multiplier="${th_proxdist_coupling}"/>
     </joint>
@@ -228,5 +228,5 @@
       <parent link="thumb1_left" />
       <child link="thumb2_left"/>
-      <limit effort="100" velocity="${50*M_PI/180}" lower="${-14.94*M_PI/180}" upper="${14.94*M_PI/180}" />
+      <limit effort="100" velocity="${50*M_PI/180}" lower="${0.0*M_PI/180}" upper="${85.0*M_PI/180}" />
     </joint>
   </xacro:unless>

File: meka_description/urdf/H2R4_r_hand_defs.urdf.xacro (robot description, xacro)
@@ -8,6 +8,6 @@
   <property name="proxmid_coupling" value="0.3" />
   <property name="middist_coupling" value="0.3" />
-  <property name="th_palmprox_coupling" value="0.5" />
-  <property name="th_proxdist_coupling" value="0.5" />
+  <property name="th_palmprox_coupling" value="0.4" />
+  <property name="th_proxdist_coupling" value="0.4" />
   <macro name="m3_r_palm" params="side parent reflect *origin use_mimic:=false">
   <joint name="palm_joint_right" type="fixed">
@@ -82,9 +82,9 @@
 <!-- Start Thumb -->
     <joint name="right_hand_j0" type="revolute">
-      <axis xyz="0 0 -1" />
-      <origin xyz="-0.02 0.028 -0.03" rpy="0 0 0" />
+      <axis xyz="0 0 1" />
+      <origin xyz="-0.02 0.028 -0.03" rpy="0 0 ${-M_PI/2.0}" />
       <parent link="palm_right"/>
       <child link="thumb0_right"/>
-      <limit effort="100" velocity="${20.0*M_PI/180}" lower="${-40*M_PI/180}" upper="${15*M_PI/180}" />
+      <limit effort="100" velocity="${20.0*M_PI/180}" lower="${0.0*M_PI/180}" upper="${120.0*M_PI/180}" />
     </joint>
     <link name="thumb0_right">
@@ -146,10 +146,10 @@
       <parent link="palm_right" />
       <child link="thumb_motor_right"/>
-      <limit effort="100" velocity="${50*M_PI/180}" lower="${0*M_PI/180}" upper="${120.0*M_PI/180.0}" />
+      <limit effort="100" velocity="${50*M_PI/180}" lower="${0*M_PI/180}" upper="${170.0*M_PI/180.0}" />
     </joint>
     <link name="thumb_motor_right"/>
     <joint name="right_hand_j1a" type="revolute">
       <axis xyz="0 -1 0"/>
-      <limit effort="100" velocity="${75*M_PI/180}" lower="${-80.919*M_PI/180}" upper="${80.91*M_PI/180}" />
+      <limit effort="100" velocity="${75*M_PI/180}" lower="${0.0*M_PI/180}" upper="${85.0*M_PI/180}" />
       <origin xyz="-0.018 0 0" rpy="0 0 0" />
       <parent link="thumb0_right"/>
@@ -161,5 +161,5 @@
     <joint name="right_hand_j1" type="revolute">
       <axis xyz="0 -1 0"/>
-      <limit effort="100" velocity="${75*M_PI/180}" lower="${-80.919*M_PI/180}" upper="${80.91*M_PI/180}" />
+      <limit effort="100" velocity="${75*M_PI/180}" lower="${0.0*M_PI/180}" upper="${85.0*M_PI/180}" />
       <origin xyz="-0.018 0 0" rpy="0 0 0" />
       <parent link="thumb0_right"/>
@@ -219,5 +219,5 @@
       <parent link="thumb1_right" />
       <child link="thumb2_right"/>
-      <limit effort="100" velocity="${50*M_PI/180}" lower="${-14.94*M_PI/180}" upper="${14.94*M_PI/180}" />
+      <limit effort="100" velocity="${50*M_PI/180}" lower="${0.0*M_PI/180}" upper="${85.0*M_PI/180}" />
 			<mimic joint="right_hand_j1" multiplier="${th_proxdist_coupling}"/>
     </joint>
@@ -229,5 +229,5 @@
       <parent link="thumb1_right" />
       <child link="thumb2_right"/>
-      <limit effort="100" velocity="${50*M_PI/180}" lower="${-14.94*M_PI/180}" upper="${14.94*M_PI/180}" />
+      <limit effort="100" velocity="${50*M_PI/180}" lower="${0.0*M_PI/180}" upper="${85.0*M_PI/180}" />
     </joint>
   </xacro:unless>

Commit message: Changed Chest to use Chest without neck, and lowered the head Fixed neck (stl only) and created a BB2 model (to manufacturer dims) Created primitive collision objects for head, neck and bb2

File: meka_description/robots/bie.urdf.xacro (robot description, xacro)
@@ -51,5 +51,5 @@
   </m3_l_hand>
   <m3_head side="r" reflect="1" parent="upper">
-    <origin xyz="0.0 0.0 0.31155" rpy="0 0 0" />
+    <origin xyz="0.0 0.0 0.2757" rpy="0 0 0" />
   </m3_head>
  <m3_r_arm side="r" reflect="1" parent="upper">
@@ -241,5 +241,5 @@
       <origin xyz="0 0 0" rpy="0 0 0" />
       <geometry name="upper_geom">
-       <mesh filename="package://${MESH}/A2R3/A2R3_T4_Chest_Neck.dae" />
+       <mesh filename="package://${MESH}/A2R3/A2R3_T4_Chest.dae" />
       </geometry>
     </visual>

File: meka_description/urdf/S3R1_head_defs.urdf.xacro (robot description, xacro)
@@ -25,22 +25,36 @@
       <visual>
 	      <material name="GreyA" />
-	      <!--<origin xyz="0 0 0.0" rpy="0 0 0 " />-->
 	      <origin xyz="0 0 0" rpy="0 0 0 " />
 	      <geometry name="neck_tilt_geom">
 		<!--<box size="0.01 0.01 0.01" />-->
 		<!--<mesh filename="package://${MESH}/S2R1/S2R1_SH1_neckTilt.dae" />-->
-		<mesh filename="package://${MESH}/S3R1/neck.dae" />
+		<mesh filename="package://${MESH}/S3R1/neck.stl" />
 	      </geometry>
       </visual>
+      <!-- meshes
       <collision>
 	      <origin xyz="0 0 0" rpy="0.0 0.0 0.0 " />
 	      <geometry name="neck_tilt_geom_collison">
-		      <mesh filename="package://${MESH_COLL}/S2R1/S2R1_SH1_neckTilt.stl" />
+		      <mesh filename="package://${MESH}/S3R1/neck.stl" />
 	      </geometry>
+      </collision>
+      -->
+      <!-- primitive only -->
+      <collision>
+        <origin xyz="0.0 0 0.00833" rpy="0.0 0.0 0.0 " />
+        <geometry>
+          <cylinder radius="0.034" length="0.0166" />
+        </geometry>
+      </collision>
+      <collision>
+        <origin xyz="0.0 0 0.0473" rpy="0.0 0.0 0.0 " />
+        <geometry>
+          <cylinder radius="0.03" length="0.0614" />
+        </geometry>
       </collision>
     </link>
     <joint name="head_j0" type="revolute">
       <axis xyz="0 -1 0" />
-      <origin xyz="0 0 0.152287" rpy="0 0 0" />
+      <origin xyz="0 0 0.1103" rpy="0 0 0" />
       <parent link="neck_pan"/>
       <child link="shell"/>
@@ -65,4 +79,5 @@
 	      </geometry>
       </visual>
+      <!-- meshes
       <collision>
 	      <origin xyz="0 0 0" rpy="0.0 0.0 0.0 " />
@@ -71,4 +86,18 @@
 	      </geometry>
       </collision>
+      -->
+      <!-- primitive only -->
+      <collision>
+        <origin xyz="0.0 0 0.0" rpy="1.5708 0.0  0.0 " />
+        <geometry>
+          <cylinder radius="0.0335" length="0.09" />
+        </geometry>
+      </collision>
+      <collision>
+        <origin xyz="0.005 0 0.07" rpy="0.0 0.0 0.0 " />
+        <geometry>
+          <box size="0.222 0.2 0.09" />
+        </geometry>
+      </collision>
     </link>
     <joint name="head_j2" type="revolute">
@@ -76,8 +105,8 @@
       <origin xyz="0.07975 0 0.123536" rpy="0 0 0" />
       <parent link="shell"/>
-      <child link="BB3"/>
+      <child link="BB2"/>
       <limit effort="100" velocity="${20.0*M_PI/180}" lower="${-18.0*M_PI/180}" upper="${1.0*M_PI/180}" />
     </joint>
-    <link name="BB3">
+    <link name="BB2">
       <inertial>
         <mass value="0.409" />
@@ -94,11 +123,11 @@
 	      <origin xyz="0 0 0" rpy="0 0 0 " />
 	      <geometry name="shell_geom">
-		      <mesh filename="package://${MESH}/S3R1/BB3.dae" />
+		      <mesh filename="package://${MESH}/S3R1/BB2.stl" />
 	      </geometry>
       </visual>
       <collision>
-	      <origin xyz="0 0 0" rpy="0.0 0.0 0.0 " />
+	      <origin xyz="-0.0141 0 0.0268" rpy="0.0 0.0 0.0 " />
 	      <geometry name="S3_collision">
-		      <box size="0.01 0.01 0.01" />
+		      <box size="0.0474 0.157 0.037" />
 	      </geometry>
       </collision>

Commit message: added hand controller config for grasping

File: meka_description/robots/bie.urdf.xacro (robot description, xacro)
@@ -64,5 +64,5 @@
   </meka_base>
   <meka_zlift  side="r" reflect="1" parent="dummy_3">
-    <origin xyz="0.43 0.0 0.75" rpy="0 0 0" />
+    <origin xyz="0.33 0.0 0.75" rpy="0 0 0" />
   </meka_zlift>
   <!-- Solid Base -->

Commit message: adjusted zlift limits and initial position

File: meka_description/robots/bie.urdf.xacro (robot description, xacro)
@@ -64,5 +64,5 @@
   </meka_base>
   <meka_zlift  side="r" reflect="1" parent="dummy_3">
-    <origin xyz="0.33 0.0 0.75" rpy="0 0 0" />
+    <origin xyz="0.33 0.0 0.45" rpy="0 0 0" />
   </meka_zlift>
   <!-- Solid Base -->

File: meka_description/urdf/Z1R2B_defs.urdf.xacro (robot description, xacro)
@@ -5,5 +5,4 @@
   <property name="M_PI" value="3.1415926535897931" />
   <macro name="meka_zlift" params="side parent reflect *origin">
-    <!-- Shoulder pan -->
     <joint name="zlift_j0" type="prismatic">
       <axis xyz="0 0 1" />
@@ -11,5 +10,5 @@
       <parent link="${parent}"/>
       <child link="zlift_link"/>
-      <limit lower="${0*M_PI/180}"  upper="${40107*M_PI/180}"
+      <limit lower="${0*M_PI/180}"  upper="${40.107*M_PI/180}"
              effort="30" velocity="${34.8}" /> <!-- !!! this should be changed at some point !!! -->
       <dynamics damping="10.0" />

Commit message: added rotation around yaxis for zlift. see issue #6728

File: meka_description/robots/bie.urdf.xacro (robot description, xacro)
@@ -64,5 +64,5 @@
   </meka_base>
   <meka_zlift  side="r" reflect="1" parent="dummy_3">
-    <origin xyz="0.33 0.0 0.45" rpy="0 0 0" />
+    <origin xyz="0.33 0.0 0.45" rpy="0 0.0236 0" />
   </meka_zlift>
   <!-- Solid Base -->

Commit message: corrected position of the chest_mount_assy

File: meka_description/robots/bie.urdf.xacro (robot description, xacro)
@@ -64,5 +64,5 @@
   </meka_base>
   <meka_zlift  side="r" reflect="1" parent="dummy_3">
-    <origin xyz="0.33 0.0 0.45" rpy="0 0.0236 0" />
+    <origin xyz="0.295 0.0 0.5219" rpy="0 0.0236 0" /> <!-- 0.33 0.0 0.45 -->
   </meka_zlift>
   <!-- Solid Base -->

Commit message: remove rotation of the zlift

File: meka_description/robots/bie.urdf.xacro (robot description, xacro)
@@ -64,5 +64,5 @@
   </meka_base>
   <meka_zlift  side="r" reflect="1" parent="dummy_3">
-    <origin xyz="0.295 0.0 0.5219" rpy="0 0.0236 0" /> <!-- 0.33 0.0 0.45 -->
+    <origin xyz="0.295 0.0 0.5219" rpy="0 0 0" /> <!-- 0.33 0.0 0.45 rpy="0 0.0236 0" -->
   </meka_zlift>
   <!-- Solid Base -->

Commit message: Fixed pan_base, pan_plate and festo_chest assembly placement to match real robot

File: meka_description/robots/bie.urdf.xacro (robot description, xacro)
@@ -64,9 +64,9 @@
   </meka_base>
   <meka_zlift  side="r" reflect="1" parent="dummy_3">
-    <origin xyz="0.295 0.0 0.5219" rpy="0 0 0" /> <!-- 0.33 0.0 0.45 rpy="0 0.0236 0" -->
+    <origin xyz="0.17513 0.0 0.5219" rpy="0 0 0" /> <!-- 0.33 0.0 0.45 rpy="0 0.0236 0" -->
   </meka_zlift>
   <!-- Solid Base -->
   <joint name="chest_joint" type="fixed">
-	  <origin xyz="0.1 0.0 0.0" rpy="0 0 0" />
+	  <origin xyz="0.263 0.0 0.006" rpy="0 0 0" />
     <parent link="zlift_link" />
     <child link="panplate" />
@@ -108,5 +108,5 @@
   <joint name="torso_j0" type="revolute">
     <axis xyz="0 0 1"/>
-    <origin xyz="0 0 0.1678" rpy="0 0 0" />
+    <origin xyz="0 0 0.1658" rpy="0 0 0" />
     <parent link="panplate" />
     <child link="torso" />

File: meka_description/urdf/Z1R2B_defs.urdf.xacro (robot description, xacro)
@@ -29,5 +29,5 @@
 	      <origin xyz="0 0 0" rpy="0 0 0 " />
 	      <geometry name="z_lift_geom">
-		      <mesh filename="package://${MESH}/B1R1/MB1_00_011_festo-chest_mount_assy+spacer.dae" />
+		      <mesh filename="package://${MESH}/B1R1/meka_festo-chest_mount_assy.dae" />
 	      </geometry>
       </visual>

Commit message: fixed z-lift position

File: meka_description/robots/bie.urdf.xacro (robot description, xacro)
@@ -64,5 +64,5 @@
   </meka_base>
   <meka_zlift  side="r" reflect="1" parent="dummy_3">
-    <origin xyz="0.17513 0.0 0.5219" rpy="0 0 0" /> <!-- 0.33 0.0 0.45 rpy="0 0.0236 0" -->
+    <origin xyz="0.17513 0.0 0.43" rpy="0 0 0" /> <!-- 0.33 0.0 0.45 rpy="0 0.0236 0" -->
   </meka_zlift>
   <!-- Solid Base -->
