Commit message: temporarily removed torso

File: meka_description/robots/bie_sim.urdf.xacro (robot description, xacro)
@@ -7,6 +7,6 @@
   <!-- generic simulator_gazebo plugins for starting mechanism control, ros time, ros battery -->
   <xacro:include filename="$(find meka_description)/gazebo/gazebo.urdf.xacro" />
-  <xacro:include filename="$(find meka_description)/transmissions/body.transmission.xacro" />
-  <!-- MEKA BASICS -->
+  <!--xacro:include filename="$(find meka_description)/transmissions/body.transmission.xacro" /-->
+  <!-- Meka Basics -->
   <xacro:include filename="$(find meka_description)/urdf/MEKA_BASIC.urdf.xacro" />
   <!-- Meka Base -->
@@ -16,23 +16,23 @@
   <xacro:include filename="$(find meka_description)/transmissions/Z1R2B_zlift.transmission.xacro" />
   <!-- Meka Arm -->
-  <!-- <xacro:include filename="$(find meka_description)/urdf/A2R4_r_arm_defs.urdf.xacro" />  -->
-  <!-- <xacro:include filename="$(find meka_description)/urdf/A2R4_l_arm_defs.urdf.xacro" />  -->
-  <!-- <xacro:include filename="$(find meka_description)/transmissions/A2R4_r_arm_defs.transmission.xacro" /> -->
-  <!-- <xacro:include filename="$(find meka_description)/transmissions/A2R4_l_arm_defs.transmission.xacro" /> -->
+  <!--xacro:include filename="$(find meka_description)/urdf/A2R4_r_arm_defs.urdf.xacro" /-->
+  <!--xacro:include filename="$(find meka_description)/urdf/A2R4_l_arm_defs.urdf.xacro" /-->
+  <!--xacro:include filename="$(find meka_description)/transmissions/A2R4_r_arm_defs.transmission.xacro" /-->
+  <!--xacro:include filename="$(find meka_description)/transmissions/A2R4_l_arm_defs.transmission.xacro" /-->
   <!-- Meka Hand -->
-  <!-- <xacro:include filename="$(find meka_description)/urdf/H2R4_r_hand_defs.urdf.xacro" />  -->
-  <!-- <xacro:include filename="$(find meka_description)/urdf/H2R4_l_hand_defs.urdf.xacro" />  -->
-  <!-- <xacro:include filename="$(find meka_description)/transmissions/H2R4_r_hand.transmission.xacro" /> -->
-  <!-- <xacro:include filename="$(find meka_description)/transmissions/H2R4_l_hand.transmission.xacro" /> -->
-  <!-- Meka Head -->
+  <!--xacro:include filename="$(find meka_description)/urdf/H2R4_r_hand_defs.urdf.xacro" /-->
+  <!--xacro:include filename="$(find meka_description)/urdf/H2R4_l_hand_defs.urdf.xacro" /-->
+  <!--xacro:include filename="$(find meka_description)/transmissions/H2R4_r_hand.transmission.xacro" /-->
+  <!--xacro:include filename="$(find meka_description)/transmissions/H2R4_l_hand.transmission.xacro" /-->
+  <!-- Meka Head>
   <xacro:include filename="$(find meka_description)/urdf/S3R1_head_defs.urdf.xacro" />
-  <xacro:include filename="$(find meka_description)/transmissions/S3R1_head.transmission.xacro" />
-  <!-- Import asus -->
-  <xacro:include filename="$(find meka_description)/urdf/asus_camera.urdf.xacro" />
-  <xacro:asus_camera name="xtion" parent="shell">
+  <xacro:include filename="$(find meka_description)/transmissions/S3R1_head.transmission.xacro" / -->
+  <!-- Import asus>
+  <xacro:include filename="$(find meka_description)/urdf/asus_camera.urdf.xacro" / -->
+  <!--xacro:asus_camera name="xtion" parent="shell">
     <origin xyz="0.12 0 0.06" rpy="0 0 0"/>
-  </xacro:asus_camera>
-  <!-- Extra Wheels -->
-  <!-- <xacro:include filename="$(find meka_description)/urdf/wheel_defs.urdf.xacro" />
+  </xacro:asus_camera-->
+  <!-- Extra Wheels
+  <xacro:include filename="$(find meka_description)/urdf/wheel_defs.urdf.xacro" />
   <wheel fb="front" lr="right" parent="base_link" translateX="1" translateY="-1" flipY="-1"/>
   <wheel fb="front" lr="left" parent="base_link" translateX="1" translateY="1" flipY="-1"/>

File: meka_description/transmissions/Z1R2B_zlift.transmission.xacro (robot description, xacro)
@@ -4,5 +4,5 @@
     <type>transmission_interface/SimpleTransmission</type>
     <joint name="zlift_j0">
-      <hardwareInterface>PositionJointInterface</hardwareInterface>
+      <hardwareInterface>EffortJointInterface</hardwareInterface>
     </joint>
     <actuator name="zlift_j0_motor">

File: meka_description/urdf/MEKA_BASIC.urdf.xacro (robot description, xacro)
@@ -48,10 +48,10 @@
 	</m3_l_arm>
 	<link name="base_link">
-	    <collision>
-          <origin xyz="0 0 0" rpy="0 0 0" />
-          <geometry>
-            <box size="0.8 0.6 0.025"/>
-          </geometry>
-        </collision>
+    <collision>
+      <origin xyz="0 0 0" rpy="0 0 0" />
+      <geometry>
+        <box size="0.8 0.6 0.025"/>
+      </geometry>
+    </collision>
 	</link>
 	<joint name="laser_front_joint" type="fixed">
@@ -76,170 +76,3 @@
 		<!-- 0.33 0.0 0.45 rpy="0 0.0236 0" -->
 	</meka_zlift>
-	<joint name="chest_joint" type="fixed">
-		<origin xyz="0.263 0.0 0.006" rpy="0 0 0" />
-		<parent link="zlift_link" />
-		<child link="panplate" />
-	</joint>
-	<link name="panplate">
-		<xacro:inertial_cuboid_with_pose mass="4.0" x_length="0.6" y_length="0.4" z_length="0.5">
-			<origin xyz="0 0 0" rpy="0 0 0" />
-		</xacro:inertial_cuboid_with_pose>
-		<visual>
-			<material name="GreyA" />
-			<origin xyz="0 0 0" rpy="0 0 0 " />
-			<geometry name="panplate_geom">
-				<mesh filename="package://${MESH}/T2R3/T2R3_TJ0_base.dae" />
-			</geometry>
-		</visual>
-		<!-- meshes
-	<collision><origin xyz="0 0 0" rpy="0.0 0.0 0.0 " /><geometry name="base_collision_geom"><mesh filename="package://${MESH_COLL}/T2R3/T2R3_TJ0_base.stl" /></geometry></collision>-->
-		<!-- primitive only -->
-		<collision>
-			<origin xyz="-0.11 0 0.025" rpy="0.0 0.0 0.0 " />
-			<geometry>
-				<box size="0.22 0.19 0.05" />
-			</geometry>
-		</collision>
-		<collision>
-			<origin xyz="0.0 0 0.05" rpy="0.0 0.0 0.0 " />
-			<geometry>
-				<cylinder radius="0.095" length="0.1" />
-			</geometry>
-		</collision>
-	</link>
-	<joint name="torso_j0" type="revolute">
-		<axis xyz="0 0 1"/>
-		<origin xyz="0 0 0.1658" rpy="0 0 0" />
-		<parent link="panplate" />
-		<child link="torso" />
-		<limit effort="25" velocity="${25.0*M_PI/180}" lower="${-120*M_PI/180.0}" upper="${120*M_PI/180}" />
-		<dynamics damping="1.0"/>
-	</joint>
-	<link name="torso">
-		<inertial>
-			<mass value="4.411" />
-			<origin xyz="0.00011774 0.0038073 -0.0522753" />
-			<inertia ixx="0.026360" ixy="-0.0000024" ixz="-0.0000508" iyy="0.0134266" iyz="0.0006839" izz="0.0229879" />
-		</inertial>
-		<visual>
-			<material name="GreyC" />
-			<origin xyz="0 0 0" rpy="0 0 0 " />
-			<geometry name="torso_geom">
-				<mesh filename="package://${MESH}/T2R3/T2R3_TJ1_pan.dae" />
-			</geometry>
-		</visual>
-		<!-- meshes
-	<collision><origin xyz="0 0 0" rpy="0.0 0.0 0.0 " /><geometry name="torso_collision_geom"><mesh filename="package://${MESH_COLL}/T2R3/T2R3_TJ1_pan.stl" /></geometry></collision>
-	-->
-		<!-- primitive only -->
-		<collision>
-			<origin xyz="0.0 0 -0.0615" rpy="0.0 0.0 0.0 " />
-			<geometry>
-				<cylinder radius="0.088" length="0.015" />
-			</geometry>
-		</collision>
-		<collision>
-			<origin xyz="0.0 0 -0.0615" rpy="0.0 0.0 0.0 " />
-			<geometry>
-				<box size="0.08 0.23 0.015" />
-			</geometry>
-		</collision>
-		<collision>
-			<origin xyz="0.0 0.105 0" rpy="1.5707 0.0 0.0 " />
-			<geometry>
-				<cylinder radius="0.052" length="0.02" />
-			</geometry>
-		</collision>
-		<collision>
-			<origin xyz="0.0 -0.105 0" rpy="1.5707 0.0 0.0  " />
-			<geometry>
-				<cylinder radius="0.052" length="0.02" />
-			</geometry>
-		</collision>
-	</link>
-	<joint name="torso_j1" type="revolute">
-		<axis xyz="0 1 0"/>
-		<origin xyz="0 0 0" rpy="0 0 0" />
-		<parent link="torso" />
-		<child link="mid" />
-		<limit effort="200" velocity="${10.0*M_PI/180}" lower="${-11.79349*M_PI/180}" upper="${53.29349*M_PI/180}" />
-		<dynamics damping="1.0"/>
-	</joint>
-	<link name="mid">
-		<inertial>
-			<mass value="4.934" />
-			<origin xyz="0.001179 -0.002993 0.046259"/>
-			<inertia ixx="0.041106" iyy="0.026009" izz="0.025902" ixy="0.000135" ixz="0.000505" iyz="0.002396" />
-		</inertial>
-		<visual>
-			<material name="GreyB" />
-			<origin xyz="0 0 0" rpy="0 0 0" />
-			<geometry name="mid_geom">
-				<mesh filename="package://${MESH}/T2R3/T2R3_TJ2.dae" />
-			</geometry>
-		</visual>
-		<!-- meshes
-	<collision><origin xyz="0 0 0" rpy="0.0 0.0 0.0 " /><geometry name="mid_collision_geom"><mesh filename="package://${MESH_COLL}/T2R3/T2R3_TJ2.stl" /></geometry></collision>
-	-->
-		<!-- primitive only -->
-		<collision>
-			<origin xyz="0.0 0 0.0684" rpy="0.0 0.0 0.0 " />
-			<geometry>
-				<box size="0.114 0.241 0.1368" />
-			</geometry>
-		</collision>
-		<collision>
-			<origin xyz="0.0 0.0 0" rpy="1.5707 0.0 0.0 " />
-			<geometry>
-				<cylinder radius="0.057" length="0.241" />
-			</geometry>
-		</collision>
-		<collision>
-			<origin xyz="0.0 0.0 0.1368" rpy="1.5707 0.0 0.0 " />
-			<geometry>
-				<cylinder radius="0.057" length="0.241" />
-			</geometry>
-		</collision>
-	</link>
-	<joint name="torso_j2" type="revolute">
-		<axis xyz="0 1 0"/>
-		<origin xyz="0 0 0.1397" rpy="0 0 0" />
-		<parent link="mid" />
-		<child link="upper" />
-		<limit effort="200" velocity="${10.0*M_PI/180}" lower="${-11.79349*M_PI/180}" upper="${53.29349*M_PI/180}" />
-		<dynamics damping="1.0"/>
-		<xacro:if value="$(arg torso_mimic)">
-			<mimic joint="torso_j1" multiplier="${torso_coupling}"/>
-		</xacro:if>
-	</joint>
-	<link name="upper">
-		<inertial>
-			<mass value="6.534" />
-			<origin xyz="0.008700 0.011470 0.129740"/>
-			<inertia ixx="0.069760" iyy="0.048010" izz="0.040590" ixy="-0.000400" ixz="0.001300" iyz="0.005100" />
-		</inertial>
-		<visual>
-			<material name="GreyC" />
-			<origin xyz="0 0 0" rpy="0 0 0" />
-			<geometry name="upper_geom">
-				<mesh filename="package://${MESH}/A2R3/A2R3_T4_Chest.dae" />
-			</geometry>
-		</visual>
-		<!-- meshes
-	<collision><origin xyz="0 0 0" rpy="0.0 0.0 0.0 " /><geometry name="upper_collision_geom"><mesh filename="package://${MESH_COLL}/T2R3/T2R3_TJ3_chest_waist_neck.stl" /></geometry></collision>
-		-->
-		<!-- primitive only -->
-		<collision>
-			<origin xyz="0.0 0 0.1346" rpy="0.0 0.0 0.0 " />
-			<geometry>
-				<box size="0.14 0.22 0.1978" />
-			</geometry>
-		</collision>
-		<collision>
-			<origin xyz="0.0 0.0 0.2335" rpy="1.5707 0.0 0.0 " />
-			<geometry>
-				<cylinder radius="0.0644" length="0.22" />
-			</geometry>
-		</collision>
-	</link>
 </robot>
