Commit message: camera link tf

File: meka_description/robots/bie_floka_sim.urdf.xacro (robot description, xacro)
@@ -7,5 +7,5 @@
     <xacro:arg name="_zlift" default="true"/>
     <xacro:arg name="_torso" default="true"/>
-    <xacro:arg name="_head" default="true"/>
+    <xacro:arg name="_head" default="false"/>
     <xacro:arg name="_xtion" default="true"/>
     <xacro:arg name="_r_arm" default="true"/>

File: meka_description/urdf/MEKA_BASIC.urdf.xacro (robot description, xacro)
@@ -50,4 +50,11 @@
 	<link name="laser_rear">
 	</link>
+    <joint name="camera_joint" type="fixed">
+      <origin xyz="0.045 -0.0551 0.195" rpy="${M_PI/2} -0.1 0" />
+      <child link="camera_link"/>
+      <parent link="upper"/>
+    </joint>
+    <link name="camera_link">
+    </link>
 	<!-- macro inserts -->
     <meka_base parent="${base_link}">
