Commit message: changed meka transmissions

File: meka_description/gazebo/gazebo.urdf.xacro (robot description, xacro)
@@ -1,11 +1,111 @@
 <?xml version="1.0"?>
-<robot xmlns:sensor="http://playerstage.sourceforge.net/gazebo/xmlschema/#sensor"
-       xmlns:controller="http://playerstage.sourceforge.net/gazebo/xmlschema/#controller"
-       xmlns:interface="http://playerstage.sourceforge.net/gazebo/xmlschema/#interface">
+<robot
+  xmlns:sensor="http://playerstage.sourceforge.net/gazebo/xmlschema/#sensor"
+  xmlns:controller="http://playerstage.sourceforge.net/gazebo/xmlschema/#controller"
+  xmlns:interface="http://playerstage.sourceforge.net/gazebo/xmlschema/#interface">
   <gazebo>
-    <controller:gazebo_ros_controller_manager name="gazebo_ros_controller_manager" plugin="libgazebo_ros_controller_manager.so">
+    <plugin name="gazebo_ros_control" filename="libgazebo_ros_control.so">
+      <robotNamespace></robotNamespace>
+      <robotSimType>gazebo_ros_control/DefaultRobotHWSim</robotSimType>
       <alwaysOn>true</alwaysOn>
-      <updateRate>10000.0</updateRate>
-    </controller:gazebo_ros_controller_manager>
+      <updateRate>30.0</updateRate>
+    </plugin>
+<!--
+    <plugin name="skid_steer_drive_controller" filename="libgazebo_ros_skid_steer_drive.so">
+      <alwaysOn>1</alwaysOn>
+      <updateRate>60.0</updateRate>
+      <robotNamespace>/</robotNamespace>
+      <leftFrontJoint>front_left_wheel_joint</leftFrontJoint>
+      <rightFrontJoint>front_right_wheel_joint</rightFrontJoint>
+      <leftRearJoint>back_left_wheel_joint</leftRearJoint>
+      <rightRearJoint>back_right_wheel_joint</rightRearJoint>
+      <wheelSeparation>1</wheelSeparation>
+      <wheelDiameter>${2*wheel_radius}</wheelDiameter>
+      <torque>1000</torque>
+      <broadcastTF>1</broadcastTF>
+      <odometryFrame>map</odometryFrame>
+      <commandTopic>cmd_vel</commandTopic>
+      <odometryTopic>odom</odometryTopic>
+      <robotBaseFrame>base_link</robotBaseFrame>
+      <covariance_x>0.0001</covariance_x>
+      <covariance_y>0.0001</covariance_y>
+      <covariance_z>0.0001</covariance_z>
+      <covariance_yaw>0.0001</covariance_yaw>
+    </plugin> -->
+    <plugin name="drive_controller" filename="libgazebo_ros_planar_move.so">
+      <odometryRate>60.0</odometryRate>
+      <robotNamespace>/</robotNamespace>
+      <commandTopic>cmd_vel</commandTopic>
+      <robotBaseFrame>base_footprint</robotBaseFrame>
+    </plugin>
+    <plugin name="mimic_right_j1a" filename="libroboticsgroup_gazebo_mimic_joint_plugin.so">
+      <joint>right_hand_j1</joint>
+      <mimicJoint>right_hand_j1a</mimicJoint>
+      <multiplier>${th_palmprox_coupling}</multiplier>
+      <sensitiveness>0.0</sensitiveness>
+    </plugin>
+    <plugin name="mimic_right_j1b" filename="libroboticsgroup_gazebo_mimic_joint_plugin.so">
+      <joint>right_hand_j1</joint>
+      <mimicJoint>right_hand_j1b</mimicJoint>
+      <multiplier>${th_proxdist_coupling}</multiplier>
+      <sensitiveness>0.0</sensitiveness>
+    </plugin>
+    <!-- j2 -->
+    <plugin name="mimic_right_j2a" filename="libroboticsgroup_gazebo_mimic_joint_plugin.so">
+      <joint>right_hand_j2</joint>
+      <mimicJoint>right_hand_j2a</mimicJoint>
+      <multiplier>${palmprox_coupling}</multiplier>
+      <sensitiveness>0.0</sensitiveness>
+    </plugin>
+    <plugin name="mimic_right_j2b" filename="libroboticsgroup_gazebo_mimic_joint_plugin.so">
+      <joint>right_hand_j2</joint>
+      <mimicJoint>right_hand_j2b</mimicJoint>
+      <multiplier>${proxmid_coupling}</multiplier>
+      <sensitiveness>0.0</sensitiveness>
+    </plugin>
+    <plugin name="mimic_right_j2c" filename="libroboticsgroup_gazebo_mimic_joint_plugin.so">
+      <joint>right_hand_j2</joint>
+      <mimicJoint>right_hand_j2c</mimicJoint>
+      <multiplier>${middist_coupling}</multiplier>
+      <sensitiveness>0.0</sensitiveness>
+    </plugin>
+    <!-- j3 -->
+   <plugin name="mimic_right_j3a" filename="libroboticsgroup_gazebo_mimic_joint_plugin.so">
+      <joint>right_hand_j3</joint>
+      <mimicJoint>right_hand_j3a</mimicJoint>
+      <multiplier>${palmprox_coupling}</multiplier>
+      <sensitiveness>0.0</sensitiveness>
+    </plugin>
+    <plugin name="mimic_right_j3b" filename="libroboticsgroup_gazebo_mimic_joint_plugin.so">
+      <joint>right_hand_j3</joint>
+      <mimicJoint>right_hand_j3b</mimicJoint>
+      <multiplier>${proxmid_coupling}</multiplier>
+      <sensitiveness>0.0</sensitiveness>
+    </plugin>
+    <plugin name="mimic_right_j3c" filename="libroboticsgroup_gazebo_mimic_joint_plugin.so">
+      <joint>right_hand_j3</joint>
+      <mimicJoint>right_hand_j3c</mimicJoint>
+      <multiplier>${middist_coupling}</multiplier>
+      <sensitiveness>0.0</sensitiveness>
+    </plugin>
+    <!-- j4 -->
+    <plugin name="mimic_right_j4a" filename="libroboticsgroup_gazebo_mimic_joint_plugin.so">
+      <joint>right_hand_j4</joint>
+      <mimicJoint>right_hand_j4a</mimicJoint>
+      <multiplier>${palmprox_coupling}</multiplier>
+      <sensitiveness>0.0</sensitiveness>
+    </plugin>
+    <plugin name="mimic_right_j4b" filename="libroboticsgroup_gazebo_mimic_joint_plugin.so">
+      <joint>right_hand_j4</joint>
+      <mimicJoint>right_hand_j4b</mimicJoint>
+      <multiplier>${proxmid_coupling}</multiplier>
+      <sensitiveness>0.0</sensitiveness>
+    </plugin>
+    <plugin name="mimic_right_j4c" filename="libroboticsgroup_gazebo_mimic_joint_plugin.so">
+      <joint>right_hand_j4</joint>
+      <mimicJoint>right_hand_j4c</mimicJoint>
+      <multiplier>${middist_coupling}</multiplier>
+      <sensitiveness>0.0</sensitiveness>
+    </plugin>
   </gazebo>
 </robot>

File: meka_description/robots/bie.urdf.xacro (robot description, xacro)
@@ -10,25 +10,29 @@
  <xacro:arg name="hand_mimic" default="true"/>
  <xacro:arg name="torso_mimic" default="true"/>
-<!-- synergy vector -->
- <xacro:property name="torso_coupling" value="1.0" />
-<!-- generic simulator_gazebo plugins for starting mechanism control, ros time, ros battery -->
+  <!-- synergy vector -->
+  <xacro:property name="torso_coupling" value="1.0" />
+  <!-- generic simulator_gazebo plugins for starting mechanism control, ros time, ros battery -->
   <xacro:include filename="$(find meka_description)/gazebo/gazebo.urdf.xacro" />
-  <!--<xacro:include filename="$(find meka_description)/transmissions/uta.transmission.xacro" />-->
-<!-- Meka Base -->
+  <xacro:include filename="$(find meka_description)/transmissions/body.transmission.xacro" />
+  <!-- Meka Base -->
   <xacro:include filename="$(find meka_description)/urdf/B1R2B_defs.urdf.xacro" />
-<!-- Meka Zlift -->
+  <!-- Meka Zlift -->
   <xacro:include filename="$(find meka_description)/urdf/Z1R2B_defs.urdf.xacro" />
-<!-- Meka Arm -->
+  <xacro:include filename="$(find meka_description)/transmissions/Z1R2B_zlift.transmission.xacro" />
+  <!-- Meka Arm -->
   <xacro:include filename="$(find meka_description)/urdf/A2R4_r_arm_defs.urdf.xacro" />
-  <xacro:include filename="$(find meka_description)/urdf/A2R4_l_arm_defs.urdf.xacro" />
+  <!-- <xacro:include filename="$(find meka_description)/urdf/A2R4_l_arm_defs.urdf.xacro" />  -->
+  <xacro:include filename="$(find meka_description)/transmissions/A2R4_r_arm_defs.transmission.xacro" />
+  <!-- <xacro:include filename="$(find meka_description)/transmissions/A2R4_l_arm_defs.transmission.xacro" />  -->
   <!-- Meka Hand -->
   <xacro:include filename="$(find meka_description)/urdf/H2R4_r_hand_defs.urdf.xacro" />
-  <xacro:include filename="$(find meka_description)/urdf/H2R4_l_hand_defs.urdf.xacro" />
-<!-- Meka Head -->
+  <!-- <xacro:include filename="$(find meka_description)/urdf/H2R4_l_hand_defs.urdf.xacro" />  -->
+  <xacro:include filename="$(find meka_description)/transmissions/H2R4_r_hand.transmission.xacro" />
+  <!-- <xacro:include filename="$(find meka_description)/transmissions/H2R4_l_hand.transmission.xacro" />  -->
+  <!-- Meka Head -->
   <xacro:include filename="$(find meka_description)/urdf/S3R1_head_defs.urdf.xacro" />
-  <!-- john added transmissions -->
-  <!-- <xacro:include filename="$(find meka_description)/transmissions/A2R4_r_arm_defs.transmission.xacro" /> -->
-  <!--<xacro:include filename="$(find meka_description)/transmissions/H2R2_r_hand_defs.transmission.xacro" />-->
-  <!--<xacro:include filename="$(find meka_description)/transmissions/S2R1_head_defs.transmission.xacro" />-->
+  <xacro:include filename="$(find meka_description)/transmissions/S3R1_head.transmission.xacro" />
+  <!-- Import asus -->
+  <xacro:include filename="$(find tobi_description)/urdf/asus_camera.urdf.xacro" />
    <property name="M_PI" value="3.1415926535897931" />
   <material name="GreyA"> <!-- darkest -->
@@ -43,5 +47,5 @@
   <!-- john added transmissions -->
   <m3_r_arm_transmission side="r" reflect="1" parent="upper"/>
-  <m3_r_hand_transmission/>
+  <m3_l_arm_transmission side="l" reflect="1" parent="upper"/>
   <m3_r_hand side="r" reflect="1" parent="handmount_RIGHT" use_mimic="$(arg hand_mimic)">
     <origin xyz="0.0 0.0 0.0" rpy="0 0 0" />
@@ -63,5 +67,5 @@
     <origin xyz="0.0 0.0 0.0" rpy="0 0 0" />
   </meka_base>
-  <meka_zlift  side="r" reflect="1" parent="dummy_3">
+  <meka_zlift  side="r" reflect="1" parent="base_link">
     <origin xyz="0.17513 0.0 0.43" rpy="0 0 0" /> <!-- 0.33 0.0 0.45 rpy="0 0.0236 0" -->
   </meka_zlift>
@@ -74,7 +78,7 @@
   <link name="panplate">
     <inertial>
-      <mass value="1000" />
+      <mass value="30" />
       <origin xyz="0 0 0" />
-      <inertia ixx="100"  ixy="0"  ixz="0" iyy="100" iyz="0" izz="100" />
+      <inertia ixx="1"  ixy="0"  ixz="0" iyy="1" iyz="0" izz="1" />
     </inertial>
     <visual>

File: meka_description/transmissions/A2R4_l_arm_defs.transmission.xacro (robot description, xacro)
@@ -1,24 +1,31 @@
 <?xml version="1.0"?>
-<robot xmlns:sensor="http://playerstage.sourceforge.net/gazebo/xmlschema/#sensor"
-       xmlns:controller="http://playerstage.sourceforge.net/gazebo/xmlschema/#controller"
-       xmlns:interface="http://playerstage.sourceforge.net/gazebo/xmlschema/#interface">
+<robot
+  xmlns:sensor="http://playerstage.sourceforge.net/gazebo/xmlschema/#sensor"
+  xmlns:controller="http://playerstage.sourceforge.net/gazebo/xmlschema/#controller"
+  xmlns:interface="http://playerstage.sourceforge.net/gazebo/xmlschema/#interface">
   <macro name="m3_l_shoulder_transmission" params="side parent reflect">
     <!-- Shoulder pan -->
     <transmission name="left_arm_t0" type="pr2_mechanism_model/SimpleTransmission">
+      <type>transmission_interface/SimpleTransmission</type>
       <actuator name="left_arm_a0" />
-      <joint name="left_arm_j0" />
-      <mechanicalReduction>1</mechanicalReduction>
+      <joint name="left_arm_j0">
+        <hardwareInterface>PositionJointInterface</hardwareInterface>
+      </joint>
     </transmission>
     <!-- Shoulder lift -->
     <transmission name="left_arm_t1" type="pr2_mechanism_model/SimpleTransmission">
+      <type>transmission_interface/SimpleTransmission</type>
       <actuator name="left_arm_a1" />
-      <joint name="left_arm_j1" />
-      <mechanicalReduction>1</mechanicalReduction>
+      <joint name="left_arm_j1">
+        <hardwareInterface>PositionJointInterface</hardwareInterface>
+      </joint>
     </transmission>
     <!-- Upperarm roll: internal fixed attchment point for upper arm -->
     <transmission name="left_arm_t2" type="pr2_mechanism_model/SimpleTransmission">
+      <type>transmission_interface/SimpleTransmission</type>
       <actuator name="left_arm_a2" />
-      <joint name="left_arm_j2" />
-      <mechanicalReduction>1</mechanicalReduction>
+      <joint name="left_arm_j2">
+        <hardwareInterface>PositionJointInterface</hardwareInterface>
+      </joint>
     </transmission>
   </macro>
@@ -26,13 +33,23 @@
   <macro name="m3_l_upper_arm_transmission" params="side parent reflect">
     <transmission name="left_arm_t3" type="pr2_mechanism_model/SimpleTransmission">
-      <actuator name="left_arm_a3" />
-      <joint name="left_arm_j3" />
+      <type>transmission_interface/SimpleTransmission</type>
+      <actuator name="left_arm_a3">
+        <hardwareInterface>PositionJointInterface</hardwareInterface>
+      </actuator>
+      <joint name="left_arm_j3">
+        <hardwareInterface>PositionJointInterface</hardwareInterface>
+      </joint>
       <mechanicalReduction>1</mechanicalReduction>
     </transmission>
     <!-- Elbow flex -->
     <transmission name="left_arm_t4" type="pr2_mechanism_model/SimpleTransmission">
-      <actuator name="left_arm_a4" />
-      <joint name="left_arm_j4" />
-      <mechanicalReduction>1</mechanicalReduction>
+      <type>transmission_interface/SimpleTransmission</type>
+      <actuator name="left_arm_a4">
+        <hardwareInterface>PositionJointInterface</hardwareInterface>
+        <mechanicalReduction>1</mechanicalReduction>
+      </actuator>
+      <joint name="left_arm_j4">
+        <hardwareInterface>PositionJointInterface</hardwareInterface>
+      </joint>
     </transmission>
   </macro>
@@ -40,19 +57,29 @@
   <macro name="m3_l_forearm_transmission" params="side parent reflect">
     <transmission name="left_arm_t5" type="pr2_mechanism_model/SimpleTransmission">
-      <actuator name="left_arm_a5" />
-      <joint name="left_arm_j5" />
-      <mechanicalReduction>1</mechanicalReduction>
+      <type>transmission_interface/SimpleTransmission</type>
+      <actuator name="left_arm_a5">
+        <hardwareInterface>PositionJointInterface</hardwareInterface>
+        <mechanicalReduction>1</mechanicalReduction>
+      </actuator>
+      <joint name="left_arm_j5">
+        <hardwareInterface>PositionJointInterface</hardwareInterface>
+      </joint>
     </transmission>
     <!-- Wrist flex -->
     <transmission name="left_arm_t6" type="pr2_mechanism_model/SimpleTransmission">
-      <actuator name="left_arm_a6" />
-      <joint name="left_arm_j6" />
-      <mechanicalReduction>1</mechanicalReduction>
+      <type>transmission_interface/SimpleTransmission</type>
+      <actuator name="left_arm_a6">
+        <hardwareInterface>PositionJointInterface</hardwareInterface>
+        <mechanicalReduction>1</mechanicalReduction>
+      </actuator>
+      <joint name="left_arm_j6">
+        <hardwareInterface>PositionJointInterface</hardwareInterface>
+      </joint>
     </transmission>
   </macro>
   <macro name="m3_l_arm_transmission" params="side parent reflect">
     <m3_l_shoulder_transmission side="${side}" reflect="${reflect}" parent="${parent}"/>
-    <m3_l_upper_arm_transmission side="${side}" reflect="${reflect}" parent="bicep_LEFT" />
-    <m3_l_forearm_transmission side="${side}" reflect="${reflect}" parent="wrist_LEFT" />
+    <m3_l_upper_arm_transmission side="${side}" reflect="${reflect}" parent="bicep_left" />
+    <m3_l_forearm_transmission side="${side}" reflect="${reflect}" parent="wrist_left" />
   </macro>
 </robot>

File: meka_description/transmissions/A2R4_r_arm_defs.transmission.xacro (robot description, xacro)
@@ -1,24 +1,31 @@
 <?xml version="1.0"?>
-<robot xmlns:sensor="http://playerstage.sourceforge.net/gazebo/xmlschema/#sensor"
-       xmlns:controller="http://playerstage.sourceforge.net/gazebo/xmlschema/#controller"
-       xmlns:interface="http://playerstage.sourceforge.net/gazebo/xmlschema/#interface">
+<robot
+  xmlns:sensor="http://playerstage.sourceforge.net/gazebo/xmlschema/#sensor"
+  xmlns:controller="http://playerstage.sourceforge.net/gazebo/xmlschema/#controller"
+  xmlns:interface="http://playerstage.sourceforge.net/gazebo/xmlschema/#interface">
   <macro name="m3_r_shoulder_transmission" params="side parent reflect">
     <!-- Shoulder pan -->
     <transmission name="right_arm_t0" type="pr2_mechanism_model/SimpleTransmission">
+      <type>transmission_interface/SimpleTransmission</type>
       <actuator name="right_arm_a0" />
-      <joint name="right_arm_j0" />
-      <mechanicalReduction>1</mechanicalReduction>
+      <joint name="right_arm_j0">
+        <hardwareInterface>PositionJointInterface</hardwareInterface>
+      </joint>
     </transmission>
     <!-- Shoulder lift -->
     <transmission name="right_arm_t1" type="pr2_mechanism_model/SimpleTransmission">
+      <type>transmission_interface/SimpleTransmission</type>
       <actuator name="right_arm_a1" />
-      <joint name="right_arm_j1" />
-      <mechanicalReduction>1</mechanicalReduction>
+      <joint name="right_arm_j1">
+        <hardwareInterface>PositionJointInterface</hardwareInterface>
+      </joint>
     </transmission>
     <!-- Upperarm roll: internal fixed attchment point for upper arm -->
     <transmission name="right_arm_t2" type="pr2_mechanism_model/SimpleTransmission">
+      <type>transmission_interface/SimpleTransmission</type>
       <actuator name="right_arm_a2" />
-      <joint name="right_arm_j2" />
-      <mechanicalReduction>1</mechanicalReduction>
+      <joint name="right_arm_j2">
+        <hardwareInterface>PositionJointInterface</hardwareInterface>
+      </joint>
     </transmission>
   </macro>
@@ -26,13 +33,23 @@
   <macro name="m3_r_upper_arm_transmission" params="side parent reflect">
     <transmission name="right_arm_t3" type="pr2_mechanism_model/SimpleTransmission">
-      <actuator name="right_arm_a3" />
-      <joint name="right_arm_j3" />
+      <type>transmission_interface/SimpleTransmission</type>
+      <actuator name="right_arm_a3">
+        <hardwareInterface>PositionJointInterface</hardwareInterface>
+      </actuator>
+      <joint name="right_arm_j3">
+        <hardwareInterface>PositionJointInterface</hardwareInterface>
+      </joint>
       <mechanicalReduction>1</mechanicalReduction>
     </transmission>
     <!-- Elbow flex -->
     <transmission name="right_arm_t4" type="pr2_mechanism_model/SimpleTransmission">
-      <actuator name="right_arm_a4" />
-      <joint name="right_arm_j4" />
-      <mechanicalReduction>1</mechanicalReduction>
+      <type>transmission_interface/SimpleTransmission</type>
+      <actuator name="right_arm_a4">
+        <hardwareInterface>PositionJointInterface</hardwareInterface>
+        <mechanicalReduction>1</mechanicalReduction>
+      </actuator>
+      <joint name="right_arm_j4">
+        <hardwareInterface>PositionJointInterface</hardwareInterface>
+      </joint>
     </transmission>
   </macro>
@@ -40,13 +57,23 @@
   <macro name="m3_r_forearm_transmission" params="side parent reflect">
     <transmission name="right_arm_t5" type="pr2_mechanism_model/SimpleTransmission">
-      <actuator name="right_arm_a5" />
-      <joint name="right_arm_j5" />
-      <mechanicalReduction>1</mechanicalReduction>
+      <type>transmission_interface/SimpleTransmission</type>
+      <actuator name="right_arm_a5">
+        <hardwareInterface>PositionJointInterface</hardwareInterface>
+        <mechanicalReduction>1</mechanicalReduction>
+      </actuator>
+      <joint name="right_arm_j5">
+        <hardwareInterface>PositionJointInterface</hardwareInterface>
+      </joint>
     </transmission>
     <!-- Wrist flex -->
     <transmission name="right_arm_t6" type="pr2_mechanism_model/SimpleTransmission">
-      <actuator name="right_arm_a6" />
-      <joint name="right_arm_j6" />
-      <mechanicalReduction>1</mechanicalReduction>
+      <type>transmission_interface/SimpleTransmission</type>
+      <actuator name="right_arm_a6">
+        <hardwareInterface>PositionJointInterface</hardwareInterface>
+        <mechanicalReduction>1</mechanicalReduction>
+      </actuator>
+      <joint name="right_arm_j6">
+        <hardwareInterface>PositionJointInterface</hardwareInterface>
+      </joint>
     </transmission>
   </macro>
