Commit message: changed meka transmissions

File: meka_description/urdf/B1R2B_defs.urdf.xacro (robot description, xacro)
@@ -2,89 +2,26 @@
 <robot xmlns:sensor="http://playerstage.sourceforge.net/gazebo/xmlschema/#sensor"
        xmlns:controller="http://playerstage.sourceforge.net/gazebo/xmlschema/#controller"
-       xmlns:interface="http://playerstage.sourceforge.net/gazebo/xmlschema/#interface">
+       xmlns:interface="http://playerstage.sourceforge.net/gazebo/xmlschema/#interface"
+       xmlns:xacro="http://playerstage.sourceforge.net/gazebo/xmlschema/#interface">
   <property name="M_PI" value="3.1415926535897931" />
+  <xacro:macro name="inertial_cuboid_with_pose" params="mass x_length y_length z_length *origin">
+    <inertial>
+      <xacro:insert_block name="origin"/>
+      <mass value="${mass}" />
+      <inertia ixx="${(1/12) * mass * (y_length*y_length + z_length*z_length)}" ixy="0.0" ixz="0.0"
+               iyy="${(1/12) * mass * (x_length*x_length + z_length*z_length)}" iyz="0.0"
+               izz="${(1/12) * mass * (x_length*x_length + y_length*y_length)}" />
+    </inertial>
+  </xacro:macro>
   <macro name="meka_base" params="side parent reflect *origin">
-    <joint name="X" type="fixed">  <!-- was prismatic -->
-      <axis xyz="1 0 0" />
+     <joint name="fixed_base_joint" type="fixed">
       <insert_block name="origin" />
+      <child link="fixed_base"/>
       <parent link="${parent}"/>
-      <child link="dummy_1"/>
-      <!--limit lower="${reflect*M_PI/4-1.5}"  upper="${reflect*M_PI/4+1.5}"
-             effort="30" velocity="${3.48}" />
-      <dynamics damping="10.0" />
-      <safety_controller k_position="100" k_velocity="10"
-                         soft_lower_limit="${reflect*M_PI/4-1.5+0.15}"
-                         soft_upper_limit="${reflect*M_PI/4+1.5-0.15}" /-->
     </joint>
-    <link name="dummy_1">
-      <inertial>
-        <mass value="25.799322" />
-        <origin xyz="0.0 0.0 0.0" rpy="0 0 0"/>
-        <inertia ixx="0.866179142480"  ixy="-0.06086507933"  ixz="-0.12118061183"
-                 iyy="0.87421714893"  iyz="-0.05886609911"
-                 izz="0.27353821674" />
-      </inertial>
-      <visual>
-	      <material name="GreyA" />
-	      <origin xyz="0 0 0" rpy="0 0 0 " />
-	      <geometry name="b1r1_1_geom">
-		      <box size="0.01 0.01 0.01" />
-	      </geometry>
-      </visual>
-      <collision>
-	      <origin xyz="0 0 0" rpy="0.0 0.0 0.0 " />
-	      <geometry name="b1r1_1_collision_geom">
-		      <box size="0.01 0.01 0.01" />
-	      </geometry>
-      </collision>
-    </link>
-    <joint name="Y" type="fixed"> <!-- was prismatic -->
-      <axis xyz="0 1 0"/>
-      <!-- limit lower="-0.5236" upper="1.3963"
-             effort="30" velocity="${3.47}" />
-      <safety_controller k_position="100" k_velocity="10"
-                         soft_lower_limit="${-0.5236+0.17}" soft_upper_limit="${1.3963-0.05}" />
-      <dynamics damping="10.0" / -->
-      <origin xyz="0 0 0" rpy="0 0 0" />
-      <parent link="dummy_1"/>
-      <child link="dummy_2"/>
-    </joint>
-    <link name="dummy_2">
-      <inertial>
-        <mass value="2.74988" />
-        <origin xyz="0.0 0.0 0.0" rpy="0 0 0"/>
-        <inertia ixx="0.02105584615" ixy="0.00496704022"  ixz="-0.00194808955"
-                 iyy="0.02127223737" iyz="0.00110425490"
-                 izz="0.01975753814" />
-      </inertial>
-      <visual>
-	      <material name="GreyB" />
-	      <origin xyz="0 0 0" rpy="0 0 0 " />
-	      <geometry name="b1r1_2_geom">
-		      <box size="0.01 0.01 0.01" />
-	      </geometry>
-      </visual>
-      <collision>
-	      <origin xyz="0 0 0" rpy="0.0 0.0 0.0 " />
-	      <geometry name="b1r1_2_collision_geom">
-		      <box size="0.01 0.01 0.01" />
-	      </geometry>
-      </collision>
-    </link>
-    <joint name="yaw" type="fixed">  <!-- was revolute -->
-      <axis xyz="0 0 1" />
-      <origin xyz="0 0.0 0.0" rpy="0 -0.017856194 0" />
-      <parent link="dummy_2" />
-      <child link="dummy_3"/>
-      <!-- limit lower="${reflect*1.55-2.35}" upper="${reflect*1.55+2.35}" effort="30" velocity="${5.45}" />
-      <safety_controller k_position="100" k_velocity="2" soft_lower_limit="${reflect*1.55-2.35+0.15}" soft_upper_limit="${reflect*1.55+2.35-0.15}" />
-      <dynamics damping="0.1" / -->
-    </joint>
-  <link name="dummy_3">
-	  <inertial>
-		  <mass value="1000" />
-		  <origin xyz="0 0 0" />
-		  <inertia ixx="1000"  ixy="0"  ixz="0" iyy="1000" iyz="0" izz="1000" />
-	  </inertial>
+  <link name="fixed_base">
+	  <xacro:inertial_cuboid_with_pose mass="100.0" x_length="0.6" y_length="0.4" z_length="0.5">
+      <origin xyz="0 0 0.25" rpy="0 0 0" />
+    </xacro:inertial_cuboid_with_pose>
 	  <visual>
 		  <material name="GreyC" />
@@ -101,12 +38,5 @@
 		  </geometry>
 	  </visual>
-	  <!--<collision>
-		  <origin xyz="0 0 0" rpy="0.0 0.0 0.0 " />
-		  <geometry name="b1r1_3_geom">
-			  <mesh filename="package://${MESH_COLL}/B1R1/MB1_00_000_meka_mobile_base+backpack+zlift.stl" />
-		  </geometry>
-	  </collision>-->
-    <!-- primitive meshes only -->
-    <collision>
+	  <collision>
 		  <origin xyz="0 0 0.2" rpy="0.0 0.0 0.0 " />
 		  <geometry>

File: meka_description/urdf/H2R4_l_hand_defs.urdf.xacro (robot description, xacro)
@@ -191,5 +191,10 @@
       <limit effort="100" velocity="${50*M_PI/180}" lower="${0*M_PI/180}" upper="${170.0*M_PI/180.0}" />
     </joint>
-    <link name="thumb_motor_left"/>
+    <link name="thumb_motor_left">
+      <inertial>
+        <mass value="2e-06"/>
+        <inertia ixx="1.1e-09" ixy="0" ixz="0" iyy="1.1e-09" iyz="0" izz="1.1e-09"/>
+		  </inertial>
+    </link>
     <joint name="left_hand_j1a" type="revolute">
       <axis xyz="0 -1 0"/>
@@ -315,5 +320,10 @@
         <limit effort="100" velocity="${50*M_PI/180}" lower="${0*M_PI/180}" upper="${300.0*M_PI/180.0}" />
       </joint>
-      <link name="index_motor_left"/>
+      <link name="index_motor_left">
+        <inertial>
+          <mass value="2e-06"/>
+          <inertia ixx="1.1e-09" ixy="0" ixz="0" iyy="1.1e-09" iyz="0" izz="1.1e-09"/>
+        </inertial>
+      </link>
       <joint name="left_hand_j2a" type="revolute">
         <axis xyz="0 1 0" />
@@ -503,5 +513,10 @@
         <limit effort="100" velocity="${50*M_PI/180}" lower="${0*M_PI/180}" upper="${300.0*M_PI/180}" />
       </joint>
-    <link name="ring_motor_left"/>
+    <link name="ring_motor_left">
+        <inertial>
+          <mass value="2e-06"/>
+          <inertia ixx="1.1e-09" ixy="0" ixz="0" iyy="1.1e-09" iyz="0" izz="1.1e-09"/>
+        </inertial>
+      </link>
     <joint name="left_hand_j3a" type="revolute">
       <axis xyz="0 1 0" />
@@ -692,5 +707,10 @@
         <limit effort="100" velocity="${50*M_PI/180}" lower="${0*M_PI/180}" upper="${300.0*M_PI/180}" />
       </joint>
-    <link name="pinky_motor_left"/>
+    <link name="pinky_motor_left">
+        <inertial>
+          <mass value="2e-06"/>
+          <inertia ixx="1.1e-09" ixy="0" ixz="0" iyy="1.1e-09" iyz="0" izz="1.1e-09"/>
+        </inertial>
+      </link>
     <joint name="left_hand_j4a" type="revolute">
       <axis xyz="0 1 0" />

File: meka_description/urdf/H2R4_r_hand_defs.urdf.xacro (robot description, xacro)
@@ -192,5 +192,10 @@
       <limit effort="100" velocity="${50*M_PI/180}" lower="${0*M_PI/180}" upper="${170.0*M_PI/180.0}" />
     </joint>
-    <link name="thumb_motor_right"/>
+    <link name="thumb_motor_right">
+        <inertial>
+          <mass value="2e-06"/>
+          <inertia ixx="1.1e-09" ixy="0" ixz="0" iyy="1.1e-09" iyz="0" izz="1.1e-09"/>
+        </inertial>
+      </link>
     <joint name="right_hand_j1a" type="revolute">
       <axis xyz="0 -1 0"/>
@@ -316,5 +321,10 @@
         <limit effort="100" velocity="${50*M_PI/180}" lower="${0*M_PI/180}" upper="${300.0*M_PI/180.0}" />
       </joint>
-      <link name="index_motor_right"/>
+      <link name="index_motor_right">
+        <inertial>
+          <mass value="2e-06"/>
+          <inertia ixx="1.1e-09" ixy="0" ixz="0" iyy="1.1e-09" iyz="0" izz="1.1e-09"/>
+        </inertial>
+      </link>
       <joint name="right_hand_j2a" type="revolute">
         <axis xyz="0 1 0" />
@@ -504,5 +514,10 @@
         <limit effort="100" velocity="${50*M_PI/180}" lower="${0*M_PI/180}" upper="${300.0*M_PI/180}" />
       </joint>
-    <link name="ring_motor_right"/>
+    <link name="ring_motor_right">
+        <inertial>
+          <mass value="2e-06"/>
+          <inertia ixx="1.1e-09" ixy="0" ixz="0" iyy="1.1e-09" iyz="0" izz="1.1e-09"/>
+        </inertial>
+      </link>
     <joint name="right_hand_j3a" type="revolute">
       <axis xyz="0 1 0" />
@@ -693,5 +708,10 @@
         <limit effort="100" velocity="${50*M_PI/180}" lower="${0*M_PI/180}" upper="${300.0*M_PI/180}" />
       </joint>
-    <link name="pinky_motor_right"/>
+    <link name="pinky_motor_right">
+        <inertial>
+          <mass value="2e-06"/>
+          <inertia ixx="1.1e-09" ixy="0" ixz="0" iyy="1.1e-09" iyz="0" izz="1.1e-09"/>
+        </inertial>
+      </link>
     <joint name="right_hand_j4a" type="revolute">
       <axis xyz="0 1 0" />

Commit message: fixed models to prevent the robot from falling over in gazebo

File: meka_description/gazebo/gazebo.urdf.xacro (robot description, xacro)
@@ -33,11 +33,12 @@
       <covariance_yaw>0.0001</covariance_yaw>
     </plugin> -->
-    <plugin name="drive_controller" filename="libgazebo_ros_planar_move.so">
-      <odometryRate>60.0</odometryRate>
-      <robotNamespace>/</robotNamespace>
+    <plugin name="object_controller" filename="libgazebo_ros_planar_move.so">
       <commandTopic>cmd_vel</commandTopic>
+      <odometryTopic>odom</odometryTopic>
+      <odometryFrame>odom</odometryFrame>
+      <odometryRate>20.0</odometryRate>
       <robotBaseFrame>base_link</robotBaseFrame>
     </plugin>
-    <plugin name="mimic_right_j1a" filename="libroboticsgroup_gazebo_mimic_joint_plugin.so">
+    <!--plugin name="mimic_right_j1a" filename="libroboticsgroup_gazebo_mimic_joint_plugin.so">
       <joint>right_hand_j1</joint>
       <mimicJoint>right_hand_j1a</mimicJoint>
@@ -51,5 +52,4 @@
       <sensitiveness>0.0</sensitiveness>
     </plugin>
-    <!-- j2 -->
     <plugin name="mimic_right_j2a" filename="libroboticsgroup_gazebo_mimic_joint_plugin.so">
       <joint>right_hand_j2</joint>
@@ -70,5 +70,4 @@
       <sensitiveness>0.0</sensitiveness>
     </plugin>
-    <!-- j3 -->
    <plugin name="mimic_right_j3a" filename="libroboticsgroup_gazebo_mimic_joint_plugin.so">
       <joint>right_hand_j3</joint>
@@ -89,5 +88,4 @@
       <sensitiveness>0.0</sensitiveness>
     </plugin>
-    <!-- j4 -->
     <plugin name="mimic_right_j4a" filename="libroboticsgroup_gazebo_mimic_joint_plugin.so">
       <joint>right_hand_j4</joint>
@@ -107,5 +105,5 @@
       <multiplier>${middist_coupling}</multiplier>
       <sensitiveness>0.0</sensitiveness>
-    </plugin>
+    </plugin-->
   </gazebo>
   <gazebo reference="base_link">

File: meka_description/robots/bie.urdf.xacro (robot description, xacro)
@@ -21,12 +21,12 @@
   <xacro:include filename="$(find meka_description)/transmissions/Z1R2B_zlift.transmission.xacro" />
   <!-- Meka Arm -->
-  <xacro:include filename="$(find meka_description)/urdf/A2R4_r_arm_defs.urdf.xacro" />
+  <!--xacro:include filename="$(find meka_description)/urdf/A2R4_r_arm_defs.urdf.xacro" /-->
   <!-- <xacro:include filename="$(find meka_description)/urdf/A2R4_l_arm_defs.urdf.xacro" />  -->
-  <xacro:include filename="$(find meka_description)/transmissions/A2R4_r_arm_defs.transmission.xacro" />
+  <!--xacro:include filename="$(find meka_description)/transmissions/A2R4_r_arm_defs.transmission.xacro" /-->
   <!-- <xacro:include filename="$(find meka_description)/transmissions/A2R4_l_arm_defs.transmission.xacro" />  -->
   <!-- Meka Hand -->
-  <xacro:include filename="$(find meka_description)/urdf/H2R4_r_hand_defs.urdf.xacro" />
+  <!--xacro:include filename="$(find meka_description)/urdf/H2R4_r_hand_defs.urdf.xacro" /-->
   <!-- <xacro:include filename="$(find meka_description)/urdf/H2R4_l_hand_defs.urdf.xacro" />  -->
-  <xacro:include filename="$(find meka_description)/transmissions/H2R4_r_hand.transmission.xacro" />
+  <!--xacro:include filename="$(find meka_description)/transmissions/H2R4_r_hand.transmission.xacro" /-->
   <!-- <xacro:include filename="$(find meka_description)/transmissions/H2R4_l_hand.transmission.xacro" />  -->
   <!-- Meka Head -->
@@ -43,4 +43,13 @@
     <color rgba="0.7 0.7 0.7 1.0"/>
   </material>
+  <xacro:macro name="inertial_cuboid_with_pose" params="mass x_length y_length z_length *origin">
+    <inertial>
+      <xacro:insert_block name="origin"/>
+      <mass value="${mass}" />
+      <inertia ixx="${(1/12) * mass * (y_length*y_length + z_length*z_length)}" ixy="0.0" ixz="0.0"
+               iyy="${(1/12) * mass * (x_length*x_length + z_length*z_length)}" iyz="0.0"
+               izz="${(1/12) * mass * (x_length*x_length + y_length*y_length)}" />
+    </inertial>
+  </xacro:macro>
   <!-- john added transmissions -->
   <m3_r_arm_transmission side="r" reflect="1" parent="upper"/>
@@ -61,5 +70,12 @@
     <origin xyz="0.0 0.18465 0.2337" rpy="0 0 0" />
   </m3_l_arm>
-  <link name="base_link" />
+  <link name="base_link" >
+       <collision>
+          <origin xyz="0 0 0" rpy="0 0 0" />
+          <geometry>
+            <box size="1.035 1.185 0.025"/>
+          </geometry>
+        </collision>
+        </link>
   <meka_base  side="r" reflect="1" parent="base_link">
     <origin xyz="0.0 0.0 0.0" rpy="0 0 0" />
@@ -75,9 +91,7 @@
   </joint>
   <link name="panplate">
-    <inertial>
-      <mass value="30" />
-      <origin xyz="0 0 0" />
-      <inertia ixx="1"  ixy="0"  ixz="0" iyy="1" iyz="0" izz="1" />
-    </inertial>
+<xacro:inertial_cuboid_with_pose mass="20.0" x_length="0.6" y_length="0.4" z_length="0.5">
+      <origin xyz="0 0 0" rpy="0 0 0" />
+    </xacro:inertial_cuboid_with_pose>
     <visual>
       <material name="GreyA" />
