Commit message: made gazebo compatible

File: meka_description/gazebo/gazebo.urdf.xacro (robot description, xacro)
@@ -10,4 +10,10 @@
       <alwaysOn>true</alwaysOn>
       <updateRate>30.0</updateRate>
+    </plugin>
+    <plugin filename="libroboticsgroup_gazebo_mimic_joint_plugin.so" name="mimic_torso">
+        <joint>torso_j1</joint>
+        <mimicJoint>torso_j2</mimicJoint>
+        <multiplier>1.0</multiplier>
+        <!--offset>0.0</offset-->
     </plugin>
 <!--

File: meka_description/transmissions/A2R4_l_arm_defs.transmission.xacro (robot description, xacro)
@@ -35,10 +35,9 @@
       <type>transmission_interface/SimpleTransmission</type>
       <actuator name="left_arm_a3">
-        <hardwareInterface>PositionJointInterface</hardwareInterface>
+          <mechanicalReduction>1</mechanicalReduction>
       </actuator>
       <joint name="left_arm_j3">
         <hardwareInterface>PositionJointInterface</hardwareInterface>
       </joint>
-      <mechanicalReduction>1</mechanicalReduction>
     </transmission>
     <!-- Elbow flex -->
@@ -46,5 +45,4 @@
       <type>transmission_interface/SimpleTransmission</type>
       <actuator name="left_arm_a4">
-        <hardwareInterface>PositionJointInterface</hardwareInterface>
         <mechanicalReduction>1</mechanicalReduction>
       </actuator>
@@ -59,5 +57,4 @@
       <type>transmission_interface/SimpleTransmission</type>
       <actuator name="left_arm_a5">
-        <hardwareInterface>PositionJointInterface</hardwareInterface>
         <mechanicalReduction>1</mechanicalReduction>
       </actuator>
@@ -70,5 +67,4 @@
       <type>transmission_interface/SimpleTransmission</type>
       <actuator name="left_arm_a6">
-        <hardwareInterface>PositionJointInterface</hardwareInterface>
         <mechanicalReduction>1</mechanicalReduction>
       </actuator>

File: meka_description/transmissions/A2R4_r_arm_defs.transmission.xacro (robot description, xacro)
@@ -35,10 +35,9 @@
       <type>transmission_interface/SimpleTransmission</type>
       <actuator name="right_arm_a3">
-        <hardwareInterface>PositionJointInterface</hardwareInterface>
+          <mechanicalReduction>1</mechanicalReduction>
       </actuator>
       <joint name="right_arm_j3">
         <hardwareInterface>PositionJointInterface</hardwareInterface>
       </joint>
-      <mechanicalReduction>1</mechanicalReduction>
     </transmission>
     <!-- Elbow flex -->
@@ -46,5 +45,4 @@
       <type>transmission_interface/SimpleTransmission</type>
       <actuator name="right_arm_a4">
-        <hardwareInterface>PositionJointInterface</hardwareInterface>
         <mechanicalReduction>1</mechanicalReduction>
       </actuator>
@@ -59,5 +57,4 @@
       <type>transmission_interface/SimpleTransmission</type>
       <actuator name="right_arm_a5">
-        <hardwareInterface>PositionJointInterface</hardwareInterface>
         <mechanicalReduction>1</mechanicalReduction>
       </actuator>
@@ -70,5 +67,4 @@
       <type>transmission_interface/SimpleTransmission</type>
       <actuator name="right_arm_a6">
-        <hardwareInterface>PositionJointInterface</hardwareInterface>
         <mechanicalReduction>1</mechanicalReduction>
       </actuator>

File: meka_description/transmissions/H2R4_l_hand.transmission.xacro (robot description, xacro)
@@ -9,5 +9,4 @@
     </joint>
     <actuator name="left_hand_j0_motor">
-      <hardwareInterface>PositionJointInterface</hardwareInterface>
       <mechanicalReduction>1</mechanicalReduction>
     </actuator>
@@ -19,5 +18,4 @@
     </joint>
     <actuator name="left_hand_j1_motor">
-      <hardwareInterface>PositionJointInterface</hardwareInterface>
       <mechanicalReduction>1</mechanicalReduction>
     </actuator>
@@ -29,5 +27,4 @@
     </joint>
     <actuator name="left_hand_j2_motor">
-      <hardwareInterface>PositionJointInterface</hardwareInterface>
       <mechanicalReduction>1</mechanicalReduction>
     </actuator>
@@ -39,5 +36,4 @@
     </joint>
     <actuator name="left_hand_j3_motor">
-      <hardwareInterface>PositionJointInterface</hardwareInterface>
       <mechanicalReduction>1</mechanicalReduction>
     </actuator>
@@ -49,5 +45,4 @@
     </joint>
     <actuator name="left_hand_j4_motor">
-      <hardwareInterface>PositionJointInterface</hardwareInterface>
       <mechanicalReduction>1</mechanicalReduction>
     </actuator>

File: meka_description/transmissions/H2R4_r_hand.transmission.xacro (robot description, xacro)
@@ -9,5 +9,4 @@
     </joint>
     <actuator name="right_hand_j0_motor">
-      <hardwareInterface>PositionJointInterface</hardwareInterface>
       <mechanicalReduction>1</mechanicalReduction>
     </actuator>
@@ -19,5 +18,4 @@
     </joint>
     <actuator name="right_hand_j1_motor">
-      <hardwareInterface>PositionJointInterface</hardwareInterface>
       <mechanicalReduction>1</mechanicalReduction>
     </actuator>
@@ -29,5 +27,4 @@
     </joint>
     <actuator name="right_hand_j2_motor">
-      <hardwareInterface>PositionJointInterface</hardwareInterface>
       <mechanicalReduction>1</mechanicalReduction>
     </actuator>
@@ -39,5 +36,4 @@
     </joint>
     <actuator name="right_hand_j3_motor">
-      <hardwareInterface>PositionJointInterface</hardwareInterface>
       <mechanicalReduction>1</mechanicalReduction>
     </actuator>
@@ -49,5 +45,4 @@
     </joint>
     <actuator name="right_hand_j4_motor">
-      <hardwareInterface>PositionJointInterface</hardwareInterface>
       <mechanicalReduction>1</mechanicalReduction>
     </actuator>

File: meka_description/transmissions/S3R1_head.transmission.xacro (robot description, xacro)
@@ -7,5 +7,4 @@
     </joint>
     <actuator name="head_j0_motor">
-      <hardwareInterface>PositionJointInterface</hardwareInterface>
       <mechanicalReduction>1</mechanicalReduction>
     </actuator>
@@ -17,5 +16,4 @@
     </joint>
     <actuator name="head_j1_motor">
-      <hardwareInterface>PositionJointInterface</hardwareInterface>
       <mechanicalReduction>1</mechanicalReduction>
     </actuator>

File: meka_description/transmissions/Z1R2B_zlift.transmission.xacro (robot description, xacro)
@@ -7,5 +7,4 @@
     </joint>
     <actuator name="zlift_j0_motor">
-      <hardwareInterface>PositionJointInterface</hardwareInterface>
       <mechanicalReduction>1</mechanicalReduction>
     </actuator>

File: meka_description/transmissions/body.transmission.xacro (robot description, xacro)
@@ -7,5 +7,4 @@
     </joint>
     <actuator name="torso_j0_motor">
-      <hardwareInterface>PositionJointInterface</hardwareInterface>
       <mechanicalReduction>1</mechanicalReduction>
     </actuator>
@@ -17,15 +16,4 @@
     </joint>
     <actuator name="torso_j1_motor">
-      <hardwareInterface>PositionJointInterface</hardwareInterface>
-      <mechanicalReduction>1</mechanicalReduction>
-    </actuator>
-  </transmission>
-  <transmission name="torso_j2_trans">
-    <type>transmission_interface/SimpleTransmission</type>
-    <joint name="torso_j2">
-      <hardwareInterface>PositionJointInterface</hardwareInterface>
-    </joint>
-    <actuator name="torso_j2_motor">
-      <hardwareInterface>PositionJointInterface</hardwareInterface>
       <mechanicalReduction>1</mechanicalReduction>
     </actuator>

File: meka_description/urdf/A2R4_l_arm_defs.urdf.xacro (robot description, xacro)
@@ -2,5 +2,5 @@
 <robot xmlns:sensor="http://playerstage.sourceforge.net/gazebo/xmlschema/#sensor"
        xmlns:controller="http://playerstage.sourceforge.net/gazebo/xmlschema/#controller"
-       xmlns:interface="http://playerstage.sourceforge.net/gazebo/xmlschema/#interface">
+       xmlns:interface="http://ros.org/wiki/xacro">
   <property name="M_PI" value="3.1415926535897931" />
   <property name="VELOCITY_LIMIT_SCALE" value="0.6" />
@@ -38,9 +38,9 @@
     <link name="shoulderupper_LEFT">
       <inertial>
-        <mass value="2.5799322" />
+        <mass value="2.0310" />
         <origin xyz="-0.001201 0.024513 -0.098231" rpy="0 0 0"/>
-        <inertia ixx="0.866179142480"  ixy="-0.06086507933"  ixz="-0.12118061183"
-                 iyy="0.87421714893"  iyz="-0.05886609911"
-                 izz="0.27353821674" />
+        <inertia xx="0.003461" ixy="0.000428" ixz="0.000002"
+	             iyy="0.003097" iyz="0.000000"
+	             zz="0.005416" />
       </inertial>
       <visual>

File: meka_description/urdf/A2R4_r_arm_defs.urdf.xacro (robot description, xacro)
@@ -2,5 +2,5 @@
 <robot xmlns:sensor="http://playerstage.sourceforge.net/gazebo/xmlschema/#sensor"
        xmlns:controller="http://playerstage.sourceforge.net/gazebo/xmlschema/#controller"
-       xmlns:interface="http://playerstage.sourceforge.net/gazebo/xmlschema/#interface">
+       xmlns:interface="http://ros.org/wiki/xacro">
   <property name="M_PI" value="3.1415926535897931" />
   <macro name="m3_r_shoulder" params="side parent reflect *origin">
@@ -17,11 +17,8 @@
       <inertial>
         <mass value="2.0310" />
-	<origin xyz="-0.010946 0.025127 0.000022"/>
-	<inertia ixx="0.003461"
-	iyy="0.003097"
-	izz="0.005416"
-	ixy="0.000428"
-	ixz="0.000002"
-	iyz="0.000000" />
+	    <origin xyz="-0.010946 0.025127 0.000022"/>
+	    <inertia ixx="0.003461" ixy="0.000428" ixz="0.000002"
+	             iyy="0.003097" iyz="0.000000"
+	             zz="0.005416" />
       </inertial>
       <visual>

File: meka_description/urdf/B1R2B_defs.urdf.xacro (robot description, xacro)
@@ -4,5 +4,5 @@
        xmlns:interface="http://playerstage.sourceforge.net/gazebo/xmlschema/#interface"
        xmlns:xacro="http://playerstage.sourceforge.net/gazebo/xmlschema/#interface">
-  <property name="M_PI" value="3.1415926535897931" />
+  <xacro:property name="M_PI" value="3.1415926535897931" />
   <xacro:macro name="inertial_cuboid_with_pose" params="mass x_length y_length z_length *origin">
     <inertial>
@@ -14,13 +14,13 @@
     </inertial>
   </xacro:macro>
-  <macro name="meka_base" params="side parent reflect *origin">
+  <xacro:macro name="meka_base" params="side parent reflect *origin">
      <joint name="fixed_base_joint" type="fixed">
-      <insert_block name="origin" />
+      <xacro:insert_block name="origin" />
       <child link="fixed_base"/>
       <parent link="${parent}"/>
     </joint>
   <link name="fixed_base">
-	  <xacro:inertial_cuboid_with_pose mass="100.0" x_length="0.6" y_length="0.4" z_length="0.5">
-      <origin xyz="0 0 0.25" rpy="0 0 0" />
+	  <xacro:inertial_cuboid_with_pose mass="120.0" x_length="0.6" y_length="0.4" z_length="0.5">
+      <origin xyz="-0.10 0 0.2" rpy="0 0 0" />
     </xacro:inertial_cuboid_with_pose>
 	  <visual>
@@ -94,4 +94,4 @@
 	  </collision>
   </link>
-  </macro>
+  </xacro:macro>
 </robot>

File: meka_description/urdf/MEKA_BASIC.urdf.xacro (robot description, xacro)
@@ -13,5 +13,4 @@
   	<xacro:property name="torso_coupling" value="1.0" />
 	<material name="GreyA">
-		<!-- darkest -->
 		<color rgba="0.3 0.3 0.3 1.0"/>
 	</material>
@@ -49,4 +48,10 @@
 	</m3_l_arm>
 	<link name="base_link">
+	    <collision>
+          <origin xyz="0 0 0" rpy="0 0 0" />
+          <geometry>
+            <box size="0.8 0.6 0.025"/>
+          </geometry>
+        </collision>
 	</link>
 	<joint name="laser_front_joint" type="fixed">
@@ -71,5 +76,4 @@
 		<!-- 0.33 0.0 0.45 rpy="0 0.0236 0" -->
 	</meka_zlift>
-	<!-- Solid Base -->
 	<joint name="chest_joint" type="fixed">
 		<origin xyz="0.263 0.0 0.006" rpy="0 0 0" />
@@ -78,5 +82,5 @@
 	</joint>
 	<link name="panplate">
-		<xacro:inertial_cuboid_with_pose mass="20.0" x_length="0.6" y_length="0.4" z_length="0.5">
+		<xacro:inertial_cuboid_with_pose mass="4.0" x_length="0.6" y_length="0.4" z_length="0.5">
 			<origin xyz="0 0 0" rpy="0 0 0" />
 		</xacro:inertial_cuboid_with_pose>
