Commit message: reverted sim

File: meka_description/gazebo/gazebo.urdf.xacro (robot description, xacro)
@@ -3,5 +3,6 @@
   xmlns:sensor="http://playerstage.sourceforge.net/gazebo/xmlschema/#sensor"
   xmlns:controller="http://playerstage.sourceforge.net/gazebo/xmlschema/#controller"
-  xmlns:interface="http://playerstage.sourceforge.net/gazebo/xmlschema/#interface">
+  xmlns:interface="http://playerstage.sourceforge.net/gazebo/xmlschema/#interface"
+  xmlns:xacro="http://playerstage.sourceforge.net/gazebo/xmlschema/#interface">
   <gazebo>
     <plugin name="gazebo_ros_control" filename="libgazebo_ros_control.so">
@@ -42,90 +43,94 @@
       <recover_pitch_velocity_p_gain>10.0</recover_pitch_velocity_p_gain>
       <recover_z_velocity_p_gain>50.0</recover_z_velocity_p_gain>
-      <x_velocity_limit_max>0.5</x_velocity_limit_max>
-      <x_velocity_limit_min>-0.5</x_velocity_limit_min>
-      <y_velocity_limit_max>0.5</y_velocity_limit_max>
-      <y_velocity_limit_min>-0.5</y_velocity_limit_min>
-      <rot_velocity_limit_max>0.5</rot_velocity_limit_max>
-      <rot_velocity_limit_min>-0.5</rot_velocity_limit_min>
-      <x_acceleration_limit_max>1.5</x_acceleration_limit_max>
-      <x_acceleration_limit_min>-1.5</x_acceleration_limit_min>
-      <y_acceleration_limit_max>1.0</y_acceleration_limit_max>
-      <y_acceleration_limit_min>-1.0</y_acceleration_limit_min>
-      <rot_acceleration_limit_max>0.5</rot_acceleration_limit_max>
-      <rot_acceleration_limit_min>-0.5</rot_acceleration_limit_min>
+      <x_velocity_limit_max>2.0</x_velocity_limit_max>
+      <x_velocity_limit_min>-2.0</x_velocity_limit_min>
+      <y_velocity_limit_max>2.0</y_velocity_limit_max>
+      <y_velocity_limit_min>-2.0</y_velocity_limit_min>
+      <rot_velocity_limit_max>1.5</rot_velocity_limit_max>
+      <rot_velocity_limit_min>-1.5</rot_velocity_limit_min>
+      <x_acceleration_limit_max>2.0</x_acceleration_limit_max>
+      <x_acceleration_limit_min>-2.0</x_acceleration_limit_min>
+      <y_acceleration_limit_max>2.0</y_acceleration_limit_max>
+      <y_acceleration_limit_min>-2.0</y_acceleration_limit_min>
+      <rot_acceleration_limit_max>1.5</rot_acceleration_limit_max>
+      <rot_acceleration_limit_min>-1.5</rot_acceleration_limit_min>
       <tilt_angle_par_max_velocity>0</tilt_angle_par_max_velocity>
     </plugin>
-    <plugin name="mimic_torso" filename="libroboticsgroup_gazebo_mimic_joint_plugin.so">
-        <joint>torso_j1</joint>
-        <mimicJoint>torso_j2</mimicJoint>
-        <multiplier>1.0</multiplier>
-        <!--offset>0.0</offset-->
-    </plugin>
-    <plugin name="mimic_right_j1a" filename="libroboticsgroup_gazebo_mimic_joint_plugin.so">
-      <joint>right_hand_j1</joint>
-      <mimicJoint>right_hand_j1a</mimicJoint>
-      <multiplier>${th_palmprox_coupling}</multiplier>
-      <sensitiveness>0.0</sensitiveness>
-    </plugin>
-    <plugin name="mimic_right_j1b" filename="libroboticsgroup_gazebo_mimic_joint_plugin.so">
-      <joint>right_hand_j1</joint>
-      <mimicJoint>right_hand_j1b</mimicJoint>
-      <multiplier>${th_proxdist_coupling}</multiplier>
-      <sensitiveness>0.0</sensitiveness>
-    </plugin>
-    <plugin name="mimic_right_j2a" filename="libroboticsgroup_gazebo_mimic_joint_plugin.so">
-      <joint>right_hand_j2</joint>
-      <mimicJoint>right_hand_j2a</mimicJoint>
-      <multiplier>${palmprox_coupling}</multiplier>
-      <sensitiveness>0.0</sensitiveness>
-    </plugin>
-    <plugin name="mimic_right_j2b" filename="libroboticsgroup_gazebo_mimic_joint_plugin.so">
-      <joint>right_hand_j2</joint>
-      <mimicJoint>right_hand_j2b</mimicJoint>
-      <multiplier>${proxmid_coupling}</multiplier>
-      <sensitiveness>0.0</sensitiveness>
-    </plugin>
-    <plugin name="mimic_right_j2c" filename="libroboticsgroup_gazebo_mimic_joint_plugin.so">
-      <joint>right_hand_j2</joint>
-      <mimicJoint>right_hand_j2c</mimicJoint>
-      <multiplier>${middist_coupling}</multiplier>
-      <sensitiveness>0.0</sensitiveness>
-    </plugin>
-   <plugin name="mimic_right_j3a" filename="libroboticsgroup_gazebo_mimic_joint_plugin.so">
-      <joint>right_hand_j3</joint>
-      <mimicJoint>right_hand_j3a</mimicJoint>
-      <multiplier>${palmprox_coupling}</multiplier>
-      <sensitiveness>0.0</sensitiveness>
-    </plugin>
-    <plugin name="mimic_right_j3b" filename="libroboticsgroup_gazebo_mimic_joint_plugin.so">
-      <joint>right_hand_j3</joint>
-      <mimicJoint>right_hand_j3b</mimicJoint>
-      <multiplier>${proxmid_coupling}</multiplier>
-      <sensitiveness>0.0</sensitiveness>
-    </plugin>
-    <plugin name="mimic_right_j3c" filename="libroboticsgroup_gazebo_mimic_joint_plugin.so">
-      <joint>right_hand_j3</joint>
-      <mimicJoint>right_hand_j3c</mimicJoint>
-      <multiplier>${middist_coupling}</multiplier>
-      <sensitiveness>0.0</sensitiveness>
-    </plugin>
-    <plugin name="mimic_right_j4a" filename="libroboticsgroup_gazebo_mimic_joint_plugin.so">
-      <joint>right_hand_j4</joint>
-      <mimicJoint>right_hand_j4a</mimicJoint>
-      <multiplier>${palmprox_coupling}</multiplier>
-      <sensitiveness>0.0</sensitiveness>
-    </plugin>
-    <plugin name="mimic_right_j4b" filename="libroboticsgroup_gazebo_mimic_joint_plugin.so">
-      <joint>right_hand_j4</joint>
-      <mimicJoint>right_hand_j4b</mimicJoint>
-      <multiplier>${proxmid_coupling}</multiplier>
-      <sensitiveness>0.0</sensitiveness>
-    </plugin>
-    <plugin name="mimic_right_j4c" filename="libroboticsgroup_gazebo_mimic_joint_plugin.so">
-      <joint>right_hand_j4</joint>
-      <mimicJoint>right_hand_j4c</mimicJoint>
-      <multiplier>${middist_coupling}</multiplier>
-      <sensitiveness>0.0</sensitiveness>
-    </plugin>
+    <xacro:if value="$(arg _torso)">
+        <plugin name="mimic_torso" filename="libroboticsgroup_gazebo_mimic_joint_plugin.so">
+            <joint>torso_j1</joint>
+            <mimicJoint>torso_j2</mimicJoint>
+            <multiplier>1.0</multiplier>
+            <!--offset>0.0</offset-->
+        </plugin>
+    </xacro:if>
+    <xacro:if value="$(arg _r_hand)">
+        <plugin name="mimic_right_j1a" filename="libroboticsgroup_gazebo_mimic_joint_plugin.so">
+          <joint>right_hand_j1</joint>
+          <mimicJoint>right_hand_j1a</mimicJoint>
+          <multiplier>${th_palmprox_coupling}</multiplier>
+          <sensitiveness>0.0</sensitiveness>
+        </plugin>
+        <plugin name="mimic_right_j1b" filename="libroboticsgroup_gazebo_mimic_joint_plugin.so">
+          <joint>right_hand_j1</joint>
+          <mimicJoint>right_hand_j1b</mimicJoint>
+          <multiplier>${th_proxdist_coupling}</multiplier>
+          <sensitiveness>0.0</sensitiveness>
+        </plugin>
+        <plugin name="mimic_right_j2a" filename="libroboticsgroup_gazebo_mimic_joint_plugin.so">
+          <joint>right_hand_j2</joint>
+          <mimicJoint>right_hand_j2a</mimicJoint>
+          <multiplier>${palmprox_coupling}</multiplier>
+          <sensitiveness>0.0</sensitiveness>
+        </plugin>
+        <plugin name="mimic_right_j2b" filename="libroboticsgroup_gazebo_mimic_joint_plugin.so">
+          <joint>right_hand_j2</joint>
+          <mimicJoint>right_hand_j2b</mimicJoint>
+          <multiplier>${proxmid_coupling}</multiplier>
+          <sensitiveness>0.0</sensitiveness>
+        </plugin>
+        <plugin name="mimic_right_j2c" filename="libroboticsgroup_gazebo_mimic_joint_plugin.so">
+          <joint>right_hand_j2</joint>
+          <mimicJoint>right_hand_j2c</mimicJoint>
+          <multiplier>${middist_coupling}</multiplier>
+          <sensitiveness>0.0</sensitiveness>
+        </plugin>
+       <plugin name="mimic_right_j3a" filename="libroboticsgroup_gazebo_mimic_joint_plugin.so">
+          <joint>right_hand_j3</joint>
+          <mimicJoint>right_hand_j3a</mimicJoint>
+          <multiplier>${palmprox_coupling}</multiplier>
+          <sensitiveness>0.0</sensitiveness>
+        </plugin>
+        <plugin name="mimic_right_j3b" filename="libroboticsgroup_gazebo_mimic_joint_plugin.so">
+          <joint>right_hand_j3</joint>
+          <mimicJoint>right_hand_j3b</mimicJoint>
+          <multiplier>${proxmid_coupling}</multiplier>
+          <sensitiveness>0.0</sensitiveness>
+        </plugin>
+        <plugin name="mimic_right_j3c" filename="libroboticsgroup_gazebo_mimic_joint_plugin.so">
+          <joint>right_hand_j3</joint>
+          <mimicJoint>right_hand_j3c</mimicJoint>
+          <multiplier>${middist_coupling}</multiplier>
+          <sensitiveness>0.0</sensitiveness>
+        </plugin>
+        <plugin name="mimic_right_j4a" filename="libroboticsgroup_gazebo_mimic_joint_plugin.so">
+          <joint>right_hand_j4</joint>
+          <mimicJoint>right_hand_j4a</mimicJoint>
+          <multiplier>${palmprox_coupling}</multiplier>
+          <sensitiveness>0.0</sensitiveness>
+        </plugin>
+        <plugin name="mimic_right_j4b" filename="libroboticsgroup_gazebo_mimic_joint_plugin.so">
+          <joint>right_hand_j4</joint>
+          <mimicJoint>right_hand_j4b</mimicJoint>
+          <multiplier>${proxmid_coupling}</multiplier>
+          <sensitiveness>0.0</sensitiveness>
+        </plugin>
+        <plugin name="mimic_right_j4c" filename="libroboticsgroup_gazebo_mimic_joint_plugin.so">
+          <joint>right_hand_j4</joint>
+          <mimicJoint>right_hand_j4c</mimicJoint>
+          <multiplier>${middist_coupling}</multiplier>
+          <sensitiveness>0.0</sensitiveness>
+        </plugin>
+  </xacro:if>
   </gazebo>
   <gazebo reference="laser_front">

File: meka_description/robots/bie.urdf.xacro (robot description, xacro)
@@ -5,4 +5,13 @@
        xmlns:xacro="http://playerstage.sourceforge.net/gazebo/xmlschema/#interface"
        name="meka" >
+    <xacro:arg name="_head" default="true"/>
+    <xacro:arg name="_r_arm" default="true"/>
+    <xacro:arg name="_l_arm" default="true"/>
+    <xacro:arg name="_r_hand" default="true"/>
+    <xacro:arg name="_l_hand" default="true"/>
+    <xacro:arg name="_torso" default="true"/>
+    <xacro:arg name="_zlift" default="true"/>
+    <xacro:arg name="_caster_hubs" default="true"/>
+  <xacro:property name="hw_interface" value="hardware_interface/PositionJointInterface" />
   <xacro:property name="M_PI" value="3.1415926535897931" />
   <xacro:property name="MESH" value="meka_description/meshes/mid_res" />

File: meka_description/robots/bie_sim.urdf.xacro (robot description, xacro)
@@ -5,4 +5,13 @@
        xmlns:xacro="http://playerstage.sourceforge.net/gazebo/xmlschema/#interface"
        name="meka" >
+    <xacro:arg name="_head" default="false"/>
+    <xacro:arg name="_r_arm" default="false"/>
+    <xacro:arg name="_l_arm" default="false"/>
+    <xacro:arg name="_r_hand" default="false"/>
+    <xacro:arg name="_l_hand" default="false"/>
+    <xacro:arg name="_torso" default="false"/>
+    <xacro:arg name="_zlift" default="false"/>
+    <xacro:arg name="_caster_hubs" default="true"/>
+  <xacro:property name="hw_interface" value="hardware_interface/PositionJointInterface" />
   <xacro:property name="M_PI" value="3.1415926535897931" />
   <xacro:property name="MESH" value="meka_description/meshes/mid_res" />

File: meka_description/transmissions/A2R4_arm_defs.transmission.xacro (robot description, xacro)
@@ -10,5 +10,5 @@
       <actuator name="${lr}_arm_a0" />
       <joint name="${lr}_arm_j0">
-        <hardwareInterface>hardware_interface/PositionJointInterface</hardwareInterface>
+        <hardwareInterface>${hw_interface}</hardwareInterface>
       </joint>
     </transmission>
@@ -18,5 +18,5 @@
       <actuator name="${lr}_arm_a1" />
       <joint name="${lr}_arm_j1">
-        <hardwareInterface>hardware_interface/PositionJointInterface</hardwareInterface>
+        <hardwareInterface>${hw_interface}</hardwareInterface>
       </joint>
     </transmission>
@@ -26,5 +26,5 @@
       <actuator name="${lr}_arm_a2" />
       <joint name="${lr}_arm_j2">
-        <hardwareInterface>hardware_interface/PositionJointInterface</hardwareInterface>
+        <hardwareInterface>${hw_interface}</hardwareInterface>
       </joint>
     </transmission>
@@ -38,5 +38,5 @@
       </actuator>
       <joint name="${lr}_arm_j3">
-        <hardwareInterface>hardware_interface/PositionJointInterface</hardwareInterface>
+        <hardwareInterface>${hw_interface}</hardwareInterface>
       </joint>
     </transmission>
@@ -48,5 +48,5 @@
       </actuator>
       <joint name="${lr}_arm_j4">
-        <hardwareInterface>hardware_interface/PositionJointInterface</hardwareInterface>
+        <hardwareInterface>${hw_interface}</hardwareInterface>
       </joint>
     </transmission>
@@ -60,5 +60,5 @@
       </actuator>
       <joint name="${lr}_arm_j5">
-        <hardwareInterface>hardware_interface/PositionJointInterface</hardwareInterface>
+        <hardwareInterface>${hw_interface}</hardwareInterface>
       </joint>
     </transmission>
@@ -70,5 +70,5 @@
       </actuator>
       <joint name="${lr}_arm_j6">
-        <hardwareInterface>hardware_interface/PositionJointInterface</hardwareInterface>
+        <hardwareInterface>${hw_interface}</hardwareInterface>
       </joint>
     </transmission>

File: meka_description/transmissions/H2R4_hand.transmission.xacro (robot description, xacro)
@@ -7,5 +7,5 @@
     <type>transmission_interface/SimpleTransmission</type>
     <joint name="${lr}_hand_j0">
-      <hardwareInterface>hardware_interface/PositionJointInterface</hardwareInterface>
+      <hardwareInterface>${hw_interface}</hardwareInterface>
     </joint>
     <actuator name="${lr}_hand_j0_motor">
@@ -16,5 +16,5 @@
     <type>transmission_interface/SimpleTransmission</type>
     <joint name="${lr}_hand_j1">
-      <hardwareInterface>hardware_interface/PositionJointInterface</hardwareInterface>
+      <hardwareInterface>${hw_interface}</hardwareInterface>
     </joint>
     <actuator name="${lr}_hand_j1_motor">
@@ -25,5 +25,5 @@
     <type>transmission_interface/SimpleTransmission</type>
     <joint name="${lr}_hand_j2">
-      <hardwareInterface>hardware_interface/PositionJointInterface</hardwareInterface>
+      <hardwareInterface>${hw_interface}</hardwareInterface>
     </joint>
     <actuator name="${lr}_hand_j2_motor">
@@ -34,5 +34,5 @@
     <type>transmission_interface/SimpleTransmission</type>
     <joint name="${lr}_hand_j3">
-      <hardwareInterface>hardware_interface/PositionJointInterface</hardwareInterface>
+      <hardwareInterface>${hw_interface}</hardwareInterface>
     </joint>
     <actuator name="${lr}_hand_j3_motor">
@@ -43,5 +43,5 @@
     <type>transmission_interface/SimpleTransmission</type>
     <joint name="${lr}_hand_j4">
-      <hardwareInterface>hardware_interface/PositionJointInterface</hardwareInterface>
+      <hardwareInterface>${hw_interface}</hardwareInterface>
     </joint>
     <actuator name="${lr}_hand_j4_motor">

File: meka_description/transmissions/S3R1_head.transmission.xacro (robot description, xacro)
@@ -4,5 +4,5 @@
     <type>transmission_interface/SimpleTransmission</type>
     <joint name="head_j0">
-      <hardwareInterface>hardware_interface/PositionJointInterface</hardwareInterface>
+      <hardwareInterface>${hw_interface}</hardwareInterface>
     </joint>
     <actuator name="head_j0_motor">
@@ -13,5 +13,5 @@
     <type>transmission_interface/SimpleTransmission</type>
     <joint name="head_j1">
-      <hardwareInterface>hardware_interface/PositionJointInterface</hardwareInterface>
+      <hardwareInterface>${hw_interface}</hardwareInterface>
     </joint>
     <actuator name="head_j1_motor">

File: meka_description/transmissions/T2R3_torso.transmission.xacro (robot description, xacro)
@@ -4,5 +4,5 @@
     <type>transmission_interface/SimpleTransmission</type>
     <joint name="torso_j0">
-      <hardwareInterface>hardware_interface/PositionJointInterface</hardwareInterface>
+      <hardwareInterface>${hw_interface}</hardwareInterface>
     </joint>
     <actuator name="torso_j0_motor">
@@ -13,5 +13,5 @@
     <type>transmission_interface/SimpleTransmission</type>
     <joint name="torso_j1">
-      <hardwareInterface>hardware_interface/PositionJointInterface</hardwareInterface>
+      <hardwareInterface>${hw_interface}</hardwareInterface>
     </joint>
     <actuator name="torso_j1_motor">

File: meka_description/transmissions/Z1R2_zlift.transmission.xacro (robot description, xacro)
@@ -4,5 +4,5 @@
     <type>transmission_interface/SimpleTransmission</type>
     <joint name="zlift_j0">
-      <hardwareInterface>hardware_interface/PositionJointInterface</hardwareInterface>
+      <hardwareInterface>${hw_interface}</hardwareInterface>
     </joint>
     <actuator name="zlift_j0_motor">

File: meka_description/urdf/MEKA_BASIC.urdf.xacro (robot description, xacro)
@@ -7,12 +7,4 @@
  	<xacro:arg name="hand_mimic" default="true"/>
  	<xacro:arg name="torso_mimic" default="true"/>
- 	<xacro:arg name="_head" default="true"/>
- 	<xacro:arg name="_r_arm" default="true"/>
- 	<xacro:arg name="_l_arm" default="true"/>
- 	<xacro:arg name="_r_hand" default="true"/>
- 	<xacro:arg name="_l_hand" default="true"/>
- 	<xacro:arg name="_torso" default="true"/>
- 	<xacro:arg name="_zlift" default="true"/>
- 	<xacro:arg name="_caster_hubs" default="true"/>
     <xacro:property name="base_link" value="base_link" />
     <xacro:macro name="inertial_cuboid_with_pose" params="mass x_length y_length z_length *origin">
@@ -37,10 +29,10 @@
 	</material>
     <link name="${base_link}">
-        <!--collision>
+        <collision>
           <origin xyz="0 0 0" rpy="0 0 0" />
           <geometry>
             <box size="0.8 0.6 0.025"/>
           </geometry>
-        </collision-->
+        </collision>
 	</link>
 	<joint name="laser_front_joint" type="fixed">
