Commit message: added meka body to sim

File: meka_description/gazebo/gazebo.urdf.xacro (robot description, xacro)
@@ -39,20 +39,20 @@
       <odometryRate>20.0</odometryRate>
       <robotBaseFrame>base_link</robotBaseFrame>
-      <joint_state_idel_sec>3.0</joint_state_idel_sec>
-      <recover_roll_velocity_p_gain>10.0</recover_roll_velocity_p_gain>
-      <recover_pitch_velocity_p_gain>10.0</recover_pitch_velocity_p_gain>
-      <recover_z_velocity_p_gain>50.0</recover_z_velocity_p_gain>
-      <x_velocity_limit_max>2.0</x_velocity_limit_max>
-      <x_velocity_limit_min>-2.0</x_velocity_limit_min>
-      <y_velocity_limit_max>2.0</y_velocity_limit_max>
-      <y_velocity_limit_min>-2.0</y_velocity_limit_min>
-      <rot_velocity_limit_max>1.5</rot_velocity_limit_max>
-      <rot_velocity_limit_min>-1.5</rot_velocity_limit_min>
-      <x_acceleration_limit_max>2.0</x_acceleration_limit_max>
-      <x_acceleration_limit_min>-2.0</x_acceleration_limit_min>
-      <y_acceleration_limit_max>2.0</y_acceleration_limit_max>
-      <y_acceleration_limit_min>-2.0</y_acceleration_limit_min>
-      <rot_acceleration_limit_max>1.5</rot_acceleration_limit_max>
-      <rot_acceleration_limit_min>-1.5</rot_acceleration_limit_min>
+      <joint_state_idel_sec>2.0</joint_state_idel_sec>
+      <recover_roll_velocity_p_gain>1.0</recover_roll_velocity_p_gain>
+      <recover_pitch_velocity_p_gain>1.0</recover_pitch_velocity_p_gain>
+      <recover_z_velocity_p_gain>5.0</recover_z_velocity_p_gain>
+      <x_velocity_limit_max>4.0</x_velocity_limit_max>
+      <x_velocity_limit_min>-4.0</x_velocity_limit_min>
+      <y_velocity_limit_max>4.0</y_velocity_limit_max>
+      <y_velocity_limit_min>-4.0</y_velocity_limit_min>
+      <rot_velocity_limit_max>3.0</rot_velocity_limit_max>
+      <rot_velocity_limit_min>-3.0</rot_velocity_limit_min>
+      <x_acceleration_limit_max>3.0</x_acceleration_limit_max>
+      <x_acceleration_limit_min>-3.0</x_acceleration_limit_min>
+      <y_acceleration_limit_max>3.0</y_acceleration_limit_max>
+      <y_acceleration_limit_min>-3.0</y_acceleration_limit_min>
+      <rot_acceleration_limit_max>2.0</rot_acceleration_limit_max>
+      <rot_acceleration_limit_min>-2.0</rot_acceleration_limit_min>
       <tilt_angle_par_max_velocity>0</tilt_angle_par_max_velocity>
     </plugin>

File: meka_description/robots/bie_sim.urdf.xacro (robot description, xacro)
@@ -5,11 +5,11 @@
        xmlns:xacro="http://playerstage.sourceforge.net/gazebo/xmlschema/#interface"
        name="meka" >
-    <xacro:arg name="_head" default="false"/>
-    <xacro:arg name="_r_arm" default="false"/>
-    <xacro:arg name="_l_arm" default="false"/>
-    <xacro:arg name="_r_hand" default="false"/>
-    <xacro:arg name="_l_hand" default="false"/>
-    <xacro:arg name="_torso" default="false"/>
-    <xacro:arg name="_zlift" default="false"/>
+    <xacro:arg name="_zlift" default="true"/>
+    <xacro:arg name="_torso" default="true"/>
+    <xacro:arg name="_head" default="true"/>
+    <xacro:arg name="_r_arm" default="true"/>
+    <xacro:arg name="_l_arm" default="true"/>
+    <xacro:arg name="_r_hand" default="true"/>
+    <xacro:arg name="_l_hand" default="true"/>
     <xacro:arg name="_caster_hubs" default="false"/>
   <xacro:property name="hw_interface" value="hardware_interface/PositionJointInterface" />

File: meka_description/transmissions/H2R4_hand.transmission.xacro (robot description, xacro)
@@ -4,49 +4,49 @@
        xmlns:interface="http://playerstage.sourceforge.net/gazebo/xmlschema/#interface">
   <macro name="m3_hand_transmission" params="lr">
-  <transmission name="${lr}_hand_j0_trans">
-    <type>transmission_interface/SimpleTransmission</type>
-    <joint name="${lr}_hand_j0">
-      <hardwareInterface>${hw_interface}</hardwareInterface>
-    </joint>
-    <actuator name="${lr}_hand_j0_motor">
-      <mechanicalReduction>1</mechanicalReduction>
-    </actuator>
-  </transmission>
-   <transmission name="${lr}_hand_j1_trans">
-    <type>transmission_interface/SimpleTransmission</type>
-    <joint name="${lr}_hand_j1">
-      <hardwareInterface>${hw_interface}</hardwareInterface>
-    </joint>
-    <actuator name="${lr}_hand_j1_motor">
-      <mechanicalReduction>1</mechanicalReduction>
-    </actuator>
-  </transmission>
-   <transmission name="${lr}_hand_j2_trans">
-    <type>transmission_interface/SimpleTransmission</type>
-    <joint name="${lr}_hand_j2">
-      <hardwareInterface>${hw_interface}</hardwareInterface>
-    </joint>
-    <actuator name="${lr}_hand_j2_motor">
-      <mechanicalReduction>1</mechanicalReduction>
-    </actuator>
-  </transmission>
-   <transmission name="${lr}_hand_j3_trans">
-    <type>transmission_interface/SimpleTransmission</type>
-    <joint name="${lr}_hand_j3">
-      <hardwareInterface>${hw_interface}</hardwareInterface>
-    </joint>
-    <actuator name="${lr}_hand_j3_motor">
-      <mechanicalReduction>1</mechanicalReduction>
-    </actuator>
-  </transmission>
-   <transmission name="${lr}_hand_j4_trans">
-    <type>transmission_interface/SimpleTransmission</type>
-    <joint name="${lr}_hand_j4">
-      <hardwareInterface>${hw_interface}</hardwareInterface>
-    </joint>
-    <actuator name="${lr}_hand_j4_motor">
-      <mechanicalReduction>1</mechanicalReduction>
-    </actuator>
-  </transmission>
+      <transmission name="${lr}_hand_j0_trans">
+        <type>transmission_interface/SimpleTransmission</type>
+        <joint name="${lr}_hand_j0">
+          <hardwareInterface>${hw_interface}</hardwareInterface>
+        </joint>
+        <actuator name="${lr}_hand_j0_motor">
+          <mechanicalReduction>1</mechanicalReduction>
+        </actuator>
+      </transmission>
+       <transmission name="${lr}_hand_j1_trans">
+        <type>transmission_interface/SimpleTransmission</type>
+        <joint name="${lr}_hand_j1">
+          <hardwareInterface>${hw_interface}</hardwareInterface>
+        </joint>
+        <actuator name="${lr}_hand_j1_motor">
+          <mechanicalReduction>1</mechanicalReduction>
+        </actuator>
+      </transmission>
+       <transmission name="${lr}_hand_j2_trans">
+        <type>transmission_interface/SimpleTransmission</type>
+        <joint name="${lr}_hand_j2">
+          <hardwareInterface>${hw_interface}</hardwareInterface>
+        </joint>
+        <actuator name="${lr}_hand_j2_motor">
+          <mechanicalReduction>1</mechanicalReduction>
+        </actuator>
+      </transmission>
+       <transmission name="${lr}_hand_j3_trans">
+        <type>transmission_interface/SimpleTransmission</type>
+        <joint name="${lr}_hand_j3">
+          <hardwareInterface>${hw_interface}</hardwareInterface>
+        </joint>
+        <actuator name="${lr}_hand_j3_motor">
+          <mechanicalReduction>1</mechanicalReduction>
+        </actuator>
+      </transmission>
+       <transmission name="${lr}_hand_j4_trans">
+        <type>transmission_interface/SimpleTransmission</type>
+        <joint name="${lr}_hand_j4">
+          <hardwareInterface>${hw_interface}</hardwareInterface>
+        </joint>
+        <actuator name="${lr}_hand_j4_motor">
+          <mechanicalReduction>1</mechanicalReduction>
+        </actuator>
+      </transmission>
   </macro>
 </robot>

File: meka_description/transmissions/S3R1_head.transmission.xacro (robot description, xacro)
@@ -1,21 +1,23 @@
 <?xml version="1.0"?>
 <robot>
-  <transmission name="head_j0_trans">
-    <type>transmission_interface/SimpleTransmission</type>
-    <joint name="head_j0">
-      <hardwareInterface>${hw_interface}</hardwareInterface>
-    </joint>
-    <actuator name="head_j0_motor">
-      <mechanicalReduction>1</mechanicalReduction>
-    </actuator>
-  </transmission>
-   <transmission name="head_j1_trans">
-    <type>transmission_interface/SimpleTransmission</type>
-    <joint name="head_j1">
-      <hardwareInterface>${hw_interface}</hardwareInterface>
-    </joint>
-    <actuator name="head_j1_motor">
-      <mechanicalReduction>1</mechanicalReduction>
-    </actuator>
-  </transmission>
+    <macro name="m3_head_transmission">
+        <transmission name="head_j0_trans">
+            <type>transmission_interface/SimpleTransmission</type>
+            <joint name="head_j0">
+              <hardwareInterface>${hw_interface}</hardwareInterface>
+            </joint>
+            <actuator name="head_j0_motor">
+              <mechanicalReduction>1</mechanicalReduction>
+            </actuator>
+        </transmission>
+        <transmission name="head_j1_trans">
+            <type>transmission_interface/SimpleTransmission</type>
+            <joint name="head_j1">
+              <hardwareInterface>${hw_interface}</hardwareInterface>
+            </joint>
+            <actuator name="head_j1_motor">
+              <mechanicalReduction>1</mechanicalReduction>
+            </actuator>
+        </transmission>
+    </macro>
 </robot>

File: meka_description/transmissions/T2R3_torso.transmission.xacro (robot description, xacro)
@@ -1,4 +1,5 @@
 <?xml version="1.0"?>
 <robot>
+ <macro name="m3_torso_transmission">
   <transmission name="torso_j0_trans">
     <type>transmission_interface/SimpleTransmission</type>
@@ -19,3 +20,4 @@
     </actuator>
   </transmission>
+ </macro>
 </robot>

File: meka_description/transmissions/Z1R2_zlift.transmission.xacro (robot description, xacro)
@@ -1,4 +1,5 @@
 <?xml version="1.0"?>
 <robot>
+<macro name="m3_zlift_transmission">
   <transmission name="zlift_j0_trans">
     <type>transmission_interface/SimpleTransmission</type>
@@ -10,3 +11,4 @@
     </actuator>
   </transmission>
+</macro>
 </robot>

File: meka_description/urdf/MEKA_BASIC.urdf.xacro (robot description, xacro)
@@ -54,4 +54,5 @@
 		<origin xyz="0.0 0.0 0.0" rpy="0 0 0" />
 	</meka_base>
+	<!-- zlift -->
 	<xacro:if value="$(arg _zlift)">
 	    <meka_zlift parent="${base_link}">
@@ -59,35 +60,43 @@
 		    <!-- 0.33 0.0 0.45 rpy="0 0.0236 0" -->
 	    </meka_zlift>
-	</xacro:if>
-	<xacro:if value="$(arg _torso)">
-	    <meka_torso parent="zlift_link">
-		    <origin xyz="0.263 0.0 0.006" rpy="0 0 0" />
-	    </meka_torso>
-	</xacro:if>
-	<xacro:if value="$(arg _head)">
-	    <m3_head parent="upper">
-		    <origin xyz="0.0 0.0 0.2757" rpy="0 0 0" />
-	    </m3_head>
-	</xacro:if>
-	<xacro:if value="$(arg _r_arm)">
-	    <m3_arm side="R" lr="right" reflect="1" rotate="0" parent="upper">
-		    <origin xyz="0.0 -0.18465 0.2337" rpy="0 0 0" />
-	    </m3_arm>
-	</xacro:if>
-	<xacro:if value="$(arg _l_arm)">
-	    <m3_arm side="L" lr="left" reflect="-1" rotate="1" parent="upper">
-		    <origin xyz="0.0 0.18465 0.2337" rpy="0 0 0" />
-	    </m3_arm>
-	</xacro:if>
-	<xacro:if value="$(arg _l_hand)">
-	    <m3_hand lr="left" reflect="1" parent="handmount_left" use_mimic="$(arg hand_mimic)">
-		    <origin xyz="0.0 0.0 0.0" rpy="0 0 0" />
-	    </m3_hand>
+	    <m3_zlift_transmission />
+	    <!-- torso -->
+	    <xacro:if value="$(arg _torso)">
+	        <meka_torso parent="zlift_link">
+		        <origin xyz="0.263 0.0 0.006" rpy="0 0 0" />
+	        </meka_torso>
+	        <m3_torso_transmission />
+	        <xacro:if value="$(arg _head)">
+	            <m3_head parent="upper">
+		            <origin xyz="0.0 0.0 0.2757" rpy="0 0 0" />
+	            </m3_head>
+	            <m3_head_transmission />
+	        </xacro:if>
+	        <xacro:if value="$(arg _r_arm)">
+	            <m3_arm side="R" lr="right" reflect="1" rotate="0" parent="upper">
+		            <origin xyz="0.0 -0.18465 0.2337" rpy="0 0 0" />
+	            </m3_arm>
+	            <!-- transmissions inserted in arm urdf -->
+	            <xacro:if value="$(arg _r_hand)">
+	                <m3_hand lr="right" reflect="-1" parent="handmount_right" use_mimic="$(arg hand_mimic)">
+		                <origin xyz="0.0 0.0 0.0" rpy="0 0 0" />
+	                </m3_hand>
+	            <!-- transmissions inserted in hand urdf -->
+	            </xacro:if>
+	        </xacro:if>
+	        <xacro:if value="$(arg _l_arm)">
+	            <m3_arm side="L" lr="left" reflect="-1" rotate="1" parent="upper">
+		            <origin xyz="0.0 0.18465 0.2337" rpy="0 0 0" />
+	            </m3_arm>
+	            <!-- transmissions inserted in arm urdf -->
+	            <xacro:if value="$(arg _l_hand)">
+	                <m3_hand lr="left" reflect="1" parent="handmount_left" use_mimic="$(arg hand_mimic)">
+		                <origin xyz="0.0 0.0 0.0" rpy="0 0 0" />
+	                </m3_hand>
+	                <!-- transmissions inserted in hand urdf -->
+                </xacro:if>
+	        </xacro:if>
+        </xacro:if>
     </xacro:if>
-	<xacro:if value="$(arg _r_hand)">
-	    <m3_hand lr="right" reflect="-1" parent="handmount_right" use_mimic="$(arg hand_mimic)">
-		    <origin xyz="0.0 0.0 0.0" rpy="0 0 0" />
-	    </m3_hand>
-	</xacro:if>
 	<xacro:if value="$(arg _caster_hubs)">
         <m3_caster_hub l="0.2678" alpha="${M_PI/6}" fb="front" lr="right" parent="${base_link}" />

Commit message: added mimic for left hand

File: meka_description/gazebo/gazebo.urdf.xacro (robot description, xacro)
@@ -129,4 +129,72 @@
           <joint>right_hand_j4</joint>
           <mimicJoint>right_hand_j4c</mimicJoint>
+          <multiplier>${middist_coupling}</multiplier>
+          <sensitiveness>0.0</sensitiveness>
+        </plugin>
+  </xacro:if>
+  <xacro:if value="$(arg _l_hand)">
+        <plugin name="mimic_left_j1a" filename="libroboticsgroup_gazebo_mimic_joint_plugin.so">
+          <joint>left_hand_j1</joint>
+          <mimicJoint>left_hand_j1a</mimicJoint>
+          <multiplier>${th_palmprox_coupling}</multiplier>
+          <sensitiveness>0.0</sensitiveness>
+        </plugin>
+        <plugin name="mimic_left_j1b" filename="libroboticsgroup_gazebo_mimic_joint_plugin.so">
+          <joint>left_hand_j1</joint>
+          <mimicJoint>left_hand_j1b</mimicJoint>
+          <multiplier>${th_proxdist_coupling}</multiplier>
+          <sensitiveness>0.0</sensitiveness>
+        </plugin>
+        <plugin name="mimic_left_j2a" filename="libroboticsgroup_gazebo_mimic_joint_plugin.so">
+          <joint>left_hand_j2</joint>
+          <mimicJoint>left_hand_j2a</mimicJoint>
+          <multiplier>${palmprox_coupling}</multiplier>
+          <sensitiveness>0.0</sensitiveness>
+        </plugin>
+        <plugin name="mimic_left_j2b" filename="libroboticsgroup_gazebo_mimic_joint_plugin.so">
+          <joint>left_hand_j2</joint>
+          <mimicJoint>left_hand_j2b</mimicJoint>
+          <multiplier>${proxmid_coupling}</multiplier>
+          <sensitiveness>0.0</sensitiveness>
+        </plugin>
+        <plugin name="mimic_left_j2c" filename="libroboticsgroup_gazebo_mimic_joint_plugin.so">
+          <joint>left_hand_j2</joint>
+          <mimicJoint>left_hand_j2c</mimicJoint>
+          <multiplier>${middist_coupling}</multiplier>
+          <sensitiveness>0.0</sensitiveness>
+        </plugin>
+       <plugin name="mimic_left_j3a" filename="libroboticsgroup_gazebo_mimic_joint_plugin.so">
+          <joint>left_hand_j3</joint>
+          <mimicJoint>left_hand_j3a</mimicJoint>
+          <multiplier>${palmprox_coupling}</multiplier>
+          <sensitiveness>0.0</sensitiveness>
+        </plugin>
+        <plugin name="mimic_left_j3b" filename="libroboticsgroup_gazebo_mimic_joint_plugin.so">
+          <joint>left_hand_j3</joint>
+          <mimicJoint>left_hand_j3b</mimicJoint>
+          <multiplier>${proxmid_coupling}</multiplier>
+          <sensitiveness>0.0</sensitiveness>
+        </plugin>
+        <plugin name="mimic_left_j3c" filename="libroboticsgroup_gazebo_mimic_joint_plugin.so">
+          <joint>left_hand_j3</joint>
+          <mimicJoint>left_hand_j3c</mimicJoint>
+          <multiplier>${middist_coupling}</multiplier>
+          <sensitiveness>0.0</sensitiveness>
+        </plugin>
+        <plugin name="mimic_left_j4a" filename="libroboticsgroup_gazebo_mimic_joint_plugin.so">
+          <joint>left_hand_j4</joint>
+          <mimicJoint>left_hand_j4a</mimicJoint>
+          <multiplier>${palmprox_coupling}</multiplier>
+          <sensitiveness>0.0</sensitiveness>
+        </plugin>
+        <plugin name="mimic_left_j4b" filename="libroboticsgroup_gazebo_mimic_joint_plugin.so">
+          <joint>left_hand_j4</joint>
+          <mimicJoint>left_hand_j4b</mimicJoint>
+          <multiplier>${proxmid_coupling}</multiplier>
+          <sensitiveness>0.0</sensitiveness>
+        </plugin>
+        <plugin name="mimic_left_j4c" filename="libroboticsgroup_gazebo_mimic_joint_plugin.so">
+          <joint>left_hand_j4</joint>
+          <mimicJoint>left_hand_j4c</mimicJoint>
           <multiplier>${middist_coupling}</multiplier>
           <sensitiveness>0.0</sensitiveness>
