Commit message: further tuning for gazebo simulation. Navigation and body movements fixed now.

File: meka_description/gazebo/gazebo.urdf.xacro (robot description, xacro)
@@ -34,5 +34,5 @@
     </plugin-->
     <plugin name="object_controller" filename="libgazebo_ros_planar_move.so">
-      <commandTopic>cmd_vel</commandTopic>
+      <commandTopic>smooth_cmd_vel</commandTopic>
       <odometryTopic>odom</odometryTopic>
       <odometryFrame>odom</odometryFrame>
@@ -40,7 +40,7 @@
       <robotBaseFrame>base_link</robotBaseFrame>
       <joint_state_idel_sec>2.0</joint_state_idel_sec>
-      <recover_roll_velocity_p_gain>1.0</recover_roll_velocity_p_gain>
+      <recover_roll_velocity_p_gain>50.0</recover_roll_velocity_p_gain>
       <recover_pitch_velocity_p_gain>50.0</recover_pitch_velocity_p_gain>
-      <recover_z_velocity_p_gain>50.0</recover_z_velocity_p_gain>
+      <recover_z_velocity_p_gain>1.0</recover_z_velocity_p_gain>
       <x_velocity_limit_max>4.0</x_velocity_limit_max>
       <x_velocity_limit_min>-4.0</x_velocity_limit_min>
@@ -55,5 +55,5 @@
       <rot_acceleration_limit_max>2.0</rot_acceleration_limit_max>
       <rot_acceleration_limit_min>-2.0</rot_acceleration_limit_min>
-      <tilt_angle_par_max_velocity>0</tilt_angle_par_max_velocity>
+      <tilt_angle_par_max_velocity>1</tilt_angle_par_max_velocity>
     </plugin>
     <xacro:if value="$(arg _torso)">
@@ -206,5 +206,5 @@
       <pose>0 0 0 0 0 0</pose>
       <visualize>false</visualize>
-      <update_rate>40</update_rate>
+      <update_rate>30</update_rate>
       <ray>
         <scan>
@@ -227,5 +227,5 @@
         </noise>
       </ray>
-      <plugin name="laser_front_sick" filename="libgazebo_ros_gpu_laser.so">
+      <plugin name="laser_front_hokuyo" filename="libgazebo_ros_gpu_laser.so">
         <topicName>/scan_front</topicName>
         <frameName>laser_front</frameName>
@@ -249,5 +249,5 @@
         <range>
           <min>0.2</min>
-          <max>8.0</max>
+          <max>25.0</max>
           <resolution>0.005759587</resolution>
         </range>
@@ -255,8 +255,8 @@
           <type>gaussian</type>
           <mean>0.0</mean>
-          <stddev>0.015</stddev>
+          <stddev>0.03</stddev>
         </noise>
       </ray>
-      <plugin name="laser_front_sick" filename="libgazebo_ros_gpu_laser.so">
+      <plugin name="laser_rear_sick" filename="libgazebo_ros_gpu_laser.so">
         <topicName>/scan_rear</topicName>
         <frameName>laser_rear</frameName>

File: meka_description/robots/bie_sim.urdf.xacro (robot description, xacro)
@@ -8,4 +8,5 @@
     <xacro:arg name="_torso" default="true"/>
     <xacro:arg name="_head" default="true"/>
+    <xacro:arg name="_xtion" default="true"/>
     <xacro:arg name="_r_arm" default="true"/>
     <xacro:arg name="_l_arm" default="true"/>
@@ -39,9 +40,13 @@
   <xacro:include filename="$(find meka_description)/transmissions/S3R1_head.transmission.xacro" />
   <!-- Import asus-->
+  <xacro:if value="$(arg _head)">
+  <xacro:if value="$(arg _xtion)">
   <xacro:include filename="$(find meka_description)/urdf/asus_camera.urdf.xacro" />
   <xacro:asus_camera name="xtion" parent="shell">
     <origin xyz="0.12 0 0.06" rpy="0 0 0"/>
   </xacro:asus_camera>
+  </xacro:if>
+  </xacro:if>
   <!-- Extra Wheels -->
-  <xacro:include filename="$(find meka_description)/urdf/wheel_defs.urdf.xacro" />
+  <!--<xacro:include filename="$(find meka_description)/urdf/wheel_defs.urdf.xacro" />-->
 </robot>

File: meka_description/urdf/A2R4_arm_defs.urdf.xacro (robot description, xacro)
@@ -303,11 +303,7 @@
     </joint>
     <link name="w_differential_${lr}">
-      <inertial>
-        <mass value="0.278" />
-        <origin xyz="0 0 0" />
-        <inertia ixx="0" ixy="0" ixz="0"
-                 iyy="0" iyz="0"
-                 izz="0" />
-      </inertial>
+		<xacro:inertial_cuboid_with_pose mass="1.5" x_length="0.1" y_length="0.1" z_length="0.2">
+			<origin xyz="0 0 0.0" rpy="0 0 0" />
+		</xacro:inertial_cuboid_with_pose>
       <visual>
 	      <material name="GreyB" />
@@ -333,11 +329,7 @@
     </joint>
     <link name="handmount_${lr}">
-      <inertial>
-        <mass value="0.093" />
-        <origin xyz="0 0 0" />
-        <inertia ixx="0" ixy="0" ixz="0"
-                 iyy="0" iyz="0"
-                 izz="0" />
-      </inertial>
+		<xacro:inertial_cuboid_with_pose mass="0.5" x_length="0.2" y_length="0.2" z_length="0.1">
+			<origin xyz="0 0 0.0" rpy="0 0 0" />
+		</xacro:inertial_cuboid_with_pose>
       <visual>
 	      <material name="GreyA" />

File: meka_description/urdf/S3R1_head_defs.urdf.xacro (robot description, xacro)
@@ -2,5 +2,6 @@
 <robot xmlns:sensor="http://playerstage.sourceforge.net/gazebo/xmlschema/#sensor"
        xmlns:controller="http://playerstage.sourceforge.net/gazebo/xmlschema/#controller"
-       xmlns:interface="http://playerstage.sourceforge.net/gazebo/xmlschema/#interface">
+       xmlns:interface="http://playerstage.sourceforge.net/gazebo/xmlschema/#interface"
+       xmlns:xacro="http://playerstage.sourceforge.net/gazebo/xmlschema/#interface">
   <property name="M_PI" value="3.1415926535897931" />
   <macro name="m3_neck" params="parent *origin">
@@ -14,14 +15,7 @@
     </joint>
     <link name="neck_pan">
-      <inertial>
-        <mass value="0.940" />
-	<origin xyz="0.000061 0.003310 0.028798"/>
-	<inertia ixx="0.001395"
-	iyy="0.001345"
-	izz="0.000392"
-	ixy="-0.000000"
-	ixz="-0.000000"
-	iyz="-0.000085" />
-      </inertial>
+		<xacro:inertial_cuboid_with_pose mass="0.1" x_length="0.1" y_length="0.1" z_length="0.05">
+			<origin xyz="0 0 0.0" rpy="0 0 0" />
+		</xacro:inertial_cuboid_with_pose>
       <visual>
 	      <material name="GreyA" />
@@ -63,14 +57,7 @@
     </joint>
     <link name="shell">
-      <inertial>
-        <mass value="0.409" />
-	<origin xyz="0.0 0.0 0.0"/>
-	<inertia ixx="0.0"
-        iyy="0.0"
-        izz="0.0"
-        ixy="0.0"
-        ixz="0.0"
-        iyz="0.0" />
-      </inertial>
+		<xacro:inertial_cuboid_with_pose mass="1.0" x_length="0.2" y_length="0.2" z_length="0.1">
+			<origin xyz="0 0 0.0" rpy="0 0 0" />
+		</xacro:inertial_cuboid_with_pose>
       <visual>
 	      <material name="GreyB" />
@@ -102,6 +89,5 @@
       </collision>
     </link>
-     <joint name="head_xtion_dummy" type="revolute">
-	<limit effort="100" velocity="${75*M_PI/180}" lower="${-56.0*M_PI/180}" upper="${56.0*M_PI/180}" />
+     <joint name="head_xtion_dummy" type="fixed">
 	<origin xyz="0.0865 0.0095 0.0542" rpy="-1.49304175558102 0.0465121191942754 -1.5830006092006217"/>
       <axis xyz="0 0 1"/>
@@ -111,16 +97,9 @@
     <link name="_xtion_link">
 	<parent link="shell"/>
-	<inertial>
-        <mass value="0.1" />
-	<origin xyz="0.0 0.0 0.0"/>
-      <inertia ixx="0.0"
-          iyy="0.0"
-          izz="0.0"
-          ixy="0.0"
-          ixz="0.0"
-          iyz="0.0" />
-      </inertial>
+		<xacro:inertial_cuboid_with_pose mass="0.1" x_length="0.1" y_length="0.1" z_length="0.05">
+			<origin xyz="0 0 0.0" rpy="0 0 0" />
+		</xacro:inertial_cuboid_with_pose>
     </link>
-     <joint name="head_xtion_dummy2" type="revolute">
+     <joint name="head_xtion_dummy2" type="fixed">
 	<limit effort="100" velocity="${75*M_PI/180}" lower="${-56.0*M_PI/180}" upper="${56.0*M_PI/180}" />
 	<origin xyz="-0.04 0 0" rpy="0 -1.5708 1.5708"/>
@@ -131,14 +110,7 @@
     <link name="xtion_link">
 	<parent link="_xtion_link"/>
-	<inertial>
-        <mass value="0.1" />
-	<origin xyz="0.0 0.0 0.0"/>
-      <inertia ixx="0.0"
-          iyy="0.0"
-          izz="0.0"
-          ixy="0.0"
-          ixz="0.0"
-          iyz="0.0" />
-      </inertial>
+		<xacro:inertial_cuboid_with_pose mass="0.1" x_length="0.1" y_length="0.1" z_length="0.05">
+			<origin xyz="0 0 0.0" rpy="0 0 0" />
+		</xacro:inertial_cuboid_with_pose>
     </link>
     <!--joint name="head_j2" type="revolute">

File: meka_description/urdf/T2R3_torso_defs.urdf.xacro (robot description, xacro)
@@ -100,9 +100,7 @@
 	</joint>
 	<link name="mid">
-		<inertial>
-			<mass value="4.934" />
-			<origin xyz="0.001179 -0.002993 0.046259"/>
-			<inertia ixx="0.041106" iyy="0.026009" izz="0.025902" ixy="0.000135" ixz="0.000505" iyz="0.002396" />
-		</inertial>
+		<xacro:inertial_cuboid_with_pose mass="5.0" x_length="0.2" y_length="0.4" z_length="0.5">
+			<origin xyz="0 0 0.01" rpy="0 0 0" />
+		</xacro:inertial_cuboid_with_pose>
 		<visual>
 			<material name="GreyB" />
@@ -147,9 +145,7 @@
 	</joint>
 	<link name="upper">
-		<inertial>
-			<mass value="6.534" />
-			<origin xyz="0.008700 0.011470 0.129740"/>
-			<inertia ixx="0.069760" iyy="0.048010" izz="0.040590" ixy="-0.000400" ixz="0.001300" iyz="0.005100" />
-		</inertial>
+		<xacro:inertial_cuboid_with_pose mass="3.0" x_length="0.2" y_length="0.4" z_length="0.6">
+			<origin xyz="0 0 0.01" rpy="0 0 0" />
+		</xacro:inertial_cuboid_with_pose>
 		<visual>
 			<material name="GreyC" />

File: meka_description/urdf/asus_camera.urdf.xacro (robot description, xacro)
@@ -9,9 +9,7 @@
       </joint>
       <link name="${name}_linkgz">
-        <inertial>
-          <mass value="0.200" />
-          <origin xyz="0 0 0" rpy="0 0 0" />
-          <inertia ixx="5.8083e-4" ixy="0" ixz="0" iyy="3.0833e-5" iyz="0" izz="5.9083e-4" />
-        </inertial>
+		<xacro:inertial_cuboid_with_pose mass="0.2" x_length="0.05" y_length="0.15" z_length="0.05">
+			<origin xyz="0 0 0.0" rpy="0 0 0" />
+		</xacro:inertial_cuboid_with_pose>
         <visual>
           <origin xyz="0 0 0" rpy="0 0 0" />
